File: camera_main_sch_brd.brd (EAGLE design)
At the start: 110 x 110 mm, 98 parts, among them CN1 USB C CON, CN2 50 PIN 0.5MM, CN3 31 PIN FPC, CN4 10/100 RJ45, CN5 USB A, CN6 NO FIT, U1 10CL016YF484C6G, U11 USBLC6-2SC6, U12 TPS70925, U2 OSD32MP157C-512M-BAA, U3 STM32L431RBT, U4 TLV61046A, U5 AS4C32M16SA, U6 AS4C32M16SA, U7 ACT2861, U9 FT232H

Commit message: Progress, new names
Parts:
- removed C48, C49: 100nF 16V, CAPACITORS:0402
- added C38: 10uF 50V, CAPACITORS:1210
- added C39, C40: 100nF 16V, CAPACITORS:0603
- added C41, C42, C43: 100nF 100V, CAPACITORS:0603
- added CN7: uSD, CONNECTORs:114-00841-68
- added CN8: NO FIT, CONNECTORs:TSM-103-DV
- added D1, D5, D6: B0540W, DIODES:SOD-123
- added D7, D8: PESD5Z5.0, DIODES:SC-79
- added D9: 20V TVS, DIODES:DO214AC
- added Q2: SI7489DP, TRANSISTORs:SO8_POWERPAK
- added R26, R33, R34, R35, R36, R37, R38: 10k, r_0603:0603
- added R27, R28, R29, R30, R31, R32: 10R, r_0603:0603
- added R39, R40: 10k, r_0402:0402
- added R44: 1.0k, r_0603:0603
- added R45: 100k, r_0603:0603
- added R46: 22k, r_0603:0603
- added TP1, TP2: 2MM_TEST_POINT, MISC:2MM_TEST_PAD
- added U13: FT230X, ICs:SSOP16-4MM
- added U14: 3.3V BUCK, ICs:TI_MICROSIP_10
- added U15: STUSB4500, ICs:QFN24
- added U8: USBLC6-2SC6, ICs:SOT23-6
- C18: value 10pF 100V -> 22uF 10V; device CAPACITORS:0603 -> CAPACITORS:1206
- C19: value 100nF 50V -> 22uF 10V; device CAPACITORS:0603 -> CAPACITORS:1206
- C44: value 2.2uF 25V -> 100nF 100V
- C45: value 2.2uF 25V -> 1uF 25V
- C46, C47: value 100nF 16V -> 1uF 25V; device CAPACITORS:0402 -> CAPACITORS:0603
- CN4: value 10/100 RJ45 -> Gb RJ45 + MAG; device CONNECTORs:ARJC02 -> CONNECTORs:0857931020
- U12: value TPS70925 -> Gb PHY; device ICs:SOT23-5 -> ICs:QFN48_7X7
- moved C44 206.2 mm to (57.5, -90.8), turned to 0 degrees
- moved C2 193.5 mm to (-11.9, -86.6)
- moved C3 193.5 mm to (-26.6, -91.4)
- moved C4 193.5 mm to (-23.1, -91.4)
- moved C5 193.5 mm to (-19.6, -91.4)
- moved C6 193.5 mm to (-16.1, -91.4)
- moved L2 193.5 mm to (-21.6, -81.6)
- moved R1 193.5 mm to (-12.6, -91.4)
- moved R19 193.5 mm to (-16.1, -94.6)
- moved R2 193.5 mm to (-9.12, -91.4)
- moved R3 193.5 mm to (-26.6, -94.6)
- moved R4 193.5 mm to (-23.1, -94.6)
- moved R5 193.5 mm to (-19.6, -94.6)
- moved U4 193.5 mm to (-26.4, -81.9)
- moved SCR1 159.7 mm to (-125.2, -154.1)
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Connections:
- removed net PR_VBAT: C44.2, U12.1, U12.3
- removed net USB_IN_N1: U11.1
- removed net USB_IN_P1: U11.3
- removed net USB_N1: U11.6, U9.6
- removed net USB_P1: U11.4, U9.7
- removed net USB_VBUS_SW: C36.1, R14.1, R16.1
- new net 3V3_SLP: C18.2, C19.2, C2.2, CN3.21, CN8.1, L2.1, R39.2, U14.6, U14.7, U3.1, U3.13, U3.19, U3.32, U3.48, U3.64, U4.6
- new net FT232H_USB_DM: U2.K18, U9.6
- new net FT232H_USB_DP: U2.K17, U9.7
- new net MEM_USB_DM: U11.6, U2.J17
- new net MEM_USB_DP: U11.4, U2.J18
- new net MP1_EEPROM_WP: TP1.1, U2.P4
- new net MP1_PMIC_!PONKEYIN: U2.D3
- new net MP1_SOFT_!RESET: R26.1, U2.M3
- new net MP1_UART_RX: U13.1
- new net MP1_UART_TX: U13.4
- new net MP1_USB_VBUS: CN5.1, U11.5, U2.K9
- new net N$19: R29.1, R32.2, U2.J6
- new net N$26: U2.G7, U2.H7, U2.J7, U2.K3, U2.K4, U2.K7, U2.L4, U2.L7, U2.M4, U2.M7
- new net N$29: R28.1, R31.2, U2.H6
- new net N$30: C38.2, D1.K, D5.K, D6.K, U14.3, U14.4
- new net N$31: CN4.11, U12.2
- new net N$33: U13.9, U8.3
- new net N$34: U13.8, U8.1
- new net N$35: U2.J8, U2.J9
- new net N$36: R27.1, R30.2, U2.G6
- new net N$37: U2.G10, U2.G9
- new net N$38: CN5.3, U11.3
- new net N$39: CN5.2, U11.1
- new net N$40: U2.K1, U2.K2
- new net N$41: U2.M1, U2.M2
- new net N$42: CN4.4, U12.5
- new net N$43: CN4.5, U12.6
- new net N$44: R40.2, U3.60
- new net N$45: CN4.3, U12.7
- new net N$46: CN4.2, U12.8
- new net N$47: CN4.8, U12.10
- new net N$48: CN4.9, U12.11
- new net N$50: R44.1, U15.18
- new net N$51: Q2.4, R45.1, R46.2
- new net N$52: R46.1, U15.16
- new net N$53: C45.2, U15.23
- new net N$54: C46.2, U15.21
- new net N$55: C41.2, CN4.7
- new net N$56: C42.2, CN4.1
- new net N$57: C43.2, CN4.6
- new net N$58: C44.2, CN4.12
- new net SD_CLK: CN7.5, R38.1, U2.V17
- new net SD_CMD: CN7.3, R37.1, U2.U18
- new net SD_D0: CN7.7, R36.1, U2.T16
- new net SD_D1: CN7.8, R35.1, U2.U16
- new net SD_D2: CN7.1, R34.1, U2.V16
- new net SD_D3: CN7.2, R33.1, U2.U17
- new net STM32_NRST: CN8.3, R39.1, U3.7
- new net STM_SWCLK: CN8.4, U3.49
- new net STM_SWDIO: CN8.5, U3.46
- new net STUSB_!ALERT: U15.19
- new net STUSB_ATTACH: U15.11
- new net STUSB_GPIO: U15.15
- new net STUSB_ORI: U15.17
- new net STUSB_PD0: U15.20
- new net STUSB_PD1: U15.14
- new net STUSB_RESET: U15.6
- new net STUSB_SCL: U15.7
- new net STUSB_SDA: U15.8
- new net USBC_CC1: CN1.A5, D7.K, U15.1, U15.2
- new net USBC_CC2: CN1.B5, D8.K, U15.4, U15.5
- new net USBC_USB_DM: CN1.A7, CN1.B7, U8.4
- new net USBC_USB_DP: CN1.A6, CN1.B6, U8.6
- new net USBC_VBUS: C47.2, CN1.A4, CN1.A9, CN1.B4, CN1.B9, D5.A, D9.K, Q2.1, Q2.2, Q2.3, R44.2, R45.2, U15.24
- new net VBUS_SWD: C36.1, Q2.5, Q2.6, Q2.7, Q2.8, Q2.PAD, R14.1, R16.1
- net 3V3: now also C39.2, C40.2, CN7.4, R26.2, R27.2, R28.2, R29.2, R33.2, R34.2, R35.2, R36.2, R37.2, R38.2, U13.10, U13.11, U13.12, U13.3, U2.H3, U2.J3; no longer CN3.21
- net 5V: now also U2.G1, U2.G2, U2.G3, U2.H1, U2.H2, U2.H8, U2.H9, U2.L8, U2.L9, U2.M8, U2.M9; no longer C2.2, L2.1, U4.6
- net 5VUSB: no longer C18.2, C19.2, U11.5
- net GND: now also C38.1, C39.1, C40.1, C41.1, C42.1, C43.1, CN1.A1, CN1.A12, CN1.B1, CN1.B12, CN1.P$1, CN1.P$10, CN1.P$11, CN1.P$12, CN1.P$13, CN1.P$14, CN1.P$15, CN1.P$16, CN1.P$17, CN1.P$18, CN1.P$19, CN1.P$2, CN1.P$20, CN1.P$21, CN1.P$22, CN1.P$23, CN1.P$24, CN1.P$25, CN1.P$26, CN1.P$27, CN1.P$28, CN1.P$3, CN1.P$4, CN1.P$5, CN1.P$6, CN1.P$7, CN1.P$8, CN1.P$9, CN4.SH1, CN4.SH2, CN5.4, CN5.SH1, CN5.SH2, CN5.SH3, CN5.SH4, CN8.6, D6.A, D7.A, D8.A, D9.A, R30.1, R31.1, R32.1, R40.1, TP2.1, U12.29, U12.PAD, U13.13, U13.5, U13.6, U14.1, U14.2, U14.PAD, U15.10, U15.12, U15.13, U15.22, U15.TAB, U2.D4, U2.E10, U2.E11, U2.E12, U2.E13, U2.E14, U2.E15, U2.E4, U2.E5, U2.E6, U2.E7, U2.E8, U2.E9, U2.F10, U2.F11, U2.F12, U2.F13, U2.F14, U2.F15, U2.F4, U2.F5, U2.F6, U2.F7, U2.F8, U2.F9, U2.G11, U2.G12, U2.G13, U2.G14, U2.G15, U2.G5, U2.H13, U2.H14, U2.H15, U2.H5, U2.J1, U2.J13, U2.J14, U2.J15, U2.J16, U2.J5, U2.K13, U2.K14, U2.K15, U2.K16, U2.K5, U2.L13, U2.L14, U2.L15, U2.L5, U2.M10, U2.M11, U2.M12, U2.M13, U2.M14, U2.M15, U2.M5, U2.N10, U2.N11, U2.N12, U2.N13, U2.N14, U2.N15, U2.N5, U2.N6, U2.N7, U2.N8, U2.N9, U2.P5, U2.P6, U2.P7, U2.P8, U3.12, U3.18, U3.31, U3.47, U3.63, U8.2; no longer C48.1, C49.1, U12.2
- net N$32: now also CN4.10, U12.3; no longer C45.2, C46.2, C47.2, C48.2, C49.2, U12.5
- net VBAT: now also D1.A
Routing:
- net USBC_USB_DM: track 0.00 -> 15.8 mm, vias 0 -> 3
- net GND: track 126.9 -> 142.4 mm, vias 109 -> 121
- net USBC_CC2: track 0.00 -> 15.3 mm, vias 0 -> 2
- net USBC_CC1: track 0.00 -> 14.4 mm, vias 0 -> 2
- net USBC_USB_DP: track 0.00 -> 13.5 mm, vias 0 -> 2
- net USB_P1: track 9.84 -> 0.00 mm
- net USB_N1: track 9.84 -> 0.00 mm
- net N$52: track 0.00 -> 9.48 mm, vias 0 -> 2
- net USBC_VBUS: track 0.00 -> 7.80 mm
- net 5VUSB: track 10.1 -> 2.50 mm
- net ACT_!IRQ: track 5.69 -> 0.00 mm, vias 1 -> 0
- net N$32: track 5.61 -> 0.00 mm, vias 5 -> 0
- net PR_VBAT: track 5.43 -> 0.00 mm, vias 1 -> 0
- net 3V3: track 29.1 -> 34.5 mm, vias 14 -> 16
- net ACT_SHIPM: track 5.03 -> 0.07 mm, vias 1 -> 0
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- added copper zone on layer 1, net USBC_VBUS
- added copper zone on layer 1, net VBUS_SWD
- removed copper zone on layer 1, net USB_VBUS_SW

Commit message: Thernet PHY added
Parts:
- removed C41, C42, C43, C44: 100nF 100V, CAPACITORS:0603
- removed U12: Gb PHY, ICs:QFN48_7X7
- added C68, C69, C70, C71: 100nF 100V, CAPACITORS:0603
- added C72, C73, C74, C75, C76, C79, C80, C81, C82, C83, C85, C87, C88: 100nF 16V, CAPACITORS:0402
- added C77, C78, C84, C86, C89: 10uF 10V, CAPACITORS:0603
- added C90, C91: 15pF 50V, CAPACITORS:0603
- added FB10, FB11, FB12, FB13, FB9: 600R, INDUCTORS:0603
- added R65, R66: 12k, r_0603:0603
- added R67, R71: NO FIT, r_0603:0603
- added R68, R69: 22R, RESISTORS:1206_ARRAY
- added R70: 4.7k, r_0603:0603
- added R72, R74, R76, R82: 1.0k, r_0603:0603
- added R73, R75, R77, R78, R79, R80, R81: 10k, r_0603:0603
- added R83, R84, R85: NOT FIT, r_0603:0603
- added U16: Gb PHY, ICs:QFN48_7X7
- added XTAL3: 25MHz, CRYSTALS:3.2X2.5SMD
- moved CN3 1.12 mm to (0.00, -45.0)
Connections:
- removed net N$31: CN4.11, U12.2
- removed net N$32: CN4.10, U12.3
- removed net N$42: CN4.4, U12.5
- removed net N$43: CN4.5, U12.6
- removed net N$45: CN4.3, U12.7
- removed net N$46: CN4.2, U12.8
- removed net N$47: CN4.8, U12.10
- removed net N$48: CN4.9, U12.11
- removed net N$55: C41.2, CN4.7
- removed net N$56: C42.2, CN4.1
- removed net N$57: C43.2, CN4.6
- removed net N$58: C44.2, CN4.12
- new net ETH_!INT: R71.1, R72.2, U16.38, U2.A4
- new net ETH_!RST: U16.42
- new net ETH_CLK125_OUT: R75.1, U16.41, U2.C15
- new net ETH_MDC: U16.36, U2.B15
- new net ETH_MDIO: R70.1, U16.37, U2.A15
- new net ETH_RXC: R69.6, R76.2, U2.C16
- new net ETH_RXD0: R68.8, R81.1, R85.2, U2.B12
- new net ETH_RXD1: R68.7, R80.1, R84.2, U2.C12
- new net ETH_RXD2: R68.6, R79.1, R83.2, U2.B5
- new net ETH_RXD3: R68.5, R78.1, R82.2, U2.C5
- new net ETH_RX_CTL: R69.5, R77.1, U2.A12
- new net ETH_TXC: U16.24, U2.B9
- new net ETH_TXD0: U16.19, U2.B7
- new net ETH_TXD1: U16.20, U2.A7
- new net ETH_TXD2: U16.21, U2.C7
- new net ETH_TXD3: U16.22, U2.A6
- new net ETH_TX_CTL: U16.25
- new net N$100: R73.2, U16.17
- new net N$101: R74.2, U16.15
- new net N$74: CN4.11, U16.2
- new net N$75: CN4.10, U16.3
- new net N$76: CN4.4, U16.5
- new net N$77: CN4.5, U16.6
- new net N$78: CN4.3, U16.7
- new net N$79: CN4.2, U16.8
- new net N$80: CN4.8, U16.10
- new net N$81: CN4.9, U16.11
- new net N$82: C68.2, CN4.7
- new net N$83: C69.2, CN4.1
- new net N$84: C70.2, CN4.6
- new net N$85: C71.2, CN4.12
- new net N$86: C74.2, C75.2, C76.2, C78.2, FB9.2, U16.16, U16.34, U16.40
- new net N$87: C72.2, C73.2, C77.2, FB10.2, U16.1, U16.12
- new net N$88: C79.2, C80.2, C81.2, C82.2, C83.2, C84.2, FB13.1, U16.18, U16.23, U16.26, U16.30, U16.39
- new net N$89: C85.2, C86.2, FB12.1, U16.44
- new net N$90: C87.2, C88.2, C89.2, FB11.1, U16.4, U16.9
- new net N$91: R65.2, R66.2, U16.48
- new net N$92: C90.2, R67.2, U16.45, XTAL3.3
- new net N$93: C91.2, R67.1, U16.46, XTAL3.1
- new net N$94: R68.4, U16.27
- new net N$95: R68.3, U16.28
- new net N$96: R68.2, U16.31
- new net N$97: R68.1, U16.32
- new net N$98: R69.4, U16.33
- new net N$99: R69.3, U16.35
- net 1V2: now also FB11.2, FB12.2, FB13.2
- net 3V3: now also FB10.1, FB9.1, R70.2, R71.2, R73.1, R75.2, R77.2, R78.2, R79.2, R80.2, R81.2
- net GND: now also C68.1, C69.1, C70.1, C71.1, C72.1, C73.1, C74.1, C75.1, C76.1, C77.1, C78.1, C79.1, C80.1, C81.1, C82.1, C83.1, C84.1, C85.1, C86.1, C87.1, C88.1, C89.1, C90.1, C91.1, R65.1, R66.1, R72.1, R74.1, R76.1, R82.1, R83.1, R84.1, R85.1, U16.29, U16.PAD; no longer C41.1, C42.1, C43.1, C44.1, U12.29, U12.PAD
Routing:
- net GND: track 142.4 -> 176.0 mm, vias 121 -> 158
- net N$86: track 0.00 -> 31.9 mm, vias 0 -> 5
- net N$88: track 0.00 -> 29.5 mm, vias 0 -> 7
- net ETH_CLK125_OUT: track 0.00 -> 20.7 mm, vias 0 -> 1
- net N$76: track 0.00 -> 19.2 mm, vias 0 -> 1
- net N$77: track 0.00 -> 19.1 mm
- net N$78: track 0.00 -> 18.7 mm
- net N$79: track 0.00 -> 18.6 mm
- net ETH_!RST: track 0.00 -> 18.4 mm
- net ETH_!INT: track 0.00 -> 18.0 mm, vias 0 -> 1
- net N$90: track 0.00 -> 16.6 mm, vias 0 -> 4
- net ETH_TXD0: track 0.00 -> 16.5 mm
- net N$80: track 0.00 -> 16.1 mm
- net ETH_MDIO: track 0.00 -> 16.0 mm, vias 0 -> 1
- net N$81: track 0.00 -> 16.0 mm, vias 0 -> 1
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
Commit message: Progress
Parts:
- removed C9: 100nF 50V, CAPACITORS:0603
- removed FB6: 150R, INDUCTORS:1206
- added C41, C42, C44: 100nF 25V, CAPACITORS:0402@1
- added C43, C55: 4.7uF 6.3V, CAPACITORS:0603
- added C48, C54: 100nF 16V, CAPACITORS:0603
- added C49, C50: 22uF 10V, CAPACITORS:1206
- added C51: 10nF 50V, CAPACITORS:0603
- added C52: 2.2nF 50V, CAPACITORS:0402
- added C53: 1uF 50V, CAPACITORS:1206
- added D2: B360A-13-F, DIODES:DO214AC
- added L3: 22uH 3.7A, INDUCTORS:SRR1260
- added R41, R47: 10k, r_0603:0603
- added R42: 2.0k, r_0603:0603
- added R43: 20k, r_0603:0603
- added U12: TPS54233D, ICs:SO8
- C10, C11, C12, C13, C14, C24, C7, C8: value 100nF 50V -> 100nF 16V
- C36, C37: value 100uF 25V -> 47uF 25V; device CAPACITORS:5MM_RADIAL_2MM_PITCH -> CAPACITORS:1206
- R10: value 2k -> 2.0k; device RESISTORS:0603 -> r_0603:0603
- R11: device RESISTORS:0603 -> r_0603:0603
- R12, R13, R6, R7, R8, R9: value 10K -> 10k; device RESISTORS:0603 -> r_0603:0603
- moved R38 90.2 mm to (-46.1, -29.9), flipped to the bottom
- moved R36 89.4 mm to (-48.4, -29.9), flipped to the bottom
- moved R37 89.2 mm to (-44.1, -29.9), flipped to the bottom
- moved R35 89.0 mm to (-49.6, -29.9), flipped to the bottom
- moved R34 87.9 mm to (-41.6, -29.9), flipped to the bottom
- moved R33 87.9 mm to (-42.9, -29.9), flipped to the bottom
- moved CN7 46.2 mm to (-45.0, -27.5)
- moved C20 9.88 mm to (-28.8, 66.8)
- moved C21 9.88 mm to (-34.0, 63.8)
- moved C22 9.88 mm to (-28.8, 64.4)
- moved C23 9.88 mm to (-23.6, 63.9)
- moved U2 9.35 mm to (-20.0, -30.0), turned to 180 degrees
- moved C37 2.55 mm to (28.0, -11.5)
- moved U1 2.50 mm to (-40.0, 22.5)
- moved U5 2.50 mm to (-32.5, 42.5)
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Connections:
- net SDRAM_!CAS renamed SDRAM0_!CAS
- net SDRAM_!CS renamed SDRAM0_!CS
- net SDRAM_!RAS renamed SDRAM0_!RAS
- net SDRAM_!WE renamed SDRAM0_!WE
- net SDRAM_A0 renamed SDRAM0_A0
- net SDRAM_A1 renamed SDRAM0_A1
- net SDRAM_A10 renamed SDRAM0_A10
- net SDRAM_A11 renamed SDRAM0_A11
- net SDRAM_A12 renamed SDRAM0_A12
- net SDRAM_A2 renamed SDRAM0_A2
- net SDRAM_A3 renamed SDRAM0_A3
- net SDRAM_A4 renamed SDRAM0_A4
- net SDRAM_A5 renamed SDRAM0_A5
- net SDRAM_A6 renamed SDRAM0_A6
- net SDRAM_A7 renamed SDRAM0_A7
- net SDRAM_A8 renamed SDRAM0_A8
- net SDRAM_A9 renamed SDRAM0_A9
- net SDRAM_BA0 renamed SDRAM0_BA0
- net SDRAM_BA1 renamed SDRAM0_BA1
- net SDRAM_CKE renamed SDRAM0_CKE
- net SDRAM_CLK renamed SDRAM0_CLK
- net SDRAM_D0 renamed SDRAM0_D0
- net SDRAM_D1 renamed SDRAM0_D1
- net SDRAM_D10 renamed SDRAM0_D10
- net SDRAM_D11 renamed SDRAM0_D11
- net SDRAM_D12 renamed SDRAM0_D12
- net SDRAM_D13 renamed SDRAM0_D13
- net SDRAM_D14 renamed SDRAM0_D14
- net SDRAM_D15 renamed SDRAM0_D15
- net SDRAM_D2 renamed SDRAM0_D2
- net SDRAM_D3 renamed SDRAM0_D3
- net SDRAM_D4 renamed SDRAM0_D4
- net SDRAM_D5 renamed SDRAM0_D5
- net SDRAM_D6 renamed SDRAM0_D6
- net SDRAM_D7 renamed SDRAM0_D7
- net SDRAM_D8 renamed SDRAM0_D8
- net SDRAM_D9 renamed SDRAM0_D9
- net SDRAM_LDM renamed SDRAM0_LDM
- net SDRAM_UDM renamed SDRAM0_UDM
- new net FT232H_3V3: C14.2, C15.2, C24.2, C7.2, C8.2, FB4.1, FB5.1, R12.2, R13.2, R6.2, R7.2, R8.2, R9.2, U10.6, U10.8, U9.12, U9.24, U9.39, U9.46
- new net N$31: C48.1, U12.1
- new net N$32: C48.2, D2.K, L3.1, U12.8
- new net N$42: R41.1, R42.2, U12.5
- new net N$43: C51.2, U12.4
- new net N$45: C52.1, R43.2
- new net N$46: C52.2, U12.6
- new net RAIL_5V_EN: R47.2, U12.3
- new net SDRAM1_!CAS: U5.F7
- new net SDRAM1_!CS: U5.G9
- new net SDRAM1_!RAS: U5.F8
- new net SDRAM1_!WE: U5.F9
- new net SDRAM1_A0: U5.H7
- new net SDRAM1_A1: U5.H8
- new net SDRAM1_A10: U5.H9
- new net SDRAM1_A11: U5.G2
- new net SDRAM1_A12: U5.G1
- new net SDRAM1_A2: U5.J8
- new net SDRAM1_A3: U5.J7
- new net SDRAM1_A4: U5.J3
- new net SDRAM1_A5: U5.J2
- new net SDRAM1_A6: U5.H3
- new net SDRAM1_A7: U5.H2
- new net SDRAM1_A8: U5.H1
- new net SDRAM1_A9: U5.G3
- new net SDRAM1_BA0: U5.G7
- new net SDRAM1_BA1: U5.G8
- new net SDRAM1_CKE: U5.F3
- new net SDRAM1_CLK: U5.F2
- new net SDRAM1_D0: U5.A8
- new net SDRAM1_D1: U5.B9
- new net SDRAM1_D10: U5.D1
- new net SDRAM1_D11: U5.C2
- new net SDRAM1_D12: U5.C1
- new net SDRAM1_D13: U5.B2
- new net SDRAM1_D14: U5.B1
- new net SDRAM1_D15: U5.A2
- new net SDRAM1_D2: U5.B8
- new net SDRAM1_D3: U5.C9
- new net SDRAM1_D4: U5.C8
- new net SDRAM1_D5: U5.D9
- new net SDRAM1_D6: U5.D8
- new net SDRAM1_D7: U5.E9
- new net SDRAM1_D8: U5.E1
- new net SDRAM1_D9: U5.D2
- new net SDRAM1_LDM: U5.E8
- new net SDRAM1_UDM: U5.F1
- net 3V3: now also C41.2, C42.2, C43.2, C44.2, U5.A7, U5.A9, U5.B3, U5.C7, U5.D3, U5.E7, U5.J9; no longer C14.2, C15.2, C24.2, C7.2, C8.2, C9.2, FB4.1, FB5.1, R12.2, R13.2, R6.2, R7.2, R8.2, R9.2, U10.6, U10.8, U9.12, U9.24, U9.39, U9.40, U9.46
- net 5V: now also C49.2, C50.2, L3.2, R41.2; no longer FB6.2
- net 5VUSB: now also C54.2, C55.2, U2.K9, U9.40; no longer FB6.1
- net GND: now also C36.1, C37.1, C41.1, C42.1, C43.1, C44.1, C49.1, C50.1, C51.1, C53.1, C54.1, C55.1, CN7.6, CN7.MNT1, CN7.MNT2, CN7.MNT3, CN7.MNT4, D2.A, R42.1, R43.1, R47.1, U12.7, U5.A1, U5.A3, U5.B7, U5.C3, U5.D7, U5.E3, U5.J1; no longer C36.2, C37.2, C9.1
- net MP1_USB_VBUS: no longer U2.K9
- net VBAT: now also C37.2, C53.2, U12.2; no longer C37.1
- net VBUS_SWD: now also C36.2; no longer C36.1
Routing:
- net MEM_USB_DP: track 0.00 -> 62.2 mm
- net MEM_USB_DM: track 0.00 -> 62.2 mm
- net GND: track 176.0 -> 236.8 mm, vias 158 -> 245
- net 2V5: track 55.2 -> 2.83 mm
- net SD_D1: track 0.00 -> 30.3 mm, vias 0 -> 2
- net SD_D0: track 0.00 -> 29.4 mm, vias 0 -> 4
- net SD_CMD: track 0.00 -> 26.1 mm, vias 0 -> 2
- net SD_CLK: track 0.00 -> 26.0 mm, vias 0 -> 2
- net SD_D3: track 0.00 -> 24.5 mm, vias 0 -> 2
- net FT232H_3V3: track 0.00 -> 23.2 mm, vias 0 -> 12
- net SD_D2: track 0.00 -> 20.6 mm, vias 0 -> 2
- net 3V3: track 46.0 -> 29.0 mm, vias 25 -> 23
- net ETH_RXC: track 6.25 -> 16.4 mm, vias 1 -> 2
- net ETH_RXD3: track 6.92 -> 16.8 mm, vias 1 -> 2
- net ETH_TXD2: track 15.2 -> 24.9 mm, vias 0 -> 1
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- added copper zone on layer 16, net VBAT
Other:
- board size 110 x 110 mm -> 113.6 x 110 mm

Commit message: Blocks are forming
Parts:
- removed MECH4, MECH5, MECH6: 6mm x 3mm, MISC:MOUNTHOLE_6X3
- removed SCR1: 128x64 White OLED, MISC:DEP_128064S
- R39, R40: device r_0402:0402 -> r_0603:0603
- moved R39 138.7 mm to (-58.6, 39.6)
- moved C53 131.8 mm to (-28.2, 42.8), flipped to the bottom, turned to 180 degrees
- moved C50 130.6 mm to (-22.5, 57.0), flipped to the bottom, turned to 180 degrees
- moved R40 126.3 mm to (-9.00, 34.4)
- moved C49 125.3 mm to (-22.5, 54.6), flipped to the bottom, turned to 180 degrees
- moved R43 121.5 mm to (-41.6, 41.5), flipped to the bottom, turned to 180 degrees
- moved C52 119.9 mm to (-39.1, 41.5), flipped to the bottom, turned to 180 degrees
- moved C51 118.5 mm to (-31.5, 38.2), flipped to the bottom, turned to 90 degrees
- moved C18 117.8 mm to (19.0, 35.2), turned to 180 degrees
- moved C19 115.8 mm to (19.0, 33.0), turned to 180 degrees
- moved R42 113.8 mm to (-36.6, 39.0), flipped to the bottom
- moved D6 113.5 mm to (22.2, 27.4), turned to 270 degrees
- moved D1 113.3 mm to (18.8, 21.6), turned to 90 degrees
- moved R47 110.1 mm to (-29.1, 41.1), flipped to the bottom
- moved R41 109.9 mm to (-36.6, 37.8), flipped to the bottom, turned to 180 degrees
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Connections:
- net 3V3: no longer C4.2
- net 3V3_SLP: now also C4.2
Routing:
- net MEM_USB_DM: track 62.2 -> 4.25 mm
- net MEM_USB_DP: track 62.2 -> 6.96 mm
- net GND: track 236.8 -> 276.8 mm, vias 245 -> 280
- net 5V: track 7.78 -> 39.7 mm, vias 11 -> 16
- net SD_D1: track 30.3 -> 3.38 mm
- net SD_D0: track 29.4 -> 3.38 mm, vias 4 -> 2
- net SD_CMD: track 26.1 -> 2.68 mm, vias 2 -> 1
- net SD_CLK: track 26.0 -> 2.66 mm, vias 2 -> 1
- net SD_D3: track 24.5 -> 3.34 mm
- net SD_D2: track 20.6 -> 2.70 mm, vias 2 -> 1
- net USBC_USB_DM: track 15.8 -> 2.91 mm, vias 3 -> 1
- net N$32: track 0.00 -> 12.7 mm
- net VDISP: track 0.00 -> 12.6 mm, vias 0 -> 2
- net USBC_CC2: track 15.3 -> 2.65 mm, vias 2 -> 0
- net RAIL_5V_EN: track 0.00 -> 12.5 mm
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- removed copper zone on layer 16, net VBAT
Other:
- board size 113.6 x 110 mm -> 133 x 133 mm

Commit message: Pushed to fusion
Parts:
- moved R26 35.5 mm to (-18.9, -63.5), turned to 270 degrees
- moved C23 6.99 mm to (-56.4, 14.6)
- moved C42 4.07 mm to (-59.8, -20.1)
- moved C41 3.81 mm to (-60.8, -18.0)
- moved C21 2.75 mm to (-59.9, 21.3)
- moved C22 1.19 mm to (-56.5, 21.3)
Other:
- outline, holes or cut-outs redrawn
