File: camera_main_sch_brd.sch (EAGLE design)
At the start: 98 parts, among them CN1 USB C CON, CN2 50 PIN 0.5MM, CN3 31 PIN FPC, CN4 10/100 RJ45, CN5 USB A, CN6 NO FIT, U1 10CL016YF484C6G, U10 93LC56B-I/SN, U11 USBLC6-2SC6, U12 TPS70925, U2 OSD32MP157C-512M-BAA, U3 STM32L431RBT, U4 TLV61046A, U5 AS4C32M16SA, U6 AS4C32M16SA, U7 ACT2861, U9 FT232H

Commit message: Progress, new names
Parts:
- removed C48, C49: 100nF 16V, CAPACITORS:CL05B104KO5NNNC
- added C38: 10uF 50V, CAPACITORS:C3225X7S1H106M250AB
- added C39, C40: 100nF 16V, CAPACITORS:CL10B104KO8WPNC
- added C41, C42, C43: 100nF 100V, CAPACITORS:06031C104KAT2A
- added CN7: uSD, CONNECTORs:114-00841-68
- added CN8: NO FIT, CONNECTORs:TSM-103-03-T-DV
- added D1, D5, D6: B0540W, DIODES:B0540W
- added D7, D8: PESD5Z5.0, DIODES:PESD5Z5.0
- added D9: 20V TVS, DIODES:SMAJ20CA-E3/61
- added Q2: SI7489DP, TRANSISTORs:SI7489DP-T1-E3
- added R26, R33, R34, R35, R36, R37, R38: 10k, r_0603:ERJ3EKF1002V
- added R27, R28, R29, R30, R31, R32: 10R, r_0603:ERJ3EKF10R0V
- added R39, R40: 10k, r_0402:ERJ-2RKF1002X
- added R44: 1.0k, r_0603:ERJ3EKF1001V
- added R45: 100k, r_0603:ERJ3EKF1003V
- added R46: 22k, r_0603:ERJ3EKF2202V
- added TP1, TP2: 2MM_TEST_POINT, MISC:2MM_TEST_POINT
- added U13: FT230X, ICs:FT230XS
- added U14: 3.3V BUCK, ICs:LMZM23600V3SILT
- added U15: STUSB4500, ICs:STUSB4500
- added U8: USBLC6-2SC6, ICs:USBLC6-2SC6
- C18: value 10pF 100V -> 22uF 10V; device CAPACITORS:06031A100FAT2A -> CAPACITORS:CL31B226MPHNNNE
- C19: value 100nF 50V -> 22uF 10V; device CAPACITORS:VJ0603Y104KXACW1BC -> CAPACITORS:CL31B226MPHNNNE
- C44: value 2.2uF 25V -> 100nF 100V; device CAPACITORS:GRM188R61E225KA12D -> CAPACITORS:06031C104KAT2A
- C45: value 2.2uF 25V -> 1uF 25V; device CAPACITORS:GRM188R61E225KA12D -> CAPACITORS:CL10A105KA8NNNC
- C46, C47: value 100nF 16V -> 1uF 25V; device CAPACITORS:CL05B104KO5NNNC -> CAPACITORS:CL10A105KA8NNNC
- CN4: value 10/100 RJ45 -> Gb RJ45 + MAG; device CONNECTORs:ARJC02-111008B -> CONNECTORs:0857931020
- U12: value TPS70925 -> Gb PHY; device ICs:TPS70925DBVR -> ICs:KSZ9131RNX
Connections:
- removed net PR_VBAT: C44.2, U12.EN, U12.VIN
- removed net USB_IN_N1: U11.D+_IN
- removed net USB_IN_P1: U11.D-_IN
- removed net USB_N1: U11.D+_OUT, U9.D-
- removed net USB_P1: U11.D-OUT, U9.D+
- removed net USB_VBUS_SW: C36.A, R14.1, R16.1
- new net 3V3_SLP: C18.2, C19.2, C2.2, CN3.21, CN8.1, L2.1, R39.2, U14.FB, U14.VOUT, U3.VBAT, U3.VDD, U3.VDDA, U4.VIN
- new net FT232H_USB_DM: U2D.USB_DM1, U9.D-
- new net FT232H_USB_DP: U2D.USB_DP1, U9.D+
- new net MEM_USB_DM: U11.D+_OUT, U2D.USB_DM2
- new net MEM_USB_DP: U11.D-OUT, U2D.USB_DP2
- new net MP1_EEPROM_WP: TP1.P$1, U2A.EEPROM_WP
- new net MP1_PMIC_!PONKEYIN: U2A.PMIC_PONKEYN
- new net MP1_SOFT_!RESET: R26.1, U2A.NRST
- new net MP1_UART_RX: U13.TXD
- new net MP1_UART_TX: U13.RXD
- new net MP1_USB_VBUS: CN5.VBUS, U11.VBUS, U2D.OTG_VBUS
- new net N$19: R29.1, R32.2, U2A.BOOT0
- new net N$26: U2A.VBAT, U2A.VDD@1, U2A.VDD@2, U2A.VDD@3, U2A.VDD@4, U2A.VDD@5, U2A.VDD@6, U2A.VDD@7, U2A.VDD@8, U2A.VDD@9
- new net N$29: R28.1, R31.2, U2A.BOOT1
- new net N$30: C38.2, D1.K, D5.K, D6.K, U14.EN, U14.VIN
- new net N$31: CN4.TD0+, U12.TXRXP_A
- new net N$33: U13.D-, U8.D-_IN
- new net N$34: U13.D+, U8.D+_IN
- new net N$35: U2A.PMIC_BSTOUT@1, U2A.PMIC_BSTOUT@2
- new net N$36: R27.1, R30.2, U2A.BOOT2
- new net N$37: U2A.PMIC_SWOUT@1, U2A.PMIC_SWOUT@2
- new net N$38: CN5.D+, U11.D-_IN
- new net N$39: CN5.D-, U11.D+_IN
- new net N$40: U2D.VREF-, U2D.VSSA
- new net N$41: U2D.VDDA, U2D.VREF+
- new net N$42: CN4.TD1+, U12.TXRXP_B
- new net N$43: CN4.TD1-, U12.TXRXM_B
- new net N$44: R40.2, U3.PH3-BOOT0
- new net N$45: CN4.TD2+, U12.TXRXP_C
- new net N$46: CN4.TD2-, U12.TXRXM_C
- new net N$47: CN4.TD3+, U12.TXRXP_D
- new net N$48: CN4.TD3-, U12.TXRXM_D
- new net N$50: R44.1, U15.VBUS_VS_DISCH
- new net N$51: Q2.G, R45.1, R46.2
- new net N$52: R46.1, U15.VBUS_EN_SNK
- new net N$53: C45.2, U15.VREG_2V7
- new net N$54: C46.2, U15.VREG_1V2
- new net N$55: C41.2, CN4.CT3
- new net N$56: C42.2, CN4.CT2
- new net N$57: C43.2, CN4.CT1
- new net N$58: C44.2, CN4.CT0
- new net SD_CLK: CN7.CLK, R38.1, U2B.PC12
- new net SD_CMD: CN7.C/R, R37.1, U2B.PD2
- new net SD_D0: CN7.D0, R36.1, U2B.PC8
- new net SD_D1: CN7.D1, R35.1, U2B.PC9
- new net SD_D2: CN7.D2, R34.1, U2B.PC10
- new net SD_D3: CN7.D3, R33.1, U2B.PC11
- new net STM32_NRST: CN8.3, R39.1, U3.NRST
- new net STM_SWCLK: CN8.4, U3.PA14
- new net STM_SWDIO: CN8.5, U3.PA13
- new net STUSB_!ALERT: U15.!ALERT
- new net STUSB_ATTACH: U15.ATTACH
- new net STUSB_GPIO: U15.GPIO
- new net STUSB_ORI: U15.A_B_SIDE
- new net STUSB_PD0: U15.POWER_OK2
- new net STUSB_PD1: U15.POWER_OK3
- new net STUSB_RESET: U15.RESET
- new net STUSB_SCL: U15.SCL
- new net STUSB_SDA: U15.SDA
- new net USBC_CC1: CN1.CC1, D7.K, U15.CC1, U15.CC1DB
- new net USBC_CC2: CN1.CC2, D8.K, U15.CC2, U15.CC2DB
- new net USBC_USB_DM: CN1.D-, U8.D-OUT
- new net USBC_USB_DP: CN1.D+, U8.D+_OUT
- new net USBC_VBUS: C47.2, CN1.VBUS, D5.A, D9.A1, Q2.S, R44.2, R45.2, U15.VDD
- new net VBUS_SWD: C36.A, Q2.D, R14.1, R16.1
- net 3V3: now also C39.2, C40.2, CN7.VCC, R26.2, R27.2, R28.2, R29.2, R33.2, R34.2, R35.2, R36.2, R37.2, R38.2, U13.!RESET, U13.3V3OUT, U13.VCC, U13.VCCIO, U2A.PMIC_VOUT4@1, U2A.PMIC_VOUT4@2; no longer CN3.21
- net 5V: now also U2A.PMIC_BSTIN@1, U2A.PMIC_BSTIN@2, U2A.PMIC_BSTIN@3, U2A.PMIC_BSTIN@4, U2A.PMIC_LDO25IN, U2A.PMIC_SWIN@1, U2A.PMIC_SWIN@2, U2A.VIN@1, U2A.VIN@2, U2A.VIN@3, U2A.VIN@4; no longer C2.2, L2.1, U4.VIN
- net 5VUSB: no longer C18.2, C19.2, U11.VBUS
- net GND: now also C38.1, C39.1, C40.1, C41.1, C42.1, C43.1, CN1.GND, CN1.SHELL, CN4.SHLD, CN5.GND, CN8.6, D6.A, D7.A, D8.A, D9.A, R30.1, R31.1, R32.1, R40.1, TP2.P$1, U12.VSS, U13.!CTS, U13.GND, U14.GND, U14.MODE/SYNC, U15.ADDR0, U15.ADDR1, U15.GND, U15.VSYS, U2A.BYPASS_REG1V8, U2A.HSE_OSC_OE, U2E.VSS@1, U2E.VSS@10, U2E.VSS@11, U2E.VSS@12, U2E.VSS@13, U2E.VSS@14, U2E.VSS@15, U2E.VSS@16, U2E.VSS@17, U2E.VSS@18, U2E.VSS@19, U2E.VSS@2, U2E.VSS@20, U2E.VSS@21, U2E.VSS@22, U2E.VSS@23, U2E.VSS@24, U2E.VSS@25, U2E.VSS@26, U2E.VSS@27, U2E.VSS@28, U2E.VSS@29, U2E.VSS@3, U2E.VSS@30, U2E.VSS@31, U2E.VSS@32, U2E.VSS@33, U2E.VSS@34, U2E.VSS@35, U2E.VSS@36, U2E.VSS@37, U2E.VSS@38, U2E.VSS@39, U2E.VSS@4, U2E.VSS@40, U2E.VSS@41, U2E.VSS@42, U2E.VSS@43, U2E.VSS@44, U2E.VSS@45, U2E.VSS@46, U2E.VSS@47, U2E.VSS@48, U2E.VSS@49, U2E.VSS@5, U2E.VSS@50, U2E.VSS@51, U2E.VSS@52, U2E.VSS@53, U2E.VSS@54, U2E.VSS@55, U2E.VSS@56, U2E.VSS@57, U2E.VSS@58, U2E.VSS@59, U2E.VSS@6, U2E.VSS@60, U2E.VSS@61, U2E.VSS@62, U2E.VSS@63, U2E.VSS@64, U2E.VSS@65, U2E.VSS@66, U2E.VSS@67, U2E.VSS@68, U2E.VSS@69, U2E.VSS@7, U2E.VSS@70, U2E.VSS@8, U2E.VSS@9, U3.VSS, U3.VSSA, U8.GND; no longer C48.1, C49.1
- net N$32: now also CN4.TD0-, U12.TXRXM_A; no longer C45.2, C46.2, C47.2, C48.2, C49.2, U12.VOUT
- net VBAT: now also D1.A
Other:
- moved on the sheet: C1, C2, C25, C26, C27, C28, C29, C3, C30, C31, C32, C33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

Commit message: Thernet PHY added
Parts:
- removed C41, C42, C43, C44: 100nF 100V, CAPACITORS:06031C104KAT2A
- removed U12: Gb PHY, ICs:KSZ9131RNX
- added C68, C69, C70, C71: 100nF 100V, CAPACITORS:06031C104KAT2A
- added C72, C73, C74, C75, C76, C79, C80, C81, C82, C83, C85, C87, C88: 100nF 16V, CAPACITORS:CL05B104KO5NNNC
- added C77, C78, C84, C86, C89: 10uF 10V, CAPACITORS:GRM188R61A106KE69D
- added C90, C91: 15pF 50V, CAPACITORS:06035A150JAT2A
- added FB10, FB11, FB12, FB13, FB9: 600R, INDUCTORS:742792651
- added R65, R66: 12k, r_0603:ERJ3EKF1202V
- added R67: NO FIT, r_0603:ERJ3EKF1004V
- added R68, R69: 22R, RESISTORS:EXB-38V220JV
- added R70: 4.7k, r_0603:ERJ3EKF4701V
- added R71: NO FIT, r_0603:ERJ3EKF1001V
- added R72, R74, R76, R82: 1.0k, r_0603:ERJ3EKF1001V
- added R73, R75, R77, R78, R79, R80, R81: 10k, r_0603:ERJ3EKF1002V
- added R83, R84, R85: NOT FIT, r_0603:ERJ3EKF1001V
- added U16: Gb PHY, ICs:KSZ9131RNX
- added XTAL3: 25MHz, CRYSTALS:TSX-322525.0000MF10P-C0
Connections:
- removed net N$31: CN4.TD0+, U12.TXRXP_A
- removed net N$32: CN4.TD0-, U12.TXRXM_A
- removed net N$42: CN4.TD1+, U12.TXRXP_B
- removed net N$43: CN4.TD1-, U12.TXRXM_B
- removed net N$45: CN4.TD2+, U12.TXRXP_C
- removed net N$46: CN4.TD2-, U12.TXRXM_C
- removed net N$47: CN4.TD3+, U12.TXRXP_D
- removed net N$48: CN4.TD3-, U12.TXRXM_D
- removed net N$55: C41.2, CN4.CT3
- removed net N$56: C42.2, CN4.CT2
- removed net N$57: C43.2, CN4.CT1
- removed net N$58: C44.2, CN4.CT0
- new net ETH_!INT: R71.1, R72.2, U16.INT_N/PME_N2/ALLPHYAD, U2C.PG12
- new net ETH_!RST: U16.!RST
- new net ETH_CLK125_OUT: R75.1, U16.CLK125_NDO/LED_MODE, U2C.PG5
- new net ETH_MDC: U16.MDC, U2B.PC1
- new net ETH_MDIO: R70.1, U16.MDIO, U2B.PA2
- new net ETH_RXC: R69.6, R76.2, U2B.PA1
- new net ETH_RXD0: R68.8, R81.1, R85.2, U2B.PC4
- new net ETH_RXD1: R68.7, R80.1, R84.2, U2B.PC5
- new net ETH_RXD2: R68.6, R79.1, R83.2, U2C.PH6
- new net ETH_RXD3: R68.5, R78.1, R82.2, U2C.PH7
- new net ETH_RX_CTL: R69.5, R77.1, U2B.PA7
- new net ETH_TXC: U16.TXC, U2C.PG4
- new net ETH_TXD0: U16.TXD0, U2C.PG13
- new net ETH_TXD1: U16.TXD1, U2C.PG14
- new net ETH_TXD2: U16.TXD2, U2B.PC2
- new net ETH_TXD3: U16.TXD3, U2C.PE2
- new net ETH_TX_CTL: U16.TX_CTL
- new net N$100: R73.2, U16.LED1/PME_N1/PHYAD0
- new net N$101: R74.2, U16.LED2/PHYAD1
- new net N$74: CN4.TD0+, U16.TXRXP_A
- new net N$75: CN4.TD0-, U16.TXRXM_A
- new net N$76: CN4.TD1+, U16.TXRXP_B
- new net N$77: CN4.TD1-, U16.TXRXM_B
- new net N$78: CN4.TD2+, U16.TXRXP_C
- new net N$79: CN4.TD2-, U16.TXRXM_C
- new net N$80: CN4.TD3+, U16.TXRXP_D
- new net N$81: CN4.TD3-, U16.TXRXM_D
- new net N$82: C68.2, CN4.CT3
- new net N$83: C69.2, CN4.CT2
- new net N$84: C70.2, CN4.CT1
- new net N$85: C71.2, CN4.CT0
- new net N$86: C74.2, C75.2, C76.2, C78.2, FB9.2, U16.DVDDH
- new net N$87: C72.2, C73.2, C77.2, FB10.2, U16.AVDDH
- new net N$88: C79.2, C80.2, C81.2, C82.2, C83.2, C84.2, FB13.1, U16.DVDDL
- new net N$89: C85.2, C86.2, FB12.1, U16.AVDDL_PLL
- new net N$90: C87.2, C88.2, C89.2, FB11.1, U16.AVDDL
- new net N$91: R65.2, R66.2, U16.ISET
- new net N$92: C90.2, R67.2, U16.XO, XTAL3.P$2
- new net N$93: C91.2, R67.1, U16.XI, XTAL3.P$1
- new net N$94: R68.4, U16.RXD3/MODE3
- new net N$95: R68.3, U16.RXD2/MODE2
- new net N$96: R68.2, U16.RXD1/MODE1
- new net N$97: R68.1, U16.RXD0/MODE0
- new net N$98: R69.4, U16.RX_CTL/CLK125_EN
- new net N$99: R69.3, U16.RXC/PHYAD2
- net 1V2: now also FB11.2, FB12.2, FB13.2
- net 3V3: now also FB10.1, FB9.1, R70.2, R71.2, R73.1, R75.2, R77.2, R78.2, R79.2, R80.2, R81.2
- net GND: now also C68.1, C69.1, C70.1, C71.1, C72.1, C73.1, C74.1, C75.1, C76.1, C77.1, C78.1, C79.1, C80.1, C81.1, C82.1, C83.1, C84.1, C85.1, C86.1, C87.1, C88.1, C89.1, C90.1, C91.1, R65.1, R66.1, R72.1, R74.1, R76.1, R82.1, R83.1, R84.1, R85.1, U16.GND, U16.VSS; no longer C41.1, C42.1, C43.1, C44.1, U12.GND, U12.VSS

Commit message: Progress
Parts:
- removed C9: 100nF 50V, CAPACITORS:VJ0603Y104KXACW1BC
- removed FB6: 150R, INDUCTORS:LI1206H151R-10
- added C41, C42, C44: 100nF 25V, CAPACITORS:MC0402B104K250CT
- added C43, C55: 4.7uF 6.3V, CAPACITORS:GRM188R60J475ME19D
- added C48, C54: 100nF 16V, CAPACITORS:CL10B104KO8WPNC
- added C49, C50: 22uF 10V, CAPACITORS:CL31B226MPHNNNE
- added C51: 10nF 50V, CAPACITORS:CL10B103KB8NCNC
- added C52: 2.2nF 50V, CAPACITORS:GCM155R71H222KA37D
- added C53: 1uF 50V, CAPACITORS:CL31B105KBHNNNE
- added D2: B360A-13-F, DIODES:B360A-13-F
- added L3: 22uH 3.7A, INDUCTORS:SRR1260-220M
- added R41, R47: 10k, r_0603:ERJ3EKF1002V
- added R42: 2.0k, r_0603:ERJ3EKF2001V
- added R43: 20k, r_0603:ERJ3EKF2002V
- added U12: TPS54233D, ICs:TPS54233D
- C10, C11, C12, C13, C14, C24, C7, C8: value 100nF 50V -> 100nF 16V; device CAPACITORS:VJ0603Y104KXACW1BC -> CAPACITORS:CL10B104KO8WPNC; FARNELL 2407338 -> (none)
- C36, C37: value 100uF 25V -> 47uF 25V; device CAPACITORS:UVY1E101MDD -> CAPACITORS:C3216X5R1E476M160AC
- R10: value 2k -> 2.0k; device RESISTORS:CRCW06032K00FKEA -> r_0603:ERJ3EKF2001V
- R11: device RESISTORS:CRCW060312K0FKEA -> r_0603:ERJ3EKF1202V
- R12, R13, R6, R7, R8, R9: value 10K -> 10k; device RESISTORS:CRCW060310K0FKEA -> r_0603:ERJ3EKF1002V
Connections:
- net SDRAM_!CAS renamed SDRAM0_!CAS
- net SDRAM_!CS renamed SDRAM0_!CS
- net SDRAM_!RAS renamed SDRAM0_!RAS
- net SDRAM_!WE renamed SDRAM0_!WE
- net SDRAM_A0 renamed SDRAM0_A0
- net SDRAM_A1 renamed SDRAM0_A1
- net SDRAM_A10 renamed SDRAM0_A10
- net SDRAM_A11 renamed SDRAM0_A11
- net SDRAM_A12 renamed SDRAM0_A12
- net SDRAM_A2 renamed SDRAM0_A2
- net SDRAM_A3 renamed SDRAM0_A3
- net SDRAM_A4 renamed SDRAM0_A4
- net SDRAM_A5 renamed SDRAM0_A5
- net SDRAM_A6 renamed SDRAM0_A6
- net SDRAM_A7 renamed SDRAM0_A7
- net SDRAM_A8 renamed SDRAM0_A8
- net SDRAM_A9 renamed SDRAM0_A9
- net SDRAM_BA0 renamed SDRAM0_BA0
- net SDRAM_BA1 renamed SDRAM0_BA1
- net SDRAM_CKE renamed SDRAM0_CKE
- net SDRAM_CLK renamed SDRAM0_CLK
- net SDRAM_D0 renamed SDRAM0_D0
- net SDRAM_D1 renamed SDRAM0_D1
- net SDRAM_D10 renamed SDRAM0_D10
- net SDRAM_D11 renamed SDRAM0_D11
- net SDRAM_D12 renamed SDRAM0_D12
- net SDRAM_D13 renamed SDRAM0_D13
- net SDRAM_D14 renamed SDRAM0_D14
- net SDRAM_D15 renamed SDRAM0_D15
- net SDRAM_D2 renamed SDRAM0_D2
- net SDRAM_D3 renamed SDRAM0_D3
- net SDRAM_D4 renamed SDRAM0_D4
- net SDRAM_D5 renamed SDRAM0_D5
- net SDRAM_D6 renamed SDRAM0_D6
- net SDRAM_D7 renamed SDRAM0_D7
- net SDRAM_D8 renamed SDRAM0_D8
- net SDRAM_D9 renamed SDRAM0_D9
- net SDRAM_LDM renamed SDRAM0_LDM
- net SDRAM_UDM renamed SDRAM0_UDM
- new net FT232H_3V3: C14.2, C15.2, C24.2, C7.2, C8.2, FB4.1, FB5.1, R12.2, R13.2, R6.2, R7.2, R8.2, R9.2, U10.ORG, U10.V+, U9.VCCD, U9.VCCIO
- new net N$31: C48.1, U12.BOOT
- new net N$32: C48.2, D2.K, L3.1, U12.PH
- new net N$42: R41.1, R42.2, U12.VSNS
- new net N$43: C51.2, U12.SS
- new net N$45: C52.1, R43.2
- new net N$46: C52.2, U12.COMP
- new net RAIL_5V_EN: R47.2, U12.EN
- new net SDRAM1_!CAS: U5.!CAS
- new net SDRAM1_!CS: U5.!CS
- new net SDRAM1_!RAS: U5.!RAS
- new net SDRAM1_!WE: U5.!WE
- new net SDRAM1_A0: U5.A0
- new net SDRAM1_A1: U5.A1
- new net SDRAM1_A10: U5.A10
- new net SDRAM1_A11: U5.A11
- new net SDRAM1_A12: U5.A12
- new net SDRAM1_A2: U5.A2
- new net SDRAM1_A3: U5.A3
- new net SDRAM1_A4: U5.A4
- new net SDRAM1_A5: U5.A5
- new net SDRAM1_A6: U5.A6
- new net SDRAM1_A7: U5.A7
- new net SDRAM1_A8: U5.A8
- new net SDRAM1_A9: U5.A9
- new net SDRAM1_BA0: U5.BA0
- new net SDRAM1_BA1: U5.BA1
- new net SDRAM1_CKE: U5.CKE
- new net SDRAM1_CLK: U5.CLK
- new net SDRAM1_D0: U5.D0
- new net SDRAM1_D1: U5.D1
- new net SDRAM1_D10: U5.D10
- new net SDRAM1_D11: U5.D11
- new net SDRAM1_D12: U5.D12
- new net SDRAM1_D13: U5.D13
- new net SDRAM1_D14: U5.D14
- new net SDRAM1_D15: U5.D15
- new net SDRAM1_D2: U5.D2
- new net SDRAM1_D3: U5.D3
- new net SDRAM1_D4: U5.D4
- new net SDRAM1_D5: U5.D5
- new net SDRAM1_D6: U5.D6
- new net SDRAM1_D7: U5.D7
- new net SDRAM1_D8: U5.D8
- new net SDRAM1_D9: U5.D9
- new net SDRAM1_LDM: U5.LDM
- new net SDRAM1_UDM: U5.UDM
- net 3V3: now also C41.2, C42.2, C43.2, C44.2, U5.VCC, U5.VCCQ; no longer C14.2, C15.2, C24.2, C7.2, C8.2, C9.2, FB4.1, FB5.1, R12.2, R13.2, R6.2, R7.2, R8.2, R9.2, U10.ORG, U10.V+, U9.VCCD, U9.VCCIO, U9.VREGIN
- net 5V: now also C49.2, C50.2, L3.2, R41.2; no longer FB6.2
- net 5VUSB: now also C54.2, C55.2, U2D.OTG_VBUS, U9.VREGIN; no longer FB6.1
- net GND: now also C36.1, C37.1, C41.1, C42.1, C43.1, C44.1, C49.1, C50.1, C51.1, C53.1, C54.1, C55.1, CN7.GND, D2.A, R42.1, R43.1, R47.1, U12.GND, U5.VSS, U5.VSSQ; no longer C36.K, C37.K, C9.1
- net MP1_USB_VBUS: no longer U2D.OTG_VBUS
- net VBAT: now also C37.2, C53.2, U12.VIN; no longer C37.A
- net VBUS_SWD: now also C36.2; no longer C36.A
Other:
- moved on the sheet: C18, C19, C24, C38, C7, C8, CN8, D1, D5, D6, R39, R40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

Commit message: Blocks are forming
Parts:
- removed MECH4, MECH5, MECH6: 6mm x 3mm, MISC:MOUNTHOLE
- removed SCR1: 128x64 White OLED, MISC:DEP_128064S-W
- R39, R40: device r_0402:ERJ-2RKF1002X -> r_0603:ERJ3EKF1002V
Connections:
- net 3V3: no longer C4.2
- net 3V3_SLP: now also C4.2
Changed lines of the file:
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@@
 <?xml version="1.0" encoding="utf-8"?>
 <!DOCTYPE eagle SYSTEM "eagle.dtd">
-<eagle version="9.6.1">
+<eagle version="9.6.2">
 <drawing>
 <settings>
@@
 <part name="U$10" library="NETS" deviceset="1V2" device=""/>
 <part name="U$34" library="NETS" deviceset="2V5" device=""/>
-<part name="SCR1" library="MISC" deviceset="DEP_128064S" device="-W" value="128x64 White OLED"/>
 <part name="CN3" library="CONNECTORs" deviceset="3-1734839-1" device="" value="31 PIN FPC"/>
 <part name="U4" library="ICs" deviceset="TLV61046A" device="DBVR" value="TLV61046A"/>
@@
 <part name="R3" library="r_0603" deviceset="ERJ3EKF1003V" device="" value="100k"/>
 <part name="GND7" library="NETS" deviceset="GND" device=""/>
-<part name="U$12" library="NETS" deviceset="3V3" device=""/>
 <part name="GND9" library="NETS" deviceset="GND" device=""/>
 <part name="C4" library="CAPACITORS" deviceset="GRM188R61E225KA12D" device="" value="2.2uF 25V"/>
@@
 <part name="MECH2" library="MISC" deviceset="MOUNTHOLE" device="" value="6mm x 3mm"/>
 <part name="MECH3" library="MISC" deviceset="MOUNTHOLE" device="" value="6mm x 3mm"/>
-<part name="MECH4" library="MISC" deviceset="MOUNTHOLE" device="" value="6mm x 3mm"/>
-<part name="MECH5" library="MISC" deviceset="MOUNTHOLE" device="" value="6mm x 3mm"/>
-<part name="MECH6" library="MISC" deviceset="MOUNTHOLE" device="" value="6mm x 3mm"/>
 <part name="U2" library="Octavo-Systems OSD32MP1" deviceset="OSD32MP157C-512M-BAA" device=""/>
 <part name="CN1" library="CONNECTORs" deviceset="12401832E402A" device="" value="USB C CON"/>
@@
 <part name="U$49" library="NETS" deviceset="3V3" device=""/>
 <part name="U$50" library="NETS" deviceset="3V3" device=""/>
-<part name="R39" library="r_0402" deviceset="ERJ-2RKF1002X" device="" value="10k"/>
+<part name="R39" library="r_0603" deviceset="ERJ3EKF1002V" device="" value="10k"/>
 <part name="CN8" library="CONNECTORs" deviceset="TSM-103-03-T-DV" device="" value="NO FIT"/>
 <part name="GND37" library="NETS" deviceset="GND" device=""/>
@@
 <part name="GND71" library="NETS" deviceset="GND" device=""/>
 <part name="GND72" library="NETS" deviceset="GND" device=""/>
-<part name="R40" library="r_0402" deviceset="ERJ-2RKF1002X" device="" value="10k"/>
+<part name="R40" library="r_0603" deviceset="ERJ3EKF1002V" device="" value="10k"/>
 <part name="GND73" library="NETS" deviceset="GND" device=""/>
 <part name="D1" library="DIODES" deviceset="B0540W" device="" value="B0540W"/>
@@
 </plain>
 <instances>
-<instance part="SCR1" gate="G$1" x="182.88" y="104.14" smashed="yes">
-<attribute name="NAME" x="167.64" y="116.84" size="1.778" layer="95"/>
-<attribute name="VALUE" x="167.64" y="114.3" size="1.778" layer="97"/>
-</instance>
 <instance part="CN3" gate="G$1" x="104.14" y="55.88" smashed="yes">
 <attribute name="NAME" x="101.6" y="101.6" size="1.778" layer="95"/>
@@
 <attribute name="VALUE" x="45.72" y="38.1" size="1.778" layer="96" align="center"/>
 </instance>
-<instance part="U$12" gate="G$1" x="170.18" y="71.12" smashed="yes">
-<attribute name="VALUE" x="170.18" y="73.66" size="1.778" layer="96" rot="R180" align="center"/>
-</instance>
 <instance part="GND9" gate="G$1" x="170.18" y="50.8" smashed="yes">
 <attribute name="VALUE" x="170.18" y="48.26" size="1.778" layer="96" align="center"/>
@@
 </segment>
 </net>
-<net name="3V3" class="0">
-<segment>
-<pinref part="U$12" gate="G$1" pin="3V3"/>
-<pinref part="C4" gate="G$1" pin="2"/>
-<wire x1="170.18" y1="68.58" x2="170.18" y2="66.04" width="0.1524" layer="91"/>
-</segment>
-</net>
 <net name="DSP_SPI_CS" class="0">
 <segment>
@@
 <pinref part="U$2" gate="G$1" pin="3V3_SLP"/>
 </segment>
+<segment>
+<pinref part="C4" gate="G$1" pin="2"/>
+<wire x1="170.18" y1="66.04" x2="170.18" y2="73.66" width="0.1524" layer="91"/>
+<wire x1="170.18" y1="73.66" x2="205.74" y2="73.66" width="0.1524" layer="91"/>
+<label x="187.96" y="73.66" size="1.778" layer="95"/>
+</segment>
 </net>
 </nets>
@@
 <attribute name="NAME" x="12.7" y="16.256" size="1.27" layer="95" align="center"/>
 </instance>
-<instance part="MECH4" gate="G$1" x="12.7" y="5.08" smashed="yes">
-<attribute name="NAME" x="12.7" y="8.636" size="1.27" layer="95" align="center"/>
-</instance>
-<instance part="MECH5" gate="G$1" x="20.32" y="12.7" smashed="yes">
-<attribute name="NAME" x="20.32" y="16.256" size="1.27" layer="95" align="center"/>
-</instance>
-<instance part="MECH6" gate="G$1" x="20.32" y="5.08" smashed="yes">
-<attribute name="NAME" x="20.32" y="8.636" size="1.27" layer="95" align="center"/>
-</instance>
 </instances>
