File: camera_main_sch_brd.sch (EAGLE design)
At the start: 195 parts, among them CN1 USB C CON, CN2 50 PIN 0.5MM, CN3 31 PIN FPC, CN4 Gb RJ45 + MAG, CN5 USB A, CN6 NO FIT, CN7 uSD, CN8 NO FIT, Q2 SI7489DP, U1 10CL016YF484C6G, U10 93LC56B-I/SN, U11 USBLC6-2SC6, U12 TPS54233D, U13 FT230X, U14 3.3V BUCK, U15 STUSB4500, U16 Gb PHY, U2 OSD32MP157C-512M-BAA, U3 STM32L431RBT, U4 TLV61046A, U5 AS4C32M16SA, U6 AS4C32M16SA, U7 ACT2861, U8 USBLC6-2SC6, U9 FT232H

Commit message: New main PCB started
Parts:
- removed C10, C11, C12, C13, C14, C24, C54, C7, C8: 100nF 16V, CAPACITORS:CL10B104KO8WPNC
- removed C15: 100nF 50V, CAPACITORS:VJ0603Y104KXACW1BC
- removed C16, C17: 18pF 50V, CAPACITORS:MC0603N180J500CT
- removed C2, C22, C43, C55: 4.7uF 6.3V, CAPACITORS:GRM188R60J475ME19D
- removed C20, C21, C23, C41, C42, C44: 100nF 25V, CAPACITORS:MC0402B104K250CT
- removed C3: 1uF 25V, CAPACITORS:CL10A105KA8NNNC
- removed C4, C5: 2.2uF 25V, CAPACITORS:GRM188R61E225KA12D
- removed C6: 100nF 16V, CAPACITORS:GCM188R71C104KA37J
- removed C68, C69, C70, C71: 100nF 100V, CAPACITORS:06031C104KAT2A
- removed C72, C73, C74, C75, C76, C79, C80, C81, C82, C83, C85, C87, C88: 100nF 16V, CAPACITORS:CL05B104KO5NNNC
- removed C77, C78, C84, C86, C89: 10uF 10V, CAPACITORS:GRM188R61A106KE69D
- removed C90, C91: 15pF 50V, CAPACITORS:06035A150JAT2A
- removed CN2: 50 PIN 0.5MM, CONNECTORs:FH52E-50S-0.5SH
- removed CN3: 31 PIN FPC, CONNECTORs:3-1734839-1
- removed CN4: Gb RJ45 + MAG, CONNECTORs:0857931020
- removed CN5: USB A, CONNECTORs:629104190121
- removed FB10, FB11, FB12, FB13, FB4, FB5, FB9: 600R, INDUCTORS:742792651
- removed L2: 15uH 0.22R, INDUCTORS:1231AS-H-150M=P3
- removed R1: 68k, r_0603:ERJ3EKF6802V
- removed R10: 2.0k, r_0603:ERJ3EKF2001V
- removed R11, R65, R66: 12k, r_0603:ERJ3EKF1202V
- removed R12, R13, R26, R6, R7, R73, R75, R77, R78, R79, R8, R80, R81, R9: 10k, r_0603:ERJ3EKF1002V
- removed R19, R5: 100R, r_0603:ERJ3EKF1000V
- removed R2, R4: 1.0M, r_0603:ERJ3EKF1004V
- removed R27, R28, R29, R30, R31, R32: 10R, r_0603:ERJ3EKF10R0V
- removed R3: 100k, r_0603:ERJ3EKF1003V
- removed R67: NO FIT, r_0603:ERJ3EKF1004V
- removed R68, R69: 22R, RESISTORS:EXB-38V220JV
- removed R70: 4.7k, r_0603:ERJ3EKF4701V
- removed R71: NO FIT, r_0603:ERJ3EKF1001V
- removed R72, R74, R76, R82: 1.0k, r_0603:ERJ3EKF1001V
- removed R83, R84, R85: NOT FIT, r_0603:ERJ3EKF1001V
- removed TP1, TP2: 2MM_TEST_POINT, MISC:2MM_TEST_POINT
- removed U10: 93LC56B-I/SN, ICs:93LC56B-I/SN
- removed U11: USBLC6-2SC6, ICs:USBLC6-2SC6
- removed U16: Gb PHY, ICs:KSZ9131RNX
- removed U2: OSD32MP157C-512M-BAA, Octavo-Systems OSD32MP1:OSD32MP157C-512M-BAA
- removed U4: TLV61046A, ICs:TLV61046ADBVR
- removed U5, U6: AS4C32M16SA, ICs:AS4C32M16SA-7BCN
- removed U9: FT232H, ICs:FT232HL
- removed XTAL2: 12MHz, CRYSTALS:ABM8-12.000MHZ-B2-T
- removed XTAL3: 25MHz, CRYSTALS:TSX-322525.0000MF10P-C0
- added MECH4, MECH5, MECH6, MECH7, MECH8: 6mm x 3mm, MISC:MOUNTHOLE
Connections:
- removed net 1V2: FB11.2, FB12.2, FB13.2, U1.VCCD_PLL1, U1.VCCD_PLL2, U1.VCCD_PLL3, U1.VCCD_PLL4, U1.VCCINT
- removed net 2V5: U1.VCCA1, U1.VCCA2, U1.VCCA3, U1.VCCA4
- removed net 5VUSB: C54.2, C55.2, U2D.OTG_VBUS, U9.VREGIN
- removed net CMV_LVDS_CLK_IN_N: CN2.P12
- removed net CMV_LVDS_CLK_IN_P: CN2.P13
- removed net CMV_LVDS_CLK_N: CN2.P49
- removed net CMV_LVDS_CLK_P: CN2.P48
- removed net CMV_LVDS_CONT_N: CN2.P15
- removed net CMV_LVDS_CONT_P: CN2.P14
- removed net CMV_LVDS_DATA_11_N: CN2.P25
- removed net CMV_LVDS_DATA_11_P: CN2.P24
- removed net CMV_LVDS_DATA_13_N: CN2.P29
- removed net CMV_LVDS_DATA_13_P: CN2.P28
- removed net CMV_LVDS_DATA_15_N: CN2.P31
- removed net CMV_LVDS_DATA_15_P: CN2.P30
- removed net CMV_LVDS_DATA_17_N: CN2.P34
- removed net CMV_LVDS_DATA_17_P: CN2.P35
- removed net CMV_LVDS_DATA_19_N: CN2.P32
- removed net CMV_LVDS_DATA_19_P: CN2.P33
- removed net CMV_LVDS_DATA_1_N: CN2.P17
- removed net CMV_LVDS_DATA_1_P: CN2.P16
- removed net CMV_LVDS_DATA_21_N: CN2.P38
- removed net CMV_LVDS_DATA_21_P: CN2.P39
- removed net CMV_LVDS_DATA_23_N: CN2.P36
- removed net CMV_LVDS_DATA_23_P: CN2.P37
- removed net CMV_LVDS_DATA_25_N: CN2.P41
- removed net CMV_LVDS_DATA_25_P: CN2.P40
- removed net CMV_LVDS_DATA_27_N: CN2.P43
- removed net CMV_LVDS_DATA_27_P: CN2.P42
- removed net CMV_LVDS_DATA_29_N: CN2.P46
- removed net CMV_LVDS_DATA_29_P: CN2.P47
- removed net CMV_LVDS_DATA_31_N: CN2.P44
- removed net CMV_LVDS_DATA_31_P: CN2.P45
- removed net CMV_LVDS_DATA_3_N: CN2.P20
- removed net CMV_LVDS_DATA_3_P: CN2.P21
- removed net CMV_LVDS_DATA_5_N: CN2.P18
- removed net CMV_LVDS_DATA_5_P: CN2.P19
- removed net CMV_LVDS_DATA_7_N: CN2.P22
- removed net CMV_LVDS_DATA_7_P: CN2.P23
- removed net CMV_LVDS_DATA_9_N: CN2.P26
- removed net CMV_LVDS_DATA_9_P: CN2.P27
- removed net DSP_D_NC: CN3.15
- removed net DSP_IREF: CN3.4, R4.2
- removed net DSP_NRESET: CN3.16
- removed net DSP_SPI_CS: CN3.17
- removed net DSP_SPI_MOSI: R5.2
- removed net DSP_SPI_SCLK: R19.2
- removed net DSP_VCOM: C5.2, CN3.3
- removed net DSP_VDISP_EN: R3.2, U4.EN
- removed net ETH_!INT: R71.1, R72.2, U16.INT_N/PME_N2/ALLPHYAD, U2C.PG12
- removed net ETH_!RST: U16.!RST
- removed net ETH_CLK125_OUT: R75.1, U16.CLK125_NDO/LED_MODE, U2C.PG5
- removed net ETH_MDC: U16.MDC, U2B.PC1
- removed net ETH_MDIO: R70.1, U16.MDIO, U2B.PA2
- removed net ETH_RXC: R69.6, R76.2, U2B.PA1
- removed net ETH_RXD0: R68.8, R81.1, R85.2, U2B.PC4
- removed net ETH_RXD1: R68.7, R80.1, R84.2, U2B.PC5
- removed net ETH_RXD2: R68.6, R79.1, R83.2, U2C.PH6
- removed net ETH_RXD3: R68.5, R78.1, R82.2, U2C.PH7
- removed net ETH_RX_CTL: R69.5, R77.1, U2B.PA7
- removed net ETH_TXC: U16.TXC, U2C.PG4
- removed net ETH_TXD0: U16.TXD0, U2C.PG13
- removed net ETH_TXD1: U16.TXD1, U2C.PG14
- removed net ETH_TXD2: U16.TXD2, U2B.PC2
- removed net ETH_TXD3: U16.TXD3, U2C.PE2
- removed net ETH_TX_CTL: U16.TX_CTL
- removed net FT232H_3V3: C14.2, C15.2, C24.2, C7.2, C8.2, FB4.1, FB5.1, R12.2, R13.2, R6.2, R7.2, R8.2, R9.2, U10.ORG, U10.V+, U9.VCCD, U9.VCCIO
- removed net FT232H_USB_DM: U2D.USB_DM1, U9.D-
- removed net FT232H_USB_DP: U2D.USB_DP1, U9.D+
- removed net FT_CLK: U9.ACBUS5
- removed net FT_D0: U9.D0
- removed net FT_D1: U9.D1
- removed net FT_D2: U9.D2
- removed net FT_D3: U9.D3
- removed net FT_D4: U9.D4
- removed net FT_D5: U9.D5
- removed net FT_D6: U9.D6
- removed net FT_D7: U9.D7
- removed net FT_EE_CLK: R7.1, U10.CLK, U9.EECLK
- removed net FT_EE_CS: R8.1, U10.CS, U9.EECS
- removed net FT_EE_DI: R10.2, U10.DI, U9.EEDATA
- removed net FT_NRST: R9.1, U9.!RESET
- removed net FT_OE: U9.ACBUS6
- removed net FT_PWRSAV1: R13.1, U9.PWRSAV#
- removed net FT_RD: U9.RD#
- removed net FT_RXF: U9.RXF#
- removed net FT_SIWU1: R12.1, U9.SIWU#
- removed net FT_TXE: U9.TXE#
- removed net FT_WR: U9.WR#
- removed net F_REQ: CN2.P1
- removed net INT1: CN2.P2
- removed net INT2: CN2.P5
- removed net MEM_USB_DM: U11.D+_OUT, U2D.USB_DM2
- removed net MEM_USB_DP: U11.D-OUT, U2D.USB_DP2
- removed net MP1_EEPROM_WP: TP1.P$1, U2A.EEPROM_WP
- removed net MP1_PMIC_!PONKEYIN: U2A.PMIC_PONKEYN
- removed net MP1_SOFT_!RESET: R26.1, U2A.NRST
- removed net MP1_USB_VBUS: CN5.VBUS, U11.VBUS
- removed net N$1: R1.2, R2.1, U4.FB
- removed net N$100: R73.2, U16.LED1/PME_N1/PHYAD0
- removed net N$101: R74.2, U16.LED2/PHYAD1
- removed net N$13: CN3.11, R5.1
- removed net N$14: CN3.12, R19.1
- removed net N$19: R29.1, R32.2, U2A.BOOT0
- removed net N$2: L2.2, U4.SW
- removed net N$26: U2A.VBAT, U2A.VDD@1, U2A.VDD@2, U2A.VDD@3, U2A.VDD@4, U2A.VDD@5, U2A.VDD@6, U2A.VDD@7, U2A.VDD@8, U2A.VDD@9
- removed net N$29: R28.1, R31.2, U2A.BOOT1
- removed net N$35: U2A.PMIC_BSTOUT@1, U2A.PMIC_BSTOUT@2
- removed net N$36: R27.1, R30.2, U2A.BOOT2
- removed net N$37: U2A.PMIC_SWOUT@1, U2A.PMIC_SWOUT@2
- removed net N$38: CN5.D+, U11.D-_IN
- removed net N$39: CN5.D-, U11.D+_IN
- removed net N$4: C13.2, U9.VCCA
- removed net N$40: U2D.VREF-, U2D.VSSA
- removed net N$41: U2D.VDDA, U2D.VREF+
- removed net N$5: C12.2, U9.VCCCORE
- removed net N$6: R11.2, U9.REF
- removed net N$7: R10.1, R6.1, U10.DO
- removed net N$74: CN4.TD0+, U16.TXRXP_A
- removed net N$75: CN4.TD0-, U16.TXRXM_A
- removed net N$76: CN4.TD1+, U16.TXRXP_B
- removed net N$77: CN4.TD1-, U16.TXRXM_B
- removed net N$78: CN4.TD2+, U16.TXRXP_C
- removed net N$79: CN4.TD2-, U16.TXRXM_C
- removed net N$8: C17.2, U9.XCSO, XTAL2.P$1
- removed net N$80: CN4.TD3+, U16.TXRXP_D
- removed net N$81: CN4.TD3-, U16.TXRXM_D
- removed net N$82: C68.2, CN4.CT3
- removed net N$83: C69.2, CN4.CT2
- removed net N$84: C70.2, CN4.CT1
- removed net N$85: C71.2, CN4.CT0
- removed net N$86: C74.2, C75.2, C76.2, C78.2, FB9.2, U16.DVDDH
- removed net N$87: C72.2, C73.2, C77.2, FB10.2, U16.AVDDH
- removed net N$88: C79.2, C80.2, C81.2, C82.2, C83.2, C84.2, FB13.1, U16.DVDDL
- removed net N$89: C85.2, C86.2, FB12.1, U16.AVDDL_PLL
- removed net N$9: C16.2, U9.XCSI, XTAL2.P$2
- removed net N$90: C87.2, C88.2, C89.2, FB11.1, U16.AVDDL
- removed net N$91: R65.2, R66.2, U16.ISET
- removed net N$92: C90.2, R67.2, U16.XO, XTAL3.P$2
- removed net N$93: C91.2, R67.1, U16.XI, XTAL3.P$1
- removed net N$94: R68.4, U16.RXD3/MODE3
- removed net N$95: R68.3, U16.RXD2/MODE2
- removed net N$96: R68.2, U16.RXD1/MODE1
- removed net N$97: R68.1, U16.RXD0/MODE0
- removed net N$98: R69.4, U16.RX_CTL/CLK125_EN
- removed net N$99: R69.3, U16.RXC/PHYAD2
- removed net PR_CMV_5V: CN2.P10, CN2.P9
- removed net SDRAM0_!CAS: U6.!CAS
- removed net SDRAM0_!CS: U6.!CS
- removed net SDRAM0_!RAS: U6.!RAS
- removed net SDRAM0_!WE: U6.!WE
- removed net SDRAM0_A0: U6.A0
- removed net SDRAM0_A1: U6.A1
- removed net SDRAM0_A10: U6.A10
- removed net SDRAM0_A11: U6.A11
- removed net SDRAM0_A12: U6.A12
- removed net SDRAM0_A2: U6.A2
- removed net SDRAM0_A3: U6.A3
- removed net SDRAM0_A4: U6.A4
- removed net SDRAM0_A5: U6.A5
- removed net SDRAM0_A6: U6.A6
- removed net SDRAM0_A7: U6.A7
- removed net SDRAM0_A8: U6.A8
- removed net SDRAM0_A9: U6.A9
- removed net SDRAM0_BA0: U6.BA0
- removed net SDRAM0_BA1: U6.BA1
- removed net SDRAM0_CKE: U6.CKE
- removed net SDRAM0_CLK: U6.CLK
- removed net SDRAM0_D0: U6.D0
- removed net SDRAM0_D1: U6.D1
- removed net SDRAM0_D10: U6.D10
- removed net SDRAM0_D11: U6.D11
- removed net SDRAM0_D12: U6.D12
- removed net SDRAM0_D13: U6.D13
- removed net SDRAM0_D14: U6.D14
- removed net SDRAM0_D15: U6.D15
- removed net SDRAM0_D2: U6.D2
- removed net SDRAM0_D3: U6.D3
- removed net SDRAM0_D4: U6.D4
- removed net SDRAM0_D5: U6.D5
- removed net SDRAM0_D6: U6.D6
- removed net SDRAM0_D7: U6.D7
- removed net SDRAM0_D8: U6.D8
- removed net SDRAM0_D9: U6.D9
- removed net SDRAM0_LDM: U6.LDM
- removed net SDRAM0_UDM: U6.UDM
- removed net SDRAM1_!CAS: U5.!CAS
- removed net SDRAM1_!CS: U5.!CS
- removed net SDRAM1_!RAS: U5.!RAS
- removed net SDRAM1_!WE: U5.!WE
- removed net SDRAM1_A0: U5.A0
- removed net SDRAM1_A1: U5.A1
- removed net SDRAM1_A10: U5.A10
- removed net SDRAM1_A11: U5.A11
- removed net SDRAM1_A12: U5.A12
- removed net SDRAM1_A2: U5.A2
- removed net SDRAM1_A3: U5.A3
- removed net SDRAM1_A4: U5.A4
- removed net SDRAM1_A5: U5.A5
- removed net SDRAM1_A6: U5.A6
- removed net SDRAM1_A7: U5.A7
- removed net SDRAM1_A8: U5.A8
- removed net SDRAM1_A9: U5.A9
- removed net SDRAM1_BA0: U5.BA0
- removed net SDRAM1_BA1: U5.BA1
- removed net SDRAM1_CKE: U5.CKE
- removed net SDRAM1_CLK: U5.CLK
- removed net SDRAM1_D0: U5.D0
- removed net SDRAM1_D1: U5.D1
- removed net SDRAM1_D10: U5.D10
- removed net SDRAM1_D11: U5.D11
- removed net SDRAM1_D12: U5.D12
- removed net SDRAM1_D13: U5.D13
- removed net SDRAM1_D14: U5.D14
- removed net SDRAM1_D15: U5.D15
- removed net SDRAM1_D2: U5.D2
- removed net SDRAM1_D3: U5.D3
- removed net SDRAM1_D4: U5.D4
- removed net SDRAM1_D5: U5.D5
- removed net SDRAM1_D6: U5.D6
- removed net SDRAM1_D7: U5.D7
- removed net SDRAM1_D8: U5.D8
- removed net SDRAM1_D9: U5.D9
- removed net SDRAM1_LDM: U5.LDM
- removed net SDRAM1_UDM: U5.UDM
- removed net SPI_EN: CN2.P7
- removed net SPI_MISO: CN2.P6
- removed net SPI_MOSI: CN2.P3
- removed net SPI_SCLK: CN2.P4
- removed net SYS_!RST: CN2.P8
- removed net VDISP: C3.2, C6.2, CN3.2, R2.2, U4.VOUT
- removed net VPHY: C11.2, FB5.2, U9.VPHY
- removed net VPLL: C10.2, FB4.2, U9.VPLL
- net 3V3: no longer C20.2, C21.2, C22.2, C23.2, C41.2, C42.2, C43.2, C44.2, FB10.1, FB9.1, R26.2, R27.2, R28.2, R29.2, R70.2, R71.2, R73.1, R75.2, R77.2, R78.2, R79.2, R80.2, R81.2, U2A.PMIC_VOUT4@1, U2A.PMIC_VOUT4@2, U5.VCC, U5.VCCQ, U6.VCC, U6.VCCQ
- net 3V3_SLP: no longer C2.2, C4.2, CN3.21, L2.1, U4.VIN
- net 5V: no longer U2A.PMIC_BSTIN@1, U2A.PMIC_BSTIN@2, U2A.PMIC_BSTIN@3, U2A.PMIC_BSTIN@4, U2A.PMIC_LDO25IN, U2A.PMIC_SWIN@1, U2A.PMIC_SWIN@2, U2A.VIN@1, U2A.VIN@2, U2A.VIN@3, U2A.VIN@4
- net GND: no longer C10.1, C11.1, C12.1, C13.1, C14.1, C15.1, C16.1, C17.1, C2.1, C20.1, C21.1, C22.1, C23.1, C24.1, C3.1, C4.1, C41.1, C42.1, C43.1, C44.1, C5.1, C54.1, C55.1, C6.1, C68.1, C69.1, C7.1, C70.1, C71.1, C72.1, C73.1, C74.1, C75.1, C76.1, C77.1, C78.1, C79.1, C8.1, C80.1, C81.1, C82.1, C83.1, C84.1, C85.1, C86.1, C87.1, C88.1, C89.1, C90.1, C91.1, CN2.GND, CN2.P11, CN2.P50, CN3.1, CN3.13, CN3.14, CN3.19, CN3.20, CN3.30, CN3.31, CN4.SHLD, CN5.GND, R1.1, R11.1, R3.1, R30.1, R31.1, R32.1, R4.1, R65.1, R66.1, R72.1, R74.1, R76.1, R82.1, R83.1, R84.1, R85.1, TP2.P$1, U1.GND, U1.GNDA1, U1.GNDA2, U1.GNDA3, U1.GNDA4, U10.GND, U11.GND, U16.GND, U16.VSS, U2A.BYPASS_REG1V8, U2A.HSE_OSC_OE, U2E.VSS@1, U2E.VSS@10, U2E.VSS@11, U2E.VSS@12, U2E.VSS@13, U2E.VSS@14, U2E.VSS@15, U2E.VSS@16, U2E.VSS@17, U2E.VSS@18, U2E.VSS@19, U2E.VSS@2, U2E.VSS@20, U2E.VSS@21, U2E.VSS@22, U2E.VSS@23, U2E.VSS@24, U2E.VSS@25, U2E.VSS@26, U2E.VSS@27, U2E.VSS@28, U2E.VSS@29, U2E.VSS@3, U2E.VSS@30, U2E.VSS@31, U2E.VSS@32, U2E.VSS@33, U2E.VSS@34, U2E.VSS@35, U2E.VSS@36, U2E.VSS@37, U2E.VSS@38, U2E.VSS@39, U2E.VSS@4, U2E.VSS@40, U2E.VSS@41, U2E.VSS@42, U2E.VSS@43, U2E.VSS@44, U2E.VSS@45, U2E.VSS@46, U2E.VSS@47, U2E.VSS@48, U2E.VSS@49, U2E.VSS@5, U2E.VSS@50, U2E.VSS@51, U2E.VSS@52, U2E.VSS@53, U2E.VSS@54, U2E.VSS@55, U2E.VSS@56, U2E.VSS@57, U2E.VSS@58, U2E.VSS@59, U2E.VSS@6, U2E.VSS@60, U2E.VSS@61, U2E.VSS@62, U2E.VSS@63, U2E.VSS@64, U2E.VSS@65, U2E.VSS@66, U2E.VSS@67, U2E.VSS@68, U2E.VSS@69, U2E.VSS@7, U2E.VSS@70, U2E.VSS@8, U2E.VSS@9, U4.GND, U5.VSS, U5.VSSQ, U6.VSS, U6.VSSQ, U9.GND, U9.TEST, XTAL2.GND
- net SD_CLK: no longer U2B.PC12
- net SD_CMD: no longer U2B.PD2
- net SD_D0: no longer U2B.PC8
- net SD_D1: no longer U2B.PC9
- net SD_D2: no longer U2B.PC10
- net SD_D3: no longer U2B.PC11
