File: sensor.brd (EAGLE design)
At the start: 40 x 50 mm, 149 parts, among them CN1 FH52E-60S-0.5SH, CN5 TC2030, U1 STM32L031G6, U18 MIC5271, U19 LM2662, U2 GMAX0505-DV, U20 MAX25300B, U21 MAX25300B, U22 MAX25300B, U23 MAX25300B, U24 3.3V BUCK, U25 MAX6627

Commit message: Sensor PCB routed and DRC passes, needs review of layer stack and diff pairs
Parts:
- removed C211: 22uF 6.3V, c_1206:1206
- added C8: 0.1uF 10V, c_0402:0402
- moved R73 2.50 mm to (-9.25, -14.6)
- moved C207 2.21 mm to (-7.00, 4.00), turned to 180 degrees
- moved R74 2.00 mm to (-7.25, -14.6)
- moved C152 1.07 mm to (-7.00, 10.6), turned to 0 degrees
- moved C246 0.79 mm to (1.62, 12.4), turned to 180 degrees
- moved C256 0.71 mm to (-16.0, -0.50), turned to 270 degrees
- moved C234 0.62 mm to (10.2, 1.88)
- moved C237 0.62 mm to (10.2, 0.88)
- moved C159 0.38 mm to (-6.75, 14.1)
- moved C233 0.25 mm to (10.2, 3.62)
- moved C238 0.25 mm to (10.2, 5.38)
- moved C239 0.25 mm to (10.2, 6.25)
- moved C240 0.25 mm to (10.2, 7.12)
- moved C242 0.25 mm to (10.2, 4.50)
- moved C254 0.25 mm to (-18.2, -1.25)
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Connections:
- net SEN_PWR_RDY renamed SEN_PWR_EN
- net GND: now also C8.1; no longer C211.1
- net SEN_CLK_IN: now also CN1.P15; no longer CN1.P18
- net SEN_PWR_3V3A: now also C8.2
- net SEN_PWR_4V1: no longer C211.2
- net SEN_SPI_!CS: now also CN1.P16; no longer CN1.P12
- net SEN_SPI_MISO: now also CN1.P17; no longer CN1.P11
- net SEN_SPI_MOSI: now also CN1.P18; no longer CN1.P10
- net SEN_SPI_SCLK: now also CN1.P11; no longer CN1.P9
- net SEN_SYS_!RESET: now also CN1.P12; no longer CN1.P17
- net SEN_TDIG0: now also CN1.P9; no longer CN1.P15
- net SEN_TDIG1: now also CN1.P10; no longer CN1.P16
- net SEN_TEMP1: now also CN1.P14; no longer CN1.P13
- net SEN_TEXP0: now also CN1.P13; no longer CN1.P14
Routing:
- net PROC_3V3: track 11.9 -> 100.4 mm, vias 7 -> 11
- net SEN_PWR_EN: track 0.00 -> 63.8 mm, vias 0 -> 2
- net SEN_SPI_SCLK: track 4.07 -> 67.6 mm, vias 1 -> 4
- net SEN_SPI_MISO: track 2.73 -> 65.1 mm, vias 1 -> 4
- net SEN_PWR_1V3A: track 21.9 -> 73.6 mm, vias 6 -> 7
- net SEN_PWR_3V6: track 18.1 -> 67.2 mm, vias 6 -> 5
- net SEN_TEMP_SPI_!CS: track 2.40 -> 50.9 mm, vias 0 -> 3
- net PROC_NRESET: track 0.00 -> 40.4 mm, vias 0 -> 2
- net SEN_PWR_3V6_EN: track 1.51 -> 41.9 mm, vias 0 -> 2
- net SEN_PWR_0V7: track 6.09 -> 45.4 mm, vias 2 -> 3
- net PROC_SWCLK: track 0.00 -> 39.0 mm, vias 0 -> 2
- net PROC_SWDIO: track 0.00 -> 37.5 mm, vias 0 -> 2
- net SEN_PWR_4V1_EN: track 1.51 -> 37.4 mm, vias 0 -> 2
- net SEN_PWR_N1V3A: track 10.0 -> 34.7 mm, vias 3 -> 4
- net SEN_TDIG0: track 0.71 -> 25.2 mm, vias 1 -> 2
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- added copper zone on layer 4, net SEN_PWR_1V3D
- added copper zone on layer 5, net SEN_PWR_3V3A

Commit message: LDO replaced for stock, BoM ordered
Parts:
- R55: value 390R -> 3.9k
- R56: value 4.7k -> 100k
- U18: value MIC5271 -> MAX1735
- moved C245 1.31 mm to (-14.8, 15.1)
- moved C244 1.08 mm to (-9.25, 14.5), turned to 270 degrees
- moved R57 0.88 mm to (-11.2, 17.4)
- moved U18 0.67 mm to (-12.0, 15.2), turned to 270 degrees
Connections:
- net GND: now also U18.1; no longer U18.2
- net N$63: now also U18.4; no longer U18.3
- net SEN_PWR_N1V3A: now also U18.5; no longer U18.4
- net SEN_PWR_N1V3A_EN: now also U18.3; no longer U18.1
- net SEN_PWR_N5V0: now also U18.2; no longer U18.5
Routing:
- net SEN_PWR_N5V0: track 17.1 -> 14.4 mm
- net N$2: track 0.00 -> 1.25 mm
- net N$1: track 0.00 -> 1.25 mm
- net SEN_PWR_N1V3A_EN: track 27.4 -> 26.4 mm
- net SEN_PWR_N1V3A: track 34.7 -> 35.6 mm
- net GND: track 196.6 -> 197.4 mm, vias 156 -> 155
- net N$63: track 4.32 -> 4.96 mm
