File: sensor.brd (EAGLE design)
At the start: 40 x 50 mm, 149 parts, among them CN1 FH52E-60S-0.5SH, CN5 TC2030, U1 STM32L031G6, U18 MAX1735, U19 LM2662, U2 GMAX0505-DV, U20 MAX25300B, U21 MAX25300B, U22 MAX25300B, U23 MAX25300B, U24 3.3V BUCK, U25 MAX6627

Commit message: Fixes for sensor PCB
Parts:
- removed C178: 4.7uF 6.3V, c_0402:0402
- removed C181, C182, C263: 22uF 6.3V, c_1206:1206
- removed C243: 2200pF 25V, c_0402:0402
- removed C265: 10uF 50V, CAPACITORS:1210
- removed C268: 0.1uF 10V, c_0402:0402
- removed MECH10: 6mm x 3mm, MISC:MOUNTHOLE_6X3
- removed R68, R71, R73, R75: 10k, r_0603:0603
- removed R72: 3k, r_0603:0603
- removed U24: 3.3V BUCK, ICs:TI_MICROSIP_10
- removed U25: MAX6627, ICs:TDFNEP8
- added C101, C102: 10uF 10V, c_1206:1206
- added C13: 0.1uF 10V, c_0402:0402
- added C87: 10uF 50V, CAPACITORS:1210
- added L1: 1uH, INDUCTORS:1008
- added MECH2: 6mm x 3mm, MISC:MOUNTHOLE_6X3
- added R11: 12k, RESISTORS:0603
- added R19: 13k, r_0603:0603
- added R20: 15k, r_0603:0603
- added R24, R4: 10k, r_0603:0603
- added U10: EMC1812T, ICs:DFN8
- added U3: MP2148, ICs:QFN6
- C1, C3, C4: value 22uF 6.3V -> 0.1uF 10V; device c_1206:1206 -> c_0402:0402
- C2: value 22uF 6.3V -> 2200pF 25V; device c_1206:1206 -> c_0402:0402
- C6, C7: value 0.1uF 10V -> 22uF 6.3V; device c_0402:0402 -> c_1206:1206
- C8: value 0.1uF 10V -> 4.7uF 6.3V
- R12: value 1.69k -> 2k
- R13: value 9.76k -> 6.2k
- R14: value 57.6k -> 36k
- R15, R17: value 10k -> 15k
- R16: value 49.9k -> 75k
- R18: value 45.3k -> 68k
- U1: value STM32L031G6 -> GMAX0505-DV; device ICs:UFQPN28 -> ICs:GMAX0505
- U2: value GMAX0505-DV -> STM32L031G6; device ICs:GMAX0505 -> ICs:UFQPN28
- moved C6 25.6 mm to (1.25, -12.0)
- moved R1 19.0 mm to (17.9, 3.12), turned to 0 degrees
- moved C2 18.0 mm to (12.6, 3.38)
- moved MECH1 18.0 mm to (17.0, 9.00)
- moved U1 17.5 mm to (0.00, 0.00), flipped to the bottom
- moved U2 17.5 mm to (11.5, 13.1), flipped to the top
- moved C1 15.8 mm to (14.2, 5.12), turned to 180 degrees
- moved C4 9.54 mm to (8.12, 12.6), turned to 0 degrees
- moved C8 8.00 mm to (2.25, 2.88), turned to 0 degrees
- moved C3 7.04 mm to (8.12, 14.6), turned to 0 degrees
- moved C7 2.02 mm to (6.12, 14.4), turned to 90 degrees
- turned R6 to 270 degrees
- renumbered C137 to C70, C149 to C65, C150 to C55, C151 to C47, C152 to C42, C153 to C38, C154 to C34, C155 to C31, C156 to C28, C157 to C25, C158 to C22, C159 to C19, C160 to C16, C161 to C66, C162 to C56, C163 to C48, C164 to C43, C165 to C39, C166 to C35, C167 to C32, C168 to C29, C169 to C26, C170 to C23, C171 to C20, C172 to C17, C173 to C14, C174 to C12, C175 to C11, C176 to C10, C177 to C9, C183 to C64, C184 to C54, C185 to C46, C186 to C41, C187 to C37, C188 to C33, C189 to C30, C190 to C27, C191 to C24, C192 to C21, C195 to C18, C196 to C15, C197 to C71, C199 to C61, C203 to C63, C206 to C67, C207 to C57, C209 to C49, C212 to C68, C213 to C58, C214 to C50, C215 to C72, C216 to C62, C218 to C69, C219 to C51, C221 to C59, C223 to C44, C224 to C60, C225 to C52, C227 to C53, C228 to C45, C230 to C40, C231 to C36, C233 to C74, C234 to C73, C235 to C75, C236 to C76, C237 to C77, C238 to C78, C239 to C79, C240 to C80, C241 to C81, C242 to C82, C244 to C105, C245 to C106, C246 to C86, C247 to C92, C248 to C97, C249 to C88, C250 to C93, C251 to C100, C252 to C98, C253 to C99, C254 to C85, C255 to C91, C256 to C96, C257 to C84, C258 to C90, C259 to C95, C260 to C83, C261 to C89, C262 to C94, C266 to C104, C267 to C103, CN5 to CN2, MECH7 to MECH3, R54 to R5, R55 to R22, R56 to R23, R57 to R21, R58 to R10, R59 to R17, R60 to R18, R61 to R9, R62 to R15, R63 to R16, R64 to R8, R65 to R13, R66 to R14, R67 to R7, R69 to R12, R70 to R6, R74 to R2, U18 to U9, U19 to U8, U20 to U7, U21 to U6, U22 to U5, U23 to U4
Connections:
- removed net 2V5SLP: CN2.1
- removed net N$67: R71.2, R72.1, U24.7
- removed net PROC_3V3: C268.2, C5.2, C6.2, C61.2, C7.2, C71.2, CN1.P7, R2.2, R73.2, R75.2, U1.1, U1.17, U1.5, U2.J16, U2.K13, U25.4
- removed net SEN_TEMP_SPI_!CS: CN1.P8, R75.1, U25.6
- new net N$3: L1.1, U3.4
- new net N$4: R19.2, R20.1, U3.1
- new net PROC_PWR: C1.2, C3.2, C4.2, C5.2, C61.2, C71.2, CN1.P7, CN2.1, R1.2, R2.2, R24.2, U1.J16, U1.K13, U10.1, U2.1, U2.17, U2.5
- new net SEN_UART_RX: CN1.P12, U2.26
- new net SEN_UART_TX: CN1.P8, U2.25
- new net TMP_ALERT: R1.1, U10.6
- new net TMP_I2C_SCL: U10.8, U2.19
- new net TMP_I2C_SDA: U10.7, U2.20
- new net TMP_THERM: R24.1, U10.4
- net GND: now also C101.1, C102.1, C13.1, C87.1, R11.1, R19.1, R4.1, U1.A11, U1.A13, U1.A7, U1.A9, U1.C16, U1.E16, U1.F12, U1.F13, U1.F14, U1.F15, U1.F5, U1.F6, U1.G12, U1.G13, U1.G14, U1.G15, U1.G16, U1.G3, U1.G4, U1.G5, U1.H1, U1.H12, U1.H13, U1.H14, U1.H15, U1.H3, U1.H4, U1.H5, U1.H6, U1.J1, U1.J15, U1.J3, U1.J4, U1.J5, U1.K1, U1.K15, U1.K17, U1.K3, U1.K4, U1.K5, U1.K6, U1.L1, U1.L3, U1.L4, U1.L5, U1.N16, U1.P16, U1.P2, U1.T10, U1.T12, U1.T14, U1.T4, U1.T6, U1.T8, U10.5, U10.EP, U2.16, U2.28, U3.2; no longer C178.1, C181.1, C182.1, C2.1, C263.1, C265.1, C268.1, R1.1, R68.1, R71.1, U1.16, U1.28, U2.A11, U2.A13, U2.A7, U2.A9, U2.C16, U2.E16, U2.F12, U2.F13, U2.F14, U2.F15, U2.F5, U2.F6, U2.G12, U2.G13, U2.G14, U2.G15, U2.G16, U2.G3, U2.G4, U2.G5, U2.H1, U2.H12, U2.H13, U2.H14, U2.H15, U2.H3, U2.H4, U2.H5, U2.H6, U2.J1, U2.J15, U2.J3, U2.J4, U2.J5, U2.K1, U2.K15, U2.K17, U2.K3, U2.K4, U2.K5, U2.K6, U2.L1, U2.L3, U2.L4, U2.L5, U2.N16, U2.P16, U2.P2, U2.T10, U2.T12, U2.T14, U2.T4, U2.T6, U2.T8, U24.1, U24.2, U24.PAD, U25.1, U25.8, U25.EP
- net N$124: now also R11.2; no longer R68.2
- net N$60: now also U1.E1; no longer U2.E1
- net N$61: now also C2.2, U1.F3, U10.2; no longer C243.2, U2.F3, U25.3
- net N$62: now also C2.1, U1.F4, U10.3; no longer C243.1, U2.F4, U25.2
- net N$70: now also U1.A4; no longer U2.A4
- net N$71: now also U1.P1; no longer U2.P1
- net N$72: now also U1.M1; no longer U2.M1
- net N$73: now also U1.G2; no longer U2.G2
- net N$74: now also U1.D1; no longer U2.D1
- net N$75: now also U1.C2; no longer U2.C2
- net N$76: now also U1.C1; no longer U2.C1
- net N$77: now also U1.A3; no longer U2.A3
- net N$78: now also U1.D2; no longer U2.D2
- net N$79: now also U1.E2; no longer U2.E2
- net PROC_BOOT0: now also R4.2, U2.27; no longer R1.2, U1.27
- net PROC_NRESET: now also U2.4; no longer U1.4
- net PROC_SWCLK: now also U2.22; no longer U1.22
- net PROC_SWDIO: now also U2.21; no longer U1.21
- net SEN_B_D0_N: now also U1.C15; no longer U2.C15
- net SEN_B_D0_P: now also U1.B15; no longer U2.B15
- net SEN_B_D12_N: now also U1.C9; no longer U2.C9
- net SEN_B_D12_P: now also U1.B9; no longer U2.B9
- net SEN_B_D15_N: now also U1.E7; no longer U2.E7
- net SEN_B_D15_P: now also U1.D7; no longer U2.D7
- net SEN_B_D18_N: now also U1.C6; no longer U2.C6
- net SEN_B_D18_P: now also U1.B6; no longer U2.B6
- net SEN_B_D21_N: now also U1.E4; no longer U2.E4
- net SEN_B_D21_P: now also U1.D4; no longer U2.D4
- net SEN_B_D3_N: now also U1.E13; no longer U2.E13
- net SEN_B_D3_P: now also U1.D13; no longer U2.D13
- net SEN_B_D6_N: now also U1.C12; no longer U2.C12
- net SEN_B_D6_P: now also U1.B12; no longer U2.B12
- net SEN_B_D9_N: now also U1.E10; no longer U2.E10
- net SEN_B_D9_P: now also U1.D10; no longer U2.D10
- net SEN_CLK_IN: now also U1.L14; no longer U2.L14
- net SEN_CLK_N: now also U1.C3; no longer U2.C3
- net SEN_CLK_P: now also U1.B3; no longer U2.B3
- net SEN_PWR_0V7: now also U1.M17; no longer U2.M17
- net SEN_PWR_0V7_EN: now also U2.10; no longer U1.10
- net SEN_PWR_1V3A: now also U1.A10, U1.C17, U1.D16, U1.J2, U1.T13, U1.T7; no longer U2.A10, U2.C17, U2.D16, U2.J2, U2.T13, U2.T7
- net SEN_PWR_1V3D: now also C101.2, C102.2, C6.2, C7.2, C8.2, L1.2, R20.2, U1.A8, U1.F16, U1.G6, U1.H16, U1.H2, U1.J6, U1.K2, U1.P17, U1.T11, U1.T5, U3.6; no longer C1.2, C178.2, C181.2, C182.2, C2.2, C263.2, C3.2, C4.2, R72.2, U2.A8, U2.F16, U2.G6, U2.H16, U2.H2, U2.J6, U2.K2, U2.P17, U2.T11, U2.T5, U24.6
- net SEN_PWR_1V3_EN: now also U2.11, U3.5; no longer U1.11, U24.4
- net SEN_PWR_3V3A: now also C13.2, U1.A12, U1.A15, U1.A5, U1.F1, U1.G1, U1.K16, U1.L2, U1.L6, U1.M16, U1.T9; no longer C8.2, U2.A12, U2.A15, U2.A5, U2.F1, U2.G1, U2.K16, U2.L2, U2.L6, U2.M16, U2.T9
- net SEN_PWR_3V3_EN: now also U2.7; no longer U1.7
- net SEN_PWR_3V6: now also U1.A14, U1.G17, U1.J17, U1.N17, U1.T15; no longer U2.A14, U2.G17, U2.J17, U2.N17, U2.T15
- net SEN_PWR_3V6_EN: now also U2.8; no longer U1.8
- net SEN_PWR_4V1: now also U1.E17, U1.L17; no longer U2.E17, U2.L17
- net SEN_PWR_4V1_EN: now also U2.9; no longer U1.9
- net SEN_PWR_EN: now also U2.12; no longer U1.12
- net SEN_PWR_N1V3A: now also U1.D17, U1.F17, U1.H17; no longer U2.D17, U2.F17, U2.H17
- net SEN_PWR_N1V3A_EN: now also U2.6; no longer U1.6
- net SEN_SPI_!CS: now also U1.L13; no longer U2.L13
- net SEN_SPI_MISO: now also U1.L12; no longer U2.L12, U25.7
- net SEN_SPI_MOSI: now also U1.K12; no longer U2.K12
- net SEN_SPI_SCLK: now also U1.J14; no longer U2.J14, U25.5
- net SEN_SYS_!RESET: now also U1.K14, U2.3; no longer CN1.P12, R73.1, U2.K14
- net SEN_TDIG0: now also U1.J12; no longer U2.J12
- net SEN_TDIG1: now also U1.J13; no longer U2.J13
- net SEN_TEMP1: now also U1.L15; no longer U2.L15
- net SEN_TEXP0: now also U1.L16; no longer U2.L16
- net SEN_T_D0_N: now also U1.R15; no longer U2.R15
- net SEN_T_D0_P: now also U1.P15; no longer U2.P15
- net SEN_T_D12_N: now also U1.R9; no longer U2.R9
- net SEN_T_D12_P: now also U1.P9; no longer U2.P9
- net SEN_T_D15_N: now also U1.N7; no longer U2.N7
- net SEN_T_D15_P: now also U1.M7; no longer U2.M7
- net SEN_T_D18_N: now also U1.R6; no longer U2.R6
- net SEN_T_D18_P: now also U1.P6; no longer U2.P6
- net SEN_T_D21_N: now also U1.N4; no longer U2.N4
- net SEN_T_D21_P: now also U1.M4; no longer U2.M4
- net SEN_T_D3_N: now also U1.N13; no longer U2.N13
- net SEN_T_D3_P: now also U1.M13; no longer U2.M13
- net SEN_T_D6_N: now also U1.R12; no longer U2.R12
- net SEN_T_D6_P: now also U1.P12; no longer U2.P12
- net SEN_T_D9_N: now also U1.N10; no longer U2.N10
- net SEN_T_D9_P: now also U1.M10; no longer U2.M10
- net SYS_PWR_5V: now also C87.2, U3.3; no longer C265.2, U24.3
Routing:
- net PROC_PWR: track 0.00 -> 117.1 mm, vias 0 -> 11
- net PROC_3V3: track 100.4 -> 0.00 mm, vias 11 -> 0
- net SEN_UART_TX: track 0.00 -> 75.6 mm, vias 0 -> 2
- net SEN_UART_RX: track 0.00 -> 71.4 mm, vias 0 -> 2
- net SEN_TEMP_SPI_!CS: track 50.9 -> 0.00 mm, vias 3 -> 0
- net SEN_SPI_MISO: track 65.1 -> 17.0 mm, vias 4 -> 2
- net SEN_SPI_SCLK: track 67.6 -> 22.5 mm, vias 4 -> 2
- net SEN_SYS_!RESET: track 23.1 -> 66.8 mm, vias 2 -> 3
- net TMP_I2C_SCL: track 0.00 -> 16.8 mm
- net TMP_I2C_SDA: track 0.00 -> 15.5 mm, vias 0 -> 2
- net PROC_NRESET: track 40.1 -> 35.0 mm
- net GND: track 197.4 -> 193.3 mm, vias 155 -> 151
- net N$67: track 3.89 -> 0.00 mm
- net TMP_THERM: track 0.00 -> 3.69 mm
- net SEN_PWR_1V3D: track 48.9 -> 45.5 mm, vias 20 -> 19
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
Commit message: Mech design and layout
Parts:
- added CN3: FH52E-60S-0.5SH, CONNECTORs:FH52E-60S-0.5SH
Connections:
- new net N$5: CN1.SH1, CN1.SH3, CN3.P1
- net GND: now also CN3.P2, CN3.P3, CN3.P39, CN3.P4, CN3.P40, CN3.P42, CN3.P43, CN3.P56, CN3.P57, CN3.P58
- net PROC_PWR: now also CN3.P55
- net SEN_B_D0_N: now also CN3.P29
- net SEN_B_D0_P: now also CN3.P30
- net SEN_B_D12_N: now also CN3.P21
- net SEN_B_D12_P: now also CN3.P22
- net SEN_B_D15_N: now also CN3.P17
- net SEN_B_D15_P: now also CN3.P18
- net SEN_B_D18_N: now also CN3.P16
- net SEN_B_D18_P: now also CN3.P15
- net SEN_B_D21_N: now also CN3.P12
- net SEN_B_D21_P: now also CN3.P11
- net SEN_B_D3_N: now also CN3.P27
- net SEN_B_D3_P: now also CN3.P28
- net SEN_B_D6_N: now also CN3.P34
- net SEN_B_D6_P: now also CN3.P33
- net SEN_B_D9_N: now also CN3.P26
- net SEN_B_D9_P: now also CN3.P25
- net SEN_CLK_IN: now also CN3.P47
- net SEN_CLK_N: now also CN3.P6
- net SEN_CLK_P: now also CN3.P5
- net SEN_PWR_EN: now also CN3.P41
- net SEN_SPI_!CS: now also CN3.P46
- net SEN_SPI_MISO: now also CN3.P45
- net SEN_SPI_MOSI: now also CN3.P44
- net SEN_SPI_SCLK: now also CN3.P51
- net SEN_TDIG0: now also CN3.P53
- net SEN_TDIG1: now also CN3.P52
- net SEN_TEMP1: now also CN3.P48
- net SEN_TEXP0: now also CN3.P49
- net SEN_T_D0_N: now also CN3.P37
- net SEN_T_D0_P: now also CN3.P38
- net SEN_T_D12_N: now also CN3.P24
- net SEN_T_D12_P: now also CN3.P23
- net SEN_T_D15_N: now also CN3.P10
- net SEN_T_D15_P: now also CN3.P9
- net SEN_T_D18_N: now also CN3.P13
- net SEN_T_D18_P: now also CN3.P14
- net SEN_T_D21_N: now also CN3.P8
- net SEN_T_D21_P: now also CN3.P7
- net SEN_T_D3_N: now also CN3.P36
- net SEN_T_D3_P: now also CN3.P35
- net SEN_T_D6_N: now also CN3.P31
- net SEN_T_D6_P: now also CN3.P32
- net SEN_T_D9_N: now also CN3.P20
- net SEN_T_D9_P: now also CN3.P19
- net SEN_UART_RX: now also CN3.P50
- net SEN_UART_TX: now also CN3.P54
- net SYS_PWR_5V: now also CN3.P59, CN3.P60, CN3.SH1, CN3.SH3

Commit message: Moved to FT600 due to IO constraints
Parts:
- removed CN1: FH52E-60S-0.5SH, CONNECTORs:FH52E-60S-0.5SH
- moved CN3 13.5 mm to (0.00, -16.5), turned to 180 degrees
- moved CN2 8.40 mm to (12.9, -22.5)
Connections:
- removed net N$5: CN1.SH1, CN1.SH3, CN3.P1
- net GND: now also CN3.P1, CN3.P38, CN3.P41, CN3.P55; no longer CN1.P19, CN1.P20, CN1.P22, CN1.P23, CN1.P4, CN1.P5, CN1.P58, CN1.P59, CN1.P6, CN1.P60, CN3.P4, CN3.P40, CN3.P43, CN3.P58
- net PROC_PWR: now also CN3.P54; no longer CN1.P7, CN3.P55
- net SEN_B_D0_N: now also CN3.P28; no longer CN1.P33, CN3.P29
- net SEN_B_D0_P: now also CN3.P29; no longer CN1.P32, CN3.P30
- net SEN_B_D12_N: now also CN3.P20; no longer CN1.P41, CN3.P21
- net SEN_B_D12_P: now also CN3.P21; no longer CN1.P40, CN3.P22
- net SEN_B_D15_N: now also CN3.P16; no longer CN1.P45, CN3.P17
- net SEN_B_D15_P: now also CN3.P17; no longer CN1.P44, CN3.P18
- net SEN_B_D18_N: now also CN3.P15; no longer CN1.P46, CN3.P16
- net SEN_B_D18_P: now also CN3.P14; no longer CN1.P47, CN3.P15
- net SEN_B_D21_N: now also CN3.P11; no longer CN1.P50, CN3.P12
- net SEN_B_D21_P: now also CN3.P10; no longer CN1.P51, CN3.P11
- net SEN_B_D3_N: now also CN3.P26; no longer CN1.P35, CN3.P27
- net SEN_B_D3_P: now also CN3.P27; no longer CN1.P34, CN3.P28
- net SEN_B_D6_N: now also CN3.P33; no longer CN1.P28, CN3.P34
- net SEN_B_D6_P: now also CN3.P32; no longer CN1.P29, CN3.P33
- net SEN_B_D9_N: now also CN3.P25; no longer CN1.P36, CN3.P26
- net SEN_B_D9_P: now also CN3.P24; no longer CN1.P37, CN3.P25
- net SEN_CLK_IN: now also CN3.P46; no longer CN1.P15, CN3.P47
- net SEN_CLK_N: now also CN3.P5; no longer CN1.P56, CN3.P6
- net SEN_CLK_P: now also CN3.P4; no longer CN1.P57, CN3.P5
- net SEN_PWR_EN: now also CN3.P40; no longer CN1.P21, CN3.P41
- net SEN_SPI_!CS: now also CN3.P45; no longer CN1.P16, CN3.P46
- net SEN_SPI_MISO: now also CN3.P44; no longer CN1.P17, CN3.P45
- net SEN_SPI_MOSI: now also CN3.P43; no longer CN1.P18, CN3.P44
- net SEN_SPI_SCLK: now also CN3.P50; no longer CN1.P11, CN3.P51
- net SEN_TDIG0: now also CN3.P52; no longer CN1.P9, CN3.P53
- net SEN_TDIG1: now also CN3.P51; no longer CN1.P10, CN3.P52
- net SEN_TEMP1: now also CN3.P47; no longer CN1.P14, CN3.P48
- net SEN_TEXP0: now also CN3.P48; no longer CN1.P13, CN3.P49
- net SEN_T_D0_N: now also CN3.P36; no longer CN1.P25, CN3.P37
- net SEN_T_D0_P: now also CN3.P37; no longer CN1.P24, CN3.P38
- net SEN_T_D12_N: now also CN3.P23; no longer CN1.P38, CN3.P24
- net SEN_T_D12_P: now also CN3.P22; no longer CN1.P39, CN3.P23
- net SEN_T_D15_N: now also CN3.P9; no longer CN1.P52, CN3.P10
- net SEN_T_D15_P: now also CN3.P8; no longer CN1.P53, CN3.P9
- net SEN_T_D18_N: now also CN3.P12; no longer CN1.P49, CN3.P13
- net SEN_T_D18_P: now also CN3.P13; no longer CN1.P48, CN3.P14
- net SEN_T_D21_N: now also CN3.P7; no longer CN1.P54, CN3.P8
- net SEN_T_D21_P: now also CN3.P6; no longer CN1.P55, CN3.P7
- net SEN_T_D3_N: now also CN3.P35; no longer CN1.P26, CN3.P36
- net SEN_T_D3_P: now also CN3.P34; no longer CN1.P27, CN3.P35
- net SEN_T_D6_N: now also CN3.P30; no longer CN1.P31, CN3.P31
- net SEN_T_D6_P: now also CN3.P31; no longer CN1.P30, CN3.P32
- net SEN_T_D9_N: now also CN3.P19; no longer CN1.P42, CN3.P20
- net SEN_T_D9_P: now also CN3.P18; no longer CN1.P43, CN3.P19
- net SEN_UART_RX: now also CN3.P49; no longer CN1.P12, CN3.P50
- net SEN_UART_TX: now also CN3.P53; no longer CN1.P8, CN3.P54
- net SYS_PWR_5V: now also CN3.P58; no longer CN1.P1, CN1.P2, CN1.P3, CN3.SH1, CN3.SH3
Routing:
- net GND: track 193.3 -> 175.5 mm, vias 151 -> 131
- net SEN_T_D21_P: track 20.3 -> 8.34 mm
- net SEN_T_D18_N: track 18.4 -> 9.63 mm
- net SYS_PWR_5V: track 23.7 -> 17.7 mm, vias 14 -> 8
- net SEN_T_D15_P: track 19.7 -> 13.7 mm
- net SEN_T_D9_P: track 21.2 -> 16.7 mm
- net SEN_T_D9_N: track 20.0 -> 15.5 mm
- net SEN_T_D3_P: track 15.2 -> 11.2 mm
- net SEN_T_D3_N: track 15.1 -> 11.1 mm
- net SEN_T_D0_P: track 17.4 -> 13.8 mm
- net SEN_T_D0_N: track 17.5 -> 13.9 mm
- net SEN_T_D6_P: track 15.0 -> 11.6 mm
- net SEN_T_D6_N: track 14.5 -> 11.1 mm
- net PROC_PWR: track 117.1 -> 114.4 mm, vias 11 -> 10
- net SEN_UART_TX: track 75.6 -> 73.1 mm
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
Commit message: Sensorboard reworked for correct connector orientation
Routing:
- net GND: track 175.5 -> 193.6 mm, vias 131 -> 151
- net PROC_PWR: track 114.4 -> 129.9 mm
- net SEN_T_D21_P: track 8.34 -> 21.8 mm
- net SEN_T_D18_N: track 9.63 -> 19.9 mm
- net PROC_SWCLK: track 34.3 -> 44.2 mm
- net PROC_SWDIO: track 34.4 -> 44.3 mm
- net PROC_NRESET: track 34.9 -> 43.6 mm
- net SEN_T_D15_P: track 13.7 -> 21.2 mm
- net SEN_T_D9_P: track 16.7 -> 22.7 mm
- net SEN_T_D9_N: track 15.5 -> 21.5 mm
- net SYS_PWR_5V: track 17.7 -> 23.3 mm, vias 8 -> 14
- net SEN_T_D3_N: track 11.1 -> 16.6 mm
- net SEN_T_D3_P: track 11.2 -> 16.7 mm
- net SEN_T_D0_P: track 13.8 -> 18.9 mm
- net SEN_T_D0_N: track 13.9 -> 19.0 mm
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