File: interface.sch (EAGLE design)
At the start: 75 parts, among them CN1 61083-103400LF, CN2 FH52E-60S-0.5SH, CN3 61083-103400LF, CN4 2.1mm DC Jack, CN5 61 PIN 0.2mm FFC, Q1 2N7002, U1 TLV3201, U2 ADJ BUCK, U24 ADJ BUCK, U27 LM2731X, U3 PI4ULS3V204ZBEX, U4 TPS54233D

Commit message: Interface PCB laid out. Needs thorough review, and FPGA pinout test
Parts:
- removed C111: 0.1uF 10V, c_0402:0402ZC104KAT2A
- removed C263: 22uF 6.3V, c_1206:C1206C226K9PACTU
- removed C265: 10uF 10V, c_1206:C1206C106K8PACTU
- removed C272, C274: 10uF 16V, c_1206:C1206C106K4PAC7210
- removed C273: 330pF 50V, c_0603:C0603C331J5GACTU
- removed D5: PMEG4010BEA, DIODES:PMEG4010BEA
- removed L6: 10uH 1.3A, INDUCTORS:IFSC1515AHER100M01
- removed R70, R71, R81: 10k, r_0603:CRCW060310K0FKTA
- removed R72: 15k, r_0603:CRCW060315K0FKEA
- removed R79: 95.3k, r_0603:CRCW060395K3FKEA
- removed R80: 13.3k, r_0603:CRCW060313K3FKEB
- removed U24: ADJ BUCK, ICs:LMZM23600SILT
- added C17: 10uF 25V, c_1206:C1206C106K3PACTU
- added C18: 68pF 100V, c_0603:06031A680JAT2A
- added C24: 0.1uF 16V, c_0603:C0603C104K4RAC7411
- added C34, C35: 22uF 10V, c_1206:C1206C226K8RAC7210
- added D4: B360A-13-F, DIODES:B360A-13-F
- added L2: 22uH, INDUCTORS:MSS1038-223MLC
- added MECH1, MECH2, MECH3, MECH4: 6mm x 3mm, MISC:MOUNTHOLE
- added R14, R19, R20, R21: 10k, r_0603:CRCW060310K0FKTA
- added R15: 21k, r_0603:CRCW060321K0FKEA
- added R18: 1.91k, r_0603:CRCW06031K91FKEA
- added U6: TPS54233D, ICs:TPS54233D
- C1, C2, C4: value 22uF 6.3V -> 0.1uF 16V; device c_1206:C1206C226K9PACTU -> c_0603:C0603C104J4REC7867
- C10: value 0.1uF 16V -> 22uF 6.3V; device c_0603:C0603C104K4RAC7411 -> c_1206:C1206C226K9PACTU
- C11: value 22uF 10V -> 22uF 6.3V; device c_1206:C1206C226K8RAC7210 -> c_1206:C1206C226K9PACTU
- C12: value 22uF 10V -> 330pF 50V; device c_1206:C1206C226K8RAC7210 -> c_0603:C0603C331J5GACTU
- C13: value 68pF 100V -> 22uF 6.3V; device c_0603:06031A680JAT2A -> c_1206:C1206C226K9PACTU
- C14: value 1800pF 50V -> 10uF 16V; device c_0603:06035C182JAT2A -> c_1206:C1206C106K4PAC7210
- C16: value 10uF 25V -> 1800pF 50V; device c_1206:C1206C106K3PACTU -> c_0603:06035C182JAT2A
- C3, C9: value 0.1uF 16V -> 10uF 10V; device c_0603:C0603C104J4REC7867 -> c_1206:C1206C106K8PACTU
- C5: value 10uF 10V -> 22uF 6.3V; device c_1206:C1206C106K8PACTU -> c_1206:C1206C226K9PACTU
- C8: value 0.1uF 16V -> 10uF 16V; device c_0603:C0603C104J4REC7867 -> c_1206:C1206C106K4PAC7210
- CN2: value FH52E-60S-0.5SH -> 61083-103400LF; device CONNECTORs:FH52E-60S-0.5SH -> CONNECTORs:61083-103400LF
- CN3: value 61083-103400LF -> FH52E-60S-0.5SH; device CONNECTORs:61083-103400LF -> CONNECTORs:FH52E-60S-0.5SH
- D1: value B360A-13-F -> PMEG4010BEA; device DIODES:B360A-13-F -> DIODES:PMEG4010BEA
- L1: value 22uH -> 10uH 1.3A; device INDUCTORS:MSS1038-223MLC -> INDUCTORS:IFSC1515AHER100M01
- R10: value 47.5k -> 15k; device r_0603:CRCW060347K5FKEA -> r_0603:CRCW060315K0FKEB
- R11: value 10k -> 95.3k; device r_0603:CRCW060310K0FKTA -> r_0603:CRCW060395K3FKEA
- R12: value 1.91k -> 13.3k; device r_0603:CRCW06031K91FKEA -> r_0603:CRCW060313K3FKEB
- R13: value 21k -> 47.5k; device r_0603:CRCW060321K0FKEA -> r_0603:CRCW060347K5FKEA
- R5: device r_0603:CRCW060315K0FKEB -> r_0603:CRCW060315K0FKEA
- R6: value 12.1k -> 10k; device r_0603:CRCW060312K1FKEB -> r_0603:CRCW060310K0FKTA
- R9: value 10k -> 12.1k; device r_0603:CRCW060310K0FKTA -> r_0603:CRCW060312K1FKEB
- U2: value ADJ BUCK -> PI4ULS3V204ZBEX; device ICs:LMZM23600SILT -> ICs:PI4ULS3V204
- U3: value PI4ULS3V204ZBEX -> ADJ BUCK; device ICs:PI4ULS3V204 -> ICs:LMZM23600SILT
- U4: value TPS54233D -> ADJ BUCK; device ICs:TPS54233D -> ICs:LMZM23600SILT
- renumbered C130 to C22, C131 to C27, C132 to C33, C133 to C21, C134 to C32, C135 to C31, C136 to C19, C138 to C20, C140 to C30, C142 to C29, C143 to C25, C144 to C28, C145 to C23, C146 to C26, R94 to R16, R95 to R17, U27 to U5
Connections:
- removed net PG_1V8: R3.2, U1.+
- new net FPGA_VCCO_EN: CN2.10, R1.2, U1.+
- net !INIT: now also CN2.9; no longer CN3.9
- net EVF_LVDS_CLK0_N: now also CN2.26; no longer CN3.26
- net EVF_LVDS_CLK0_P: now also CN2.24; no longer CN3.24
- net EVF_LVDS_CLK1_N: now also CN2.47; no longer CN3.47
- net EVF_LVDS_CLK1_P: now also CN2.49; no longer CN3.49
- net EVF_LVDS_D0_N: now also CN2.20; no longer CN3.20
- net EVF_LVDS_D0_P: now also CN2.18; no longer CN3.18
- net EVF_LVDS_D1_N: now also CN2.30; no longer CN3.30
- net EVF_LVDS_D1_P: now also CN2.32; no longer CN3.32
- net EVF_LVDS_D2_N: now also CN2.35; no longer CN3.35
- net EVF_LVDS_D2_P: now also CN2.37; no longer CN3.37
- net EVF_LVDS_D7_N: now also CN2.61; no longer CN3.61
- net EVF_LVDS_D7_P: now also CN2.63; no longer CN3.63
- net EVF_LVDS_D8_N: now also CN2.43; no longer CN3.43
- net EVF_LVDS_D8_P: now also CN2.41; no longer CN3.41
- net EVF_LVDS_D9_N: now also CN2.53; no longer CN3.53
- net EVF_LVDS_D9_P: now also CN2.55; no longer CN3.55
- net EVF_PWR_10V: now also C12.2, C14.2, D1.K, R11.2; no longer C273.2, C274.2, D5.K, R79.2
- net EVF_PWR_10V_EN: now also R8.2; no longer R81.2
- net EVF_PWR_1V8: now also C10.2, C11.2, C13.2, C4.1, R21.2, R9.2, U2.VCCB, U4.VOUT; no longer C4.2, C6.2, C7.2, C9.1, R6.2, R8.2, U2.VOUT, U3.VCCB
- net EVF_PWR_1V8_EN: now also R7.2, U4.EN; no longer R4.2, U2.EN
- net EVF_SPI_!CS: now also U2.B4; no longer U3.B4
- net EVF_SPI_MISO: now also U2.B3; no longer U3.B3
- net EVF_SPI_MOSI: now also U2.B2; no longer U3.B2
- net EVF_SPI_SCLK: now also U2.B1; no longer U3.B1
- net EVF_SYS_!RESET: now also R21.1; no longer R8.1
- net FPGA_EVF_SPI_!CS: now also CN2.25, U2.A4; no longer CN3.25, U3.A4
- net FPGA_EVF_SPI_MISO: now also CN2.23, U2.A3; no longer CN3.23, U3.A3
- net FPGA_EVF_SPI_MOSI: now also CN2.19, U2.A2; no longer CN3.19, U3.A2
- net FPGA_EVF_SPI_SCLK: now also CN2.17, U2.A1; no longer CN3.17, U3.A1
- net FPGA_EVF_SYS_!RESET: now also CN2.29, R20.1; no longer CN3.29, R7.1
- net GND: now also C1.2, C10.1, C14.1, C17.1, C18.1, C2.2, C3.1, C34.1, C35.1, C4.2, C8.1, C9.1, CN2.15, CN2.16, CN2.21, CN2.22, CN2.27, CN2.28, CN2.33, CN2.34, CN2.39, CN2.40, CN2.45, CN2.46, CN2.51, CN2.52, CN2.65, CN2.66, CN2.71, CN2.72, CN2.77, CN2.85, CN2.86, CN2.91, CN2.92, CN3.P1, CN3.P2, CN3.P3, CN3.P38, CN3.P39, CN3.P41, CN3.P42, CN3.P55, CN3.P56, CN3.P57, D4.A, R10.1, R14.1, R15.1, R18.1, R20.2, R6.1, R7.1, R8.1, U3.MODE/SYNC, U4.MODE/SYNC, U6.GND; no longer C1.1, C111.1, C12.1, C16.1, C2.1, C263.1, C265.1, C272.1, C274.1, C3.2, C4.1, C8.2, C9.2, CN2.P1, CN2.P2, CN2.P3, CN2.P38, CN2.P39, CN2.P41, CN2.P42, CN2.P55, CN2.P56, CN2.P57, CN3.15, CN3.16, CN3.21, CN3.22, CN3.27, CN3.28, CN3.33, CN3.34, CN3.39, CN3.40, CN3.45, CN3.46, CN3.51, CN3.52, CN3.65, CN3.66, CN3.71, CN3.72, CN3.77, CN3.85, CN3.86, CN3.91, CN3.92, D1.A, R13.1, R5.1, R7.2, R70.1, R71.1, R80.1, R81.1, R9.1, U2.MODE/SYNC, U24.GND, U24.MODE/SYNC
- net N$1: now also R10.2, R9.1, U4.FB; no longer R5.2, R6.1, U2.FB
- net N$10: now also C16.1, R15.2; no longer C14.1, R13.2
- net N$100: now also CN2.73; no longer CN3.73
- net N$101: now also CN2.75; no longer CN3.75
- net N$102: now also CN2.81; no longer CN3.81
- net N$103: now also CN2.83; no longer CN3.83
- net N$104: now also CN2.87; no longer CN3.87
- net N$105: now also CN2.89; no longer CN3.89
- net N$11: now also U6.SS; no longer U4.SS
- net N$116: now also CN2.14; no longer CN3.14
- net N$119: now also D1.A, L1.2; no longer D5.A, L6.2
- net N$121: now also C12.1, R11.1, R12.2; no longer C273.1, R79.1, R80.2
- net N$125: now also CN2.36; no longer CN3.36
- net N$126: now also CN2.38; no longer CN3.38
- net N$127: now also CN2.42; no longer CN3.42
- net N$128: now also CN2.44; no longer CN3.44
- net N$129: now also CN2.48; no longer CN3.48
- net N$130: now also CN2.50; no longer CN3.50
- net N$131: now also CN2.54; no longer CN3.54
- net N$132: now also CN2.56; no longer CN3.56
- net N$133: now also CN2.62; no longer CN3.62
- net N$134: now also CN2.64; no longer CN3.64
- net N$135: now also CN2.68; no longer CN3.68
- net N$136: now also CN2.70; no longer CN3.70
- net N$137: now also CN2.74; no longer CN3.74
- net N$138: now also CN2.76; no longer CN3.76
- net N$139: now also CN2.82; no longer CN3.82
- net N$140: now also CN2.84; no longer CN3.84
- net N$141: now also CN2.88; no longer CN3.88
- net N$142: now also CN2.90; no longer CN3.90
- net N$2: now also R3.2; no longer R1.2
- net N$3: now also CN2.31; no longer CN3.31
- net N$4: now also C24.1, D4.K, L2.1, U6.PH; no longer C10.1, D1.K, L1.1, U4.PH
- net N$5: now also C24.2, U6.BOOT; no longer C10.2, U4.BOOT
- net N$6: now also C17.2, R13.2, U6.VIN; no longer C16.2, R10.2, U4.VIN
- net N$67: now also R5.1, R6.2, U3.FB; no longer R71.2, R72.1, U24.FB
- net N$7: now also R13.1, R14.2, U6.EN; no longer R10.1, R9.2, U4.EN
- net N$79: now also CN2.13; no longer CN3.13
- net N$8: now also R18.2, R19.1, U6.VSNS; no longer R11.1, R12.2, U4.VSNS
- net N$9: now also C16.2, C18.2, U6.COMP; no longer C13.2, C14.2, U4.COMP
- net N$98: now also CN2.67; no longer CN3.67
- net N$99: now also CN2.69; no longer CN3.69
- net PG_MODULE: now also CN2.11; no longer CN3.11
- net PMOD_D0: now also CN2.1; no longer CN3.1
- net PMOD_D1: now also CN2.2; no longer CN3.2
- net PMOD_D2: now also CN2.3; no longer CN3.3
- net PMOD_D3: now also CN2.4; no longer CN3.4
- net PMOD_D4: now also CN2.5; no longer CN3.5
- net PMOD_D5: now also CN2.6; no longer CN3.6
- net PMOD_D6: now also CN2.7; no longer CN3.7
- net PMOD_D7: now also CN2.8; no longer CN3.8
- net SEN_B_D0_N: now also CN3.P28; no longer CN2.P28
- net SEN_B_D0_P: now also CN3.P29; no longer CN2.P29
- net SEN_B_D12_N: now also CN3.P20; no longer CN2.P20
- net SEN_B_D12_P: now also CN3.P21; no longer CN2.P21
- net SEN_B_D15_N: now also CN3.P16; no longer CN2.P16
- net SEN_B_D15_P: now also CN3.P17; no longer CN2.P17
- net SEN_B_D18_N: now also CN3.P15; no longer CN2.P15
- net SEN_B_D18_P: now also CN3.P14; no longer CN2.P14
- net SEN_B_D21_N: now also CN3.P11; no longer CN2.P11
- net SEN_B_D21_P: now also CN3.P10; no longer CN2.P10
- net SEN_B_D3_N: now also CN3.P26; no longer CN2.P26
- net SEN_B_D3_P: now also CN3.P27; no longer CN2.P27
- net SEN_B_D6_N: now also CN3.P33; no longer CN2.P33
- net SEN_B_D6_P: now also CN3.P32; no longer CN2.P32
- net SEN_B_D9_N: now also CN3.P25; no longer CN2.P25
- net SEN_B_D9_P: now also CN3.P24; no longer CN2.P24
- net SEN_CLK_IN: now also CN3.P46; no longer CN2.P46
- net SEN_CLK_N: now also CN3.P5; no longer CN2.P5
- net SEN_CLK_P: now also CN3.P4; no longer CN2.P4
- net SEN_PWR_EN: now also CN3.P40; no longer CN2.P40
- net SEN_SPI_!CS: now also CN3.P45; no longer CN2.P45
- net SEN_SPI_MISO: now also CN3.P44; no longer CN2.P44
- net SEN_SPI_MOSI: now also CN3.P43; no longer CN2.P43
- net SEN_SPI_SCLK: now also CN3.P50; no longer CN2.P50
- net SEN_SYS_!RESET: now also CN3.P49; no longer CN2.P49
- net SEN_TDIG0: now also CN3.P52; no longer CN2.P52
- net SEN_TDIG1: now also CN3.P51; no longer CN2.P51
- net SEN_TEMP1: now also CN3.P47; no longer CN2.P47
- net SEN_TEMP_SPI_!CS: now also CN3.P53; no longer CN2.P53
- net SEN_TEXP0: now also CN3.P48; no longer CN2.P48
- net SEN_T_D0_N: now also CN3.P36; no longer CN2.P36
- net SEN_T_D0_P: now also CN3.P37; no longer CN2.P37
- net SEN_T_D12_N: now also CN3.P23; no longer CN2.P23
- net SEN_T_D12_P: now also CN3.P22; no longer CN2.P22
- net SEN_T_D15_N: now also CN3.P9; no longer CN2.P9
- net SEN_T_D15_P: now also CN3.P8; no longer CN2.P8
- net SEN_T_D18_N: now also CN3.P12; no longer CN2.P12
- net SEN_T_D18_P: now also CN3.P13; no longer CN2.P13
- net SEN_T_D21_N: now also CN3.P7; no longer CN2.P7
- net SEN_T_D21_P: now also CN3.P6; no longer CN2.P6
- net SEN_T_D3_N: now also CN3.P35; no longer CN2.P35
- net SEN_T_D3_P: now also CN3.P34; no longer CN2.P34
- net SEN_T_D6_N: now also CN3.P30; no longer CN2.P30
- net SEN_T_D6_P: now also CN3.P31; no longer CN2.P31
- net SEN_T_D9_N: now also CN3.P19; no longer CN2.P19
- net SEN_T_D9_P: now also CN3.P18; no longer CN2.P18
- net SYS_PWR_2V5: now also C2.1, C5.2, C6.2, C7.2, CN2.78, CN2.79, CN2.80, CN3.P54, R5.2, U2.EN, U2.VCCA, U3.VOUT; no longer C1.2, C2.2, C263.2, C8.1, CN2.P54, CN3.10, CN3.78, CN3.79, CN3.80, R72.2, U24.VOUT, U3.EN, U3.VCCA
- net SYS_PWR_5V: now also C1.1, C3.2, C34.2, C35.2, C8.2, C9.2, CN2.12, CN2.57, CN2.58, CN2.59, CN2.60, CN3.P58, CN3.P59, CN3.P60, L1.1, L2.2, R19.2, U3.VIN, U4.VIN; no longer C11.2, C111.2, C12.2, C265.2, C272.2, C3.1, C5.2, CN2.P58, CN2.P59, CN2.P60, CN3.12, CN3.57, CN3.58, CN3.59, CN3.60, L1.2, L6.1, R11.2, U2.VIN, U24.VIN
- net SYS_VCCO_EN: now also R4.2, U3.EN; no longer R70.2, U24.EN
Other:
- note added: "2021.10.18 - GSWDH LTD. IMAGE SENSOR INTERFACE REVISION 1.0.0 DESIGN BY GEORGE WALLER AT GSWDH LTD. GEORGEWALLER@GSWDH.CO.UK CONFIDENTIAL. FOR THE INTENDED READER ONLY."
- note removed: "2021.10.18 - GSWDH LTD. IMAGE SENSOR MODULE REVISION 1.0.0 DESIGN BY GEORGE WALLER AT GSWDH LTD. GEORGEWALLER@GSWDH.CO.UK CONFIDENTIAL. FOR THE INTENDED READER ONLY."

Commit message: Interface modified with in stock components
Parts:
- removed C10, C11: 22uF 6.3V, c_1206:C1206C226K9PACTU
- removed C2, C4: 0.1uF 16V, c_0603:C0603C104J4REC7867
- removed C9: 10uF 10V, c_1206:C1206C106K8PACTU
- removed R16, R17: 10k, r_0603:CRCW060310K0FKTA
- removed U2: PI4ULS3V204ZBEX, ICs:PI4ULS3V204
- removed U4: ADJ BUCK, ICs:LMZM23600SILT
- added C36: 100pF 25V, c_0603:06033A101FAT2A
- added CN6: PCB Tab, CONNECTORs:PCB_TAB_SMALL
- added L3, L5: 2.2uH 3A, INDUCTORS:IFSC1515AHER2R2M01
- added MECH5, MECH6: 6mm x 3mm, MISC:MOUNTHOLE
- added R22: 10R, r_0603:CRCW060310R0FKTA
- added R23, R25: 1.5k, r_0603:CRCW06031K50FKEB
- added R24, R26: 680R, r_0603:CRCW0603680RFKEB
- added U7: PAM2312, ICs:PAM2312
- C13, C5, C7: value 22uF 6.3V -> 10uF 10V; device c_1206:C1206C226K9PACTU -> c_1206:C1206C106K8PACTU
- C6: value 22uF 6.3V -> 100pF 25V; device c_1206:C1206C226K9PACTU -> c_0603:06033A101FAT2A
- CN4: value 2.1mm DC Jack -> PCB Tab; device CONNECTORs:PJ-202AH -> CONNECTORs:PCB_TAB_SMALL
- L2: device INDUCTORS:MSS1038-223MLC -> INDUCTORS:ECS-MPIL0630-220MC
- R10: value 15k -> 150k; device r_0603:CRCW060315K0FKEB -> r_0603:CRCW0603150KFKEB
- R4: value 10k -> 200k; device r_0603:CRCW060310K0FKTA -> r_0603:CRCW0603200KFKEB
- R5: value 15k -> 100k; device r_0603:CRCW060315K0FKEA -> r_0603:CRCW0603100KFKEB
- R6: value 10k -> 475k; device r_0603:CRCW060310K0FKTA -> r_0603:CRCW0603475KFKTA
- R7: value 10k -> 1.5k; device r_0603:CRCW060310K0FKTA -> r_0603:CRCW06031K50FKEB
- R9: value 12.1k -> 680R; device r_0603:CRCW060312K1FKEB -> r_0603:CRCW0603680RFKEB
- U3: value ADJ BUCK -> PAM2312; device ICs:LMZM23600SILT -> ICs:PAM2312
Connections:
- removed net N$1: R10.2, R9.1, U4.FB
- removed net N$36: CN1.81
- removed net N$67: R5.1, R6.2, U3.FB
- removed net N$79: CN2.13
- new net N$14: L3.1, U7.SW
- new net N$15: C36.1, R10.2, R6.1, U7.FB
- new net N$17: L5.1, U3.SW
- new net N$18: C6.1, R4.1, R5.2, U3.FB
- net EVF_PWR_10V_EN: now also CN1.81
- net EVF_PWR_1V8: now also C3.2, C6.2, L5.2, R4.2; no longer C10.2, C11.2, C13.2, C4.1, R16.2, R9.2, U2.VCCB, U4.VOUT
- net EVF_PWR_1V8_EN: now also CN2.13, U3.EN; no longer R7.2, U4.EN
- net EVF_SPI_!CS: now also R25.2, R26.2; no longer R16.1, U2.B4
- net EVF_SPI_MISO: now also R22.2; no longer R17.1, U2.B3
- net EVF_SPI_MOSI: now also R23.2, R24.2; no longer U2.B2
- net EVF_SPI_SCLK: now also R7.2, R9.2; no longer U2.B1
- net FPGA_EVF_SPI_!CS: now also R26.1; no longer U2.A4
- net FPGA_EVF_SPI_MISO: now also R22.1; no longer U2.A3
- net FPGA_EVF_SPI_MOSI: now also R24.1; no longer U2.A2
- net FPGA_EVF_SPI_SCLK: now also R9.1; no longer U2.A1
- net GND: now also CN6.1, R23.1, R25.1, R5.1, U7.GND; no longer C10.1, C11.1, C2.2, C4.2, C6.1, C9.1, CN4.GND, R17.2, R4.1, R6.1, U2.GND, U3.MODE/SYNC, U4.GND, U4.MODE/SYNC
- net N$12: now also CN4.1; no longer CN4.V+
- net SYS_PWR_2V5: now also C36.2, L3.2, R6.2; no longer C2.1, C5.2, C6.2, R5.2, U2.EN, U2.VCCA, U3.VOUT
- net SYS_PWR_5V: now also C13.2, C5.2, U7.VIN; no longer C3.2, C9.2, U4.VIN
- net SYS_VCCO_EN: now also U7.EN; no longer R4.2, U3.EN
