File: sensor.sch (EAGLE design)
At the start: 149 parts, among them CN1 FH52E-60S-0.5SH, CN5 TC2030, U1 STM32L031G6, U18 MIC5271, U19 LM2662, U2 GMAX0505-DV, U20 MAX25300B, U21 MAX25300B, U22 MAX25300B, U23 MAX25300B, U24 3.3V BUCK, U25 MAX6627

Commit message: Sensor PCB routed and DRC passes, needs review of layer stack and diff pairs
Parts:
- removed C211: 22uF 6.3V, c_1206:C1206C226K9PACTU
- added C8: 0.1uF 10V, c_0402:0402ZD104KAT2A
Connections:
- net SEN_PWR_RDY renamed SEN_PWR_EN
- net GND: now also C8.1; no longer C211.1
- net SEN_CLK_IN: now also CN1.P15; no longer CN1.P18
- net SEN_PWR_3V3A: now also C8.2
- net SEN_PWR_4V1: no longer C211.2
- net SEN_SPI_!CS: now also CN1.P16; no longer CN1.P12
- net SEN_SPI_MISO: now also CN1.P17; no longer CN1.P11
- net SEN_SPI_MOSI: now also CN1.P18; no longer CN1.P10
- net SEN_SPI_SCLK: now also CN1.P11; no longer CN1.P9
- net SEN_SYS_!RESET: now also CN1.P12; no longer CN1.P17
- net SEN_TDIG0: now also CN1.P9; no longer CN1.P15
- net SEN_TDIG1: now also CN1.P10; no longer CN1.P16
- net SEN_TEMP1: now also CN1.P14; no longer CN1.P13
- net SEN_TEXP0: now also CN1.P13; no longer CN1.P14
Changed lines of the file:
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@@
 <part name="C209" library="c_0402" deviceset="0402ZD104KAT2A" device="" value="0.1uF 10V"/>
 <part name="GND227" library="NETS" deviceset="GND" device=""/>
-<part name="C211" library="c_1206" deviceset="C1206C226K9PACTU" device="" value="22uF 6.3V"/>
-<part name="GND229" library="NETS" deviceset="GND" device=""/>
 <part name="C212" library="c_0402" deviceset="0402ZD104KAT2A" device="" value="0.1uF 10V"/>
 <part name="C213" library="c_0402" deviceset="04026D475KAT2A" device="" value="4.7uF 6.3V"/>
@@
 <part name="R1" library="r_0603" deviceset="CRCW060310K0FKTA" device="" value="10k"/>
 <part name="GND10" library="NETS" deviceset="GND" device=""/>
+<part name="C8" library="c_0402" deviceset="0402ZD104KAT2A" device="" value="0.1uF 10V"/>
+<part name="GND11" library="NETS" deviceset="GND" device=""/>
 </parts>
 <sheets>
@@
 </segment>
 <segment>
-<pinref part="CN1" gate="G$1" pin="P17"/>
-<wire x1="93.98" y1="33.02" x2="129.54" y2="33.02" width="0.1524" layer="91"/>
-<label x="96.52" y="33.02" size="1.778" layer="95"/>
+<pinref part="CN1" gate="G$1" pin="P12"/>
+<wire x1="93.98" y1="45.72" x2="129.54" y2="45.72" width="0.1524" layer="91"/>
+<label x="96.52" y="45.72" size="1.778" layer="95"/>
 </segment>
 </net>
@@
 </segment>
 <segment>
-<pinref part="CN1" gate="G$1" pin="P18"/>
-<wire x1="93.98" y1="30.48" x2="129.54" y2="30.48" width="0.1524" layer="91"/>
-<label x="96.52" y="30.48" size="1.778" layer="95"/>
+<pinref part="CN1" gate="G$1" pin="P15"/>
+<wire x1="93.98" y1="38.1" x2="129.54" y2="38.1" width="0.1524" layer="91"/>
+<label x="96.52" y="38.1" size="1.778" layer="95"/>
 </segment>
 </net>
@@
 </segment>
 <segment>
-<pinref part="CN1" gate="G$1" pin="P15"/>
-<wire x1="93.98" y1="38.1" x2="129.54" y2="38.1" width="0.1524" layer="91"/>
-<label x="96.52" y="38.1" size="1.778" layer="95"/>
+<pinref part="CN1" gate="G$1" pin="P9"/>
+<wire x1="93.98" y1="53.34" x2="129.54" y2="53.34" width="0.1524" layer="91"/>
+<label x="96.52" y="53.34" size="1.778" layer="95"/>
 </segment>
 </net>
@@
 </segment>
 <segment>
-<pinref part="CN1" gate="G$1" pin="P16"/>
-<wire x1="93.98" y1="35.56" x2="129.54" y2="35.56" width="0.1524" layer="91"/>
-<label x="96.52" y="35.56" size="1.778" layer="95"/>
+<pinref part="CN1" gate="G$1" pin="P10"/>
+<wire x1="93.98" y1="50.8" x2="129.54" y2="50.8" width="0.1524" layer="91"/>
+<label x="96.52" y="50.8" size="1.778" layer="95"/>
 </segment>
 </net>
@@
 </segment>
 <segment>
+<pinref part="CN1" gate="G$1" pin="P13"/>
+<wire x1="93.98" y1="43.18" x2="129.54" y2="43.18" width="0.1524" layer="91"/>
+<label x="96.52" y="43.18" size="1.778" layer="95"/>
+</segment>
+</net>
+<net name="SEN_TEMP1" class="0">
+<segment>
+<pinref part="U2" gate="A" pin="TEXP1"/>
+<wire x1="-104.14" y1="106.68" x2="-144.78" y2="106.68" width="0.1524" layer="91"/>
+<label x="-142.24" y="106.68" size="1.778" layer="95"/>
+</segment>
+<segment>
 <pinref part="CN1" gate="G$1" pin="P14"/>
 <wire x1="93.98" y1="40.64" x2="129.54" y2="40.64" width="0.1524" layer="91"/>
 <label x="96.52" y="40.64" size="1.778" layer="95"/>
-</segment>
-</net>
-<net name="SEN_TEMP1" class="0">
-<segment>
-<pinref part="U2" gate="A" pin="TEXP1"/>
-<wire x1="-104.14" y1="106.68" x2="-144.78" y2="106.68" width="0.1524" layer="91"/>
-<label x="-142.24" y="106.68" size="1.778" layer="95"/>
-</segment>
-<segment>
-<pinref part="CN1" gate="G$1" pin="P13"/>
-<wire x1="93.98" y1="43.18" x2="129.54" y2="43.18" width="0.1524" layer="91"/>
-<label x="96.52" y="43.18" size="1.778" layer="95"/>
 </segment>
 </net>
@@
 </segment>
 <segment>
-<pinref part="CN1" gate="G$1" pin="P12"/>
-<wire x1="93.98" y1="45.72" x2="129.54" y2="45.72" width="0.1524" layer="91"/>
-<label x="96.52" y="45.72" size="1.778" layer="95"/>
+<pinref part="CN1" gate="G$1" pin="P16"/>
+<wire x1="93.98" y1="35.56" x2="129.54" y2="35.56" width="0.1524" layer="91"/>
+<label x="96.52" y="35.56" size="1.778" layer="95"/>
 </segment>
 </net>
@@
 </segment>
 <segment>
-<pinref part="CN1" gate="G$1" pin="P9"/>
-<wire x1="93.98" y1="53.34" x2="129.54" y2="53.34" width="0.1524" layer="91"/>
-<label x="96.52" y="53.34" size="1.778" layer="95"/>
+<pinref part="CN1" gate="G$1" pin="P11"/>
+<wire x1="93.98" y1="48.26" x2="129.54" y2="48.26" width="0.1524" layer="91"/>
+<label x="96.52" y="48.26" size="1.778" layer="95"/>
 </segment>
 </net>
@@
 </segment>
 <segment>
-<pinref part="CN1" gate="G$1" pin="P10"/>
-<wire x1="93.98" y1="50.8" x2="129.54" y2="50.8" width="0.1524" layer="91"/>
-<label x="96.52" y="50.8" size="1.778" layer="95"/>
+<pinref part="CN1" gate="G$1" pin="P18"/>
+<wire x1="93.98" y1="30.48" x2="129.54" y2="30.48" width="0.1524" layer="91"/>
+<label x="96.52" y="30.48" size="1.778" layer="95"/>
 </segment>
 </net>
@@
 </segment>
 <segment>
-<pinref part="CN1" gate="G$1" pin="P11"/>
-<wire x1="93.98" y1="48.26" x2="129.54" y2="48.26" width="0.1524" layer="91"/>
-<label x="96.52" y="48.26" size="1.778" layer="95"/>
+<pinref part="CN1" gate="G$1" pin="P17"/>
+<wire x1="93.98" y1="33.02" x2="129.54" y2="33.02" width="0.1524" layer="91"/>
+<label x="96.52" y="33.02" size="1.778" layer="95"/>
 </segment>
 </net>
@@
 </segment>
 </net>
-<net name="SEN_PWR_RDY" class="0">
+<net name="SEN_PWR_EN" class="0">
 <segment>
 <pinref part="CN1" gate="G$1" pin="P21"/>
@@
 <attribute name="VALUE" x="45.72" y="-43.18" size="1.778" layer="96" align="center"/>
 </instance>
-<instance part="C211" gate="G$1" x="38.1" y="-30.48" smashed="yes" rot="R90">
-<attribute name="NAME" x="35.56" y="-30.48" size="1.27" layer="95" rot="R90" align="center"/>
-<attribute name="VALUE" x="40.64" y="-30.48" size="1.27" layer="96" rot="R90" align="center"/>
-</instance>
-<instance part="GND229" gate="G$1" x="38.1" y="-40.64" smashed="yes">
-<attribute name="VALUE" x="38.1" y="-43.18" size="1.778" layer="96" align="center"/>
-</instance>
 <instance part="C212" gate="G$1" x="60.96" y="-5.08" smashed="yes" rot="R90">
 <attribute name="NAME" x="58.42" y="-5.08" size="1.27" layer="95" rot="R90" align="center"/>
@@
 <instance part="GND235" gate="G$1" x="60.96" y="35.56" smashed="yes">
 <attribute name="VALUE" x="60.96" y="33.02" size="1.778" layer="96" align="center"/>
+</instance>
+<instance part="C8" gate="G$1" x="-30.48" y="-81.28" smashed="yes" rot="R90">
+<attribute name="NAME" x="-33.02" y="-81.28" size="1.27" layer="95" rot="R90" align="center"/>
+<attribute name="VALUE" x="-27.94" y="-81.28" size="1.27" layer="96" rot="R90" align="center"/>
+</instance>
+<instance part="GND11" gate="G$1" x="-30.48" y="-91.44" smashed="yes">
+<attribute name="VALUE" x="-30.48" y="-93.98" size="1.778" layer="96" align="center"/>
 </instance>
 </instances>
@@
 </segment>
 <segment>
-<pinref part="C211" gate="G$1" pin="1"/>
-<pinref part="GND229" gate="G$1" pin="GND"/>
-<wire x1="38.1" y1="-38.1" x2="38.1" y2="-35.56" width="0.1524" layer="91"/>
-</segment>
-<segment>
 <pinref part="C212" gate="G$1" pin="1"/>
 <pinref part="GND230" gate="G$1" pin="GND"/>
@@
 <pinref part="GND235" gate="G$1" pin="GND"/>
 <wire x1="60.96" y1="38.1" x2="60.96" y2="40.64" width="0.1524" layer="91"/>
+</segment>
+<segment>
+<pinref part="C8" gate="G$1" pin="1"/>
+<pinref part="GND11" gate="G$1" pin="GND"/>
+<wire x1="-30.48" y1="-88.9" x2="-30.48" y2="-86.36" width="0.1524" layer="91"/>
 </segment>
 </net>
@@
 <wire x1="-7.62" y1="-73.66" x2="-15.24" y2="-73.66" width="0.1524" layer="91"/>
 <wire x1="-15.24" y1="-73.66" x2="-22.86" y2="-73.66" width="0.1524" layer="91"/>
-<wire x1="-22.86" y1="-73.66" x2="-127" y2="-73.66" width="0.1524" layer="91"/>
+<wire x1="-22.86" y1="-73.66" x2="-30.48" y2="-73.66" width="0.1524" layer="91"/>
+<wire x1="-30.48" y1="-73.66" x2="-127" y2="-73.66" width="0.1524" layer="91"/>
 <wire x1="60.96" y1="-76.2" x2="60.96" y2="-73.66" width="0.1524" layer="91"/>
 <junction x="60.96" y="-73.66"/>
@@
 <wire x1="-22.86" y1="-76.2" x2="-22.86" y2="-73.66" width="0.1524" layer="91"/>
 <junction x="-22.86" y="-73.66"/>
+<pinref part="C8" gate="G$1" pin="2"/>
+<wire x1="-30.48" y1="-76.2" x2="-30.48" y2="-73.66" width="0.1524" layer="91"/>
+<junction x="-30.48" y="-73.66"/>
 </segment>
 <segment>
@@
 <wire x1="60.96" y1="-22.86" x2="53.34" y2="-22.86" width="0.1524" layer="91"/>
 <wire x1="53.34" y1="-22.86" x2="45.72" y2="-22.86" width="0.1524" layer="91"/>
-<wire x1="45.72" y1="-22.86" x2="38.1" y2="-22.86" width="0.1524" layer="91"/>
-<wire x1="38.1" y1="-22.86" x2="-127" y2="-22.86" width="0.1524" layer="91"/>
+<wire x1="45.72" y1="-22.86" x2="-127" y2="-22.86" width="0.1524" layer="91"/>
 <wire x1="60.96" y1="-25.4" x2="60.96" y2="-22.86" width="0.1524" layer="91"/>
 <junction x="60.96" y="-22.86"/>
@@
 <wire x1="45.72" y1="-25.4" x2="45.72" y2="-22.86" width="0.1524" layer="91"/>
 <junction x="45.72" y="-22.86"/>
-<pinref part="C211" gate="G$1" pin="2"/>
-<wire x1="38.1" y1="-25.4" x2="38.1" y2="-22.86" width="0.1524" layer="91"/>
-<junction x="38.1" y="-22.86"/>
 <label x="-124.46" y="-22.86" size="1.778" layer="95"/>
 </segment>

Commit message: LDO replaced for stock, BoM ordered
Parts:
- R55: value 390R -> 3.9k; device r_0603:CRCW0603390RFKEA -> r_0603:CRCW06033K90FKEA
- R56: value 4.7k -> 100k; device r_0603:CRCW06034K70FKEA -> r_0603:CRCW0603100KFKEB
- U18: value MIC5271 -> MAX1735; device ICs:MIC5271YM5-TR -> ICs:MAX1735EUK50+T
Changed lines of the file:
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@@
 <part name="C244" library="c_0603" deviceset="C0603C105K8PAC7411" device="" value="1uF 10V"/>
 <part name="C245" library="c_0603" deviceset="C0603C105K8PAC7411" device="" value="1uF 10V"/>
-<part name="R55" library="r_0603" deviceset="CRCW0603390RFKEA" device="" value="390R"/>
-<part name="R56" library="r_0603" deviceset="CRCW06034K70FKEA" device="" value="4.7k"/>
+<part name="R55" library="r_0603" deviceset="CRCW06033K90FKEA" device="" value="3.9k"/>
+<part name="R56" library="r_0603" deviceset="CRCW0603100KFKEB" device="" value="100k"/>
 <part name="R57" library="r_0603" deviceset="CRCW060310K0FKTA" device="" value="10k"/>
 <part name="U20" library="ICs" deviceset="MAX25300BATA/V+" device="" value="MAX25300B"/>
@@
 <part name="R69" library="r_0603" deviceset="CRCW06031K69FKEA" device="" value="1.69k"/>
 <part name="GND283" library="NETS" deviceset="GND" device=""/>
-<part name="U18" library="ICs" deviceset="MIC5271YM5-TR" device="" value="MIC5271"/>
+<part name="U18" library="ICs" deviceset="MAX1735EUK50+T" device="" value="MAX1735"/>
 <part name="U24" library="ICs" deviceset="LMZM23600V3SILT" device="" value="3.3V BUCK"/>
 <part name="GND284" library="NETS" deviceset="GND" device=""/>

Commit message: Interface PCB started
Other:
- note added: "2021.10.18 - GSWDH LTD. IMAGE SENSOR MODULE REVISION 1.0.0 DESIGN BY GEORGE WALLER AT GSWDH LTD. GEORGEWALLER@GSWDH.CO.UK CONFIDENTIAL. FOR THE INTENDED READER ONLY."
- note removed: "2021.09.29 - ZONE OS LTD. ANGLE MEASUREMENT DEVICE REVISION 2.1.0 DESIGN BY GEORGE WALLER AT ZONE OS LTD. GEORGE@ZONEOS.IO CONFIDENTIAL. FOR THE INTENDED READER ONLY."
Changed lines of the file:
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@@
 <description>TITLE</description>
 <plain>
-<text x="0" y="0" size="7.62" layer="97" font="vector" align="center">2021.09.29 - ZONE OS LTD.
-ANGLE MEASUREMENT DEVICE
-REVISION 2.1.0
-DESIGN BY GEORGE WALLER AT ZONE OS LTD.
-GEORGE@ZONEOS.IO
+<text x="0" y="0" size="7.62" layer="97" font="vector" align="center">2021.10.18 - GSWDH LTD.
+IMAGE SENSOR MODULE
+REVISION 1.0.0
+DESIGN BY GEORGE WALLER AT GSWDH LTD.
+GEORGEWALLER@GSWDH.CO.UK
 CONFIDENTIAL. FOR THE INTENDED READER ONLY.</text>
 <wire x1="-177.8" y1="292.1" x2="177.8" y2="292.1" width="0.1524" layer="97"/>

Commit message: Fixes for sensor PCB
Parts:
- removed C178: 4.7uF 6.3V, c_0402:04026D475KAT2A
- removed C181, C182, C263: 22uF 6.3V, c_1206:C1206C226K9PACTU
- removed C243: 2200pF 25V, c_0402:C0402C222J3GEC7411
- removed C268: 0.1uF 10V, c_0402:0402ZC104KAT2A
- removed MECH10: 6mm x 3mm, MISC:MOUNTHOLE
- removed R59, R62, R68, R71, R73, R75: 10k, r_0603:CRCW060310K0FKTA
- removed R60: 45.3k, r_0603:CRCW060345K3FKEA
- removed R63: 49.9k, r_0603:CRCW060349K9FKTA
- removed R65: 9.76k, r_0603:CRCW06039K76FKEA
- removed R66: 57.6k, r_0603:CRCW060357K6FKEA
- removed R69: 1.69k, r_0603:CRCW06031K69FKEA
- removed R72: 3k, r_0603:CRCW06033K00FKEB
- removed U24: 3.3V BUCK, ICs:LMZM23600V3SILT
- removed U25: MAX6627, ICs:MAX6627MTA+T
- added C101, C102: 10uF 10V, c_1206:C1206C106K8PACTU
- added C13: 0.1uF 10V, c_0402:0402ZD104KAT2A
- added L1: 1uH, INDUCTORS:CIGT252010EH1R0MNE
- added MECH2: 6mm x 3mm, MISC:MOUNTHOLE
- added R11: 12k, RESISTORS:CRCW060312K0FKEA
- added R12: 2k, r_0603:CRCW06032K00FKTA
- added R13: 6.2k, r_0603:CRCW06036K20FKEA
- added R14: 36k, r_0603:CRCW060336K0FKEA
- added R15, R17: 15k, r_0603:CRCW060315K0FKEB
- added R16: 75k, r_0603:CRCW060375K0FKEB
- added R18: 68k, r_0603:CRCW060368K0FKEA
- added R19: 13k, r_0603:CRCW060313K0FKEA
- added R20: 15k, r_0603:CRCW060315K0FKEA
- added R24, R4: 10k, r_0603:CRCW060310K0FKTA
- added U10: EMC1812T, ICs:EMC1812T
- added U3: MP2148, ICs:MP2148GQD-Z
- C1: value 22uF 6.3V -> 0.1uF 10V; device c_1206:C1206C226K9PACTU -> c_0402:0402ZC104KAT2A
- C2: value 22uF 6.3V -> 2200pF 25V; device c_1206:C1206C226K9PACTU -> c_0402:C0402C222J3GEC7411
- C3, C4: value 22uF 6.3V -> 0.1uF 10V; device c_1206:C1206C226K9PACTU -> c_0402:0402ZD104KAT2A
- C6, C7: value 0.1uF 10V -> 22uF 6.3V; device c_0402:0402ZD104KAT2A -> c_1206:C1206C226K9PACTU
- C8: value 0.1uF 10V -> 4.7uF 6.3V; device c_0402:0402ZD104KAT2A -> c_0402:04026D475KAT2A
- U1: value STM32L031G6 -> GMAX0505-DV; device ICs:STM32L031G6 -> ICs:GMAX0505
- U2: value GMAX0505-DV -> STM32L031G6; device ICs:GMAX0505 -> ICs:STM32L031G6
- renumbered C137 to C70, C149 to C65, C150 to C55, C151 to C47, C152 to C42, C153 to C38, C154 to C34, C155 to C31, C156 to C28, C157 to C25, C158 to C22, C159 to C19, C160 to C16, C161 to C66, C162 to C56, C163 to C48, C164 to C43, C165 to C39, C166 to C35, C167 to C32, C168 to C29, C169 to C26, C170 to C23, C171 to C20, C172 to C17, C173 to C14, C174 to C12, C175 to C11, C176 to C10, C177 to C9, C183 to C64, C184 to C54, C185 to C46, C186 to C41, C187 to C37, C188 to C33, C189 to C30, C190 to C27, C191 to C24, C192 to C21, C195 to C18, C196 to C15, C197 to C71, C199 to C61, C203 to C63, C206 to C67, C207 to C57, C209 to C49, C212 to C68, C213 to C58, C214 to C50, C215 to C72, C216 to C62, C218 to C69, C219 to C51, C221 to C59, C223 to C44, C224 to C60, C225 to C52, C227 to C53, C228 to C45, C230 to C40, C231 to C36, C233 to C74, C234 to C73, C235 to C75, C236 to C76, C237 to C77, C238 to C78, C239 to C79, C240 to C80, C241 to C81, C242 to C82, C244 to C105, C245 to C106, C246 to C86, C247 to C92, C248 to C97, C249 to C88, C250 to C93, C251 to C100, C252 to C98, C253 to C99, C254 to C85, C255 to C91, C256 to C96, C257 to C84, C258 to C90, C259 to C95, C260 to C83, C261 to C89, C262 to C94, C265 to C87, C266 to C104, C267 to C103, CN5 to CN2, MECH7 to MECH3, R54 to R5, R55 to R22, R56 to R23, R57 to R21, R58 to R10, R61 to R9, R64 to R8, R67 to R7, R70 to R6, R74 to R2, U18 to U9, U19 to U8, U20 to U7, U21 to U6, U22 to U5, U23 to U4
Connections:
- removed net 2V5SLP: CN2.VCC
- removed net N$67: R71.2, R72.1, U24.FB
- removed net PROC_3V3: C268.2, C5.2, C6.2, C61.2, C7.2, C71.2, CN1.P7, R2.2, R73.2, R75.2, U1.VDD, U1.VDDA, U25.VCC, U2B.VDDIO
- removed net SEN_TEMP_SPI_!CS: CN1.P8, R75.1, U25.!CS
- new net N$3: L1.1, U3.SW
- new net N$4: R19.2, R20.1, U3.FB
- new net PROC_PWR: C1.2, C3.2, C4.2, C5.2, C61.2, C71.2, CN1.P7, CN2.VCC, R1.2, R2.2, R24.2, U10.VCC, U1B.VDDIO, U2.VDD, U2.VDDA
- new net SEN_UART_RX: CN1.P12, U2.PB7
- new net SEN_UART_TX: CN1.P8, U2.PB6
- new net TMP_ALERT: R1.1, U10.!ALERT
- new net TMP_I2C_SCL: U10.SCL, U2.PA9
- new net TMP_I2C_SDA: U10.SDA, U2.PA10
- new net TMP_THERM: R24.1, U10.ADDR
- net GND: now also C101.1, C102.1, C13.1, R11.1, R13.1, R15.1, R17.1, R19.1, R4.1, U10.GND, U1B.GNDA, U1B.GNDAD, U1B.GNDD, U2.VSS, U3.GND; no longer C178.1, C181.1, C182.1, C2.1, C263.1, C268.1, R1.1, R59.1, R62.1, R65.1, R68.1, R71.1, U1.VSS, U24.GND, U24.MODE/SYNC, U25.GND, U2B.GNDA, U2B.GNDAD, U2B.GNDD
- net N$116: now also R15.2, R16.1; no longer R62.2, R63.1
- net N$120: now also R13.2, R14.1; no longer R65.2, R66.1
- net N$124: now also R11.2, R12.1; no longer R68.2, R69.1
- net N$60: now also U1B.VRCP; no longer U2B.VRCP
- net N$61: now also C2.2, U10.DXP, U1A.VDP; no longer C243.2, U25.DXP, U2A.VDP
- net N$62: now also C2.1, U10.DXN, U1A.VDN; no longer C243.1, U25.DXN, U2A.VDN
- net N$69: now also R17.2, R18.1; no longer R59.2, R60.1
- net N$70: now also U1B.VPBP; no longer U2B.VPBP
- net N$71: now also U1B.VCLBN; no longer U2B.VCLBN
- net N$72: now also U1B.VPBN; no longer U2B.VPBN
- net N$73: now also U1B.VCLPCN; no longer U2B.VCLPCN
- net N$74: now also U1B.VREF; no longer U2B.VREF
- net N$75: now also U1B.VRS; no longer U2B.VRS
- net N$76: now also U1B.VRF; no longer U2B.VRF
- net N$77: now also U1B.VCBN; no longer U2B.VCBN
- net N$78: now also U1B.VCIBP; no longer U2B.VCIBP
- net N$79: now also U1B.VRBP; no longer U2B.VRBP
- net PROC_BOOT0: now also R4.2, U2.BOOT0; no longer R1.2, U1.BOOT0
- net PROC_NRESET: now also U2.NRST; no longer U1.NRST
- net PROC_SWCLK: now also U2.PA14; no longer U1.PA14
- net PROC_SWDIO: now also U2.PA13; no longer U1.PA13
- net SEN_B_D0_N: now also U1A.OUTB_N_0; no longer U2A.OUTB_N_0
- net SEN_B_D0_P: now also U1A.OUTB_P_0; no longer U2A.OUTB_P_0
- net SEN_B_D12_N: now also U1A.OUTB_N_12; no longer U2A.OUTB_N_12
- net SEN_B_D12_P: now also U1A.OUTB_P_12; no longer U2A.OUTB_P_12
- net SEN_B_D15_N: now also U1A.OUTB_N_15; no longer U2A.OUTB_N_15
- net SEN_B_D15_P: now also U1A.OUTB_P_15; no longer U2A.OUTB_P_15
- net SEN_B_D18_N: now also U1A.OUTB_N_18; no longer U2A.OUTB_N_18
- net SEN_B_D18_P: now also U1A.OUTB_P_18; no longer U2A.OUTB_P_18
- net SEN_B_D21_N: now also U1A.OUTB_N_21; no longer U2A.OUTB_N_21
- net SEN_B_D21_P: now also U1A.OUTB_P_21; no longer U2A.OUTB_P_21
- net SEN_B_D3_N: now also U1A.OUTB_N_3; no longer U2A.OUTB_N_3
- net SEN_B_D3_P: now also U1A.OUTB_P_3; no longer U2A.OUTB_P_3
- net SEN_B_D6_N: now also U1A.OUTB_N_6; no longer U2A.OUTB_N_6
- net SEN_B_D6_P: now also U1A.OUTB_P_6; no longer U2A.OUTB_P_6
- net SEN_B_D9_N: now also U1A.OUTB_N_9; no longer U2A.OUTB_N_9
- net SEN_B_D9_P: now also U1A.OUTB_P_9; no longer U2A.OUTB_P_9
- net SEN_CLK_IN: now also U1A.CLK_REF; no longer U2A.CLK_REF
- net SEN_CLK_N: now also U1A.CLKN_OUT; no longer U2A.CLKN_OUT
- net SEN_CLK_P: now also U1A.CLKP_OUT; no longer U2A.CLKP_OUT
- net SEN_PWR_0V7: now also R12.2, U1B.VDDCL; no longer R69.2, U2B.VDDCL
- net SEN_PWR_0V7_EN: now also U2.PA4; no longer U1.PA4
- net SEN_PWR_1V3A: now also U1B.VDD13AD; no longer U2B.VDD13AD
- net SEN_PWR_1V3D: now also C101.2, C102.2, C6.2, C7.2, C8.2, L1.2, R20.2, U1B.VDD13D, U3.OUT; no longer C1.2, C178.2, C181.2, C182.2, C2.2, C263.2, C3.2, C4.2, R72.2, U24.VOUT, U2B.VDD13D
- net SEN_PWR_1V3_EN: now also U2.PA5, U3.EN; no longer U1.PA5, U24.EN
- net SEN_PWR_3V3A: now also C13.2, R18.2, U1B.VDD33A; no longer C8.2, R60.2, U2B.VDD33A
- net SEN_PWR_3V3_EN: now also U2.PA1; no longer U1.PA1
- net SEN_PWR_3V6: now also R16.2, U1B.VDDPIX, U1B.VTXH; no longer R63.2, U2B.VDDPIX, U2B.VTXH
- net SEN_PWR_3V6_EN: now also U2.PA2; no longer U1.PA2
- net SEN_PWR_4V1: now also R14.2, U1B.VG_RSTH; no longer R66.2, U2B.VG_RSTH
- net SEN_PWR_4V1_EN: now also U2.PA3; no longer U1.PA3
- net SEN_PWR_EN: now also U2.PA6; no longer U1.PA6
- net SEN_PWR_N1V3A: now also U1B.VGRSTL, U1B.VTXL; no longer U2B.VGRSTL, U2B.VTXL
- net SEN_PWR_N1V3A_EN: now also U2.PA0; no longer U1.PA0
- net SEN_SPI_!CS: now also U1A.SPI_CS; no longer U2A.SPI_CS
- net SEN_SPI_MISO: now also U1A.SPI_MISO; no longer U25.MISO, U2A.SPI_MISO
- net SEN_SPI_MOSI: now also U1A.SPI_MOSI; no longer U2A.SPI_MOSI
- net SEN_SPI_SCLK: now also U1A.SPI_SCLK; no longer U25.SCLK, U2A.SPI_SCLK
- net SEN_SYS_!RESET: now also U1A.!SYS_RST, U2.PC15; no longer CN1.P12, R73.1, U2A.!SYS_RST
- net SEN_TDIG0: now also U1A.TDIG0; no longer U2A.TDIG0
- net SEN_TDIG1: now also U1A.TDIG1; no longer U2A.TDIG1
- net SEN_TEMP1: now also U1A.TEXP1; no longer U2A.TEXP1
- net SEN_TEXP0: now also U1A.TEXP0; no longer U2A.TEXP0
- net SEN_T_D0_N: now also U1A.OUTT_N_0; no longer U2A.OUTT_N_0
- net SEN_T_D0_P: now also U1A.OUTT_P_0; no longer U2A.OUTT_P_0
- net SEN_T_D12_N: now also U1A.OUTT_N_12; no longer U2A.OUTT_N_12
- net SEN_T_D12_P: now also U1A.OUTT_P_12; no longer U2A.OUTT_P_12
- net SEN_T_D15_N: now also U1A.OUTT_N_15; no longer U2A.OUTT_N_15
- net SEN_T_D15_P: now also U1A.OUTT_P_15; no longer U2A.OUTT_P_15
- net SEN_T_D18_N: now also U1A.OUTT_N_18; no longer U2A.OUTT_N_18
- net SEN_T_D18_P: now also U1A.OUTT_P_18; no longer U2A.OUTT_P_18
- net SEN_T_D21_N: now also U1A.OUTT_N_21; no longer U2A.OUTT_N_21
- net SEN_T_D21_P: now also U1A.OUTT_P_21; no longer U2A.OUTT_P_21
- net SEN_T_D3_N: now also U1A.OUTT_N_3; no longer U2A.OUTT_N_3
- net SEN_T_D3_P: now also U1A.OUTT_P_3; no longer U2A.OUTT_P_3
- net SEN_T_D6_N: now also U1A.OUTT_N_6; no longer U2A.OUTT_N_6
- net SEN_T_D6_P: now also U1A.OUTT_P_6; no longer U2A.OUTT_P_6
- net SEN_T_D9_N: now also U1A.OUTT_N_9; no longer U2A.OUTT_N_9
- net SEN_T_D9_P: now also U1A.OUTT_P_9; no longer U2A.OUTT_P_9
- net SYS_PWR_5V: now also U3.VIN; no longer U24.VIN
Other:
- note added: "2022.07.12 - GSWDH LTD. IMAGE SENSOR MODULE REVISION 1.1.0 DESIGN BY GEORGE WALLER AT GSWDH LTD. GEORGEWALLER@GSWDH.CO.UK CONFIDENTIAL. FOR THE INTENDED READER ONLY."
- note removed: "2021.10.18 - GSWDH LTD. IMAGE SENSOR MODULE REVISION 1.0.0 DESIGN BY GEORGE WALLER AT GSWDH LTD. GEORGEWALLER@GSWDH.CO.UK CONFIDENTIAL. FOR THE INTENDED READER ONLY."

Commit message: Mech design and layout
Parts:
- added CN3: FH52E-60S-0.5SH, CONNECTORs:FH52E-60S-0.5SH
Connections:
- new net N$5: CN1.GND, CN3.P1
- net GND: now also CN3.P2, CN3.P3, CN3.P39, CN3.P4, CN3.P40, CN3.P42, CN3.P43, CN3.P56, CN3.P57, CN3.P58
- net PROC_PWR: now also CN3.P55
- net SEN_B_D0_N: now also CN3.P29
- net SEN_B_D0_P: now also CN3.P30
- net SEN_B_D12_N: now also CN3.P21
- net SEN_B_D12_P: now also CN3.P22
- net SEN_B_D15_N: now also CN3.P17
- net SEN_B_D15_P: now also CN3.P18
- net SEN_B_D18_N: now also CN3.P16
- net SEN_B_D18_P: now also CN3.P15
- net SEN_B_D21_N: now also CN3.P12
- net SEN_B_D21_P: now also CN3.P11
- net SEN_B_D3_N: now also CN3.P27
- net SEN_B_D3_P: now also CN3.P28
- net SEN_B_D6_N: now also CN3.P34
- net SEN_B_D6_P: now also CN3.P33
- net SEN_B_D9_N: now also CN3.P26
- net SEN_B_D9_P: now also CN3.P25
- net SEN_CLK_IN: now also CN3.P47
- net SEN_CLK_N: now also CN3.P6
- net SEN_CLK_P: now also CN3.P5
- net SEN_PWR_EN: now also CN3.P41
- net SEN_SPI_!CS: now also CN3.P46
- net SEN_SPI_MISO: now also CN3.P45
- net SEN_SPI_MOSI: now also CN3.P44
- net SEN_SPI_SCLK: now also CN3.P51
- net SEN_TDIG0: now also CN3.P53
- net SEN_TDIG1: now also CN3.P52
- net SEN_TEMP1: now also CN3.P48
- net SEN_TEXP0: now also CN3.P49
- net SEN_T_D0_N: now also CN3.P37
- net SEN_T_D0_P: now also CN3.P38
- net SEN_T_D12_N: now also CN3.P24
- net SEN_T_D12_P: now also CN3.P23
- net SEN_T_D15_N: now also CN3.P10
- net SEN_T_D15_P: now also CN3.P9
- net SEN_T_D18_N: now also CN3.P13
- net SEN_T_D18_P: now also CN3.P14
- net SEN_T_D21_N: now also CN3.P8
- net SEN_T_D21_P: now also CN3.P7
- net SEN_T_D3_N: now also CN3.P36
- net SEN_T_D3_P: now also CN3.P35
- net SEN_T_D6_N: now also CN3.P31
- net SEN_T_D6_P: now also CN3.P32
- net SEN_T_D9_N: now also CN3.P20
- net SEN_T_D9_P: now also CN3.P19
- net SEN_UART_RX: now also CN3.P50
- net SEN_UART_TX: now also CN3.P54
- net SYS_PWR_5V: now also CN3.GND, CN3.P59, CN3.P60
