File: power.brd (EAGLE design)
At the start: 136 x 136 mm, 37 parts, among them CN1 21700, CN2 21700, CN3 21700, CN4 21700, CN5 15PIN 0.5MM, Q6 IRLML6244, Q7 IRLML6244, U17 MAX17320G20+

Commit message: Battery PCB done
Parts:
- removed C122, C123, C124: 100nF 16V, CAPACITORS:0603
- removed C125, C126, C127, C128: 470nF 25V, CAPACITORS:0603
- removed C129: 10nF 50V, CAPACITORS:0603
- removed Q6, Q7: IRLML6244, TRANSISTORs:SOT23-3
- removed R38: 0R01, RESISTORS:1206
- removed R41, R42, R43: 47R, r_0603:0603
- removed R47: 10R, r_0603:0603
- removed R48, R49, R50: 1.0k, r_0603:0603
- removed R51, R53: 100R, r_0603:0603
- removed R52: 10k, r_0603:0603
- removed U17: MAX17320G20+, ICs:TQFN24
- added C10: 10nF 50V, CAPACITORS:0603
- added C3, C4, C5: 100nF 16V, CAPACITORS:0603
- added C6, C7, C8, C9: 470nF 25V, CAPACITORS:0603
- added Q1, Q2: IRLML6244, TRANSISTORs:SOT23-3
- added R10, R12, R6: 1.0k, r_0603:0603
- added R11: 10k, r_0603:0603
- added R2, R3, R4, R5: 47R, r_0603:0603
- added R7, R9: 100R, r_0603:0603
- added R8: 0R01, RESISTORS:1206
- added U1: MAX17320G20+, ICs:TQFN24
- R1: value 47R -> 10R
- moved MECH4 141.2 mm to (-27.5, 65.0)
- moved MECH5 119.1 mm to (27.5, -65.0)
- moved MECH3 107.6 mm to (-65.0, 10.0)
- moved F1 57.1 mm to (-15.2, 38.1), turned to 180 degrees
- moved MECH2 55.0 mm to (27.5, 65.0)
- moved R1 7.25 mm to (22.9, 54.6), turned to 180 degrees
- moved C2 5.15 mm to (23.1, 49.5), turned to 90 degrees
- moved C1 4.44 mm to (23.1, 52.2), turned to 90 degrees
Connections:
- net BMS_I2C_SCL: now also U1.8; no longer U17.8
- net BMS_I2C_SDA: now also U1.9; no longer U17.9
- net BMS_NALERT: now also U1.7; no longer U17.7
- net BMS_TH1: now also R11.2, U1.10; no longer R52.2, U17.10
- net GND: now also R8.1, U1.14; no longer C126.2, C129.1, R38.1, U17.14
- net N$1: now also C3.1, C4.2, R5.2, U1.21; no longer C1.1, C122.2, R41.2, U17.21
- net N$2: now also C1.1, R3.2, U1.23; no longer C123.1, R42.2, U17.23
- net N$3: now also C3.2, R4.2, U1.22; no longer C1.2, R1.2, U17.22
- net N$36: now also R1.1, R2.1; no longer R43.1, R47.1
- net N$38: now also C5.2, C6.1, R1.2, U1.1; no longer C124.2, C125.1, R47.2, U17.1
- net N$39: now also C1.2, R2.2, U1.24; no longer C123.2, R43.2, U17.24
- net N$4: now also R3.1; no longer R42.1
- net N$41: now also C6.2, U1.2; no longer C125.2, U17.2
- net N$42: now also Q1.3; no longer Q7.3
- net N$43: now also Q2.1, R9.2; no longer Q6.1, R51.2
- net N$45: now also R6.2, U1.11; no longer R48.2, U17.11
- net N$46: now also C10.2, R12.1, U1.6; no longer C129.2, R49.1, U17.6
- net N$47: now also R10.1, U1.5; no longer R50.1, U17.5
- net N$48: now also C7.1, U1.12; no longer C126.1, U17.12
- net N$49: now also C8.1, U1.17; no longer C127.1, U17.17
- net N$5: now also R4.1; no longer R1.1
- net N$55: now also C9.1, U1.13; no longer C128.1, U17.13
- net N$56: now also R9.1, U1.4; no longer R51.1, U17.4
- net N$57: now also Q1.2, Q2.2; no longer Q6.2, Q7.2
- net N$58: now also Q1.1, R7.2; no longer Q7.1, R53.2
- net N$59: now also R7.1, U1.3; no longer R53.1, U17.3
- net PACK_MID: now also R5.1; no longer R41.1
- net PGND: now also C10.1, C4.1, C5.1, C7.2, C8.2, C9.2, R11.1, R6.1, R8.2, U1.15, U1.16, U1.18, U1.19, U1.20, U1.PAD; no longer C122.1, C124.1, C127.2, C128.2, R38.2, R48.1, R52.1, U17.15, U17.16, U17.18, U17.19, U17.20, U17.PAD
- net PWR_VPACK: now also Q2.3, R10.2, R12.2; no longer Q6.3, R49.2, R50.2
Routing:
- net PACK_MID: track 21.9 -> 205.8 mm, vias 0 -> 1
- net N$36: track 7.13 -> 141.5 mm, vias 0 -> 9
- net N$5: track 21.9 -> 129.9 mm, vias 0 -> 1
- net N$4: track 21.9 -> 52.8 mm, vias 0 -> 1
- net N$59: track 9.78 -> 40.2 mm
- net N$56: track 13.2 -> 37.6 mm
- net GND: track 7.89 -> 31.5 mm, vias 2 -> 0
- net PGND: track 22.6 -> 44.3 mm, vias 6 -> 17
- net PWR_VPACK: track 19.0 -> 36.7 mm, vias 2 -> 0
- net BMS_NALERT: track 5.92 -> 21.2 mm, vias 0 -> 2
- net BMS_I2C_SCL: track 5.92 -> 20.9 mm
- net BMS_I2C_SDA: track 5.92 -> 20.2 mm
- net N$3: track 0.00 -> 6.74 mm
- net N$38: track 2.10 -> 6.91 mm
- net N$1: track 4.19 -> 7.05 mm
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- added copper zone on layer 1, net PGND

Commit message: debug board done
Parts:
- added R13: 10R, r_0603:0603
Connections:
- new net N$6: R13.2, U1.15
- net PGND: now also R13.1; no longer U1.15
Routing:
- net PGND: track 44.3 -> 23.4 mm
- net N$6: track 0.00 -> 17.7 mm
Changed lines of the file:
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@@
 </layers>
 <board>
-<fusionsync huburn="a.YnVzaW5lc3M6bXl1Y2wxNDk2" projecturn="a.YnVzaW5lc3M6bXl1Y2wxNDk2IzIwMjExMjA3NDc0MjU0MzI2" f3durn="urn:adsk.wipprod:dm.lineage:-o3MW2fXTlyFglXsuSGDiA" pcbguid="" lastpulledtime="2022-04-18T10:55:57Z" lastsyncedchangeguid="" latestrevisionid="20f91420-efc4-4c1a-9ffb-bc58426cf1a7" lastsyncedrevisionid="20f91420-efc4-4c1a-9ffb-bc58426cf1a7" lastboardhashguid="8f3bba5c-4b1b-cbbf-cbcb-a6c4245ae9e2" lastpushedtime="2022-12-11T09:33:34Z" linktopcb3d="true"/>
+<fusionsync huburn="a.YnVzaW5lc3M6bXl1Y2wxNDk2" projecturn="a.YnVzaW5lc3M6bXl1Y2wxNDk2IzIwMjExMjA3NDc0MjU0MzI2" f3durn="urn:adsk.wipprod:dm.lineage:-o3MW2fXTlyFglXsuSGDiA" pcbguid="" lastpulledtime="2022-04-18T10:55:57Z" lastsyncedchangeguid="" latestrevisionid="71ad996f-8101-4d6b-b739-1cdb66934eb4" lastsyncedrevisionid="71ad996f-8101-4d6b-b739-1cdb66934eb4" lastboardhashguid="7e5822f3-6512-944f-913a-f4c7bde74239" lastpushedtime="2022-12-12T08:45:35Z" linktopcb3d="true"/>
 <plain>
 <wire x1="-24" y1="31" x2="24" y2="31" width="0" layer="20" locked="yes"/>
@@
 <element name="MECH3" library="MISC" package="MOUNTHOLE_6X3" value="6mm x 3mm" x="-65" y="10" smashed="yes"/>
 <element name="MECH6" library="MISC" package="MOUNTHOLE_6X3" value="6mm x 3mm" x="65" y="-5" smashed="yes"/>
+<element name="R13" library="r_0603" package="0603" value="10R" x="4.875" y="39" smashed="yes" rot="R90">
+<attribute name="DIGIKEY" value="P10.0HCT-ND" x="4.875" y="39" size="1.778" layer="27" rot="R90" display="off"/>
+<attribute name="FARNELL" value="" x="4.875" y="39" size="1.778" layer="27" rot="R90" display="off"/>
+<attribute name="NAME" x="4.125" y="37.5" size="1.016" layer="25" rot="R90"/>
+<attribute name="PRICE_PER" value="0.10000" x="4.875" y="39" size="1.778" layer="27" rot="R90" display="off"/>
+</element>
 </elements>
 <signals>
@@
 <signal name="PGND">
 <contactref element="R8" pad="2"/>
-<contactref element="U1" pad="15"/>
 <contactref element="C5" pad="1"/>
 <contactref element="R6" pad="1"/>
@@
 <wire x1="2.875" y1="38.25" x2="3.75" y2="37.375" width="0.5" layer="1"/>
 <via x="3.75" y="37.375" extent="1-16" drill="0.5"/>
-<wire x1="17.25" y1="46.42" x2="17.25" y2="42.125" width="0.15" layer="1"/>
-<wire x1="17.25" y1="42.125" x2="15.125" y2="40" width="0.15" layer="1"/>
 <wire x1="2.875" y1="38.375" x2="2.75" y2="38.25" width="0.15" layer="1"/>
-<wire x1="15.125" y1="40" x2="3.375" y2="40" width="0.15" layer="1"/>
-<wire x1="3.375" y1="40" x2="2.875" y2="39.5" width="0.15" layer="1"/>
-<wire x1="2.875" y1="39.5" x2="2.875" y2="38.375" width="0.15" layer="1"/>
 <contactref element="C7" pad="2"/>
 <contactref element="C10" pad="1"/>
@@
 <vertex x="-100" y="-100"/>
 </polygon>
+<contactref element="R13" pad="1"/>
 </signal>
 <signal name="BMS_TH1">
@@
 <contactref element="CN5" pad="9"/>
 </signal>
+<signal name="N$6">
+<contactref element="U1" pad="15"/>
+<contactref element="R13" pad="2"/>
+<wire x1="17.25" y1="46.42" x2="17.25" y2="42.125" width="0.15" layer="1"/>
+<wire x1="5.125" y1="40" x2="4.875" y2="39.75" width="0.15" layer="1"/>
+<wire x1="17.25" y1="42.125" x2="15.125" y2="40" width="0.15" layer="1"/>
+<wire x1="15.125" y1="40" x2="5.125" y2="40" width="0.15" layer="1"/>
+</signal>
 </signals>

Commit message: New format working on
Parts:
- removed CN1, CN2, CN3, CN4: 21700, CONNECTORs:1122
- removed MECH1, MECH2, MECH4, MECH5: 6mm x 3mm, MISC:MOUNTHOLE_6X3
- added MECH7, MECH8: 6mm x 3mm, MISC:MOUNTHOLE_6X3
- moved MECH6 55.2 mm to (27.0, 35.0)
- moved MECH3 45.5 mm to (-27.0, 35.0)
- moved C1 38.8 mm to (48.2, 22.6)
- moved C10 38.8 mm to (38.2, 22.6)
- moved C2 38.8 mm to (48.2, 19.9)
- moved C3 38.8 mm to (48.2, 17.1)
- moved C4 38.8 mm to (48.2, 14.4)
- moved C5 38.8 mm to (45.2, 24.2)
- moved C6 38.8 mm to (44.5, 22.2)
- moved C7 38.8 mm to (39.2, 16.1)
- moved C8 38.8 mm to (43.4, 14.6)
- moved C9 38.8 mm to (41.0, 14.6)
- moved R1 38.8 mm to (48.0, 25.0)
- moved R10 38.8 mm to (41.5, 23.4)
- moved R11 38.8 mm to (36.6, 18.2)
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Connections:
- net N$36: no longer CN1.+
- net N$4: no longer CN1.-, CN2.+
- net N$5: no longer CN2.-, CN3.+
- net PACK_MID: no longer CN3.-, CN4.+
- net PGND: no longer CN4.-
Routing:
- net PACK_MID: track 205.8 -> 0.00 mm, vias 1 -> 0
- net N$36: track 141.5 -> 0.00 mm, vias 9 -> 0
- net N$5: track 129.9 -> 0.00 mm, vias 1 -> 0
- net N$4: track 52.8 -> 0.00 mm, vias 1 -> 0
- net N$59: track 40.2 -> 0.00 mm
- net N$56: track 37.6 -> 0.00 mm
- net PWR_VPACK: track 36.7 -> 0.00 mm
- net GND: track 31.5 -> 0.00 mm
- net PGND: track 23.4 -> 0.00 mm, vias 17 -> 1
- net BMS_NALERT: track 21.2 -> 0.00 mm, vias 2 -> 0
- net BMS_I2C_SCL: track 20.9 -> 0.00 mm
- net BMS_I2C_SDA: track 20.2 -> 0.00 mm
- net N$6: track 17.7 -> 0.00 mm
- net N$39: track 7.27 -> 0.00 mm
- net N$1: track 7.05 -> 0.00 mm
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Other:
- board size 136 x 136 mm -> 156 x 76 mm

Commit message: Progress
Parts:
- added CN1, CN2: 21700, CONNECTORs:1122
- moved R13 57.0 mm to (42.2, -23.9)
- moved R8 57.0 mm to (39.6, -23.1)
- moved CN5 49.2 mm to (47.4, 21.9), turned to 270 degrees
- moved MECH3 37.2 mm to (-57.0, 57.0)
- moved MECH6 37.2 mm to (57.0, 57.0)
- moved MECH7 37.2 mm to (-57.0, -57.0)
- moved MECH8 37.2 mm to (57.0, -57.0)
- moved C1 31.9 mm to (49.0, -9.25)
- moved C10 31.9 mm to (39.0, -9.25)
- moved C2 31.9 mm to (49.0, -12.0)
- moved C3 31.9 mm to (49.0, -14.8)
- moved C4 31.9 mm to (49.0, -17.5)
- moved C5 31.9 mm to (46.0, -7.62)
- moved C6 31.9 mm to (45.2, -9.62)
- moved C7 31.9 mm to (40.0, -15.8)
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Connections:
- net N$5: now also CN2.+
- net PACK_MID: now also CN1.+, CN2.-
- net PGND: now also CN1.-
Other:
- board size 156 x 76 mm -> 120 x 120 mm

Commit message: Progress
Parts:
- removed C1: 100nF 16V, CAPACITORS:0603
- removed R2: 47R, r_0603:0603
- added CN3: 21700, CONNECTORs:21700_TABBED
- CN1, CN2: device CONNECTORs:1122 -> CONNECTORs:21700_TABBED
- F1: value 1A Fast -> 20A; device FUSES:1206 -> FUSES:0678H
- Q1, Q2: value IRLML6244 -> SIRA36DP-T1-GE3; device TRANSISTORs:SOT23-3 -> TRANSISTORs:SO8_POWERPAK
- moved F1 85.1 mm to (38.5, 50.0), flipped to the bottom, turned to 0 degrees
- moved R7 80.1 mm to (38.8, 40.4), turned to 180 degrees
- moved R9 76.5 mm to (38.8, 38.6), turned to 180 degrees
- moved Q1 72.0 mm to (31.4, 40.5), turned to 180 degrees
- moved Q2 68.0 mm to (31.4, 35.2), turned to 180 degrees
- moved CN2 62.2 mm to (0.00, -43.0)
- moved R8 44.5 mm to (35.2, 21.1)
- moved R13 44.4 mm to (32.8, 19.5), turned to 180 degrees
- moved R6 28.0 mm to (46.6, 11.5), turned to 270 degrees
- moved R11 27.2 mm to (47.9, 11.5), turned to 270 degrees
- moved C7 25.8 mm to (45.2, 9.50), turned to 180 degrees
- moved C9 24.7 mm to (43.6, 7.38), turned to 180 degrees
- moved C10 23.1 mm to (51.1, 10.4), turned to 270 degrees
- moved C8 22.6 mm to (43.6, 5.38), turned to 180 degrees
- moved R12 20.1 mm to (51.9, 8.38), turned to 0 degrees
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Connections:
- removed net N$36: F1.1, R1.1, R2.1
- removed net N$4: R3.1
- net N$2: no longer C1.1
- net N$39: now also CN3.P1, CN3.P10, CN3.P11, CN3.P12, CN3.P13, CN3.P14, CN3.P15, CN3.P16, CN3.P17, CN3.P18, CN3.P19, CN3.P2, CN3.P20, CN3.P21, CN3.P22, CN3.P23, CN3.P24, CN3.P25, CN3.P3, CN3.P4, CN3.P5, CN3.P6, CN3.P7, CN3.P8, CN3.P9, F1.1, R1.1, R3.1; no longer C1.2, R2.2
- net N$42: now also Q1.1, Q1.2
- net N$43: now also Q2.4; no longer Q2.1
- net N$5: now also CN2.P1, CN2.P10, CN2.P11, CN2.P12, CN2.P13, CN2.P14, CN2.P15, CN2.P16, CN2.P17, CN2.P18, CN2.P19, CN2.P2, CN2.P20, CN2.P21, CN2.P22, CN2.P23, CN2.P24, CN2.P25, CN2.P3, CN2.P4, CN2.P5, CN2.P6, CN2.P7, CN2.P8, CN2.P9, CN3.N, CN3.N1, CN3.N10, CN3.N11, CN3.N12, CN3.N13, CN3.N14, CN3.N15, CN3.N16, CN3.N17, CN3.N18, CN3.N19, CN3.N2, CN3.N20, CN3.N21, CN3.N22, CN3.N23, CN3.N24, CN3.N3, CN3.N4, CN3.N5, CN3.N6, CN3.N7, CN3.N8, CN3.N9; no longer CN2.+
- net N$57: now also Q1.5, Q1.6, Q1.7, Q1.8, Q1.PAD, Q2.5, Q2.6, Q2.7, Q2.8, Q2.PAD; no longer Q1.2, Q2.2
- net N$58: now also Q1.4; no longer Q1.1
- net PACK_MID: now also CN1.P1, CN1.P10, CN1.P11, CN1.P12, CN1.P13, CN1.P14, CN1.P15, CN1.P16, CN1.P17, CN1.P18, CN1.P19, CN1.P2, CN1.P20, CN1.P21, CN1.P22, CN1.P23, CN1.P24, CN1.P25, CN1.P3, CN1.P4, CN1.P5, CN1.P6, CN1.P7, CN1.P8, CN1.P9, CN2.N, CN2.N1, CN2.N10, CN2.N11, CN2.N12, CN2.N13, CN2.N14, CN2.N15, CN2.N16, CN2.N17, CN2.N18, CN2.N19, CN2.N2, CN2.N20, CN2.N21, CN2.N22, CN2.N23, CN2.N24, CN2.N3, CN2.N4, CN2.N5, CN2.N6, CN2.N7, CN2.N8, CN2.N9; no longer CN1.+, CN2.-
- net PGND: now also CN1.N, CN1.N1, CN1.N10, CN1.N11, CN1.N12, CN1.N13, CN1.N14, CN1.N15, CN1.N16, CN1.N17, CN1.N18, CN1.N19, CN1.N2, CN1.N20, CN1.N21, CN1.N22, CN1.N23, CN1.N24, CN1.N3, CN1.N4, CN1.N5, CN1.N6, CN1.N7, CN1.N8, CN1.N9; no longer CN1.-
- net PWR_VPACK: now also Q2.1, Q2.2
Routing:
- net PACK_MID: track 0.00 -> 142.0 mm
- net N$39: track 0.00 -> 75.7 mm
- net N$5: track 0.00 -> 60.4 mm
- net N$59: track 0.00 -> 48.1 mm
- net N$56: track 0.00 -> 46.2 mm
- net N$57: track 0.00 -> 32.0 mm
- net GND: track 0.00 -> 30.3 mm
- net PWR_VPACK: track 0.00 -> 28.5 mm
- net N$6: track 0.00 -> 25.7 mm
- net BMS_NALERT: track 0.00 -> 25.1 mm, vias 0 -> 2
- net BMS_I2C_SCL: track 0.00 -> 25.0 mm
- net BMS_I2C_SDA: track 0.00 -> 24.4 mm
- net PGND: track 0.00 -> 14.3 mm, vias 0 -> 39
- net N$1: track 0.00 -> 7.05 mm
- net N$58: track 0.00 -> 6.89 mm, vias 0 -> 2
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- added copper zone on layer 1, net GND
- added copper zone on layer 1, net N$42
- added copper zone on layer 16, net N$42
- added copper zone on layer 1, net PWR_VPACK
Other:
- outline, holes or cut-outs redrawn
- board text added: "gswdh.co.uk"
- board text added: "gswdh.co.uk camera power PCB rev 1.0.0 2023.04.08"
