File: power.brd (EAGLE design)
At the start: 120 x 120 mm, 34 parts, among them CN1 21700, CN2 21700, CN3 21700, CN5 15PIN 0.5MM, Q1 SIRA36DP-T1-GE3, Q2 SIRA36DP-T1-GE3, U1 MAX17320G20+

Commit message: Correct FPGA footprint routed. A lot of work to length match, optimise and review
Parts:
- moved MECH8 20.0 mm to (47.0, -57.0)
Changed lines of the file:
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@@
 <layer number="14" name="Route14" color="1" fill="6" visible="no" active="no"/>
 <layer number="15" name="Route15" color="4" fill="6" visible="no" active="no"/>
-<layer number="16" name="Bottom" color="9" fill="1" visible="yes" active="yes"/>
+<layer number="16" name="Bottom" color="9" fill="1" visible="no" active="yes"/>
 <layer number="17" name="Pads" color="2" fill="1" visible="yes" active="yes"/>
 <layer number="18" name="Vias" color="2" fill="1" visible="yes" active="yes"/>
@@
 <layer number="20" name="Dimension" color="15" fill="1" visible="yes" active="yes"/>
 <layer number="21" name="tPlace" color="7" fill="1" visible="yes" active="yes"/>
-<layer number="22" name="bPlace" color="14" fill="1" visible="yes" active="yes"/>
+<layer number="22" name="bPlace" color="14" fill="1" visible="no" active="yes"/>
 <layer number="23" name="tOrigins" color="15" fill="1" visible="yes" active="yes"/>
-<layer number="24" name="bOrigins" color="14" fill="1" visible="yes" active="yes"/>
+<layer number="24" name="bOrigins" color="14" fill="1" visible="no" active="yes"/>
 <layer number="25" name="tNames" color="7" fill="1" visible="yes" active="yes"/>
-<layer number="26" name="bNames" color="14" fill="1" visible="yes" active="yes"/>
+<layer number="26" name="bNames" color="14" fill="1" visible="no" active="yes"/>
 <layer number="27" name="tValues" color="7" fill="1" visible="no" active="yes"/>
 <layer number="28" name="bValues" color="14" fill="1" visible="no" active="yes"/>
@@
 <layer number="43" name="vRestrict" color="2" fill="10" visible="no" active="yes"/>
 <layer number="44" name="Drills" color="7" fill="1" visible="no" active="yes"/>
-<layer number="45" name="Holes" color="7" fill="1" visible="yes" active="yes"/>
+<layer number="45" name="Holes" color="7" fill="1" visible="no" active="yes"/>
 <layer number="46" name="Milling" color="3" fill="1" visible="no" active="yes"/>
 <layer number="47" name="Measures" color="7" fill="1" visible="no" active="yes"/>
@@
 <element name="MECH6" library="MISC" package="MOUNTHOLE_6X3" value="6mm x 3mm" x="47" y="57" smashed="yes"/>
 <element name="MECH7" library="MISC" package="MOUNTHOLE_6X3" value="6mm x 3mm" x="-47" y="-57" smashed="yes"/>
-<element name="MECH8" library="MISC" package="MOUNTHOLE_6X3" value="6mm x 3mm" x="27" y="-57" smashed="yes"/>
+<element name="MECH8" library="MISC" package="MOUNTHOLE_6X3" value="6mm x 3mm" x="47" y="-57" smashed="yes"/>
 <element name="CN1" library="CONNECTORs" package="21700_TABBED" value="21700" x="-43" y="10" locked="yes" smashed="yes" rot="MR180">
 <attribute name="DIGIKEY" value="" x="-43" y="10" locked="yes" size="1.778" layer="28" rot="MR180" display="off"/>
@@
 <contactref element="Q2" pad="4"/>
 <contactref element="R9" pad="2"/>
-<wire x1="37.25" y1="37.875" x2="34.765" y2="37.875" width="0.15" layer="1"/>
-<wire x1="34.045" y1="37.155" x2="34.765" y2="37.875" width="0.15" layer="1"/>
+<wire x1="37.25" y1="37.875" x2="35.14" y2="37.875" width="0.15" layer="1"/>
+<wire x1="34.045" y1="37.155" x2="34.42" y2="37.155" width="0.15" layer="1"/>
+<wire x1="35.14" y1="37.875" x2="34.42" y2="37.155" width="0.15" layer="1"/>
 <wire x1="37.25" y1="37.875" x2="38" y2="38.625" width="0.15" layer="1"/>
 </signal>
@@
 <wire x1="52.625" y1="8.375" x2="52.625" y2="7.125" width="0.15" layer="1"/>
 <wire x1="52.625" y1="8.375" x2="52.625" y2="17" width="0.15" layer="1"/>
-<wire x1="38.25" y1="26.875" x2="38.125" y2="27" width="0.15" layer="1"/>
 <wire x1="52.625" y1="17" x2="42.75" y2="26.875" width="0.15" layer="1"/>
 <wire x1="42.75" y1="26.875" x2="38.25" y2="26.875" width="0.15" layer="1"/>
+<wire x1="38.25" y1="26.875" x2="38.125" y2="27" width="0.15" layer="1"/>
 </signal>
 <signal name="BMS_NALERT">

Commit message: MIPI length matched DRC passes
Parts:
- moved CN1 20.0 mm to (-43.0, -10.0)
- moved CN2 10.0 mm to (10.0, -43.0)
Routing:
- net PACK_MID: track 143.8 -> 130.0 mm
- net N$4: track 61.0 -> 57.5 mm
- net N$1: track 4.32 -> 5.57 mm
