File: power.brd (EAGLE design)
At the start: 120 x 120 mm, 34 parts, among them CN1 21700, CN2 21700, CN3 21700, CN5 15PIN 0.5MM, Q1 SIRA36DP-T1-GE3, Q2 SIRA36DP-T1-GE3, U1 MAX17320G20+

Commit message: Added extra decoupling to the PLL PSU
Parts:
- removed CN5: 15PIN 0.5MM, CONNECTORs:SFV15R-1STE1HLF
- removed F1: 20A, FUSES:0678H
- added CN4: 15PIN 0.5MM, CONNECTORs:SFV15R-1STE1HLF
- CN1, CN2, CN3: device CONNECTORs:21700_TABBED -> CONNECTORs:1122
- moved R7 55.7 mm to (-16.9, 37.9), flipped to the bottom, turned to 0 degrees
- moved R9 51.2 mm to (-12.1, 44.4), flipped to the bottom, turned to 90 degrees
- moved R4 48.4 mm to (26.4, 43.1), flipped to the bottom, turned to 0 degrees
- moved C4 47.8 mm to (24.4, 43.9), flipped to the bottom, turned to 270 degrees
- moved R5 47.8 mm to (26.4, 41.9), flipped to the bottom, turned to 0 degrees
- moved Q1 47.7 mm to (-15.5, 49.5), flipped to the bottom, turned to 90 degrees
- moved R3 47.1 mm to (26.4, 40.4), flipped to the bottom, turned to 0 degrees
- moved C2 46.6 mm to (24.4, 41.1), flipped to the bottom, turned to 270 degrees
- moved C8 46.2 mm to (19.6, 44.9), flipped to the bottom, turned to 90 degrees
- moved R2 46.1 mm to (26.4, 37.6), flipped to the bottom, turned to 0 degrees
- moved C1 45.7 mm to (24.4, 38.4), flipped to the bottom, turned to 270 degrees
- moved R1 45.7 mm to (26.4, 36.4), flipped to the bottom, turned to 0 degrees
- moved C9 45.6 mm to (17.6, 44.9), flipped to the bottom, turned to 90 degrees
- moved C10 45.4 mm to (14.6, 37.4), flipped to the bottom, turned to 180 degrees
- moved R8 45.3 mm to (3.88, 53.8), flipped to the bottom, turned to 0 degrees
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Connections:
- removed net N$39: CN3.P1, CN3.P10, CN3.P11, CN3.P12, CN3.P13, CN3.P14, CN3.P15, CN3.P16, CN3.P17, CN3.P18, CN3.P19, CN3.P2, CN3.P20, CN3.P21, CN3.P22, CN3.P23, CN3.P24, CN3.P25, CN3.P3, CN3.P4, CN3.P5, CN3.P6, CN3.P7, CN3.P8, CN3.P9, F1.1, R1.1, R2.1
- net BMS_BUS_RSVD_1: now also CN4.8; no longer CN5.8
- net BMS_BUS_RSVD_2: now also CN4.7; no longer CN5.9
- net BMS_I2C_SCL: now also CN4.11; no longer CN5.5
- net BMS_I2C_SDA: now also CN4.10; no longer CN5.6
- net BMS_NALERT: now also CN4.9; no longer CN5.7
- net GND: now also CN4.1, CN4.2, CN4.3, CN4.4, CN4.5, CN4.6; no longer CN5.10, CN5.11, CN5.12, CN5.13, CN5.14, CN5.15
- net N$4: now also CN2.+, CN3.-; no longer CN2.P1, CN2.P10, CN2.P11, CN2.P12, CN2.P13, CN2.P14, CN2.P15, CN2.P16, CN2.P17, CN2.P18, CN2.P19, CN2.P2, CN2.P20, CN2.P21, CN2.P22, CN2.P23, CN2.P24, CN2.P25, CN2.P3, CN2.P4, CN2.P5, CN2.P6, CN2.P7, CN2.P8, CN2.P9, CN3.N, CN3.N1, CN3.N10, CN3.N11, CN3.N12, CN3.N13, CN3.N14, CN3.N15, CN3.N16, CN3.N17, CN3.N18, CN3.N19, CN3.N2, CN3.N20, CN3.N21, CN3.N22, CN3.N23, CN3.N24, CN3.N3, CN3.N4, CN3.N5, CN3.N6, CN3.N7, CN3.N8, CN3.N9
- net N$42: now also CN3.+, R1.1, R2.1; no longer F1.2
- net PACK_MID: now also CN1.+, CN2.-; no longer CN1.P1, CN1.P10, CN1.P11, CN1.P12, CN1.P13, CN1.P14, CN1.P15, CN1.P16, CN1.P17, CN1.P18, CN1.P19, CN1.P2, CN1.P20, CN1.P21, CN1.P22, CN1.P23, CN1.P24, CN1.P25, CN1.P3, CN1.P4, CN1.P5, CN1.P6, CN1.P7, CN1.P8, CN1.P9, CN2.N, CN2.N1, CN2.N10, CN2.N11, CN2.N12, CN2.N13, CN2.N14, CN2.N15, CN2.N16, CN2.N17, CN2.N18, CN2.N19, CN2.N2, CN2.N20, CN2.N21, CN2.N22, CN2.N23, CN2.N24, CN2.N3, CN2.N4, CN2.N5, CN2.N6, CN2.N7, CN2.N8, CN2.N9
- net PGND: now also CN1.-; no longer CN1.N, CN1.N1, CN1.N10, CN1.N11, CN1.N12, CN1.N13, CN1.N14, CN1.N15, CN1.N16, CN1.N17, CN1.N18, CN1.N19, CN1.N2, CN1.N20, CN1.N21, CN1.N22, CN1.N23, CN1.N24, CN1.N3, CN1.N4, CN1.N5, CN1.N6, CN1.N7, CN1.N8, CN1.N9
- net PWR_VPACK: now also CN4.12, CN4.13, CN4.14, CN4.15; no longer CN5.1, CN5.2, CN5.3, CN5.4
Routing:
- net PACK_MID: track 130.0 -> 1.25 mm
- net N$39: track 66.9 -> 0.00 mm
- net N$4: track 57.5 -> 0.00 mm
- net N$42: track 0.00 -> 54.5 mm, vias 29 -> 0
- net N$59: track 48.1 -> 41.0 mm
- net N$58: track 6.89 -> 0.06 mm, vias 2 -> 0
- net BMS_NALERT: track 25.1 -> 29.8 mm
- net N$56: track 46.2 -> 42.3 mm
- net BMS_I2C_SDA: track 24.4 -> 27.7 mm
- net PWR_VPACK: track 28.5 -> 25.9 mm
- net N$43: track 4.56 -> 2.09 mm
- net BMS_I2C_SCL: track 25.0 -> 26.8 mm
- net N$6: track 25.7 -> 23.9 mm
- net GND: track 30.3 -> 29.5 mm
- net PGND: vias 38 -> 28
- added copper zone on layer 16, net GND
- added copper zone on layer 16, net PWR_VPACK
- removed copper zone on layer 1, net GND
- removed copper zone on layer 1, net N$42
- removed copper zone on layer 16, net N$42
- removed copper zone on layer 1, net PWR_VPACK
Other:
- outline, holes or cut-outs redrawn
- board text added: "gswdh.co.uk camera power PCB rev 1.2.0 2023.09.22"
- board text removed: "gswdh.co.uk camera power PCB rev 1.1.0 2023.09.01"

Commit message: Power PCB connector now in correct orientation
Parts:
- moved CN4 0.40 mm to (-0.38, 48.4), turned to 90 degrees
- moved R8 0.38 mm to (4.25, 53.8)
Connections:
- net BMS_BUS_RSVD_2: now also CN4.9; no longer CN4.7
- net BMS_I2C_SCL: now also CN4.5; no longer CN4.11
- net BMS_I2C_SDA: now also CN4.6; no longer CN4.10
- net BMS_NALERT: now also CN4.7; no longer CN4.9
- net GND: now also CN4.10, CN4.11, CN4.12, CN4.13, CN4.14, CN4.15; no longer CN4.1, CN4.2, CN4.3, CN4.4, CN4.5, CN4.6
- net PWR_VPACK: now also CN4.1, CN4.2, CN4.3, CN4.4; no longer CN4.12, CN4.13, CN4.14, CN4.15
Routing:
- net PWR_VPACK: track 25.9 -> 17.4 mm
- net BMS_NALERT: track 29.8 -> 24.0 mm
- net BMS_I2C_SDA: track 27.7 -> 22.6 mm
- net BMS_I2C_SCL: track 26.8 -> 22.6 mm
Changed lines of the file:
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@@
 <attribute name="PRICE_PER" value="0.08" x="40.75" y="49.75" size="1.778" layer="28" rot="MR270" display="off"/>
 </element>
-<element name="R8" library="RESISTORS" package="1206" value="0R01" x="3.875" y="53.75" smashed="yes" rot="MR0">
-<attribute name="DIGIKEY" value="CRF1206-FZ-R010ELFCT-ND" x="26.5" y="11.75" size="1.778" layer="28" rot="MR0" display="off"/>
-<attribute name="HEIGHT" value="0.65" x="26.5" y="11.75" size="1.778" layer="28" rot="MR0" display="off"/>
-<attribute name="NAME" x="6.25" y="52.75" size="0.5" layer="26" rot="MR90"/>
-<attribute name="PRICE_PER" value="0.42" x="26.5" y="11.75" size="1.778" layer="28" rot="MR0" display="off"/>
+<element name="R8" library="RESISTORS" package="1206" value="0R01" x="4.25" y="53.75" smashed="yes" rot="MR0">
+<attribute name="DIGIKEY" value="CRF1206-FZ-R010ELFCT-ND" x="26.875" y="11.75" size="1.778" layer="28" rot="MR0" display="off"/>
+<attribute name="HEIGHT" value="0.65" x="26.875" y="11.75" size="1.778" layer="28" rot="MR0" display="off"/>
+<attribute name="NAME" x="6.625" y="52.75" size="0.5" layer="26" rot="MR90"/>
+<attribute name="PRICE_PER" value="0.42" x="26.875" y="11.75" size="1.778" layer="28" rot="MR0" display="off"/>
 </element>
 <element name="C5" library="CAPACITORS" package="0603" value="100nF 16V" x="22.625" y="36.625" smashed="yes" rot="MR90">
@@
 <attribute name="PRICE_PER" value="0.10000" x="26.375" y="41.875" size="1.778" layer="28" rot="MR0" display="off"/>
 </element>
-<element name="CN4" library="CONNECTORs" package="SFV15R-1STE1HLF" value="15PIN 0.5MM" x="0" y="48.5" smashed="yes" rot="MR180">
-<attribute name="DIGIKEY" value="609-4311-1-ND" x="0" y="48.5" size="1.778" layer="28" rot="MR180" display="off"/>
-<attribute name="HEIGHT" value="1.8" x="0" y="48.5" size="1.778" layer="28" rot="MR180" display="off"/>
-<attribute name="NAME" x="-6.75" y="45.625" size="1" layer="26" rot="MR180"/>
-<attribute name="PRICE_PER" value="0.46" x="0" y="48.5" size="1.778" layer="28" rot="MR180" display="off"/>
+<element name="CN4" library="CONNECTORs" package="SFV15R-1STE1HLF" value="15PIN 0.5MM" x="-0.375" y="48.375" smashed="yes" rot="MR90">
+<attribute name="DIGIKEY" value="609-4311-1-ND" x="-0.375" y="48.375" size="1.778" layer="28" rot="MR90" display="off"/>
+<attribute name="HEIGHT" value="1.8" x="-0.375" y="48.375" size="1.778" layer="28" rot="MR90" display="off"/>
+<attribute name="NAME" x="2.5" y="41.625" size="1" layer="26" rot="MR90"/>
+<attribute name="PRICE_PER" value="0.46" x="-0.375" y="48.375" size="1.778" layer="28" rot="MR90" display="off"/>
 </element>
 </elements>
@@
 <wire x1="18.25" y1="43.33" x2="18.25" y2="54.25" width="0.15" layer="16"/>
 <wire x1="18.25" y1="54.25" x2="16.75" y2="55.75" width="0.15" layer="16"/>
-<wire x1="2.375" y1="54.75" x2="2.375" y2="53.75" width="0.15" layer="16"/>
+<wire x1="2.75" y1="55.125" x2="2.75" y2="53.75" width="0.15" layer="16"/>
 <wire x1="16.75" y1="55.75" x2="3.375" y2="55.75" width="0.15" layer="16"/>
-<wire x1="3.375" y1="55.75" x2="2.375" y2="54.75" width="0.15" layer="16"/>
-<contactref element="CN4" pad="1"/>
-<contactref element="CN4" pad="2"/>
-<contactref element="CN4" pad="3"/>
-<contactref element="CN4" pad="4"/>
-<contactref element="CN4" pad="5"/>
-<contactref element="CN4" pad="6"/>
+<wire x1="3.375" y1="55.75" x2="2.75" y2="55.125" width="0.15" layer="16"/>
+<contactref element="CN4" pad="10"/>
+<contactref element="CN4" pad="11"/>
+<contactref element="CN4" pad="12"/>
+<contactref element="CN4" pad="13"/>
+<contactref element="CN4" pad="14"/>
+<contactref element="CN4" pad="15"/>
 </signal>
 <signal name="N$38">
@@
 <wire x1="16.92" y1="40" x2="15.5" y2="40" width="0.15" layer="16"/>
 <wire x1="15.5" y1="40" x2="14.875" y2="39.375" width="0.15" layer="16"/>
-<contactref element="CN4" pad="11"/>
 <wire x1="14.875" y1="39.375" x2="9.95073125" y2="39.375" width="0.15" layer="16"/>
-<wire x1="9.95073125" y1="39.375" x2="7.5" y2="41.82573125" width="0.15" layer="16"/>
-<wire x1="7.5" y1="41.82573125" x2="7.5" y2="50.75" width="0.15" layer="16"/>
-<wire x1="7.5" y1="50.75" x2="6.875" y2="51.375" width="0.15" layer="16"/>
-<wire x1="6.875" y1="51.375" x2="1.7068" y2="51.375" width="0.15" layer="16"/>
-<wire x1="1.5" y1="50.375" x2="1.5" y2="51.1682" width="0.15" layer="16"/>
-<wire x1="1.5" y1="51.1682" x2="1.7068" y2="51.375" width="0.15" layer="16"/>
+<wire x1="-1" y1="47" x2="-1.125" y2="46.875" width="0.15" layer="16"/>
+<wire x1="-1.125" y1="46.875" x2="-2.25" y2="46.875" width="0.15" layer="16"/>
+<contactref element="CN4" pad="5"/>
+<wire x1="9.95073125" y1="39.375" x2="2.32573125" y2="47" width="0.15" layer="16"/>
+<wire x1="2.32573125" y1="47" x2="-1" y2="47" width="0.15" layer="16"/>
 </signal>
 <signal name="BMS_I2C_SDA">
@@
 <wire x1="16.92" y1="40.5" x2="15.5" y2="40.5" width="0.15" layer="16"/>
 <wire x1="15.5" y1="40.5" x2="14.75" y2="39.75" width="0.15" layer="16"/>
-<contactref element="CN4" pad="10"/>
-<wire x1="1.375" y1="51.75" x2="1" y2="51.375" width="0.15" layer="16"/>
-<wire x1="1" y1="51.375" x2="1" y2="50.375" width="0.15" layer="16"/>
 <wire x1="14.75" y1="39.75" x2="10" y2="39.75" width="0.15" layer="16"/>
-<wire x1="10" y1="39.75" x2="7.875" y2="41.875" width="0.15" layer="16"/>
-<wire x1="7.875" y1="41.875" x2="7.875" y2="51" width="0.15" layer="16"/>
-<wire x1="7.875" y1="51" x2="7.125" y2="51.75" width="0.15" layer="16"/>
-<wire x1="7.125" y1="51.75" x2="1.375" y2="51.75" width="0.15" layer="16"/>
+<contactref element="CN4" pad="6"/>
+<wire x1="10" y1="39.75" x2="2.375" y2="47.375" width="0.15" layer="16"/>
+<wire x1="2.375" y1="47.375" x2="-2.25" y2="47.375" width="0.15" layer="16"/>
 </signal>
 <signal name="N$2">
@@
 <contactref element="Q2" pad="2"/>
 <polygon width="0.15" layer="16" thermals="no">
-<vertex x="3.75" y="51.125"/>
+<vertex x="3.75" y="47.625"/>
 <vertex x="3.75" y="38.875"/>
 <vertex x="-12.75" y="38.875"/>
 <vertex x="-12.75" y="47.625"/>
-<vertex x="1.875" y="47.625"/>
-<vertex x="1.875" y="51.125"/>
 </polygon>
 <wire x1="16.625" y1="35.875" x2="17.875" y2="35.875" width="0.15" layer="16"/>
-<contactref element="CN4" pad="12"/>
-<contactref element="CN4" pad="13"/>
-<contactref element="CN4" pad="14"/>
-<contactref element="CN4" pad="15"/>
 <wire x1="5.75" y1="41.625" x2="3.25" y2="41.625" width="0.15" layer="16"/>
 <wire x1="3.25" y1="41.625" x2="3" y2="41.875" width="0.15" layer="16"/>
-<wire x1="3" y1="41.875" x2="3" y2="50.375" width="0.15" layer="16"/>
 <wire x1="16.625" y1="35.875" x2="11.5" y2="35.875" width="0.15" layer="16"/>
 <wire x1="11.5" y1="35.875" x2="5.75" y2="41.625" width="0.15" layer="16"/>
+<contactref element="CN4" pad="1"/>
+<contactref element="CN4" pad="2"/>
+<contactref element="CN4" pad="3"/>
+<contactref element="CN4" pad="4"/>
 </signal>
 <signal name="BMS_NALERT">
@@
 <wire x1="16.92" y1="39.5" x2="15.42426875" y2="39.5" width="0.15" layer="16"/>
 <wire x1="15.42426875" y1="39.5" x2="14.92426875" y2="39" width="0.15" layer="16"/>
-<contactref element="CN4" pad="9"/>
 <wire x1="11" y1="39" x2="10.875" y2="38.875" width="0.15" layer="16"/>
 <via x="10.875" y="38.875" extent="1-16" drill="0.3"/>
@@
 <via x="10.875" y="40.375" extent="1-16" drill="0.3"/>
 <wire x1="10.875" y1="40.375" x2="9.875" y2="40.375" width="0.15" layer="16"/>
-<wire x1="0.5" y1="51.5" x2="0.5" y2="50.375" width="0.15" layer="16"/>
 <wire x1="14.92426875" y1="39" x2="11" y2="39" width="0.15" layer="16"/>
-<wire x1="9.875" y1="40.375" x2="8.25" y2="42" width="0.15" layer="16"/>
-<wire x1="8.25" y1="42" x2="8.25" y2="51.125" width="0.15" layer="16"/>
-<wire x1="1.125" y1="52.125" x2="0.5" y2="51.5" width="0.15" layer="16"/>
-<wire x1="8.25" y1="51.125" x2="7.25" y2="52.125" width="0.15" layer="16"/>
-<wire x1="7.25" y1="52.125" x2="1.125" y2="52.125" width="0.15" layer="16"/>
-</signal>
-<signal name="BMS_BUS_RSVD_1">
-<contactref element="CN4" pad="8"/>
-</signal>
-<signal name="BMS_BUS_RSVD_2">
+<wire x1="-1" y1="47.75" x2="-1.125" y2="47.875" width="0.15" layer="16"/>
+<wire x1="-1.125" y1="47.875" x2="-2.25" y2="47.875" width="0.15" layer="16"/>
 <contactref element="CN4" pad="7"/>
+<wire x1="9.875" y1="40.375" x2="2.5" y2="47.75" width="0.15" layer="16"/>
+<wire x1="2.5" y1="47.75" x2="-1" y2="47.75" width="0.15" layer="16"/>
 </signal>
 <signal name="N$6">
@@
 <wire x1="20.83" y1="40.5" x2="20.83" y2="41" width="0" layer="19" extent="16-16"/>
 </signal>
+<signal name="BMS_BUS_RSVD_1">
+<contactref element="CN4" pad="8"/>
+</signal>
+<signal name="BMS_BUS_RSVD_2">
+<contactref element="CN4" pad="9"/>
+</signal>
 </signals>

Commit message: Power PCB updated
Parts:
- removed CN4: 15PIN 0.5MM, CONNECTORs:SFV15R-1STE1HLF
- added CN5: 15PIN 0.5MM, CONNECTORs:SFV15R-1STE1HLF
- moved Q1 66.5 mm to (37.4, 9.12), flipped to the top, turned to 0 degrees
- moved Q2 59.2 mm to (37.4, 14.4), flipped to the top, turned to 0 degrees
- moved R7 57.9 mm to (32.2, 7.25), flipped to the top
- moved R9 54.6 mm to (32.2, 12.5), flipped to the top, turned to 0 degrees
- moved R8 39.2 mm to (35.0, 29.5), flipped to the top, turned to 270 degrees
- moved R13 36.4 mm to (33.4, 30.4), flipped to the top, turned to 270 degrees
- moved R6 16.9 mm to (27.0, 31.8), flipped to the top, turned to 90 degrees
- moved C7 16.0 mm to (28.4, 33.8), flipped to the top, turned to 0 degrees
- moved C9 15.3 mm to (30.0, 35.9), flipped to the top, turned to 0 degrees
- moved R11 15.1 mm to (25.8, 31.8), flipped to the top, turned to 90 degrees
- moved C8 12.5 mm to (30.0, 37.9), flipped to the top, turned to 0 degrees
- moved R1 9.58 mm to (21.5, 44.6), flipped to the top, turned to 270 degrees
- moved C10 9.07 mm to (22.5, 32.9), flipped to the top, turned to 90 degrees
- moved R2 7.88 mm to (22.8, 44.6), flipped to the top, turned to 270 degrees
- moved U1 7.88 mm to (25.9, 37.1), flipped to the top, turned to 0 degrees
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Connections:
- net BMS_BUS_RSVD_1: now also CN5.8; no longer CN4.8
- net BMS_BUS_RSVD_2: now also CN5.7; no longer CN4.9
- net BMS_I2C_SCL: now also CN5.11; no longer CN4.5
- net BMS_I2C_SDA: now also CN5.10; no longer CN4.6
- net BMS_NALERT: now also CN5.9; no longer CN4.7
- net GND: now also CN5.1, CN5.2, CN5.3, CN5.4, CN5.5, CN5.6; no longer CN4.10, CN4.11, CN4.12, CN4.13, CN4.14, CN4.15
- net PWR_VPACK: now also CN5.12, CN5.13, CN5.14, CN5.15; no longer CN4.1, CN4.2, CN4.3, CN4.4
Routing:
- net PACK_MID: track 1.25 -> 200.9 mm, vias 0 -> 1
- net N$4: track 0.00 -> 118.5 mm, vias 0 -> 1
- net N$42: track 54.5 -> 75.4 mm, vias 0 -> 26
- net GND: track 29.4 -> 16.2 mm
- net PWR_VPACK: track 17.4 -> 27.3 mm
- net N$6: track 23.9 -> 14.7 mm
- net N$56: track 42.3 -> 35.2 mm
- net PGND: track 13.3 -> 16.0 mm, vias 28 -> 34
- net BMS_I2C_SCL: track 22.6 -> 24.6 mm
- net N$57: track 32.0 -> 30.3 mm
- net N$59: track 41.0 -> 42.6 mm
- net N$58: track 0.06 -> 1.72 mm
- net BMS_I2C_SDA: track 22.6 -> 24.0 mm
- net N$3: track 11.0 -> 12.3 mm
- net BMS_NALERT: track 24.0 -> 24.7 mm
- added copper zone on layer 1, net GND
- added copper zone on layer 1, net N$42
- added copper zone on layer 1, net PWR_VPACK
- removed copper zone on layer 16, net GND
- removed copper zone on layer 16, net PWR_VPACK
Other:
- outline, holes or cut-outs redrawn
- board text added: "gswdh.co.uk camera power PCB rev 1.2.0 2023.10.24"
- board text removed: "gswdh.co.uk camera power PCB rev 1.2.0 2023.09.22"

Commit message: Fixed ETH RX CTL and CLK bug. Mved USB and WTH resets to PL
Other:
- outline, holes or cut-outs redrawn
Changed lines of the file:
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@@
 <setting verticaltext="up"/>
 </settings>
-<grid distance="0.125" unitdist="mm" unit="mm" style="lines" multiple="1" display="yes" altdistance="0.0625" altunitdist="mm" altunit="mm"/>
+<grid distance="0.01" unitdist="mm" unit="mm" style="lines" multiple="1" display="yes" altdistance="0.0625" altunitdist="mm" altunit="mm"/>
 <layers>
 <layer number="1" name="Top" color="4" fill="1" visible="yes" active="yes"/>
@@
 </layers>
 <board>
-<fusionsync huburn="a.YnVzaW5lc3M6bXl1Y2wxNDk2" projecturn="a.YnVzaW5lc3M6bXl1Y2wxNDk2IzIwMjExMjA3NDc0MjU0MzI2" f3durn="urn:adsk.wipprod:dm.lineage:fSLqUUoyRPS3Y_nTmPxjag" pcbguid="" lastpulledtime="" lastsyncedchangeguid="" latestrevisionid="e6377d3b-3d46-4d91-8665-f750c05ee5dd" lastsyncedrevisionid="e6377d3b-3d46-4d91-8665-f750c05ee5dd" lastboardhashguid="592efbe1-0410-9761-83a9-80d70b0fd50a" lastpushedtime="2023-10-24T12:27:45Z" linktopcb3d="true"/>
+<fusionsync huburn="a.YnVzaW5lc3M6bXl1Y2wxNDk2" projecturn="a.YnVzaW5lc3M6bXl1Y2wxNDk2IzIwMjExMjA3NDc0MjU0MzI2" f3durn="urn:adsk.wipprod:dm.lineage:fSLqUUoyRPS3Y_nTmPxjag" pcbguid="" lastpulledtime="" lastsyncedchangeguid="" latestrevisionid="d7a7c983-fb24-4705-bd6c-139b3cd3fb53" lastsyncedrevisionid="d7a7c983-fb24-4705-bd6c-139b3cd3fb53" lastboardhashguid="f4c80b79-bbe1-e5b1-3553-b7d58f142774" lastpushedtime="2023-11-30T13:24:19Z" linktopcb3d="true"/>
 <plain>
 <wire x1="-49" y1="60" x2="-60" y2="49" width="0" layer="20" curve="90"/>
@@
 <wire x1="-49" y1="-60" x2="49" y2="-60" width="0" layer="20"/>
 <wire x1="60" y1="-49" x2="60" y2="49" width="0" layer="20"/>
-<circle x="0" y="0" radius="29" width="0.0001" layer="20"/>
 <wire x1="57" y1="29" x2="57" y2="21" width="0" layer="20"/>
 <wire x1="57" y1="21" x2="58" y2="20" width="0" layer="20" curve="90"/>
@@
 <wire x1="59" y1="29" x2="58" y2="30" width="0" layer="20" curve="90"/>
 <wire x1="58" y1="30" x2="57" y2="29" width="0" layer="20" curve="90"/>
+<wire x1="-30.55918125" y1="12.44556875" x2="-31.4" y2="10.1" width="0" layer="20"/>
+<wire x1="-24.747209375" y1="15.11871875" x2="-30.55918125" y2="12.44556875" width="0" layer="20" curve="90.600938"/>
+<wire x1="-32.1711" y1="7.333209375" x2="-28.95" y2="1.81" width="0" layer="20" curve="90.600864"/>
+<wire x1="-32.1711" y1="7.333209375" x2="-31.53" y2="9.73" width="0" layer="20"/>
+<wire x1="-28.95" y1="1.81" x2="-24.747209375" y2="15.11871875" width="0" layer="20" curve="332.156305"/>
+<wire x1="-31.4" y1="10.1" x2="-31.53" y2="9.73" width="0" layer="20"/>
 </plain>
 <attributes>
@@
 <attribute name="DIGIKEY" value="36-1122-ND" x="-44.5" y="8" size="1.778" layer="28" rot="MR270" display="off"/>
 <attribute name="HEIGHT" value="22" x="-44.5" y="8" size="1.778" layer="28" rot="MR270" display="off"/>
-<attribute name="NAME" x="-39.5" y="-2.25" size="0.5" layer="22" rot="MR270"/>
+<attribute name="NAME" x="-57.25" y="-33.5" size="0.5" layer="22" rot="MR180"/>
 <attribute name="PRICE_PER" value="4.1" x="-44.5" y="8" size="1.778" layer="28" rot="MR270" display="off"/>
 </element>
@@
 <attribute name="DIGIKEY" value="36-1122-ND" x="0" y="-46.5" size="1.778" layer="28" rot="MR180" display="off"/>
 <attribute name="HEIGHT" value="22" x="0" y="-46.5" size="1.778" layer="28" rot="MR180" display="off"/>
-<attribute name="NAME" x="-18.25" y="-49.375" size="0.5" layer="22" rot="MR180"/>
+<attribute name="NAME" x="-41.125" y="-58.25" size="0.5" layer="22" rot="MR270"/>
 <attribute name="PRICE_PER" value="4.1" x="0" y="-46.5" size="1.778" layer="28" rot="MR180" display="off"/>
 </element>
@@
 <attribute name="DIGIKEY" value="36-1122-ND" x="44.5" y="8" size="1.778" layer="28" rot="MR90" display="off"/>
 <attribute name="HEIGHT" value="22" x="44.5" y="8" size="1.778" layer="28" rot="MR90" display="off"/>
-<attribute name="NAME" x="48.375" y="10.875" size="0.5" layer="22" rot="MR90"/>
+<attribute name="NAME" x="56.375" y="-33.125" size="0.5" layer="22" rot="MR180"/>
 <attribute name="PRICE_PER" value="4.1" x="44.5" y="8" size="1.778" layer="28" rot="MR90" display="off"/>
 </element>
@@
 <via x="34.75" y="32.5" extent="1-16" drill="0.5"/>
 <polygon width="0.15" layer="1" thermals="no" rank="6">
-<vertex x="-60" y="60"/>
-<vertex x="60" y="60"/>
+<vertex x="-60" y="70.83"/>
+<vertex x="60" y="70.83"/>
 <vertex x="60" y="-60"/>
 <vertex x="-60" y="-60"/>
