File: power.brd (EAGLE design)
At the start: 120 x 120 mm, 33 parts, among them CN1 21700, CN2 21700, CN3 21700, CN5 15PIN 0.5MM, Q1 SIRA36DP-T1-GE3, Q2 SIRA36DP-T1-GE3, U1 MAX17320G20+

Commit message: Power PCB updated and ready for manufacture
Parts:
- added C11, C3: 0.1uF 16V, c_0402:0402
- added C12: 2.2uF 6.3V, c_0603:0603
- added C13: 1uF 25V, c_0603:0603
- added D1: VDMR10A1, OPTO:VDMX10A1
- added Q10, Q3, Q4, Q5, Q6, Q7, Q8, Q9: BSS123, TRANSISTORs:SOT23-3
- added R14, R15, R16, R17, R18, R19, R20, R21: 1k, r_0402:0402
- added R22, R23, R24, R25, R26, R27, R28, R29, R30, R31: 10k, r_0402:0402
- added TP1, TP2, TP3, TP4: TEST_POINT_SQUARE, MISC:OSPREY_HSS_PAD
- added U2: TCA6408AQPWRQ1, ICs:TSSOP16
- added U3: TPS70918, ICs:SOT23-5
- moved MECH3 18.0 mm to (-35.0, 53.0)
- moved MECH6 18.0 mm to (35.0, 53.0)
- moved MECH7 11.0 mm to (-53.0, -42.0)
- moved MECH8 11.0 mm to (53.0, -42.0)
- moved C1 3.98 mm to (21.0, 45.7)
- moved C10 3.98 mm to (20.0, 36.0)
- moved C2 3.98 mm to (23.8, 45.7)
- moved C4 3.98 mm to (26.5, 45.7)
- moved C5 3.98 mm to (19.2, 44.0)
- moved C6 3.98 mm to (20.0, 42.0)
- moved C7 3.98 mm to (25.9, 36.9)
- moved C8 3.98 mm to (27.5, 41.0)
- moved C9 3.98 mm to (27.5, 39.0)
- moved R1 3.98 mm to (19.0, 47.7)
- moved R10 3.98 mm to (19.2, 39.2)
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Connections:
- removed net BMS_BUS_RSVD_1: CN5.8
- removed net BMS_BUS_RSVD_2: CN5.7
- new net N$10: D1.5, R18.1
- new net N$11: D1.10, R19.1
- new net N$12: D1.9, R20.1
- new net N$13: D1.1, R21.1
- new net N$18: Q3.2, R14.1
- new net N$19: Q4.2, R15.1
- new net N$20: Q5.2, R16.1
- new net N$21: Q6.2, R17.1
- new net N$26: Q7.2, R21.2
- new net N$27: Q8.2, R20.2
- new net N$28: Q9.2, R19.2
- new net N$29: Q10.2, R18.2
- new net N$44: R30.1, U2.13
- new net N$5: D1.7, R14.2
- new net N$50: R31.1, U2.3
- new net N$7: D1.6, R15.2
- new net N$8: D1.4, R16.2
- new net N$9: D1.2, R17.2
- new net PWR_BMS_1V8: C11.2, C12.2, C3.2, R30.2, R31.2, TP1.1, U2.1, U2.16, U3.5
- new net SVNSEG_A: Q3.1, R22.2, U2.6
- new net SVNSEG_B: Q4.1, R23.2, U2.7
- new net SVNSEG_C: Q5.1, R24.2, U2.11
- new net SVNSEG_D: Q6.1, R25.2, U2.10
- new net SVNSEG_DP: Q10.1, R29.2, U2.12
- new net SVNSEG_E: Q7.1, R26.2, U2.9
- new net SVNSEG_F: Q8.1, R27.2, U2.5
- new net SVNSEG_G: Q9.1, R28.2, U2.4
- net BMS_I2C_SCL: now also TP2.1, U2.14
- net BMS_I2C_SDA: now also TP3.1, U2.15
- net GND: now also C11.1, C12.1, C13.1, C3.1, Q10.3, Q3.3, Q4.3, Q5.3, Q6.3, Q7.3, Q8.3, Q9.3, R22.1, R23.1, R24.1, R25.1, R26.1, R27.1, R28.1, R29.1, TP4.1, U2.2, U2.8, U3.2
- net PWR_VPACK: now also C13.2, D1.3, D1.8, U3.1, U3.3
Routing:
- net PWR_VPACK: track 27.3 -> 231.7 mm
- net GND: track 16.2 -> 157.8 mm, vias 0 -> 18
- net SVNSEG_E: track 0.00 -> 60.7 mm
- net SVNSEG_D: track 0.00 -> 57.0 mm
- net BMS_I2C_SCL: track 24.6 -> 80.3 mm, vias 0 -> 3
- net BMS_I2C_SDA: track 24.0 -> 79.0 mm, vias 0 -> 3
- net SVNSEG_C: track 0.00 -> 53.3 mm
- net SVNSEG_DP: track 0.00 -> 49.8 mm
- net SVNSEG_G: track 0.00 -> 25.1 mm
- net SVNSEG_F: track 0.00 -> 21.4 mm
- net PWR_BMS_1V8: track 0.00 -> 20.7 mm, vias 0 -> 1
- net SVNSEG_A: track 0.00 -> 17.6 mm
- net SVNSEG_B: track 0.00 -> 15.6 mm
- net N$56: track 35.2 -> 40.4 mm
- net N$44: track 0.00 -> 5.02 mm
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- added copper zone on layer 16, net GND
Other:
- outline, holes or cut-outs redrawn
- board text added: "gswdh.co.uk camera power PCB rev 1.2.2 2024.09.15"
- board text removed: "gswdh.co.uk camera power PCB rev 1.2.0 2023.10.24"

Commit message: Added I2C test points
Parts:
- Q10, Q3, Q4, Q5, Q6, Q7, Q8, Q9: value BSS123 -> DMN2005K-7

Commit message: started on power pcb
Parts:
- removed CN1, CN2: 21700, CONNECTORs:1122
- removed D1: VDMR10A1, OPTO:VDMX10A1
- removed MECH7: 6mm x 3mm, MISC:MOUNTHOLE_6X3
- removed Q10, Q3, Q4, Q5, Q6, Q7, Q8, Q9: DMN2005K-7, TRANSISTORs:SOT23-3
- removed R19: 1k, r_0402:0402
- removed R22, R24, R26, R27, R28, R29, R30, R31: 10k, r_0402:0402
- removed TP1, TP2, TP3, TP4: TEST_POINT_SQUARE, MISC:OSPREY_HSS_PAD
- added C14, C18, C19, C22, C24, C25, C26: 22uF 50V, CAPACITORS:2220
- added C15, C16: 47pF 25V, c_0402:0402
- added C17, C23, C27: 10uF 50V, CAPACITORS:1210
- added C20: 0.1uF 50V, c_0603:0603
- added C21: 100nF 16V, CAPACITORS:0603
- added CN10, CN11, CN12, CN15, CN16, CN17, CN18, CN21, CN22, CN23, CN24, CN4, CN6, CN9: 21700 CLIP, CONNECTORs:KEYSTONE_247
- added MECH10, MECH2, MECH4: 6mm x 3mm, MISC:MOUNTHOLE_6X3
- added U5: NCS20071, ICs:SOT23-5
- added U6: LTM8055, ICs:BGA121-1.27MM
- C11, C3: value 0.1uF 16V -> 47pF 25V
- C12: value 2.2uF 6.3V -> 10uF 50V; device c_0603:0603 -> CAPACITORS:1210
- C13: value 1uF 25V -> 22uF 50V; device c_0603:0603 -> CAPACITORS:2220
- CN3: value 21700 -> 21700 CLIP; device CONNECTORs:1122 -> CONNECTORs:KEYSTONE_247
- CN5: value 15PIN 0.5MM -> 21700 CLIP; device CONNECTORs:SFV15R-1STE1HLF -> CONNECTORs:KEYSTONE_247
- R13: value 10R -> 0R082; device r_0603:0603 -> RESISTORS:2512
- R14: value 1k -> 150k
- R15: value 1k -> 12k
- R16, R18: value 1k -> 10k
- R17: value 1k -> 45.3k
- R20: value 1k -> 75k
- R21: value 1k -> 5.1k
- R23: value 10k -> 45.3k
- U2: value TCA6408AQPWRQ1 -> LTM8055; device ICs:TSSOP16 -> ICs:BGA121-1.27MM
- U3: value TPS70918 -> STM32G030C8; device ICs:SOT23-5 -> ICs:QFP48
- moved MECH3 175.5 mm to (37.0, -107.0), turned to 90 degrees
- moved MECH8 174.1 mm to (-37.0, 107.0), turned to 90 degrees
- moved U3 136.9 mm to (-3.75, -87.9), flipped to the bottom, turned to 0 degrees
- moved R4 107.6 mm to (-5.00, -55.4), flipped to the bottom, turned to 180 degrees
- moved C4 106.0 mm to (-3.00, -56.1), flipped to the bottom, turned to 90 degrees
- moved R5 104.6 mm to (-5.00, -52.6), flipped to the bottom, turned to 180 degrees
- moved R3 101.5 mm to (-5.00, -49.9), flipped to the bottom, turned to 180 degrees
- moved C2 100.0 mm to (-3.00, -50.6), flipped to the bottom, turned to 90 degrees
- moved C8 98.4 mm to (1.75, -54.0), flipped to the bottom, turned to 270 degrees
- moved R2 98.2 mm to (-5.00, -47.1), flipped to the bottom, turned to 180 degrees
- moved R8 97.0 mm to (3.75, -63.4), flipped to the bottom, turned to 180 degrees
- moved C1 96.6 mm to (-3.00, -47.9), flipped to the bottom, turned to 90 degrees
- moved R1 96.6 mm to (-5.00, -45.9), flipped to the bottom, turned to 180 degrees
- moved C9 96.0 mm to (3.75, -54.0), flipped to the bottom, turned to 270 degrees
- moved U1 92.7 mm to (2.50, -50.1), flipped to the bottom, turned to 270 degrees
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Connections:
- removed net N$13: D1.1, R21.1
- removed net N$19: Q4.2, R15.1
- removed net N$20: Q5.2, R16.1
- removed net N$21: Q6.2, R17.1
- removed net N$26: Q7.2, R21.2
- removed net N$29: Q10.2, R18.2
- removed net N$42: CN3.+, Q1.1, Q1.2, Q1.3, R1.1, R2.1
- removed net N$44: R30.1, U2.13
- removed net N$50: R31.1, U2.3
- removed net N$6: R13.2, U1.15
- removed net N$8: D1.4, R16.2
- removed net N$9: D1.2, R17.2
- removed net PACK_MID: CN1.+, CN2.-, R4.1, R5.1
- removed net PWR_BMS_1V8: C11.2, C12.2, C3.2, R30.2, R31.2, TP1.1, U2.1, U2.16, U3.5
- removed net PWR_VPACK: C13.2, CN5.12, CN5.13, CN5.14, CN5.15, D1.3, D1.8, Q2.1, Q2.2, Q2.3, R10.2, R12.2, U3.1, U3.3
- removed net SVNSEG_A: Q3.1, R22.2, U2.6
- removed net SVNSEG_B: Q4.1, R23.2, U2.7
- removed net SVNSEG_C: Q5.1, R24.2, U2.11
- removed net SVNSEG_D: Q6.1, R25.2, U2.10
- removed net SVNSEG_DP: Q10.1, R29.2, U2.12
- removed net SVNSEG_E: Q7.1, R26.2, U2.9
- removed net SVNSEG_F: Q8.1, R27.2, U2.5
- removed net SVNSEG_G: Q9.1, R28.2, U2.4
- new net CHRG_ENABLE: R25.1, U2.L4
- new net CHRG_IOUT_CTL: R18.1, U5.3
- new net N$17: U2.F1, U2.G2
- new net N$22: CN11.1, CN11.2, CN11.3, CN4.1, CN4.2, CN4.3, CN6.1, CN6.2, CN6.3, CN9.1, CN9.2, CN9.3, R4.1
- new net N$23: R20.1, R21.1, U6.J1
- new net N$25: CN10.1, CN10.2, CN10.3, CN12.1, CN12.2, CN12.3, CN15.1, CN15.2, CN15.3, CN17.1, CN17.2, CN17.3, R5.1
- new net N$32: CN16.1, CN16.2, CN16.3, CN18.1, CN18.2, CN18.3, CN21.1, CN21.2, CN21.3, CN23.1, CN23.2, CN23.3, R3.1
- new net N$35: U6.F1, U6.G2
- new net N$36: C16.2, U6.K1
- new net N$63: C2.1, C21.2, R5.2, U1.22
- new net PWR_BAT_VPACK: C17.2, C27.2, Q2.1, Q2.2, Q2.3, R10.2, R12.2, R13.2, U2.D1, U6.F10, U6.F11, U6.G10, U6.G11, U6.H10, U6.H11, U6.J10, U6.J11, U6.K10, U6.K11, U6.L10, U6.L11, U6.L9
- new net PWR_SYS_19V: C18.2, C19.2, C22.2, C24.2, R20.2, U6.A1, U6.A2, U6.A3, U6.A4, U6.A5, U6.A6, U6.B1, U6.B2, U6.B3, U6.B4, U6.B5, U6.B6, U6.C1, U6.C2, U6.C3, U6.C4, U6.C5, U6.C6, U6.D1
- new net PWR_SYS_19V_EN: R16.1, U6.L4
- new net PWR_SYS_VIN_COND: C12.2, C20.2, C23.2, U2.F10, U2.F11, U2.G10, U2.G11, U2.H10, U2.H11, U2.J10, U2.J11, U2.K10, U2.K11, U2.L10, U2.L11, U2.L9, U5.5
- net BMS_I2C_SCL: no longer CN5.11, TP2.1, U2.14
- net BMS_I2C_SDA: no longer CN5.10, TP3.1, U2.15
- net BMS_NALERT: no longer CN5.9
- net GND: now also C14.1, C15.1, C16.1, C17.1, C18.1, C19.1, C20.1, C22.1, C23.1, C24.1, C25.1, C26.1, C27.1, R15.2, R16.2, R17.1, R18.2, R21.2, R25.2, U2.A10, U2.A11, U2.A7, U2.A8, U2.A9, U2.B10, U2.B11, U2.B7, U2.B8, U2.B9, U2.C10, U2.C11, U2.C7, U2.C8, U2.C9, U2.D10, U2.D11, U2.D2, U2.D3, U2.D4, U2.D5, U2.D6, U2.D7, U2.D8, U2.D9, U2.E1, U2.E10, U2.E11, U2.E2, U2.E3, U2.E4, U2.E5, U2.E6, U2.E7, U2.E8, U2.E9, U2.F2, U2.F3, U2.F4, U2.F5, U2.F6, U2.F7, U2.F8, U2.F9, U2.G3, U2.G4, U2.G5, U2.G6, U2.G7, U2.G8, U2.G9, U2.H2, U2.H3, U2.H4, U2.H5, U2.H6, U2.H7, U2.H8, U2.H9, U2.J3, U2.J4, U2.J5, U2.J6, U2.J7, U2.J8, U2.J9, U2.K3, U2.K4, U2.K5, U2.K6, U2.K7, U2.K8, U2.K9, U2.L1, U2.L5, U2.L6, U2.L7, U2.L8, U5.2, U6.A10, U6.A11, U6.A7, U6.A8, U6.A9, U6.B10, U6.B11, U6.B7, U6.B8, U6.B9, U6.C10, U6.C11, U6.C7, U6.C8, U6.C9, U6.D10, U6.D11, U6.D2, U6.D3, U6.D4, U6.D5, U6.D6, U6.D7, U6.D8, U6.D9, U6.E1, U6.E10, U6.E11, U6.E2, U6.E3, U6.E4, U6.E5, U6.E6, U6.E7, U6.E8, U6.E9, U6.F2, U6.F3, U6.F4, U6.F5, U6.F6, U6.F7, U6.F8, U6.F9, U6.G3, U6.G4, U6.G5, U6.G6, U6.G7, U6.G8, U6.G9, U6.H2, U6.H3, U6.H4, U6.H5, U6.H6, U6.H7, U6.H8, U6.H9, U6.J3, U6.J4, U6.J5, U6.J6, U6.J7, U6.J8, U6.J9, U6.K3, U6.K4, U6.K5, U6.K6, U6.K7, U6.K8, U6.K9, U6.L1, U6.L5, U6.L6, U6.L7, U6.L8; no longer CN5.1, CN5.2, CN5.3, CN5.4, CN5.5, CN5.6, Q10.3, Q3.3, Q4.3, Q5.3, Q6.3, Q7.3, Q8.3, Q9.3, R22.1, R24.1, R25.1, R26.1, R27.1, R28.1, R29.1, TP4.1, U2.2, U2.8, U3.2
- net N$10: now also R17.2, U2.H1; no longer D1.5, R18.1
- net N$11: now also C3.2, U2.J2; no longer D1.10, R19.1
- net N$12: now also U2.K2, U5.1, U5.4; no longer D1.9, R20.1
- net N$18: now also C11.2, U2.K1; no longer Q3.2, R14.1
- net N$27: now also R23.2, U6.H1; no longer Q8.2, R20.2
- net N$28: now also C15.2, U6.J2; no longer Q9.2, R19.2
- net N$3: now also C21.1; no longer C2.1, R5.2, U1.22
- net N$4: now also C13.2, C14.2, C25.2, C26.2, R13.1, R14.2, U2.A1, U2.A2, U2.A3, U2.A4, U2.A5, U2.A6, U2.B1, U2.B2, U2.B3, U2.B4, U2.B5, U2.B6, U2.C1, U2.C2, U2.C3, U2.C4, U2.C5, U2.C6; no longer CN2.+, CN3.-, R3.1
- net N$5: now also CN22.1, CN22.2, CN22.3, CN24.1, CN24.2, CN24.3, Q1.1, Q1.2, Q1.3, R1.1, R2.1; no longer D1.7, R14.2
- net N$7: now also R14.1, R15.1, U2.J1; no longer D1.6, R15.2
- net PGND: now also CN3.1, CN3.2, CN3.3, CN5.1, CN5.2, CN5.3, U1.15; no longer CN1.-, R13.1
Routing:
- net PWR_VPACK: track 231.7 -> 0.00 mm
- net PACK_MID: track 200.7 -> 0.00 mm, vias 3 -> 0
- net GND: track 157.8 -> 8.58 mm, vias 18 -> 41
- net N$4: track 119.6 -> 0.00 mm, vias 3 -> 1
- net BMS_I2C_SCL: track 80.3 -> 0.00 mm, vias 3 -> 0
- net BMS_I2C_SDA: track 79.0 -> 0.00 mm, vias 3 -> 0
- net N$42: track 75.7 -> 0.00 mm, vias 19 -> 0
- net SVNSEG_E: track 60.7 -> 0.00 mm
- net SVNSEG_D: track 57.0 -> 0.00 mm
- net SVNSEG_C: track 53.3 -> 0.00 mm
- net SVNSEG_DP: track 49.8 -> 0.00 mm
- net N$59: track 46.4 -> 11.7 mm
- net N$57: track 30.3 -> 0.00 mm
- net N$56: track 40.4 -> 11.2 mm
- net BMS_NALERT: track 25.9 -> 0.00 mm, vias 2 -> 0
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- removed copper zone on layer 1, net GND
- removed copper zone on layer 16, net GND
- removed copper zone on layer 1, net N$42
- removed copper zone on layer 1, net PGND
- removed copper zone on layer 1, net PWR_VPACK
Other:
- board size 120 x 120 mm -> 80 x 220 mm
- board text removed: "gswdh.co.uk"
- board text removed: "gswdh.co.uk camera power PCB rev 1.2.2 2024.09.15"
