File: power.sch (EAGLE design)
At the start: 38 parts, among them CN1 21700, CN2 21700, CN3 21700, CN4 21700, CN5 15PIN 0.5MM, Q1 IRLML6244, Q2 IRLML6244, U1 MAX17320G20+

Commit message: New format working on
Parts:
- removed CN1, CN2, CN3, CN4: 21700, CONNECTORs:KEYSTONE1122
- removed MECH1, MECH2, MECH3, MECH4, MECH5, MECH6: 6mm x 3mm, MISC:MOUNTHOLE
Connections:
- net N$36: no longer CN1.V+
- net N$4: no longer CN1.V-, CN2.V+
- net N$5: no longer CN2.V-, CN3.V+
- net PACK_MID: no longer CN3.V-, CN4.V+
- net PGND: no longer CN4.V-
Changed lines of the file:
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@@
 <part name="R7" library="r_0603" deviceset="ERJ3EKF1000V" device="" value="100R"/>
 <part name="F1" library="FUSES" deviceset="SF-1206F100-2" device="" value="1A Fast"/>
-<part name="MECH1" library="MISC" deviceset="MOUNTHOLE" device="" value="6mm x 3mm"/>
-<part name="MECH4" library="MISC" deviceset="MOUNTHOLE" device="" value="6mm x 3mm"/>
-<part name="MECH2" library="MISC" deviceset="MOUNTHOLE" device="" value="6mm x 3mm"/>
-<part name="MECH5" library="MISC" deviceset="MOUNTHOLE" device="" value="6mm x 3mm"/>
-<part name="CN1" library="CONNECTORs" deviceset="KEYSTONE1122" device="" value="21700"/>
-<part name="CN2" library="CONNECTORs" deviceset="KEYSTONE1122" device="" value="21700"/>
-<part name="CN4" library="CONNECTORs" deviceset="KEYSTONE1122" device="" value="21700"/>
 <part name="R4" library="r_0603" deviceset="ERJ3EKF47R0V" device="" value="47R"/>
 <part name="C3" library="CAPACITORS" deviceset="CL10B104KO8WPNC" device="" value="100nF 16V"/>
 <part name="C2" library="CAPACITORS" deviceset="CL10B104KO8WPNC" device="" value="100nF 16V"/>
-<part name="CN3" library="CONNECTORs" deviceset="KEYSTONE1122" device="" value="21700"/>
 <part name="CN5" library="CONNECTORs" deviceset="SFV15R-1STE1HLF" device="" value="15PIN 0.5MM"/>
 <part name="GND4" library="NETS" deviceset="GND" device=""/>
-<part name="MECH3" library="MISC" deviceset="MOUNTHOLE" device="" value="6mm x 3mm"/>
-<part name="MECH6" library="MISC" deviceset="MOUNTHOLE" device="" value="6mm x 3mm"/>
 <part name="U$2" library="NETS" deviceset="PGND" device=""/>
 <part name="R13" library="r_0603" deviceset="ERJ3EKF10R0V" device="" value="10R"/>
@@
 <attribute name="VALUE" x="-48.26" y="73.66" size="1.27" layer="96" rot="R90" align="center"/>
 </instance>
-<instance part="MECH1" gate="G$1" x="-154.94" y="-236.22" smashed="yes">
-<attribute name="NAME" x="-154.94" y="-232.664" size="1.27" layer="95" align="center"/>
-</instance>
-<instance part="MECH4" gate="G$1" x="-147.32" y="-236.22" smashed="yes">
-<attribute name="NAME" x="-147.32" y="-232.664" size="1.27" layer="95" align="center"/>
-</instance>
-<instance part="MECH2" gate="G$1" x="-154.94" y="-243.84" smashed="yes">
-<attribute name="NAME" x="-154.94" y="-240.284" size="1.27" layer="95" align="center"/>
-</instance>
-<instance part="MECH5" gate="G$1" x="-147.32" y="-243.84" smashed="yes">
-<attribute name="NAME" x="-147.32" y="-240.284" size="1.27" layer="95" align="center"/>
-</instance>
-<instance part="CN1" gate="G$1" x="-50.8" y="7.62" smashed="yes">
-<attribute name="NAME" x="-54.61" y="7.62" size="1.778" layer="95" rot="R90" align="center"/>
-<attribute name="VALUE" x="-46.99" y="7.62" size="1.778" layer="96" rot="R90" align="center"/>
-</instance>
-<instance part="CN2" gate="G$1" x="-50.8" y="-7.62" smashed="yes">
-<attribute name="NAME" x="-54.61" y="-7.62" size="1.778" layer="95" rot="R90" align="center"/>
-<attribute name="VALUE" x="-46.99" y="-7.62" size="1.778" layer="96" rot="R90" align="center"/>
-</instance>
-<instance part="CN4" gate="G$1" x="-50.8" y="-38.1" smashed="yes">
-<attribute name="NAME" x="-54.61" y="-38.1" size="1.778" layer="95" rot="R90" align="center"/>
-<attribute name="VALUE" x="-46.99" y="-38.1" size="1.778" layer="96" rot="R90" align="center"/>
-</instance>
 <instance part="R4" gate="G$1" x="-43.18" y="-15.24" smashed="yes">
 <attribute name="NAME" x="-43.18" y="-12.7" size="1.27" layer="95" align="center"/>
@@
 <attribute name="VALUE" x="-33.02" y="-7.62" size="1.27" layer="96" rot="R90" align="center"/>
 </instance>
-<instance part="CN3" gate="G$1" x="-50.8" y="-22.86" smashed="yes">
-<attribute name="NAME" x="-54.61" y="-22.86" size="1.778" layer="95" rot="R90" align="center"/>
-<attribute name="VALUE" x="-46.99" y="-22.86" size="1.778" layer="96" rot="R90" align="center"/>
-</instance>
 <instance part="CN5" gate="G$1" x="91.44" y="22.86" smashed="yes">
 <attribute name="NAME" x="86.36" y="48.26" size="1.778" layer="95"/>
@@
 <instance part="GND4" gate="G$1" x="101.6" y="0" smashed="yes">
 <attribute name="VALUE" x="101.6" y="-2.54" size="1.778" layer="96" align="center"/>
-</instance>
-<instance part="MECH3" gate="G$1" x="-154.94" y="-251.46" smashed="yes">
-<attribute name="NAME" x="-154.94" y="-247.904" size="1.27" layer="95" align="center"/>
-</instance>
-<instance part="MECH6" gate="G$1" x="-147.32" y="-251.46" smashed="yes">
-<attribute name="NAME" x="-147.32" y="-247.904" size="1.27" layer="95" align="center"/>
 </instance>
 <instance part="U$2" gate="G$1" x="43.18" y="17.78" smashed="yes">
@@
 <junction x="-50.8" y="38.1"/>
 <pinref part="F1" gate="G$1" pin="1"/>
-<pinref part="CN1" gate="G$1" pin="V+"/>
 <wire x1="-50.8" y1="12.7" x2="-50.8" y2="15.24" width="0.1524" layer="91"/>
 <junction x="-50.8" y="15.24"/>
@@
 <segment>
 <pinref part="R5" gate="G$1" pin="1"/>
-<pinref part="CN3" gate="G$1" pin="V-"/>
 <wire x1="-48.26" y1="-30.48" x2="-50.8" y2="-30.48" width="0.1524" layer="91"/>
 <wire x1="-50.8" y1="-30.48" x2="-50.8" y2="-27.94" width="0.1524" layer="91"/>
-<pinref part="CN4" gate="G$1" pin="V+"/>
 <wire x1="-50.8" y1="-33.02" x2="-50.8" y2="-30.48" width="0.1524" layer="91"/>
 <junction x="-50.8" y="-30.48"/>
@@
 <segment>
 <pinref part="U$28" gate="G$1" pin="PGND"/>
-<pinref part="CN4" gate="G$1" pin="V-"/>
 <wire x1="-50.8" y1="-45.72" x2="-50.8" y2="-43.18" width="0.1524" layer="91"/>
 </segment>
@@
 <segment>
 <pinref part="R3" gate="G$1" pin="1"/>
-<pinref part="CN1" gate="G$1" pin="V-"/>
 <wire x1="-48.26" y1="0" x2="-50.8" y2="0" width="0.1524" layer="91"/>
 <wire x1="-50.8" y1="0" x2="-50.8" y2="2.54" width="0.1524" layer="91"/>
-<pinref part="CN2" gate="G$1" pin="V+"/>
 <wire x1="-50.8" y1="-2.54" x2="-50.8" y2="0" width="0.1524" layer="91"/>
 <junction x="-50.8" y="0"/>
@@
 <segment>
 <pinref part="R4" gate="G$1" pin="1"/>
-<pinref part="CN2" gate="G$1" pin="V-"/>
 <wire x1="-48.26" y1="-15.24" x2="-50.8" y2="-15.24" width="0.1524" layer="91"/>
 <wire x1="-50.8" y1="-15.24" x2="-50.8" y2="-12.7" width="0.1524" layer="91"/>
-<pinref part="CN3" gate="G$1" pin="V+"/>
 <wire x1="-50.8" y1="-17.78" x2="-50.8" y2="-15.24" width="0.1524" layer="91"/>
 <junction x="-50.8" y="-15.24"/>

Commit message: Progress
Parts:
- added CN1, CN2: 21700, CONNECTORs:KEYSTONE1122
Connections:
- net N$5: now also CN2.V+
- net PACK_MID: now also CN1.V+, CN2.V-
- net PGND: now also CN1.V-
Other:
- note added: "YYYY.MM.DD - GSWDH LTD. CAMERA POWER PCB REVISION 1.x.x DESIGN BY GEORGE WALLER, GSWDH LTD. GEORGEWALLER@GSWDH.CO.UK CONFIDENTIAL. FOR THE INTENDED READER ONLY."
- note removed: "YYYY.MM.DD - GSWDH LTD. CAMERA MAIN PCB REVISION 1.x.x DESIGN BY GEORGE WALLER, GSWDH LTD. GEORGEWALLER@GSWDH.CO.UK CONFIDENTIAL. FOR THE INTENDED READER ONLY."
Changed lines of the file:
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@@
 <part name="U$2" library="NETS" deviceset="PGND" device=""/>
 <part name="R13" library="r_0603" deviceset="ERJ3EKF10R0V" device="" value="10R"/>
+<part name="CN1" library="CONNECTORs" deviceset="KEYSTONE1122" device="" value="21700"/>
+<part name="CN2" library="CONNECTORs" deviceset="KEYSTONE1122" device="" value="21700"/>
 </parts>
 <sheets>
@@
 <plain>
 <text x="0" y="0" size="7.62" layer="97" font="vector" align="center">YYYY.MM.DD - GSWDH LTD.
-CAMERA MAIN PCB
+CAMERA POWER PCB
 REVISION 1.x.x
 DESIGN BY GEORGE WALLER, GSWDH LTD.
@@
 <attribute name="VALUE" x="-5.08" y="-78.74" size="1.27" layer="96" rot="R90" align="center"/>
 </instance>
+<instance part="CN1" gate="G$1" x="-50.8" y="-38.1" smashed="yes">
+<attribute name="NAME" x="-54.61" y="-38.1" size="1.778" layer="95" rot="R90" align="center"/>
+<attribute name="VALUE" x="-46.99" y="-38.1" size="1.778" layer="96" rot="R90" align="center"/>
+</instance>
+<instance part="CN2" gate="G$1" x="-50.8" y="-22.86" smashed="yes">
+<attribute name="NAME" x="-54.61" y="-22.86" size="1.778" layer="95" rot="R90" align="center"/>
+<attribute name="VALUE" x="-46.99" y="-22.86" size="1.778" layer="96" rot="R90" align="center"/>
+</instance>
 </instances>
 <busses>
@@
 <wire x1="-50.8" y1="-33.02" x2="-50.8" y2="-30.48" width="0.1524" layer="91"/>
 <junction x="-50.8" y="-30.48"/>
+<pinref part="CN1" gate="G$1" pin="V+"/>
+<pinref part="CN2" gate="G$1" pin="V-"/>
 </segment>
 </net>
@@
 <pinref part="U$28" gate="G$1" pin="PGND"/>
 <wire x1="-50.8" y1="-45.72" x2="-50.8" y2="-43.18" width="0.1524" layer="91"/>
+<pinref part="CN1" gate="G$1" pin="V-"/>
 </segment>
 <segment>
@@
 <wire x1="-50.8" y1="-17.78" x2="-50.8" y2="-15.24" width="0.1524" layer="91"/>
 <junction x="-50.8" y="-15.24"/>
-</segment>
-</net>
+<pinref part="CN2" gate="G$1" pin="V+"/>
+</segment>
+</net>

Commit message: Progress
Parts:
- removed C1: 100nF 16V, CAPACITORS:CL10B104KO8WPNC
- removed R2: 47R, r_0603:ERJ3EKF47R0V
- added CN3: 21700, CONNECTORs:21700_TAB
- CN1, CN2: device CONNECTORs:KEYSTONE1122 -> CONNECTORs:21700_TAB
- F1: value 1A Fast -> 20A; device FUSES:SF-1206F100-2 -> FUSES:0678H9200-02
- Q1, Q2: value IRLML6244 -> SIRA36DP-T1-GE3; device TRANSISTORs:IRLML6244TRPBF -> TRANSISTORs:SIRA36DP-T1-GE3
Connections:
- removed net N$36: F1.1, R1.1, R2.1
- removed net N$4: R3.1
- net N$2: no longer C1.1
- net N$39: now also CN3.V+, F1.1, R1.1, R3.1; no longer C1.2, R2.2
- net N$5: now also CN3.V-
Other:
- moved on the sheet: CN5
