File: power.sch (EAGLE design)
At the start: 29 parts, among them CN1 21700, CN2 21700, CN3 21700, CN5 15PIN 0.5MM, Q1 SIRA36DP-T1-GE3, Q2 SIRA36DP-T1-GE3, U1 MAX17320G20+

Commit message: Passing DRC
Parts:
- removed C3: 100nF 16V, CAPACITORS:CL10B104KO8WPNC
- added C1: 100nF 16V, CAPACITORS:CL10B104KO8WPNC
- added R2: 47R, r_0603:ERJ3EKF47R0V
Connections:
- removed net N$5: CN2.V+, CN3.V-, R4.1
- new net N$4: CN2.V+, CN3.V-, R3.1
- net N$1: now also C1.2, R2.2, U1.BATTS; no longer C3.1, C4.2, R5.2, U1.CELL1
- net N$2: now also C1.1
- net N$3: now also C4.2, R5.2, U1.CELL1; no longer C3.2
- net N$39: now also R2.1; no longer R3.1, U1.BATTS
- net PACK_MID: now also R4.1
Other:
- moved on the sheet: CN2, CN3, R4, R5

Commit message: Debug and power board ready for outputs
Other:
- note added: "2023.07.25- GSWDH LTD. CAMERA POWER PCB REVISION 1.0.0 DESIGN BY GEORGE WALLER, GSWDH LTD. GEORGEWALLER@GSWDH.CO.UK CONFIDENTIAL. FOR THE INTENDED READER ONLY."
- note removed: "YYYY.MM.DD - GSWDH LTD. CAMERA POWER PCB REVISION 1.x.x DESIGN BY GEORGE WALLER, GSWDH LTD. GEORGEWALLER@GSWDH.CO.UK CONFIDENTIAL. FOR THE INTENDED READER ONLY."
Changed lines of the file:
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@@
 <drawing>
 <settings>
-<setting alwaysvectorfont="no"/>
+<setting alwaysvectorfont="yes"/>
 <setting keepoldvectorfont="yes"/>
 <setting verticaltext="up"/>
@@
 <description>TITLE</description>
 <plain>
-<text x="0" y="0" size="7.62" layer="97" font="vector" align="center">YYYY.MM.DD - GSWDH LTD.
+<text x="0" y="0" size="7.62" layer="97" font="vector" align="center">2023.07.25- GSWDH LTD.
 CAMERA POWER PCB
-REVISION 1.x.x
+REVISION 1.0.0
 DESIGN BY GEORGE WALLER, GSWDH LTD.
 GEORGEWALLER@GSWDH.CO.UK

Commit message: Updated schematic front page on power
Other:
- note added: "2023.09.01- GSWDH LTD. CAMERA POWER PCB REVISION 1.1.0 DESIGN BY GEORGE WALLER, GSWDH LTD. GEORGEWALLER@GSWDH.CO.UK CONFIDENTIAL. FOR THE INTENDED READER ONLY."
- note removed: "2023.07.25- GSWDH LTD. CAMERA POWER PCB REVISION 1.0.0 DESIGN BY GEORGE WALLER, GSWDH LTD. GEORGEWALLER@GSWDH.CO.UK CONFIDENTIAL. FOR THE INTENDED READER ONLY."
Changed lines of the file:
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@@
 <description>TITLE</description>
 <plain>
-<text x="0" y="0" size="7.62" layer="97" font="vector" align="center">2023.07.25- GSWDH LTD.
+<text x="0" y="0" size="7.62" layer="97" font="vector" align="center">2023.09.01- GSWDH LTD.
 CAMERA POWER PCB
-REVISION 1.0.0
+REVISION 1.1.0
 DESIGN BY GEORGE WALLER, GSWDH LTD.
 GEORGEWALLER@GSWDH.CO.UK
