File: power.sch (EAGLE design)
At the start: 30 parts, among them CN1 21700, CN2 21700, CN3 21700, CN5 15PIN 0.5MM, Q1 SIRA36DP-T1-GE3, Q2 SIRA36DP-T1-GE3, U1 MAX17320G20+

Commit message: Added extra decoupling to the PLL PSU
Parts:
- removed F1: 20A, FUSES:0678H9200-02
- CN1, CN2, CN3: device CONNECTORs:21700_TAB -> CONNECTORs:KEYSTONE1122
- renumbered CN5 to CN4
Connections:
- removed net N$39: CN3.V+, F1.1, R1.1, R2.1
- net BMS_BUS_RSVD_2: now also CN4.7; no longer CN4.9
- net BMS_I2C_SCL: now also CN4.11; no longer CN4.5
- net BMS_I2C_SDA: now also CN4.10; no longer CN4.6
- net BMS_NALERT: now also CN4.9; no longer CN4.7
- net GND: now also CN4.1, CN4.2, CN4.3, CN4.4, CN4.5, CN4.6; no longer CN4.10, CN4.11, CN4.12, CN4.13, CN4.14, CN4.15
- net N$42: now also CN3.V+, R1.1, R2.1; no longer F1.2
- net PWR_VPACK: now also CN4.12, CN4.13, CN4.14, CN4.15; no longer CN4.1, CN4.2, CN4.3, CN4.4
Changed lines of the file:
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@@
 <part name="Q1" library="TRANSISTORs" deviceset="SIRA36DP-T1-GE3" device="" value="SIRA36DP-T1-GE3"/>
 <part name="R7" library="r_0603" deviceset="ERJ3EKF1000V" device="" value="100R"/>
-<part name="F1" library="FUSES" deviceset="0678H9200-02" device="" value="20A"/>
 <part name="C2" library="CAPACITORS" deviceset="CL10B104KO8WPNC" device="" value="100nF 16V"/>
-<part name="CN5" library="CONNECTORs" deviceset="SFV15R-1STE1HLF" device="" value="15PIN 0.5MM"/>
 <part name="GND4" library="NETS" deviceset="GND" device=""/>
 <part name="U$2" library="NETS" deviceset="PGND" device=""/>
 <part name="R13" library="r_0603" deviceset="ERJ3EKF10R0V" device="" value="10R"/>
-<part name="CN1" library="CONNECTORs" deviceset="21700_TAB" device="" value="21700"/>
-<part name="CN2" library="CONNECTORs" deviceset="21700_TAB" device="" value="21700"/>
-<part name="CN3" library="CONNECTORs" deviceset="21700_TAB" device="" value="21700"/>
+<part name="CN1" library="CONNECTORs" deviceset="KEYSTONE1122" device="" value="21700"/>
+<part name="CN2" library="CONNECTORs" deviceset="KEYSTONE1122" device="" value="21700"/>
+<part name="CN3" library="CONNECTORs" deviceset="KEYSTONE1122" device="" value="21700"/>
 <part name="R2" library="r_0603" deviceset="ERJ3EKF47R0V" device="" value="47R"/>
 <part name="C1" library="CAPACITORS" deviceset="CL10B104KO8WPNC" device="" value="100nF 16V"/>
 <part name="R4" library="r_0603" deviceset="ERJ3EKF47R0V" device="" value="47R"/>
 <part name="R5" library="r_0603" deviceset="ERJ3EKF47R0V" device="" value="47R"/>
+<part name="CN4" library="CONNECTORs" deviceset="SFV15R-1STE1HLF" device="" value="15PIN 0.5MM"/>
 </parts>
 <sheets>
@@
 <attribute name="VALUE" x="-5.08" y="78.74" size="1.27" layer="96" rot="R90" align="center"/>
 </instance>
-<instance part="F1" gate="G$1" x="-50.8" y="73.66" smashed="yes" rot="R90">
-<attribute name="NAME" x="-53.34" y="73.66" size="1.27" layer="95" rot="R90" align="center"/>
-<attribute name="VALUE" x="-48.26" y="73.66" size="1.27" layer="96" rot="R90" align="center"/>
-</instance>
 <instance part="C2" gate="G$1" x="-35.56" y="-7.62" smashed="yes" rot="R90">
 <attribute name="NAME" x="-38.1" y="-7.62" size="1.27" layer="95" rot="R90" align="center"/>
 <attribute name="VALUE" x="-33.02" y="-7.62" size="1.27" layer="96" rot="R90" align="center"/>
 </instance>
-<instance part="CN5" gate="G$1" x="137.16" y="22.86" smashed="yes" rot="MR0">
-<attribute name="NAME" x="142.24" y="48.26" size="1.778" layer="95" rot="MR0"/>
-<attribute name="VALUE" x="142.24" y="45.72" size="1.778" layer="96" rot="MR0"/>
-</instance>
 <instance part="GND4" gate="G$1" x="127" y="0" smashed="yes" rot="MR0">
 <attribute name="VALUE" x="127" y="-2.54" size="1.778" layer="96" rot="MR0" align="center"/>
@@
 <attribute name="NAME" x="-43.18" y="-12.7" size="1.27" layer="95" align="center"/>
 <attribute name="VALUE" x="-43.18" y="-17.78" size="1.27" layer="96" align="center"/>
+</instance>
+<instance part="CN4" gate="G$1" x="137.16" y="22.86" smashed="yes" rot="R180">
+<attribute name="NAME" x="132.08" y="48.26" size="1.778" layer="95"/>
+<attribute name="VALUE" x="132.08" y="45.72" size="1.778" layer="96"/>
 </instance>
 </instances>
@@
 </segment>
 <segment>
-<pinref part="CN5" gate="G$1" pin="11"/>
 <wire x1="129.54" y1="15.24" x2="127" y2="15.24" width="0.1524" layer="91"/>
 <wire x1="127" y1="15.24" x2="127" y2="12.7" width="0.1524" layer="91"/>
-<pinref part="CN5" gate="G$1" pin="12"/>
 <wire x1="127" y1="12.7" x2="127" y2="10.16" width="0.1524" layer="91"/>
 <wire x1="127" y1="10.16" x2="127" y2="7.62" width="0.1524" layer="91"/>
 <wire x1="127" y1="7.62" x2="127" y2="5.08" width="0.1524" layer="91"/>
 <wire x1="127" y1="5.08" x2="127" y2="2.54" width="0.1524" layer="91"/>
+<junction x="127" y="12.7"/>
 <wire x1="129.54" y1="12.7" x2="127" y2="12.7" width="0.1524" layer="91"/>
-<junction x="127" y="12.7"/>
-<pinref part="CN5" gate="G$1" pin="14"/>
+<junction x="127" y="7.62"/>
 <wire x1="129.54" y1="7.62" x2="127" y2="7.62" width="0.1524" layer="91"/>
-<junction x="127" y="7.62"/>
-<pinref part="CN5" gate="G$1" pin="13"/>
+<junction x="127" y="10.16"/>
 <wire x1="129.54" y1="10.16" x2="127" y2="10.16" width="0.1524" layer="91"/>
-<junction x="127" y="10.16"/>
-<pinref part="CN5" gate="G$1" pin="15"/>
-<wire x1="129.54" y1="5.08" x2="127" y2="5.08" width="0.1524" layer="91"/>
 <junction x="127" y="5.08"/>
 <pinref part="GND4" gate="G$1" pin="GND"/>
-<pinref part="CN5" gate="G$1" pin="10"/>
+<wire x1="129.54" y1="5.08" x2="127" y2="5.08" width="0.1524" layer="91"/>
 <wire x1="129.54" y1="17.78" x2="127" y2="17.78" width="0.1524" layer="91"/>
 <wire x1="127" y1="17.78" x2="127" y2="15.24" width="0.1524" layer="91"/>
 <junction x="127" y="15.24"/>
+<pinref part="CN4" gate="G$1" pin="1"/>
+<pinref part="CN4" gate="G$1" pin="2"/>
+<pinref part="CN4" gate="G$1" pin="3"/>
+<pinref part="CN4" gate="G$1" pin="4"/>
+<pinref part="CN4" gate="G$1" pin="5"/>
+<pinref part="CN4" gate="G$1" pin="6"/>
 </segment>
 </net>
@@
 </segment>
 </net>
-<net name="N$39" class="0">
-<segment>
-<wire x1="-50.8" y1="68.58" x2="-50.8" y2="38.1" width="0.1524" layer="91"/>
-<wire x1="-50.8" y1="38.1" x2="-50.8" y2="15.24" width="0.1524" layer="91"/>
-<pinref part="R1" gate="G$1" pin="1"/>
-<wire x1="-48.26" y1="38.1" x2="-50.8" y2="38.1" width="0.1524" layer="91"/>
-<junction x="-50.8" y="38.1"/>
-<pinref part="F1" gate="G$1" pin="1"/>
-<pinref part="CN3" gate="G$1" pin="V+"/>
-<wire x1="-50.8" y1="12.7" x2="-50.8" y2="15.24" width="0.1524" layer="91"/>
-<junction x="-50.8" y="15.24"/>
-<wire x1="-50.8" y1="15.24" x2="-48.26" y2="15.24" width="0.1524" layer="91"/>
-<pinref part="R2" gate="G$1" pin="1"/>
-</segment>
-</net>
 <net name="PACK_MID" class="0">
 <segment>
@@
 <net name="N$42" class="0">
 <segment>
-<wire x1="-50.8" y1="91.44" x2="-50.8" y2="78.74" width="0.1524" layer="91"/>
 <wire x1="-10.16" y1="91.44" x2="-50.8" y2="91.44" width="0.1524" layer="91"/>
 <pinref part="Q1" gate="G$1" pin="S"/>
-<pinref part="F1" gate="G$1" pin="2"/>
+<wire x1="-50.8" y1="91.44" x2="-50.8" y2="38.1" width="0.1524" layer="91"/>
+<wire x1="-50.8" y1="38.1" x2="-50.8" y2="15.24" width="0.1524" layer="91"/>
+<pinref part="R1" gate="G$1" pin="1"/>
+<wire x1="-48.26" y1="38.1" x2="-50.8" y2="38.1" width="0.1524" layer="91"/>
+<junction x="-50.8" y="38.1"/>
+<pinref part="CN3" gate="G$1" pin="V+"/>
+<wire x1="-50.8" y1="12.7" x2="-50.8" y2="15.24" width="0.1524" layer="91"/>
+<junction x="-50.8" y="15.24"/>
+<wire x1="-50.8" y1="15.24" x2="-48.26" y2="15.24" width="0.1524" layer="91"/>
+<pinref part="R2" gate="G$1" pin="1"/>
 </segment>
 </net>
@@
 </segment>
 <segment>
-<pinref part="CN5" gate="G$1" pin="5"/>
+<label x="124.46" y="30.48" size="1.778" layer="95" rot="MR0"/>
+<pinref part="CN4" gate="G$1" pin="11"/>
 <wire x1="129.54" y1="30.48" x2="93.98" y2="30.48" width="0.1524" layer="91"/>
-<label x="124.46" y="30.48" size="1.778" layer="95" rot="MR0"/>
 </segment>
 </net>
@@
 </segment>
 <segment>
-<pinref part="CN5" gate="G$1" pin="6"/>
+<label x="124.46" y="27.94" size="1.778" layer="95" rot="MR0"/>
+<pinref part="CN4" gate="G$1" pin="10"/>
 <wire x1="129.54" y1="27.94" x2="93.98" y2="27.94" width="0.1524" layer="91"/>
-<label x="124.46" y="27.94" size="1.778" layer="95" rot="MR0"/>
 </segment>
 </net>
@@
 <net name="PWR_VPACK" class="0">
 <segment>
-<pinref part="CN5" gate="G$1" pin="2"/>
 <wire x1="129.54" y1="38.1" x2="127" y2="38.1" width="0.1524" layer="91"/>
-<pinref part="CN5" gate="G$1" pin="1"/>
 <wire x1="129.54" y1="40.64" x2="127" y2="40.64" width="0.1524" layer="91"/>
 <wire x1="127" y1="40.64" x2="93.98" y2="40.64" width="0.1524" layer="91"/>
 <wire x1="127" y1="38.1" x2="127" y2="40.64" width="0.1524" layer="91"/>
 <junction x="127" y="40.64"/>
-<pinref part="CN5" gate="G$1" pin="3"/>
 <wire x1="129.54" y1="35.56" x2="127" y2="35.56" width="0.1524" layer="91"/>
 <wire x1="127" y1="35.56" x2="127" y2="38.1" width="0.1524" layer="91"/>
 <junction x="127" y="38.1"/>
-<pinref part="CN5" gate="G$1" pin="4"/>
 <wire x1="129.54" y1="33.02" x2="127" y2="33.02" width="0.1524" layer="91"/>
 <wire x1="127" y1="33.02" x2="127" y2="35.56" width="0.1524" layer="91"/>
 <junction x="127" y="35.56"/>
 <label x="124.46" y="40.64" size="1.778" layer="95" rot="MR0"/>
+<pinref part="CN4" gate="G$1" pin="12"/>
+<pinref part="CN4" gate="G$1" pin="13"/>
+<pinref part="CN4" gate="G$1" pin="14"/>
+<pinref part="CN4" gate="G$1" pin="15"/>
 </segment>
 <segment>
@@
 <net name="BMS_NALERT" class="0">
 <segment>
-<pinref part="CN5" gate="G$1" pin="7"/>
+<label x="124.46" y="25.4" size="1.778" layer="95" rot="MR0"/>
+<pinref part="CN4" gate="G$1" pin="9"/>
 <wire x1="129.54" y1="25.4" x2="93.98" y2="25.4" width="0.1524" layer="91"/>
-<label x="124.46" y="25.4" size="1.778" layer="95" rot="MR0"/>
 </segment>
 <segment>
@@
 <net name="BMS_BUS_RSVD_1" class="0">
 <segment>
-<pinref part="CN5" gate="G$1" pin="8"/>
+<label x="124.46" y="22.86" size="1.778" layer="95" rot="MR0"/>
+<pinref part="CN4" gate="G$1" pin="8"/>
 <wire x1="129.54" y1="22.86" x2="93.98" y2="22.86" width="0.1524" layer="91"/>
-<label x="124.46" y="22.86" size="1.778" layer="95" rot="MR0"/>
 </segment>
 </net>
 <net name="BMS_BUS_RSVD_2" class="0">
 <segment>
-<pinref part="CN5" gate="G$1" pin="9"/>
+<label x="124.46" y="20.32" size="1.778" layer="95" rot="MR0"/>
+<pinref part="CN4" gate="G$1" pin="7"/>
 <wire x1="129.54" y1="20.32" x2="93.98" y2="20.32" width="0.1524" layer="91"/>
-<label x="124.46" y="20.32" size="1.778" layer="95" rot="MR0"/>
-</segment>
-</net>
+</segment>
+</net>

Commit message: Power PCB connector now in correct orientation
Connections:
- net BMS_BUS_RSVD_2: now also CN4.9; no longer CN4.7
- net BMS_I2C_SCL: now also CN4.5; no longer CN4.11
- net BMS_I2C_SDA: now also CN4.6; no longer CN4.10
- net BMS_NALERT: now also CN4.7; no longer CN4.9
- net GND: now also CN4.10, CN4.11, CN4.12, CN4.13, CN4.14, CN4.15; no longer CN4.1, CN4.2, CN4.3, CN4.4, CN4.5, CN4.6
- net PWR_VPACK: now also CN4.1, CN4.2, CN4.3, CN4.4; no longer CN4.12, CN4.13, CN4.14, CN4.15
Other:
- moved on the sheet: CN4
Changed lines of the file:
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@@
 <attribute name="VALUE" x="-43.18" y="-17.78" size="1.27" layer="96" align="center"/>
 </instance>
-<instance part="CN4" gate="G$1" x="137.16" y="22.86" smashed="yes" rot="R180">
-<attribute name="NAME" x="132.08" y="48.26" size="1.778" layer="95"/>
-<attribute name="VALUE" x="132.08" y="45.72" size="1.778" layer="96"/>
+<instance part="CN4" gate="G$1" x="137.16" y="22.86" smashed="yes" rot="MR0">
+<attribute name="NAME" x="132.08" y="-2.54" size="1.778" layer="95" rot="MR180"/>
+<attribute name="VALUE" x="132.08" y="0" size="1.778" layer="96" rot="MR180"/>
 </instance>
 </instances>
@@
 <wire x1="127" y1="17.78" x2="127" y2="15.24" width="0.1524" layer="91"/>
 <junction x="127" y="15.24"/>
-<pinref part="CN4" gate="G$1" pin="1"/>
-<pinref part="CN4" gate="G$1" pin="2"/>
-<pinref part="CN4" gate="G$1" pin="3"/>
-<pinref part="CN4" gate="G$1" pin="4"/>
-<pinref part="CN4" gate="G$1" pin="5"/>
-<pinref part="CN4" gate="G$1" pin="6"/>
+<pinref part="CN4" gate="G$1" pin="10"/>
+<pinref part="CN4" gate="G$1" pin="11"/>
+<pinref part="CN4" gate="G$1" pin="12"/>
+<pinref part="CN4" gate="G$1" pin="13"/>
+<pinref part="CN4" gate="G$1" pin="14"/>
+<pinref part="CN4" gate="G$1" pin="15"/>
 </segment>
 </net>
@@
 <segment>
 <label x="124.46" y="30.48" size="1.778" layer="95" rot="MR0"/>
-<pinref part="CN4" gate="G$1" pin="11"/>
 <wire x1="129.54" y1="30.48" x2="93.98" y2="30.48" width="0.1524" layer="91"/>
+<pinref part="CN4" gate="G$1" pin="5"/>
 </segment>
 </net>
@@
 <segment>
 <label x="124.46" y="27.94" size="1.778" layer="95" rot="MR0"/>
-<pinref part="CN4" gate="G$1" pin="10"/>
 <wire x1="129.54" y1="27.94" x2="93.98" y2="27.94" width="0.1524" layer="91"/>
+<pinref part="CN4" gate="G$1" pin="6"/>
 </segment>
 </net>
@@
 <junction x="127" y="35.56"/>
 <label x="124.46" y="40.64" size="1.778" layer="95" rot="MR0"/>
-<pinref part="CN4" gate="G$1" pin="12"/>
-<pinref part="CN4" gate="G$1" pin="13"/>
-<pinref part="CN4" gate="G$1" pin="14"/>
-<pinref part="CN4" gate="G$1" pin="15"/>
+<pinref part="CN4" gate="G$1" pin="1"/>
+<pinref part="CN4" gate="G$1" pin="2"/>
+<pinref part="CN4" gate="G$1" pin="3"/>
+<pinref part="CN4" gate="G$1" pin="4"/>
 </segment>
 <segment>
@@
 <segment>
 <label x="124.46" y="25.4" size="1.778" layer="95" rot="MR0"/>
-<pinref part="CN4" gate="G$1" pin="9"/>
 <wire x1="129.54" y1="25.4" x2="93.98" y2="25.4" width="0.1524" layer="91"/>
+<pinref part="CN4" gate="G$1" pin="7"/>
 </segment>
 <segment>
@@
 <segment>
 <label x="124.46" y="22.86" size="1.778" layer="95" rot="MR0"/>
+<wire x1="129.54" y1="22.86" x2="93.98" y2="22.86" width="0.1524" layer="91"/>
 <pinref part="CN4" gate="G$1" pin="8"/>
-<wire x1="129.54" y1="22.86" x2="93.98" y2="22.86" width="0.1524" layer="91"/>
 </segment>
 </net>
@@
 <segment>
 <label x="124.46" y="20.32" size="1.778" layer="95" rot="MR0"/>
-<pinref part="CN4" gate="G$1" pin="7"/>
 <wire x1="129.54" y1="20.32" x2="93.98" y2="20.32" width="0.1524" layer="91"/>
-</segment>
-</net>
+<pinref part="CN4" gate="G$1" pin="9"/>
+</segment>
+</net>

Commit message: Power PCB updated
Parts:
- renumbered CN4 to CN5
Connections:
- net BMS_BUS_RSVD_2: now also CN5.7; no longer CN5.9
- net BMS_I2C_SCL: now also CN5.11; no longer CN5.5
- net BMS_I2C_SDA: now also CN5.10; no longer CN5.6
- net BMS_NALERT: now also CN5.9; no longer CN5.7
- net GND: now also CN5.1, CN5.2, CN5.3, CN5.4, CN5.5, CN5.6; no longer CN5.10, CN5.11, CN5.12, CN5.13, CN5.14, CN5.15
- net PWR_VPACK: now also CN5.12, CN5.13, CN5.14, CN5.15; no longer CN5.1, CN5.2, CN5.3, CN5.4
Other:
- note added: "2023.10.24- GSWDH LTD. CAMERA POWER PCB REVISION 1.2.0 DESIGN BY GEORGE WALLER, GSWDH LTD. GEORGEWALLER@GSWDH.CO.UK CONFIDENTIAL. FOR THE INTENDED READER ONLY."
- note removed: "2023.09.01- GSWDH LTD. CAMERA POWER PCB REVISION 1.1.0 DESIGN BY GEORGE WALLER, GSWDH LTD. GEORGEWALLER@GSWDH.CO.UK CONFIDENTIAL. FOR THE INTENDED READER ONLY."
Changed lines of the file:
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@@
 <part name="R4" library="r_0603" deviceset="ERJ3EKF47R0V" device="" value="47R"/>
 <part name="R5" library="r_0603" deviceset="ERJ3EKF47R0V" device="" value="47R"/>
-<part name="CN4" library="CONNECTORs" deviceset="SFV15R-1STE1HLF" device="" value="15PIN 0.5MM"/>
+<part name="CN5" library="CONNECTORs" deviceset="SFV15R-1STE1HLF" device="" value="15PIN 0.5MM"/>
 </parts>
 <sheets>
@@
 <description>TITLE</description>
 <plain>
-<text x="0" y="0" size="7.62" layer="97" font="vector" align="center">2023.09.01- GSWDH LTD.
+<text x="0" y="0" size="7.62" layer="97" font="vector" align="center">2023.10.24- GSWDH LTD.
 CAMERA POWER PCB
-REVISION 1.1.0
+REVISION 1.2.0
 DESIGN BY GEORGE WALLER, GSWDH LTD.
 GEORGEWALLER@GSWDH.CO.UK
@@
 <attribute name="VALUE" x="-43.18" y="-17.78" size="1.27" layer="96" align="center"/>
 </instance>
-<instance part="CN4" gate="G$1" x="137.16" y="22.86" smashed="yes" rot="MR0">
-<attribute name="NAME" x="132.08" y="-2.54" size="1.778" layer="95" rot="MR180"/>
-<attribute name="VALUE" x="132.08" y="0" size="1.778" layer="96" rot="MR180"/>
+<instance part="CN5" gate="G$1" x="137.16" y="22.86" smashed="yes" rot="R180">
+<attribute name="NAME" x="132.08" y="48.26" size="1.778" layer="95"/>
+<attribute name="VALUE" x="132.08" y="45.72" size="1.778" layer="96"/>
 </instance>
 </instances>
@@
 <wire x1="127" y1="5.08" x2="127" y2="2.54" width="0.1524" layer="91"/>
 <junction x="127" y="12.7"/>
+<junction x="127" y="7.62"/>
 <wire x1="129.54" y1="12.7" x2="127" y2="12.7" width="0.1524" layer="91"/>
-<junction x="127" y="7.62"/>
+<junction x="127" y="10.16"/>
 <wire x1="129.54" y1="7.62" x2="127" y2="7.62" width="0.1524" layer="91"/>
-<junction x="127" y="10.16"/>
-<wire x1="129.54" y1="10.16" x2="127" y2="10.16" width="0.1524" layer="91"/>
 <junction x="127" y="5.08"/>
 <pinref part="GND4" gate="G$1" pin="GND"/>
+<wire x1="129.54" y1="10.16" x2="127" y2="10.16" width="0.1524" layer="91"/>
 <wire x1="129.54" y1="5.08" x2="127" y2="5.08" width="0.1524" layer="91"/>
 <wire x1="129.54" y1="17.78" x2="127" y2="17.78" width="0.1524" layer="91"/>
 <wire x1="127" y1="17.78" x2="127" y2="15.24" width="0.1524" layer="91"/>
 <junction x="127" y="15.24"/>
-<pinref part="CN4" gate="G$1" pin="10"/>
-<pinref part="CN4" gate="G$1" pin="11"/>
-<pinref part="CN4" gate="G$1" pin="12"/>
-<pinref part="CN4" gate="G$1" pin="13"/>
-<pinref part="CN4" gate="G$1" pin="14"/>
-<pinref part="CN4" gate="G$1" pin="15"/>
+<pinref part="CN5" gate="G$1" pin="1"/>
+<pinref part="CN5" gate="G$1" pin="2"/>
+<pinref part="CN5" gate="G$1" pin="3"/>
+<pinref part="CN5" gate="G$1" pin="4"/>
+<pinref part="CN5" gate="G$1" pin="5"/>
+<pinref part="CN5" gate="G$1" pin="6"/>
 </segment>
 </net>
@@
 <segment>
 <label x="124.46" y="30.48" size="1.778" layer="95" rot="MR0"/>
+<pinref part="CN5" gate="G$1" pin="11"/>
 <wire x1="129.54" y1="30.48" x2="93.98" y2="30.48" width="0.1524" layer="91"/>
-<pinref part="CN4" gate="G$1" pin="5"/>
 </segment>
 </net>
@@
 <segment>
 <label x="124.46" y="27.94" size="1.778" layer="95" rot="MR0"/>
+<pinref part="CN5" gate="G$1" pin="10"/>
 <wire x1="129.54" y1="27.94" x2="93.98" y2="27.94" width="0.1524" layer="91"/>
-<pinref part="CN4" gate="G$1" pin="6"/>
 </segment>
 </net>
@@
 <junction x="127" y="35.56"/>
 <label x="124.46" y="40.64" size="1.778" layer="95" rot="MR0"/>
-<pinref part="CN4" gate="G$1" pin="1"/>
-<pinref part="CN4" gate="G$1" pin="2"/>
-<pinref part="CN4" gate="G$1" pin="3"/>
-<pinref part="CN4" gate="G$1" pin="4"/>
+<pinref part="CN5" gate="G$1" pin="12"/>
+<pinref part="CN5" gate="G$1" pin="13"/>
+<pinref part="CN5" gate="G$1" pin="14"/>
+<pinref part="CN5" gate="G$1" pin="15"/>
 </segment>
 <segment>
@@
 <segment>
 <label x="124.46" y="25.4" size="1.778" layer="95" rot="MR0"/>
+<pinref part="CN5" gate="G$1" pin="9"/>
 <wire x1="129.54" y1="25.4" x2="93.98" y2="25.4" width="0.1524" layer="91"/>
-<pinref part="CN4" gate="G$1" pin="7"/>
 </segment>
 <segment>
@@
 <segment>
 <label x="124.46" y="22.86" size="1.778" layer="95" rot="MR0"/>
+<pinref part="CN5" gate="G$1" pin="8"/>
 <wire x1="129.54" y1="22.86" x2="93.98" y2="22.86" width="0.1524" layer="91"/>
-<pinref part="CN4" gate="G$1" pin="8"/>
 </segment>
 </net>
@@
 <segment>
 <label x="124.46" y="20.32" size="1.778" layer="95" rot="MR0"/>
+<pinref part="CN5" gate="G$1" pin="7"/>
 <wire x1="129.54" y1="20.32" x2="93.98" y2="20.32" width="0.1524" layer="91"/>
-<pinref part="CN4" gate="G$1" pin="9"/>
-</segment>
-</net>
+</segment>
+</net>

Commit message: Power PCB updated and ready for manufacture
Parts:
- added C11, C3: 0.1uF 16V, c_0402:0402YD104KAT2A
- added C12: 2.2uF 6.3V, c_0603:06036D225KAT2A
- added C13: 1uF 25V, c_0603:06033C105KAT2A
- added D1: VDMR10A1, OPTO:VDMR10A1
- added Q10, Q3, Q4, Q5, Q6, Q7, Q8, Q9: BSS123, TRANSISTORs:BSS123
- added R14, R15, R16, R17, R18, R19, R20, R21: 1k, r_0402:RC0402FR-071KL
- added R22, R23, R24, R25, R26, R27, R28, R29, R30, R31: 10k, r_0402:RC0402FR-1010KL
- added TP1, TP2, TP3, TP4: TEST_POINT_SQUARE, MISC:TEST_POINT_SQUARE
- added U2: TCA6408AQPWRQ1, ICs:TCA6408AQ
- added U3: TPS70918, ICs:TPS70918DBVT
Connections:
- removed net BMS_BUS_RSVD_1: CN5.8
- removed net BMS_BUS_RSVD_2: CN5.7
- new net N$10: D1.DP, R18.1
- new net N$11: D1.G, R19.1
- new net N$12: D1.F, R20.1
- new net N$13: D1.E, R21.1
- new net N$18: Q3.D, R14.1
- new net N$19: Q4.D, R15.1
- new net N$20: Q5.D, R16.1
- new net N$21: Q6.D, R17.1
- new net N$26: Q7.D, R21.2
- new net N$27: Q8.D, R20.2
- new net N$28: Q9.D, R19.2
- new net N$29: Q10.D, R18.2
- new net N$44: R30.1, U2.!INT
- new net N$5: D1.A, R14.2
- new net N$50: R31.1, U2.!RESET
- new net N$7: D1.B, R15.2
- new net N$8: D1.C, R16.2
- new net N$9: D1.D, R17.2
- new net PWR_BMS_1V8: C11.2, C12.2, C3.2, R30.2, R31.2, TP1.P$1, U2.VCCI, U2.VCCP, U3.VOUT
- new net SVNSEG_A: Q3.G, R22.2, U2.P2
- new net SVNSEG_B: Q4.G, R23.2, U2.P3
- new net SVNSEG_C: Q5.G, R24.2, U2.P6
- new net SVNSEG_D: Q6.G, R25.2, U2.P5
- new net SVNSEG_DP: Q10.G, R29.2, U2.P7
- new net SVNSEG_E: Q7.G, R26.2, U2.P4
- new net SVNSEG_F: Q8.G, R27.2, U2.P1
- new net SVNSEG_G: Q9.G, R28.2, U2.P0
- net BMS_I2C_SCL: now also TP2.P$1, U2.SCL
- net BMS_I2C_SDA: now also TP3.P$1, U2.SDA
- net GND: now also C11.1, C12.1, C13.1, C3.1, Q10.S, Q3.S, Q4.S, Q5.S, Q6.S, Q7.S, Q8.S, Q9.S, R22.1, R23.1, R24.1, R25.1, R26.1, R27.1, R28.1, R29.1, TP4.P$1, U2.ADDR, U2.GND, U3.GND
- net PWR_VPACK: now also C13.2, D1.VCC, U3.EN, U3.VIN
Other:
- note added: "2024.09.15- GSWDH LTD. CAMERA POWER PCB REVISION 1.2.1 DESIGN BY GEORGE WALLER, GSWDH LTD. GEORGEWALLER@GSWDH.CO.UK CONFIDENTIAL. FOR THE INTENDED READER ONLY."
- note removed: "2023.10.24- GSWDH LTD. CAMERA POWER PCB REVISION 1.2.0 DESIGN BY GEORGE WALLER, GSWDH LTD. GEORGEWALLER@GSWDH.CO.UK CONFIDENTIAL. FOR THE INTENDED READER ONLY."
- moved on the sheet: C1, C10, C2, C4, C5, C6, C7, C8, C9, CN1, CN2, CN3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

Commit message: Added I2C test points
Parts:
- Q10, Q3, Q4, Q5, Q6, Q7, Q8, Q9: value BSS123 -> DMN2005K-7; device TRANSISTORs:BSS123 -> TRANSISTORs:DMN2005K-7
Other:
- moved on the sheet: D1, Q10, Q3, Q4, Q5, Q6, Q7, Q8, Q9, R14, R15, R16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
