File: main.brd (EAGLE design)
At the start: 120 x 120 mm, 514 parts, among them CN1 50 PIN 0.5MM, CN2 10067847-001RLF, CN3 632723300011, CN4 FF0881SA1, CN5 15PIN 0.5MM, CN6 31 PIN FPC, Q1 2N7002, Q2 FDN302P, Q3 2N7002, Q5 SI7489DP, SW2 TACT, SW3 TACT, SW4 TACT, SW5 TACT, SW7 TACT, SW8 SLIDE SPDT, U1 GMAX0505-DV, U10 TPS70950, U11 FT601Q, U12 CBTU02043, U13 MAX25300B, U14 ESP32, U15 MAX25300B, U16 INA180, U17 AP62301, U18 AP62301, U19 SCHMITT, U2 XC7Z014S-1CLG484C, U20 MAX25300B, U21 NOT, U22 MAX25300B, U23 SN74LVC1G3, U24 NAND, U25 EMC1812T, U26 BIPOLAR HALL, U27 LM2663, U28 ADS7867, U29 LM2663, U3 IS43TR16128CL-125KBLI, U30 LM2731X, U31 USBLC6-2SC6, U32 MAX1735, U33 MP2148, U34 TPS22917, U35 AP62301, U36 TLV61046A, U37 W25Q128JV, U38 TPS70918, U39 AP62301, U4 AP63300WU-7, U5 STM32L431RBT, U6 USB ESD, U7 ACT2861QI301-T, U8 TPS70918, U9 STUSB4500

Commit message: DRC passes. Need to length match and review
Parts:
- moved R13 4.81 mm to (6.40, -40.5), flipped to the top, turned to 180 degrees
- moved TP97 2.56 mm to (28.4, 41.5)
- moved R3 0.10 mm to (2.40, -40.2)
Routing:
- net PWR_SYS_3V3: track 124.2 -> 153.7 mm
- net PSS_FLASH_D2: track 17.6 -> 34.3 mm, vias 2 -> 3
- net PSS_FLASH_D1: track 20.5 -> 32.9 mm, vias 2 -> 3
- net PSS_FLASH_SCLK: track 16.7 -> 29.0 mm
- net PSS_FLASH_D0: track 15.8 -> 26.6 mm, vias 0 -> 2
- net N$5: track 0.00 -> 6.51 mm
- net PSS_FLASH_D3: track 12.0 -> 18.4 mm
- net GND: track 511.7 -> 517.4 mm, vias 520 -> 523
- net PSS_SD_CD: track 53.9 -> 55.8 mm
- net EVF_MIPI_A_D0_N: track 66.5 -> 68.1 mm
- net EVF_MIPI_A_D0_P: track 65.9 -> 67.4 mm
- net N$70: track 17.0 -> 18.4 mm
- net PWR_DDR3_1V35: track 38.3 -> 37.1 mm
- net N$69: track 0.00 -> 1.25 mm
- net N$68: track 0.00 -> 1.25 mm
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
Commit message: Decoupling added to FPGA
Parts:
- added C100, C104, C120, C122, C123, C124, C125, C126, C127, C128, C129, C130, C131, C132, C133, C138, C139, C140, C141, C142, C143, C144, C156, C170, C184, C186, C196, C198, C200, C258, C259, C260, C261, C262, C81, C82, C85: 0.1uF 10V, c_0402:0402
- added C101, C110, C121, C83, C84, C86: 47uF 6.3V, c_0603:0603
- added C105: 2.2uF 10V, c_0402:0402
Connections:
- net DDR_D0: now also U2.E3; no longer U2.E1
- net DDR_D12: now also U2.D3; no longer U2.E3
- net DDR_D2: now also U2.G1; no longer U2.G2
- net DDR_D8: now also U2.G2; no longer U2.G1
- net DDR_D9: now also U2.E1; no longer U2.D3
- net FT_D10: now also U2.V10; no longer U2.W10
- net FT_D6: now also U2.U12; no longer U2.V12
- net FT_D7: now also U2.V12; no longer U2.U12
- net FT_GPIO1: now also U2.W10; no longer U2.V10
- net FT_NRD: now also U2.W7; no longer U2.V7
- net FT_NWR: now also U2.V7; no longer U2.W7
- net GND: now also C100.1, C101.1, C104.1, C105.1, C110.1, C120.1, C121.1, C122.1, C123.1, C124.1, C125.1, C126.1, C127.1, C128.1, C129.1, C130.1, C131.1, C132.1, C133.1, C138.1, C139.1, C140.1, C141.1, C142.1, C143.1, C144.1, C156.1, C170.1, C184.1, C186.1, C196.1, C198.1, C200.1, C258.1, C259.1, C260.1, C261.1, C262.1, C81.1, C82.1, C83.1, C84.1, C85.1, C86.1
- net PWR_ANA_1V8: now also C104.2, C105.2
- net PWR_DDR3_1V35: now also C156.2, C170.2, C184.2, C186.2, C196.2, C198.2, C200.2
- net PWR_FPGA_1V0: now also C100.2, C101.2, C81.2, C82.2, C83.2, C84.2, C85.2, C86.2
- net PWR_SYS_1V8: now also C110.2, C120.2, C121.2, C122.2, C123.2, C124.2, C125.2, C126.2, C127.2, C128.2, C129.2, C130.2, C131.2, C132.2, C133.2
- net PWR_SYS_3V3: now also C138.2, C139.2, C140.2, C141.2, C142.2, C143.2, C144.2, C258.2, C259.2, C260.2, C261.2, C262.2
Routing:
- net GND: track 517.4 -> 560.0 mm, vias 523 -> 524
- net PWR_SYS_1V8: track 76.2 -> 89.8 mm, vias 38 -> 35
- net PWR_SYS_3V3: track 153.7 -> 165.5 mm
- net PWR_FPGA_1V0: track 25.4 -> 31.8 mm, vias 17 -> 15
- net PWR_DDR3_1V35: track 37.1 -> 42.1 mm
- net DDR_D9: track 17.2 -> 14.1 mm
- net DDR_D0: track 15.4 -> 17.7 mm
- net FT_D10: track 17.2 -> 19.0 mm
- net FT_NRD: track 24.1 -> 22.6 mm
- net FT_D7: track 22.4 -> 21.0 mm
- net PWR_ANA_1V8: track 17.2 -> 18.6 mm
- net DDR_D8: track 9.19 -> 10.5 mm
- net FPGA_JTAG_TDO: track 77.1 -> 78.4 mm
- net FPGA_JTAG_TDI: track 79.8 -> 81.0 mm
- net BTN_BTMLEFT: track 46.1 -> 44.9 mm
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
Commit message: Decoupling added to DDR3
Parts:
- added C263, C273, C275, C277: 0.1uF 10V, c_0402:0402
- added C272, C274, C276, C278: 2.2uF 10V, c_0402:0402
Connections:
- net GND: now also C263.1, C272.1, C273.1, C274.1, C275.1, C276.1, C277.1, C278.1
- net PWR_DDR3_1V35: now also C263.2, C272.2, C273.2, C274.2, C275.2, C276.2, C277.2, C278.2
Routing:
- net PWR_DDR3_1V35: track 42.1 -> 48.1 mm
- net GND: track 560.0 -> 565.7 mm
- net DDR_NRST: track 27.6 -> 30.4 mm

Commit message: DDR3 length matched
Parts:
- moved R13 2.77 mm to (4.30, -42.3)
- moved R3 1.14 mm to (2.10, -41.3)
Routing:
- net DDR_D14: track 8.30 -> 25.1 mm
- net DDR_D1: track 9.02 -> 25.0 mm
- net DDR_D10: track 9.47 -> 24.7 mm
- net DDR_D7: track 10.1 -> 25.0 mm
- net DDR_D8: track 10.7 -> 25.0 mm
- net DDR_D3: track 10.7 -> 25.0 mm
- net DDR_CKE: track 11.4 -> 25.0 mm
- net DDR_D5: track 11.4 -> 24.9 mm
- net DDR_D12: track 12.4 -> 25.1 mm
- net DDR_DQS1_P: track 11.9 -> 24.5 mm
- net DDR_D4: track 13.4 -> 25.0 mm
- net DDR_DQS1_N: track 12.6 -> 24.2 mm
- net DDR_DM0: track 13.6 -> 25.1 mm
- net DDR_D9: track 14.1 -> 25.0 mm
- net DDR_D2: track 14.6 -> 25.0 mm
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
Commit message: GMAX length matched
Parts:
- moved SW2 1.75 mm to (36.0, -36.2)
- moved SW3 1.75 mm to (-36.0, -21.2)
- moved SW4 1.75 mm to (36.0, -21.2)
- moved SW5 1.75 mm to (-36.0, -36.2)
Routing:
- net PSS_SD_D0: track 52.9 -> 75.0 mm
- net SEN_B_D0_P: track 15.8 -> 35.3 mm
- net SEN_B_D0_N: track 15.8 -> 35.3 mm
- net PSS_SD_D1: track 58.2 -> 74.9 mm
- net SEN_CLK_P: track 18.7 -> 35.0 mm
- net SEN_CLK_N: track 18.7 -> 35.0 mm
- net SEN_B_D6_P: track 19.3 -> 35.1 mm
- net SEN_B_D6_N: track 19.3 -> 34.4 mm
- net SEN_B_D18_P: track 21.0 -> 35.0 mm
- net SEN_B_D18_N: track 21.0 -> 35.0 mm
- net SEN_B_D3_N: track 21.5 -> 34.9 mm
- net SEN_B_D3_P: track 21.5 -> 34.9 mm
- net SEN_B_D21_N: track 21.5 -> 34.7 mm
- net SEN_B_D21_P: track 21.8 -> 35.0 mm
- net SEN_B_D9_N: track 22.4 -> 35.0 mm
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
Commit message: EVF Length Matched
Routing:
- net EVF_MIPI_A_D3_P: track 65.4 -> 81.6 mm
- net EVF_MIPI_A_D3_N: track 65.7 -> 81.9 mm
- net EVF_MIPI_B_D3_P: track 66.7 -> 80.6 mm
- net EVF_MIPI_B_D3_N: track 68.0 -> 81.9 mm
- net EVF_MIPI_A_D0_P: track 67.4 -> 81.2 mm
- net EVF_MIPI_A_D0_N: track 68.1 -> 81.9 mm
- net EVF_MIPI_A_D2_N: track 69.3 -> 81.8 mm
- net EVF_MIPI_A_D2_P: track 69.4 -> 81.9 mm
- net EVF_MIPI_A_D1_P: track 71.0 -> 81.4 mm
- net EVF_MIPI_A_D1_N: track 71.5 -> 82.0 mm
- net MIPI_DSI_B_HS_L0_N: track 7.73 -> 18.0 mm
- net MIPI_DSI_B_HS_L0_P: track 7.73 -> 18.0 mm
- net MIPI_DSI_A_HS_L1_N: track 7.98 -> 17.7 mm
- net MIPI_DSI_A_HS_L1_P: track 8.32 -> 18.0 mm
- net EVF_MIPI_A_CLK_P: track 72.7 -> 81.9 mm
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
Commit message: Some pullups added
Parts:
- added D15: BAT54S, DIODES:SOT23-3
- added R103: 10k, r_0402:0402
- added R105, R178, R179, R180, R181, R182: 2.2k, r_0402:0402
- C154: value 1uF 25V -> 1uF 6.3V; device CAPACITORS:0603 -> c_0402:0402
- R85: value 26.7k -> 28k; device r_0603:0603 -> r_0402:0402
- R86: device r_0603:0603 -> r_0402:0402
- moved C154 0.80 mm to (31.8, 38.4)
- moved R86 0.40 mm to (31.8, 37.5)
Connections:
- removed net N$134: U5.34
- net ACT_I2C_SCL: now also R179.1
- net ACT_I2C_SDA: now also R180.1
- net BMS_I2C_SCL: now also R105.1
- net BMS_I2C_SDA: now also R178.1
- net GND: now also D15.1, R103.1
- net MON_SYS_BUS_V: now also D15.2
- net PSS_I2C_SCL: now also R182.1
- net PSS_I2C_SDA: now also R181.1
- net PWR_SYS_1V8: now also R181.2, R182.2
- net PWR_SYS_1V8_SLP: now also D15.3, R105.2, R178.2, R179.2, R180.2
- net STUSB_RESET: now also R103.2
Routing:
- net PWR_SYS_1V8_SLP: track 315.4 -> 319.2 mm, vias 17 -> 22
- net MON_SYS_BUS_V: track 10.9 -> 13.7 mm
- net PWR_VBAT_EN: track 12.7 -> 15.4 mm
- net PWR_SYS_1V8: track 88.8 -> 90.4 mm, vias 35 -> 37
- net PMC_NRESET: track 178.0 -> 176.8 mm
- net GND: track 570.3 -> 571.3 mm, vias 524 -> 526
- net ACT_I2C_SCL: track 23.5 -> 24.5 mm
- net PSS_I2C_SDA: track 29.9 -> 30.8 mm
- net PSS_I2C_SCL: track 17.9 -> 18.5 mm
Other:
- board text added: "gswdh.co.uk camera - soke main PCB rev 1.0.0 2023.07.18"
- board text removed: "gswdh.co.uk camera - muleshoe main PCB rev 1.0.0 2023.06.20"

Commit message: Clock for FTDI fixed and SD status pins moved
Parts:
- added R183, R184, R185, R186: 10k, r_0402:0402
Connections:
- new net N$19: U2.M20
- new net N$31: U2.M19
- net BTN_BTMLEFT: now also R183.1
- net BTN_BTMRIGHT: now also R186.1
- net BTN_TOPLEFT: now also R185.1
- net BTN_TOPRIGHT: now also R184.1
- net FT_CLK: now also U2.AA9; no longer U2.AB7
- net FT_D14: now also U2.AA8; no longer U2.AA9
- net FT_NOE: now also U2.AB7; no longer U2.AA8
- net PSS_SD_CD: now also U2.U10; no longer U2.B12
- net PSS_SD_WP: now also U2.U9; no longer U2.B14
- net PWR_SYS_1V8: now also R186.2
- net PWR_SYS_3V3: now also R183.2, R184.2, R185.2
- net SEN_B_D12_N: now also U2.T17; no longer U2.N20
- net SEN_B_D12_P: now also U2.T16; no longer U2.N19
- net SEN_CLK_N: now also U2.N20; no longer U2.T17
- net SEN_CLK_P: now also U2.N19; no longer U2.T16
Routing:
- net PSS_SD_WP: track 66.6 -> 26.0 mm, vias 0 -> 2
- net PWR_SYS_3V3: track 165.2 -> 189.2 mm
- net PSS_SD_CD: track 56.0 -> 49.1 mm, vias 0 -> 2
- net FT_CLK: track 9.29 -> 11.6 mm
- net FT_NOE: track 22.0 -> 20.2 mm
- net BTN_TOPRIGHT: track 36.0 -> 37.6 mm, vias 1 -> 2
- net BTN_BTMRIGHT: track 41.7 -> 43.3 mm, vias 1 -> 2
- net FT_NWAKEUP: track 25.8 -> 27.2 mm
- net BTN_BTMLEFT: track 46.1 -> 47.4 mm
- net FPGA_DONE: track 191.5 -> 192.7 mm
- net FT_GPIO0: track 27.4 -> 28.4 mm
- net FT_D9: track 21.0 -> 22.0 mm
- net FPGA_NINIT: track 190.6 -> 191.4 mm
- net FT_D15: track 13.2 -> 13.9 mm, vias 0 -> 2
- net PWR_SYS_1V8: track 90.4 -> 91.1 mm, vias 37 -> 38
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