File: main.brd (EAGLE design)
At the start: 120 x 120 mm, 578 parts, among them CN1 50 PIN 0.5MM, CN2 10067847-001RLF, CN3 632723300011, CN4 FF0881SA1, CN5 15PIN 0.5MM, CN6 31 PIN FPC, Q1 2N7002, Q2 FDN302P, Q3 2N7002, Q5 SI7489DP, SW2 TACT, SW3 TACT, SW4 TACT, SW5 TACT, SW7 TACT, SW8 SLIDE SPDT, U1 GMAX0505-DV, U10 TPS70950, U11 FT601Q, U12 CBTU02043, U13 MAX25300B, U14 ESP32, U15 MAX25300B, U16 INA180, U17 AP62301, U18 AP62301, U19 SCHMITT, U2 XC7Z014S-1CLG484C, U20 MAX25300B, U21 NOT, U22 MAX25300B, U23 SN74LVC1G3, U24 NAND, U25 EMC1812T, U26 BIPOLAR HALL, U27 LM2663, U28 ADS7867, U29 LM2663, U3 IS43TR16128CL-125KBLI, U30 LM2731X, U31 USBLC6-2SC6, U32 MAX1735, U33 MP2148, U34 TPS22917, U35 AP62301, U36 TLV61046A, U37 W25Q128JV, U38 TPS70918, U39 AP62301, U4 AP63300WU-7, U5 STM32L431RBT, U6 USB ESD, U7 ACT2861QI301-T, U8 TPS70918, U9 STUSB4500

Commit message: DDR3 FPGA VRP/N pins fixed, pullups on the buttons corrected
Parts:
- moved R1 1.92 mm to (1.50, -33.0), turned to 90 degrees
- moved R2 0.71 mm to (2.50, -33.0), turned to 270 degrees
- moved R186 0.10 mm to (-33.0, -34.6)
Connections:
- net BTN_BTMLEFT: now also U2.G13; no longer U2.G6
- net BTN_TOPLEFT: now also U2.G6; no longer U2.G13
- net GND: now also R2.2; no longer R1.1
- net PWR_DDR3_1V35: now also R1.1; no longer R2.2
- net PWR_SYS_1V8: now also R183.2, R184.2; no longer R186.2
- net PWR_SYS_3V3: now also R186.2; no longer R183.2, R184.2
Routing:
- net PWR_SYS_3V3: track 189.2 -> 177.0 mm
- net BTN_TOPLEFT: track 64.2 -> 56.6 mm
- net PWR_SYS_1V8: track 91.1 -> 98.4 mm, vias 38 -> 37
- net BTN_BTMLEFT: track 47.4 -> 52.6 mm
- net GND: track 571.1 -> 572.9 mm

Commit message: Small changes
Parts:
- moved R178 10.9 mm to (43.1, 50.5), flipped to the top, turned to 90 degrees
- moved R105 10.9 mm to (44.0, 50.5), flipped to the top, turned to 90 degrees
- moved TP99 7.79 mm to (-36.8, -39.6), turned to 90 degrees
Routing:
- net PWR_VDISP_EN: track 56.6 -> 50.3 mm
- net PSS_FLASH_SCLK: track 29.1 -> 24.7 mm
- net GND: track 572.9 -> 570.3 mm
- net BMS_I2C_SCL: track 220.9 -> 222.1 mm
- net BMS_I2C_SDA: track 220.6 -> 221.7 mm
- net PMC_NRESET: track 176.8 -> 176.0 mm
- net FPGA_DONE: track 192.7 -> 191.8 mm
- net FPGA_NINIT: track 191.4 -> 190.5 mm
- net STUSB_SCL: track 98.6 -> 99.3 mm
- net STUSB_SDA: track 100.3 -> 101.0 mm
- net TMP_I2C_SCL: track 86.6 -> 86.0 mm

Commit message: Rev 1.0.0 ready for release
Parts:
- moved D6 7.92 mm to (-44.4, -30.6)
- moved D7 7.92 mm to (-44.4, -32.1)
- moved D9 7.92 mm to (-44.4, -33.6)
- moved R59 7.92 mm to (-41.9, -30.6)
- moved R79 7.92 mm to (-41.9, -32.1)
- moved R80 7.92 mm to (-41.9, -33.6)
Routing:
- net FPGA_LED_2: track 44.9 -> 35.7 mm
- net FPGA_LED_1: track 44.0 -> 35.9 mm
- net FPGA_LED_0: track 45.6 -> 37.5 mm
- net USBC_SS_RX2_P: track 15.9 -> 15.3 mm
- net USBC_SS_RX2_N: track 15.5 -> 15.0 mm
Other:
- board text added: "CONFIG SETTING"
- board text added: "LED_0"
- board text added: "LED_1"
- board text added: "LED_2"
- board text added: "gswdh.co.uk camera - soke main PCB rev 1.0.0 2023.07.25"
- board text removed: "gswdh.co.uk camera - soke main PCB rev 1.0.0 2023.07.18"

Commit message: SRST added to the debug port
Connections:
- net PSS_NSRST: now also CN1.P27
Routing:
- net PSS_NSRST: track 140.4 -> 185.9 mm, vias 3 -> 5
Changed lines of the file:
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@@
 <wire x1="-8.3" y1="-12.7" x2="-7.6" y2="-13.4" width="0.0889" layer="4"/>
 <wire x1="-7.6" y1="-13.4" x2="-7.6" y2="-14.5" width="0.0889" layer="4"/>
+<contactref element="CN1" pad="P27"/>
+<wire x1="-8.3" y1="-10.5" x2="-9" y2="-11.2" width="0.0889" layer="1"/>
+<wire x1="-9" y1="-11.2" x2="-9.8" y2="-11.2" width="0.0889" layer="1"/>
+<wire x1="-9.8" y1="-11.2" x2="-11.6" y2="-13" width="0.0889" layer="1"/>
+<wire x1="-25.9364125" y1="-13" x2="-25.9447625" y2="-13.00835" width="0.0889" layer="1"/>
+<via x="-36.1002875" y="-12.8002875" extent="1-16" drill="0.2"/>
+<wire x1="-36.1002875" y1="-12.8002875" x2="-36.3" y2="-13" width="0.0889" layer="16"/>
+<wire x1="-51.35" y1="-13" x2="-51.6" y2="-13.25" width="0.0889" layer="16"/>
+<via x="-51.6" y="-13.25" extent="1-16" drill="0.2"/>
+<wire x1="-51.6" y1="-13.25" x2="-52.5" y2="-13.25" width="0.0889" layer="1"/>
+<wire x1="-11.6" y1="-13" x2="-25.9364125" y2="-13" width="0.0889" layer="1"/>
+<wire x1="-36.3" y1="-13" x2="-51.35" y2="-13" width="0.0889" layer="16"/>
+<wire x1="-35.892225" y1="-13.00835" x2="-36.1002875" y2="-12.8002875" width="0.0889" layer="1"/>
+<wire x1="-25.9447625" y1="-13.00835" x2="-35.892225" y2="-13.00835" width="0.0889" layer="1"/>
 </signal>
 <signal name="FPGA_DEBUG_D0">

Commit message: Correct FPGA footprint routed. A lot of work to length match, optimise and review
Parts:
- removed C124, C126: 0.1uF 10V, c_0402:0402
- C104, C123: value 0.1uF 10V -> 47uF 6.3V; device c_0402:0402 -> c_0603:0603
- U2: device ICs:FBGA484 -> ICs:CLG484
- moved C131 17.3 mm to (6.80, -19.0)
- moved C123 16.9 mm to (5.90, -37.3), flipped to the top, turned to 180 degrees
- moved C132 13.9 mm to (0.80, -24.2), turned to 90 degrees
- moved C133 12.1 mm to (0.40, -19.8), turned to 0 degrees
- moved C104 8.83 mm to (-6.00, -37.3), flipped to the top
- moved C127 8.27 mm to (2.00, -21.4), turned to 180 degrees
- moved C138 7.57 mm to (-3.20, -21.0), turned to 270 degrees
- moved R1 7.52 mm to (8.10, -36.6), turned to 0 degrees
- moved R2 7.18 mm to (8.10, -37.5), turned to 180 degrees
- moved C128 6.53 mm to (10.0, -25.9)
- moved C86 5.71 mm to (0.80, -30.9), turned to 180 degrees
- moved C120 4.50 mm to (4.00, -29.0), turned to 90 degrees
- moved C186 4.36 mm to (-9.30, -34.2), turned to 180 degrees
- moved C83 4.21 mm to (-2.40, -27.0), turned to 0 degrees
- moved C122 4.20 mm to (3.20, -27.4), turned to 270 degrees
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Connections:
- removed net N$19: U2.M20
- removed net N$31: U2.M19
- net DDR_D0: now also U2.E1; no longer U2.E3
- net DDR_D2: now also U2.G2; no longer U2.G1
- net DDR_D4: now also U2.L2; no longer U2.L1
- net DDR_D6: now also U2.L1; no longer U2.L2
- net DDR_D8: now also U2.G1; no longer U2.G2
- net DDR_D9: now also U2.E3; no longer U2.E1
- net FT_BE0: now also U2.V4; no longer U2.U4
- net FT_BE1: now also U2.U6; no longer U2.Y5
- net FT_BE3: now also U2.U5; no longer U2.V5
- net FT_D0: now also U2.AA12; no longer U2.AB12
- net FT_D1: now also U2.AB12; no longer U2.AA12
- net FT_D10: now also U2.W10; no longer U2.V10
- net FT_D11: now also U2.AB10; no longer U2.Y10
- net FT_D12: now also U2.Y10; no longer U2.AB10
- net FT_D24: now also U2.U4; no longer U2.V4
- net FT_D29: now also U2.T6; no longer U2.R7
- net FT_D3: now also U2.AA11; no longer U2.AB11
- net FT_D30: now also U2.R7; no longer U2.T6
- net FT_D4: now also U2.AB11; no longer U2.AA11
- net FT_D6: now also U2.V12; no longer U2.U12
- net FT_D7: now also U2.U12; no longer U2.V12
- net FT_GPIO0: now also U2.W8; no longer U2.V8
- net FT_GPIO1: now also U2.V10; no longer U2.W10
- net FT_NRESET: now also U2.V8; no longer U2.Y8
- net FT_NSIWU: now also U2.Y5; no longer U2.U6
- net FT_NTXE: now also U2.V5; no longer U2.U5
- net FT_NWAKEUP: now also U2.Y8; no longer U2.W8
- net GND: no longer C124.1, C126.1
- net PWR_ANA_1V8: no longer C104.2
- net PWR_DDR3_1V35: now also C104.2, C123.2
- net PWR_SEN_0V7_EN: now also U2.A9; no longer U2.B10
- net PWR_SEN_N1V3A_EN: now also U2.B10; no longer U2.A9
- net PWR_SYS_1V8: no longer C123.2, C124.2, C126.2
Routing:
- net BTN_TOPLEFT: track 56.6 -> 108.3 mm
- net BTN_BTMLEFT: track 52.6 -> 103.9 mm, vias 3 -> 2
- net PSS_SD_D0: track 75.0 -> 47.5 mm
- net PSS_SD_D1: track 74.9 -> 48.4 mm
- net PSS_SD_CLK: track 74.7 -> 57.2 mm
- net SEN_B_D12_N: track 35.1 -> 22.5 mm
- net SEN_B_D12_P: track 35.1 -> 22.8 mm
- net N$42: track 1.41 -> 13.1 mm, vias 1 -> 2
- net N$7: track 1.41 -> 12.8 mm
- net PSS_SD_D3: track 74.8 -> 63.9 mm
- net PSS_SD_CMD: track 75.3 -> 65.3 mm
- net PSS_NRST: track 143.9 -> 153.5 mm
- net DDR_A10: track 25.0 -> 15.8 mm
- net PWR_SYS_3V3: track 177.0 -> 168.8 mm
- net BTN_BTMRIGHT: track 43.4 -> 51.3 mm, vias 2 -> 3
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
Commit message: Passes DRC
Parts:
- moved C156 0.20 mm to (-4.50, -38.8)
Routing:
- net PWR_ANA_1V8: track 18.7 -> 19.4 mm

Commit message: DDR3 length matched
Routing:
- net DDR_A10: track 15.8 -> 25.0 mm
- net DDR_A3: track 29.6 -> 25.0 mm
- net PSS_SPI_SCLK: track 170.8 -> 175.2 mm
- net DDR_D9: track 29.2 -> 24.9 mm
- net DDR_CLK_P: track 21.2 -> 24.8 mm
- net DDR_CLK_N: track 21.5 -> 24.8 mm
- net DDR_A13: track 28.0 -> 25.1 mm, vias 2 -> 4
- net DDR_D4: track 27.9 -> 25.0 mm
- net DDR_D14: track 27.6 -> 25.0 mm
- net DDR_D1: track 27.3 -> 25.0 mm
- net DDR_DM0: track 27.3 -> 25.0 mm
- net DDR_NCAS: track 27.3 -> 25.1 mm
- net DDR_A9: track 22.8 -> 25.0 mm
- net DDR_A0: track 27.2 -> 25.0 mm
- net DDR_D2: track 27.2 -> 25.0 mm
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
Commit message: MIPI length matched DRC passes
Routing:
- net MIPI_DSI_A_HS_CK_P: track 14.7 -> 20.0 mm
- net MIPI_DSI_A_HS_CK_N: track 14.7 -> 20.0 mm
- net DDR_NRAS: track 20.5 -> 25.0 mm
- net TMP_ALERT: track 92.3 -> 94.5 mm
- net MIPI_DSI_A_HS_L2_P: track 18.6 -> 20.0 mm
- net MIPI_DSI_A_HS_L2_N: track 18.6 -> 20.0 mm
- net MIPI_DSI_B_HS_L2_N: track 18.8 -> 20.0 mm
- net MIPI_DSI_B_HS_CK_N: track 19.0 -> 20.0 mm
- net MIPI_DSI_B_HS_L2_P: track 19.1 -> 20.0 mm
- net MIPI_DSI_B_HS_CK_P: track 19.3 -> 20.1 mm
