File: main.brd (EAGLE design)
At the start: 120 x 120 mm, 576 parts, among them CN1 50 PIN 0.5MM, CN2 10067847-001RLF, CN3 632723300011, CN4 FF0881SA1, CN5 15PIN 0.5MM, CN6 31 PIN FPC, Q1 2N7002, Q2 FDN302P, Q3 2N7002, Q5 SI7489DP, SW2 TACT, SW3 TACT, SW4 TACT, SW5 TACT, SW7 TACT, SW8 SLIDE SPDT, U1 GMAX0505-DV, U10 TPS70950, U11 FT601Q, U12 CBTU02043, U13 MAX25300B, U14 ESP32, U15 MAX25300B, U16 INA180, U17 AP62301, U18 AP62301, U19 SCHMITT, U2 XC7Z014S-1CLG484C, U20 MAX25300B, U21 NOT, U22 MAX25300B, U23 SN74LVC1G3, U24 NAND, U25 EMC1812T, U26 BIPOLAR HALL, U27 LM2663, U28 ADS7867, U29 LM2663, U3 IS43TR16128CL-125KBLI, U30 LM2731X, U31 USBLC6-2SC6, U32 MAX1735, U33 MP2148, U34 TPS22917, U35 AP62301, U36 TLV61046A, U37 W25Q128JV, U38 TPS70918, U39 AP62301, U4 AP63300WU-7, U5 STM32L431RBT, U6 USB ESD, U7 ACT2861QI301-T, U8 TPS70918, U9 STUSB4500

Commit message: Added extra decoupling to the PLL PSU
Parts:
- removed MECH3, MECH4: 6mm x 3mm, MISC:MOUNTHOLE_6X3
- added C124: 47uF 6.3V, c_0603:0603
- moved SCR1 8.20 mm to (0.00, -58.0)
- moved MECH5 7.21 mm to (-53.0, 53.0)
- moved MECH6 7.21 mm to (53.0, 53.0)
- moved MECH7 7.21 mm to (-53.0, -53.0)
- moved MECH8 7.21 mm to (53.0, -53.0)
- moved TP98 5.37 mm to (45.8, -55.1)
- moved CN3 5.00 mm to (57.0, -43.0)
- moved D2 2.20 mm to (51.9, -34.6), turned to 0 degrees
- moved C83 0.40 mm to (-2.00, -27.0)
- moved C105 0.20 mm to (-4.40, -28.8)
Connections:
- net GND: now also C124.1
- net PWR_ANA_1V8: now also C124.2
Routing:
- net USBC_SS_RX1_N: track 23.5 -> 3.21 mm
- net USBC_SS_RX1_P: track 22.8 -> 3.31 mm
- net USBC_SS_TX2_N: track 22.9 -> 3.88 mm
- net USBC_SS_TX2_P: track 22.2 -> 3.98 mm
- net USBC_CC2: track 17.6 -> 4.95 mm
- net USBC_CC1: track 16.6 -> 4.58 mm, vias 2 -> 1
- net PWR_ANA_1V8: track 19.4 -> 9.17 mm, vias 2 -> 3
- net USBC_SS_TX1_P: track 16.6 -> 9.54 mm
- net USBC_SS_TX1_N: track 16.3 -> 9.29 mm
- net USBC_SS_RX2_P: track 15.3 -> 8.63 mm
- net USBC_SS_RX2_N: track 15.0 -> 8.42 mm
- net GND: track 565.2 -> 559.6 mm
- net N$12: track 5.43 -> 0.00 mm, vias 1 -> 0
- net N$43: track 4.32 -> 0.00 mm
- net PWR_USBC_VBUS: track 51.8 -> 49.2 mm, vias 13 -> 12
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- added copper zone on layer 7, net PWR_ANA_1V8
- removed copper zone on layer 1, net GND
Other:
- outline, holes or cut-outs redrawn

Commit message: CN6 routed to new location closes #22
Parts:
- R95: device r_0603:0603 -> r_0402:0402
- moved C255 26.2 mm to (-22.9, -50.8)
- moved C256 24.3 mm to (-22.9, -42.1), turned to 180 degrees
- moved C257 24.0 mm to (-22.9, -40.8)
- moved CN6 22.8 mm to (-20.8, -48.0), turned to 270 degrees
- moved TP3 16.3 mm to (-33.1, -51.1)
- moved R95 12.9 mm to (-22.9, -43.1)
- moved C219 12.0 mm to (-36.9, -52.4)
- moved L9 12.0 mm to (-37.6, -55.5)
- moved R92 12.0 mm to (-30.6, -56.8)
- moved R93 12.0 mm to (-30.6, -55.5)
- moved R94 12.0 mm to (-30.6, -54.2)
- moved U36 12.0 mm to (-33.7, -55.5)
- moved C247 12.0 mm to (-33.0, -52.6)
- moved R162 3.14 mm to (-24.9, -46.9), turned to 270 degrees
- moved R163 1.92 mm to (-23.4, -47.4)
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Connections:
- net DDR_D0: now also U2.G1; no longer U2.E1
- net DDR_D8: now also U2.E1; no longer U2.G1
- net DDR_DQS0_N: now also U2.J2; no longer U2.D2
- net DDR_DQS0_P: now also U2.H2; no longer U2.C2
- net DDR_DQS1_N: now also U2.D2; no longer U2.J2
- net DDR_DQS1_P: now also U2.C2; no longer U2.H2
Routing:
- net BTN_BTMRIGHT: track 51.3 -> 75.3 mm
- net PWR_DDR3_1V35: track 50.7 -> 65.1 mm, vias 35 -> 36
- net DSP_IREF: track 10.6 -> 2.09 mm
- net PSS_SPI_MOSI: track 107.3 -> 99.1 mm
- net PSS_SPI_SCLK: track 108.1 -> 100.4 mm
- net PWR_SYS_3V3: track 168.8 -> 162.6 mm, vias 52 -> 53
- net DSP_D_NC: track 37.1 -> 32.1 mm
- net DSP_NRESET: track 37.5 -> 32.9 mm
- net PWR_VDISP_EN: track 52.1 -> 56.0 mm
- net PSS_FLASH_D3: track 20.9 -> 24.7 mm
- net DSP_SPI_NCS: track 39.9 -> 36.3 mm
- net PSS_FLASH_D2: track 35.4 -> 37.9 mm
- net GND: track 559.6 -> 558.0 mm, vias 532 -> 538
- net PSS_FLASH_SCLK: track 27.4 -> 28.9 mm
- net PSS_FLASH_D1: track 34.6 -> 36.0 mm
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
Commit message: Display is now connected to FPGA logic Closes #21
Connections:
- removed net ADC_SPI_NCS: U2.A8
- new net DSP_SPI_MOSI: CN6.11, U2.F16
- new net DSP_SPI_SCLK: CN6.12, U2.E16
- net DSP_D_NC: now also U2.D16; no longer U2.D8
- net DSP_NRESET: now also U2.D15; no longer U2.E8
- net DSP_SPI_NCS: now also U2.E15; no longer U2.E10
- net PSS_SPI_MISO: no longer U2.E9
- net PSS_SPI_MOSI: no longer CN6.11, U2.F11
- net PSS_SPI_SCLK: no longer CN6.12, U2.D6
- net SEN_SPI_NCS: no longer U2.A7
Routing:
- net PSS_SPI_SCLK: track 100.4 -> 0.00 mm, vias 5 -> 0
- net PSS_SPI_MOSI: track 99.1 -> 0.00 mm, vias 5 -> 0
- net DSP_SPI_MOSI: track 0.00 -> 38.3 mm, vias 0 -> 3
- net DSP_SPI_SCLK: track 0.00 -> 37.3 mm, vias 0 -> 3
- net TMP_ALERT: track 94.5 -> 102.4 mm, vias 3 -> 5
- net DSP_D_NC: track 32.1 -> 36.9 mm
- net DSP_NRESET: track 32.9 -> 36.8 mm
- net DSP_SPI_NCS: track 36.3 -> 38.1 mm
- net SEN_SPI_NCS: track 69.0 -> 67.3 mm
- net GND: track 558.0 -> 559.1 mm
- net PSS_SPI_MISO: track 70.4 -> 69.8 mm
- net FPGA_LED_0: track 39.2 -> 39.8 mm

Commit message: STUSB4500 now has pullups
Parts:
- added R187, R188: 2.2k, r_0402:0402
- moved D12 14.0 mm to (45.5, 57.4), turned to 270 degrees
- moved R60 11.9 mm to (45.5, 54.9), turned to 270 degrees
- moved D13 11.7 mm to (47.0, 57.4), turned to 270 degrees
- moved D14 9.71 mm to (48.5, 57.4), turned to 270 degrees
- moved R76 9.01 mm to (47.0, 54.9), turned to 270 degrees
- moved R77 6.26 mm to (48.5, 54.9), turned to 270 degrees
Connections:
- removed net STUSB_SCL: U5.23, U9.7
- removed net STUSB_SDA: U5.56, U9.8
- new net STUSB_I2C_SCL: R187.1, U5.23, U9.7
- new net STUSB_I2C_SDA: R188.1, U5.56, U9.8
- net PWR_SYS_1V8_SLP: now also R187.2, R188.2
Routing:
- net STUSB_I2C_SDA: track 0.00 -> 102.5 mm, vias 0 -> 2
- net STUSB_I2C_SCL: track 0.00 -> 102.1 mm, vias 0 -> 2
- net STUSB_SDA: track 101.0 -> 0.00 mm, vias 2 -> 0
- net STUSB_SCL: track 99.3 -> 0.00 mm, vias 2 -> 0
- net PMC_LED_STATUS: track 14.3 -> 6.04 mm
- net PMC_LED_FPGA_OK: track 12.3 -> 5.96 mm
- net PMC_LED_RUN: track 10.2 -> 6.58 mm
- net PWR_SYS_1V8_SLP: track 318.3 -> 321.4 mm

Commit message: STUSB4500 corrected digikey order number
Parts:
- U37: device ICs:SO8 -> ICs:SO8-208MIL
Routing:
- net GND: track 559.1 -> 560.0 mm
- net PSS_FLASH_SCLK: track 28.9 -> 28.0 mm
- net PSS_FLASH_NCS: track 8.58 -> 7.66 mm
- net PSS_FLASH_D3: track 24.7 -> 25.5 mm
Changed lines of the file:
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@@
 </element>
 <element name="U9" library="ICs" package="QFN24" value="STUSB4500" x="41.425" y="-38.35" smashed="yes" rot="R180">
-<attribute name="DIGIKEY" value="497-STUSB4500LQCT-ND" x="41.425" y="-38.35" size="1.778" layer="27" rot="R180" display="off"/>
+<attribute name="DIGIKEY" value="497-18060-1-ND" x="41.425" y="-38.35" size="1.778" layer="27" rot="R180" display="off"/>
 <attribute name="HEIGHT" value="1" x="41.425" y="-38.35" size="1.778" layer="27" rot="R180" display="off"/>
 <attribute name="NAME" x="39.05" y="-35.85" size="0.5" layer="25"/>
@@
 <attribute name="PRICE_PER" value="0.08" x="35.9" y="-46.2" size="0.5" layer="27" display="off"/>
 </element>
-<element name="U37" library="ICs" package="SO8" value="W25Q128JV" x="-17.7" y="-38.3" smashed="yes" rot="R180">
+<element name="U37" library="ICs" package="SO8-208MIL" value="W25Q128JV" x="-17.7" y="-38.3" smashed="yes" rot="R180">
 <attribute name="DIGIKEY" value="W25Q128JVSIQ-ND" x="-17.7" y="-38.3" size="0.5" layer="27" rot="R180" display="off"/>
 <attribute name="HEIGHT" value="2" x="-17.7" y="-38.3" size="0.5" layer="27" rot="R180" display="off"/>
@@
 <wire x1="-19.4" y1="-34.6" x2="-18.7" y2="-34.6" width="0.0889" layer="1"/>
 <via x="-18.7" y="-34.6" extent="1-16" drill="0.2"/>
-<wire x1="-15" y1="-36.425" x2="-16.075" y2="-36.425" width="0.25" layer="1"/>
+<wire x1="-14.075" y1="-36.395" x2="-16.075" y2="-36.425" width="0.25" layer="1"/>
 <wire x1="-16.075" y1="-36.425" x2="-16.1" y2="-36.4" width="0.25" layer="1"/>
 <via x="-16.1" y="-36.4" extent="1-16" drill="0.3"/>
@@
 <wire x1="23" y1="-16.7" x2="23" y2="-17.1" width="0.5" layer="1"/>
 <via x="23" y="-16.7" extent="1-16" drill="0.5"/>
-<wire x1="-20.4" y1="-40.175" x2="-20.4" y2="-41.4" width="0.25" layer="1"/>
+<wire x1="-21.325" y1="-40.205" x2="-20.4" y2="-41.4" width="0.25" layer="1"/>
 <wire x1="-20.4" y1="-41.4" x2="-21.85" y2="-41.4" width="0.25" layer="1"/>
 <via x="-21.85" y="-41.4" extent="1-16" drill="0.3"/>
@@
 <contactref element="U2" pad="A1"/>
 <contactref element="U37" pad="1"/>
-<wire x1="-13.975" y1="-40.175" x2="-15" y2="-40.175" width="0.0889" layer="1"/>
+<wire x1="-13.975" y1="-40.175" x2="-14.075" y2="-40.205" width="0.0889" layer="1"/>
 <wire x1="-8.4" y1="-35.4" x2="-9.2" y2="-35.4" width="0.0889" layer="1"/>
 <wire x1="-9.2" y1="-35.4" x2="-13.975" y2="-40.175" width="0.0889" layer="1"/>
@@
 <contactref element="U2" pad="A2"/>
 <contactref element="U37" pad="5"/>
-<wire x1="-18.675" y1="-36.425" x2="-20.4" y2="-36.425" width="0.0889" layer="1"/>
+<wire x1="-18.675" y1="-36.425" x2="-21.325" y2="-36.395" width="0.0889" layer="1"/>
 <contactref element="R36" pad="1"/>
 <contactref element="R167" pad="2"/>
@@
 <via x="-22.4" y="-36.5" extent="1-16" drill="0.2"/>
 <wire x1="-22.4" y1="-36.5" x2="-22.325" y2="-36.425" width="0.0889" layer="1"/>
-<wire x1="-22.325" y1="-36.425" x2="-20.4" y2="-36.425" width="0.0889" layer="1"/>
+<wire x1="-22.325" y1="-36.425" x2="-21.325" y2="-36.395" width="0.0889" layer="1"/>
 <wire x1="-29.1" y1="-43.7" x2="-25.1" y2="-43.7" width="0.0889" layer="16"/>
 <wire x1="-8.4" y1="-34.6" x2="-10" y2="-34.6" width="0.0889" layer="1"/>
@@
 <contactref element="U37" pad="2"/>
 <via x="-15" y="-38.3" extent="1-16" drill="0.2"/>
-<wire x1="-15" y1="-38.3" x2="-15" y2="-38.925" width="0.0889" layer="1"/>
+<wire x1="-15" y1="-38.3" x2="-14.075" y2="-38.935" width="0.0889" layer="1"/>
 <wire x1="-14.79045" y1="-38.09045" x2="-14.79045" y2="-36.59045" width="0.0889" layer="16"/>
 <wire x1="-15" y1="-38.3" x2="-14.79045" y2="-38.09045" width="0.0889" layer="16"/>
@@
 <via x="-16" y="-37.7" extent="1-16" drill="0.2"/>
 <wire x1="-16" y1="-37.7" x2="-15.975" y2="-37.675" width="0.0889" layer="1"/>
-<wire x1="-15.975" y1="-37.675" x2="-15" y2="-37.675" width="0.0889" layer="1"/>
+<wire x1="-15.975" y1="-37.675" x2="-14.075" y2="-37.665" width="0.0889" layer="1"/>
 <contactref element="R169" pad="2"/>
 <contactref element="R51" pad="1"/>
@@
 <via x="-14" y="-37.7" extent="1-16" drill="0.2"/>
 <wire x1="-14" y1="-37.7" x2="-14.025" y2="-37.675" width="0.0889" layer="1"/>
-<wire x1="-14.025" y1="-37.675" x2="-15" y2="-37.675" width="0.0889" layer="1"/>
+<wire x1="-14.025" y1="-37.675" x2="-14.075" y2="-37.665" width="0.0889" layer="1"/>
 <wire x1="-29.1" y1="-41.7" x2="-25.975" y2="-41.7" width="0.0889" layer="16"/>
 <wire x1="-5.2" y1="-33" x2="-4.8" y2="-33.4" width="0.0889" layer="1"/>
@@
 <wire x1="-14.4" y1="-36.8" x2="-14.4" y2="-38.65" width="0.0889" layer="16"/>
 <wire x1="-14.625" y1="-38.875" x2="-14.4" y2="-38.65" width="0.0889" layer="16"/>
-<wire x1="-20.4" y1="-38.925" x2="-20.45" y2="-38.875" width="0.0889" layer="1"/>
+<wire x1="-21.325" y1="-38.935" x2="-20.45" y2="-38.875" width="0.0889" layer="1"/>
 <wire x1="-20.45" y1="-38.875" x2="-21.5" y2="-38.875" width="0.0889" layer="1"/>
 <contactref element="R176" pad="2"/>
@@
 <wire x1="-25.575" y1="-39.7" x2="-24.625" y2="-38.75" width="0.0889" layer="16"/>
 <via x="-21.525" y="-37.675" extent="1-16" drill="0.2"/>
-<wire x1="-20.4" y1="-37.675" x2="-21.525" y2="-37.675" width="0.0889" layer="1"/>
+<wire x1="-21.325" y1="-37.665" x2="-21.525" y2="-37.675" width="0.0889" layer="1"/>
 <wire x1="-14.75" y1="-38.625" x2="-15.625" y2="-38.625" width="0.0889" layer="16"/>
 <wire x1="-22.6" y1="-38.75" x2="-21.525" y2="-37.675" width="0.0889" layer="16"/>

Commit message: STUSB4500 I2C orientation corrected and resistors added to facilitate reversing
Parts:
- added R189, R190: 10R, r_0402:0402
- moved R187 15.6 mm to (57.4, 43.5), turned to 0 degrees
- moved R188 11.8 mm to (53.6, 42.5), turned to 180 degrees
Connections:
- new net STM_I2C2_SCL: R190.1, U5.56
- new net STM_I2C2_SDA: R189.1, U5.23
- net STUSB_I2C_SCL: now also R190.2; no longer U5.23
- net STUSB_I2C_SDA: now also R189.2; no longer U5.56
Routing:
- net STM_I2C2_SCL: track 0.00 -> 17.9 mm, vias 0 -> 2
- net STM_I2C2_SDA: track 0.00 -> 16.1 mm, vias 0 -> 2
- net STUSB_I2C_SDA: track 102.5 -> 88.2 mm, vias 2 -> 0
- net STUSB_I2C_SCL: track 102.1 -> 89.4 mm, vias 2 -> 0
- net PWR_SYS_1V8_SLP: track 321.4 -> 319.7 mm, vias 22 -> 24
- net STUSB_RESET: track 90.6 -> 90.9 mm, vias 0 -> 2
Changed lines of the file:
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@@
 <attribute name="VOLTAGE" value="6.3V" x="-4.7" y="-27.7" size="1.778" layer="28" rot="MR180" display="off"/>
 </element>
-<element name="R187" library="r_0402" package="0402" value="2.2k" x="44.4" y="34.8" smashed="yes" rot="R270">
-<attribute name="DIGIKEY" value="311-2.20KLRCT-ND" x="44.4" y="34.8" size="1.778" layer="27" rot="R270" display="off"/>
-<attribute name="HEIGHT" value="0.4" x="44.4" y="34.8" size="1.778" layer="27" rot="R270" display="off"/>
-<attribute name="NAME" x="44.9" y="35.675" size="0.508" layer="25" rot="R270"/>
-<attribute name="PRICE_PER" value="0.08" x="44.4" y="34.8" size="1.778" layer="27" rot="R270" display="off"/>
+<element name="R187" library="r_0402" package="0402" value="2.2k" x="57.4" y="43.5" smashed="yes">
+<attribute name="DIGIKEY" value="311-2.20KLRCT-ND" x="57.4" y="43.5" size="1.778" layer="27" display="off"/>
+<attribute name="HEIGHT" value="0.4" x="57.4" y="43.5" size="1.778" layer="27" display="off"/>
+<attribute name="NAME" x="56.525" y="44" size="0.508" layer="25"/>
+<attribute name="PRICE_PER" value="0.08" x="57.4" y="43.5" size="1.778" layer="27" display="off"/>
 </element>
-<element name="R188" library="r_0402" package="0402" value="2.2k" x="44.9" y="50.5" smashed="yes" rot="R90">
-<attribute name="DIGIKEY" value="311-2.20KLRCT-ND" x="44.9" y="50.5" size="1.778" layer="27" rot="R90" display="off"/>
-<attribute name="HEIGHT" value="0.4" x="44.9" y="50.5" size="1.778" layer="27" rot="R90" display="off"/>
-<attribute name="NAME" x="45.3" y="51.525" size="0.508" layer="25" rot="R90"/>
-<attribute name="PRICE_PER" value="0.08" x="44.9" y="50.5" size="1.778" layer="27" rot="R90" display="off"/>
+<element name="R188" library="r_0402" package="0402" value="2.2k" x="53.6" y="42.5" smashed="yes" rot="R180">
+<attribute name="DIGIKEY" value="311-2.20KLRCT-ND" x="53.6" y="42.5" size="1.778" layer="27" rot="R180" display="off"/>
+<attribute name="HEIGHT" value="0.4" x="53.6" y="42.5" size="1.778" layer="27" rot="R180" display="off"/>
+<attribute name="NAME" x="54.575" y="42" size="0.508" layer="25" rot="R180"/>
+<attribute name="PRICE_PER" value="0.08" x="53.6" y="42.5" size="1.778" layer="27" rot="R180" display="off"/>
+</element>
+<element name="R189" library="r_0402" package="0402" value="10R" x="55" y="43" smashed="yes" rot="R270">
+<attribute name="DIGIKEY" value="311-10.0LRCT-ND" x="55" y="43" size="1.778" layer="27" rot="R270" display="off"/>
+<attribute name="HEIGHT" value="0.4" x="55" y="43" size="1.778" layer="27" rot="R270" display="off"/>
+<attribute name="NAME" x="55.3" y="44.025" size="0.508" layer="25" rot="R90"/>
+<attribute name="PRICE_PER" value="0.08" x="55" y="43" size="1.778" layer="27" rot="R270" display="off"/>
+</element>
+<element name="R190" library="r_0402" package="0402" value="10R" x="56" y="43" smashed="yes" rot="R90">
+<attribute name="DIGIKEY" value="311-10.0LRCT-ND" x="56" y="43" size="1.778" layer="27" rot="R90" display="off"/>
+<attribute name="HEIGHT" value="0.4" x="56" y="43" size="1.778" layer="27" rot="R90" display="off"/>
+<attribute name="NAME" x="55.7" y="41.975" size="0.508" layer="25" rot="R270"/>
+<attribute name="PRICE_PER" value="0.08" x="56" y="43" size="1.778" layer="27" rot="R90" display="off"/>
 </element>
 </elements>
@@
 <wire x1="57.1" y1="-7.8" x2="57.1" y2="30.5" width="0.0889" layer="1"/>
 <wire x1="57.1" y1="30.5" x2="53.4" y2="34.2" width="0.0889" layer="1"/>
-<wire x1="53.4" y1="34.2" x2="53.4" y2="42.2" width="0.0889" layer="1"/>
+<wire x1="53.4" y1="34.2" x2="53.4" y2="39.3" width="0.0889" layer="1"/>
 <contactref element="U5" pad="41"/>
-<wire x1="52.35" y1="43.25" x2="49.75" y2="43.25" width="0.0889" layer="1"/>
-<wire x1="53.4" y1="42.2" x2="52.35" y2="43.25" width="0.0889" layer="1"/>
 <contactref element="R103" pad="2"/>
 <wire x1="43.3" y1="-21.6" x2="43.3" y2="-34.6" width="0.0889" layer="1"/>
 <wire x1="43.3" y1="-37.075" x2="43.3" y2="-34.6" width="0.0889" layer="1"/>
+<wire x1="53.4" y1="39.3" x2="54.4" y2="40.3" width="0.0889" layer="1"/>
+<via x="54.4" y="40.3" extent="1-16" drill="0.2"/>
+<wire x1="54.4" y1="40.3" x2="53.7" y2="41" width="0.0889" layer="16"/>
+<via x="53.7" y="41" extent="1-16" drill="0.2"/>
+<wire x1="53.7" y1="41" x2="51.45" y2="43.25" width="0.0889" layer="1"/>
+<wire x1="51.45" y1="43.25" x2="49.75" y2="43.25" width="0.0889" layer="1"/>
 </signal>
 <signal name="STUSB_I2C_SCL">
 <contactref element="U9" pad="7"/>
-<contactref element="U5" pad="23"/>
 <wire x1="42.675" y1="-36.45" x2="42.675" y2="-33.97645" width="0.0889" layer="1"/>
 <wire x1="42.675" y1="-33.97645" x2="43.1" y2="-33.55145" width="0.0889" layer="1"/>
@@
 <wire x1="43.1" y1="-21.5" x2="56.9" y2="-7.7" width="0.0889" layer="1"/>
 <wire x1="56.9" y1="-7.7" x2="56.9" y2="30.4" width="0.0889" layer="1"/>
-<via x="43.7" y="38.4" extent="1-16" drill="0.2"/>
-<wire x1="43.7" y1="38.4" x2="43.25" y2="37.95" width="0.0889" layer="1"/>
-<wire x1="43.25" y1="37.95" x2="43.25" y2="37.25" width="0.0889" layer="1"/>
 <wire x1="56.9" y1="30.4" x2="53.2" y2="34.1" width="0.0889" layer="1"/>
-<wire x1="53.2" y1="41.8" x2="53" y2="42" width="0.0889" layer="1"/>
-<via x="53" y="42" extent="1-16" drill="0.2"/>
-<wire x1="53.2" y1="34.1" x2="53.2" y2="41.8" width="0.0889" layer="1"/>
-<wire x1="45.2" y1="42" x2="43.7" y2="40.5" width="0.0889" layer="4"/>
-<wire x1="43.7" y1="38.4" x2="43.7" y2="40.5" width="0.0889" layer="4"/>
-<wire x1="45.2" y1="42" x2="53" y2="42" width="0.0889" layer="4"/>
 <contactref element="R187" pad="1"/>
-<wire x1="43.25" y1="37.25" x2="43.25" y2="35.85" width="0.0889" layer="1"/>
-<wire x1="43.8" y1="35.3" x2="44.4" y2="35.3" width="0.0889" layer="1"/>
-<wire x1="43.25" y1="35.85" x2="43.8" y2="35.3" width="0.0889" layer="1"/>
+<contactref element="R190" pad="2"/>
+<wire x1="53.2" y1="34.1" x2="53.2" y2="39.6364125" width="0.0889" layer="1"/>
+<wire x1="55.5" y1="43" x2="56" y2="43.5" width="0.0889" layer="1"/>
+<wire x1="53.2" y1="39.6364125" x2="55.5" y2="41.9364125" width="0.0889" layer="1"/>
+<wire x1="55.5" y1="41.9364125" x2="55.5" y2="43" width="0.0889" layer="1"/>
+<wire x1="56.9" y1="43.5" x2="56" y2="43.5" width="0.0889" layer="1"/>
 </signal>
 <signal name="STUSB_I2C_SDA">
@@
 <wire x1="42.9" y1="-21.4" x2="56.7" y2="-7.6" width="0.0889" layer="1"/>
 <wire x1="56.7" y1="-7.6" x2="56.7" y2="30.3" width="0.0889" layer="1"/>
-<contactref element="U5" pad="56"/>
-<wire x1="44.25" y1="43.15" x2="44.25" y2="48.75" width="0.0889" layer="1"/>
 <wire x1="56.7" y1="30.3" x2="53" y2="34" width="0.0889" layer="1"/>
-<wire x1="53" y1="41.4" x2="52.6" y2="41.8" width="0.0889" layer="1"/>
-<wire x1="52.6" y1="41.8" x2="52.6" y2="42.4" width="0.0889" layer="1"/>
-<via x="52.6" y="42.4" extent="1-16" drill="0.2"/>
-<wire x1="53" y1="34" x2="53" y2="41.4" width="0.0889" layer="1"/>
-<via x="44.25" y="43.15" extent="1-16" drill="0.2"/>
-<wire x1="52.6" y1="42.4" x2="52.4" y2="42.2" width="0.0889" layer="4"/>
-<wire x1="52.4" y1="42.2" x2="45.2" y2="42.2" width="0.0889" layer="4"/>
-<wire x1="45.2" y1="42.2" x2="44.25" y2="43.15" width="0.0889" layer="4"/>
 <contactref element="R188" pad="1"/>
-<wire x1="44.25" y1="48.75" x2="44.25" y2="49.35" width="0.0889" layer="1"/>
-<wire x1="44.25" y1="49.35" x2="44.9" y2="50" width="0.0889" layer="1"/>
+<contactref element="R189" pad="2"/>
+<wire x1="55" y1="41.8" x2="55" y2="42.5" width="0.0889" layer="1"/>
+<wire x1="53" y1="34" x2="53" y2="39.8" width="0.0889" layer="1"/>
+<wire x1="53" y1="39.8" x2="55" y2="41.8" width="0.0889" layer="1"/>
+<wire x1="55" y1="42.5" x2="54.1" y2="42.5" width="0.0889" layer="1"/>
 </signal>
 <signal name="STUSB_PD0">
@@
 <contactref element="R187" pad="2"/>
 <contactref element="R188" pad="2"/>
-<wire x1="44.4" y1="34.3" x2="42.2" y2="34.3" width="0.0889" layer="1"/>
-<wire x1="44.9" y1="51" x2="44" y2="51" width="0.0889" layer="1"/>
+<wire x1="53.1" y1="42.5" x2="53.1" y2="43.2" width="0.0889" layer="1"/>
+<via x="53.1" y="43.2" extent="1-16" drill="0.2"/>
+<wire x1="57.9" y1="43.5" x2="57.9" y2="42.8" width="0.0889" layer="1"/>
+<via x="57.9" y="42.8" extent="1-16" drill="0.2"/>
 </signal>
 <signal name="N$37">
@@
 <wire x1="-18" y1="-44.5" x2="-19.5" y2="-46" width="0.0889" layer="5"/>
 </signal>
+<signal name="STM_I2C2_SDA">
+<contactref element="R189" pad="1"/>
+<contactref element="U5" pad="23"/>
+<wire x1="55" y1="43.5" x2="55" y2="44.2" width="0.0889" layer="1"/>
+<via x="55" y="44.2" extent="1-16" drill="0.2"/>
+<wire x1="55" y1="44.2" x2="52.6" y2="41.8" width="0.0889" layer="4"/>
+<wire x1="46.5" y1="41.8" x2="43.8" y2="39.1" width="0.0889" layer="4"/>
+<via x="43.8" y="39.1" extent="1-16" drill="0.2"/>
+<wire x1="43.8" y1="39.1" x2="43.25" y2="38.55" width="0.0889" layer="1"/>
+<wire x1="43.25" y1="38.55" x2="43.25" y2="37.25" width="0.0889" layer="1"/>
+<wire x1="52.6" y1="41.8" x2="46.5" y2="41.8" width="0.0889" layer="4"/>
+</signal>
+<signal name="STM_I2C2_SCL">
+<contactref element="R190" pad="1"/>
+<contactref element="U5" pad="56"/>
+<wire x1="56" y1="42.5" x2="56" y2="41.8" width="0.0889" layer="1"/>
+<via x="56" y="41.8" extent="1-16" drill="0.2"/>
+<wire x1="56" y1="41.8" x2="56" y2="44.5" width="0.0889" layer="4"/>
+<wire x1="44.95" y1="48.7" x2="44.25" y2="48" width="0.0889" layer="4"/>
+<via x="44.25" y="48" extent="1-16" drill="0.2"/>
+<wire x1="56" y1="44.5" x2="51.8" y2="48.7" width="0.0889" layer="4"/>
+<wire x1="51.8" y1="48.7" x2="44.95" y2="48.7" width="0.0889" layer="4"/>
+<wire x1="44.25" y1="48.75" x2="44.25" y2="48" width="0.0889" layer="1"/>
+</signal>
 </signals>

Commit message: SPI fixed, FPGA LEDs fixed
Parts:
- R59, R79, R80: value 120 -> 2.2k
Connections:
- removed net PSS_SPI_MISO: U1.L12
- removed net PSS_SPI_MOSI: U1.K12
- removed net PSS_SPI_SCLK: U1.J14
- new net SEN_SPI_MISO: U1.L12, U2.Y21
- new net SEN_SPI_MOSI: U1.K12, U2.U22
- new net SEN_SPI_SCLK: U1.J14, U2.U19
- net SEN_SPI_NCS: now also U2.T22
Routing:
- net SEN_SPI_MISO: track 0.00 -> 101.5 mm, vias 0 -> 4
- net PSS_SPI_MISO: track 69.8 -> 0.00 mm, vias 3 -> 0
- net SEN_SPI_SCLK: track 0.00 -> 33.3 mm, vias 0 -> 4
- net SEN_SPI_NCS: track 67.3 -> 97.8 mm, vias 2 -> 3
- net SEN_SPI_MOSI: track 0.00 -> 29.2 mm, vias 0 -> 2
- net TMP_ALERT: track 102.4 -> 105.4 mm
- net PWR_SEN_3V3A_EN: track 46.8 -> 49.6 mm
- net PWR_SEN_1V3_EN: track 62.5 -> 65.3 mm
- net TMP_THERM: track 85.4 -> 88.0 mm
- net TMP_I2C_SCL: track 86.0 -> 88.6 mm
- net TMP_I2C_SDA: track 88.6 -> 91.2 mm
- net FPGA_NPROG: track 182.4 -> 181.7 mm
