File: main.brd (EAGLE design)
At the start: 120 x 120 mm, 579 parts, among them CN1 50 PIN 0.5MM, CN2 10067847-001RLF, CN3 632723300011, CN4 FF0881SA1, CN5 15PIN 0.5MM, CN6 31 PIN FPC, Q1 2N7002, Q2 FDN302P, Q3 2N7002, Q5 SI7489DP, SW2 TACT, SW3 TACT, SW4 TACT, SW5 TACT, SW7 TACT, SW8 SLIDE SPDT, U1 GMAX0505-DV, U10 TPS70950, U11 FT601Q, U12 CBTU02043, U13 MAX25300B, U14 ESP32, U15 MAX25300B, U16 INA180, U17 AP62301, U18 AP62301, U19 SCHMITT, U2 XC7Z014S-1CLG484C, U20 MAX25300B, U21 NOT, U22 MAX25300B, U23 SN74LVC1G3, U24 NAND, U25 EMC1812T, U26 BIPOLAR HALL, U27 LM2663, U28 ADS7867, U29 LM2663, U3 IS43TR16128CL-125KBLI, U30 LM2731X, U31 USBLC6-2SC6, U32 MAX1735, U33 MP2148, U34 TPS22917, U35 AP62301, U36 TLV61046A, U37 W25Q128JV, U38 TPS70918, U39 AP62301, U4 AP63300WU-7, U5 STM32L431RBT, U6 USB ESD, U7 ACT2861QI301-T, U8 TPS70918, U9 STUSB4500

Commit message: U22 now powered
Connections:
- removed net SYS_PWR_3V3: C69.2, U22.1
- net PWR_SYS_3V3: now also C69.2, U22.1
Routing:
- net PWR_SYS_3V3: track 162.9 -> 174.0 mm, vias 53 -> 54
- net SYS_PWR_3V3: track 1.05 -> 0.00 mm
Changed lines of the file:
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@@
 <wire x1="-21.625" y1="-50.75" x2="-22.375" y2="-51.5" width="0.5" layer="3"/>
 <wire x1="-21.625" y1="-41.625" x2="-21.625" y2="-50.75" width="0.5" layer="3"/>
+<contactref element="U22" pad="1"/>
+<contactref element="C69" pad="2"/>
+<wire x1="-28.925" y1="7.475" x2="-28.925" y2="8.35" width="0.25" layer="1"/>
+<wire x1="-28.925" y1="8.35" x2="-28.8" y2="8.475" width="0.25" layer="1"/>
+<wire x1="-28.8" y1="8.475" x2="-29.775" y2="8.475" width="0.5" layer="1"/>
+<wire x1="-29.775" y1="8.475" x2="-29.8" y2="8.5" width="0.5" layer="1"/>
+<via x="-29.8" y="8.5" extent="1-16" drill="0.5"/>
+<wire x1="-29.8" y1="8.5" x2="-32.3" y2="8.5" width="0.5" layer="3"/>
+<wire x1="-32.3" y1="8.5" x2="-36.9" y2="3.9" width="0.5" layer="3"/>
 </signal>
 <signal name="PSS_PMC_UART_TX">
@@
 <wire x1="-7.062225" y1="-26.5" x2="-6.537775" y2="-26.5" width="0.0889" layer="16"/>
 </signal>
-<signal name="SYS_PWR_3V3">
-<contactref element="U22" pad="1"/>
-<contactref element="C69" pad="2"/>
-<wire x1="-28.925" y1="7.475" x2="-28.925" y2="8.35" width="0.25" layer="1"/>
-<wire x1="-28.925" y1="8.35" x2="-28.8" y2="8.475" width="0.25" layer="1"/>
-</signal>
 <signal name="SEN_T_D3_P">
