File: debug.brd (EAGLE design)
At the start: 25 x 100 mm, 24 parts, among them CN1 2X10 HEADER, CN2 MICRO USB B, CN3 14 PIN 2mm, CN4 MICRO USB B, CN5 2X10 HEADER, CN6 31 PIN FPC, U1 USBLC6-2SC6, U2 USBLC6-2SC6, U3 FT231X, U7 FT231X

Commit message: Thumb button connected to wakeup, diff pair lengths fixed
Parts:
- removed CN6: 31 PIN FPC, CONNECTORs:3-1734839-1
- removed R3: 10R, r_0603:0603
- added Q1, Q2: MMBT3904, TRANSISTORs:SOT23-3
- added R5: 10k, r_0603:0603
- CN3: value 14 PIN 2mm -> 50 PIN 0.5MM; device CONNECTORs:0878331420 -> CONNECTORs:FH52E-50S-0.5SH
- R4: value 10R -> 10k
- moved CN2 71.3 mm to (51.4, -79.6), turned to 0 degrees
- moved CN4 68.3 mm to (-10.0, -23.8), turned to 0 degrees
- moved FB2 64.2 mm to (-13.8, -14.8)
- moved CN1 63.0 mm to (39.9, -19.2), turned to 270 degrees
- moved C13 62.1 mm to (53.4, -72.1), turned to 90 degrees
- moved U1 61.2 mm to (-10.0, -14.8), turned to 180 degrees
- moved FB1 61.1 mm to (48.8, -72.9), turned to 270 degrees
- moved U2 60.1 mm to (51.2, -71.4), turned to 180 degrees
- moved C1 58.3 mm to (-7.12, -14.8), turned to 180 degrees
- moved C2 53.1 mm to (-11.5, -7.75), turned to 90 degrees
- moved C10 52.7 mm to (47.1, -67.1), turned to 180 degrees
- moved C3 52.2 mm to (-10.2, -7.75), turned to 90 degrees
- moved C4 51.0 mm to (47.1, -65.9), turned to 180 degrees
- moved U7 49.1 mm to (42.0, -65.5), turned to 0 degrees
- moved CN3 48.0 mm to (0.00, 20.0), turned to 180 degrees
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Connections:
- net N$13 renamed USB_VBUS
- removed net DEBUG_GPIO_0: CN6.30
- removed net FPGA_JTAG_NRESET: CN3.13, CN6.6
- removed net FPGA_TCK: CN3.5, CN6.2
- removed net FPGA_TDI: CN3.9, CN6.5
- removed net FPGA_TDO: CN3.7, CN6.4
- removed net FPGA_TMS: CN3.3, CN6.3
- removed net N$15: R3.1, U3.20
- removed net N$16: R4.1, U3.4
- removed net STP_UART_RX: CN6.26, R3.2
- removed net STP_UART_TX: CN6.25, R4.2
- new net BMS_I2C_SCL: CN3.P25
- new net BMS_I2C_SDA: CN3.P24
- new net BMS_NINT: CN3.P23
- new net DEBUG_UART_RX: CN3.P34
- new net DEBUG_UART_TX: CN3.P35
- new net ESP32_EN: CN3.P28, Q1.2
- new net ESP32_UART_!DTR: Q2.3, R4.2, U3.1
- new net ESP32_UART_!RTS: Q1.3, R5.2, U3.2
- new net ESP32_UART_RX: CN3.P30, U3.20
- new net ESP32_UART_TX: CN3.P29, U3.4
- new net ESP_IO0: CN3.P31, Q2.2
- new net FPGA_GPIO_0: CN3.P9
- new net FPGA_GPIO_1: CN3.P12
- new net FPGA_GPIO_2: CN3.P14
- new net FPGA_GPIO_3: CN3.P10
- new net FPGA_GPIO_4: CN3.P13
- new net FPGA_GPIO_5: CN3.P11
- new net FPGA_GPIO_6: CN3.P15
- new net FPGA_JTAG_TCK: CN3.P47
- new net FPGA_JTAG_TDI: CN3.P48
- new net FPGA_JTAG_TDO: CN3.P46
- new net FPGA_JTAG_TMS: CN3.P49
- new net N$100: Q2.1, R5.1
- new net N$99: Q1.1, R4.1
- new net PMC_UART_RX: CN3.P3
- new net PMC_UART_TX: CN3.P2
- new net PSS_JTAG_MOD: CN3.P41
- new net PSS_JTAG_NTRST: CN3.P40
- new net PSS_JTAG_TCK: CN3.P42
- new net PSS_JTAG_TDI: CN3.P39
- new net PSS_JTAG_TDO: CN3.P38
- new net PSS_JTAG_TMS: CN3.P43
- new net PWR_DIG_1V8: CN3.P16, CN3.P45
- new net PWR_PSS_DCDC_1V8: CN3.P33, CN3.P37
- new net PWR_SYS_1V8_SLP: CN3.P7
- net FPGA_DEBUG_CLK: no longer CN6.13
- net FPGA_DEBUG_D0: no longer CN6.15
- net FPGA_DEBUG_D1: no longer CN6.16
- net FPGA_DEBUG_D2: no longer CN6.17
- net FPGA_DEBUG_D3: no longer CN6.18
- net FPGA_DEBUG_D4: no longer CN6.19
- net FPGA_DEBUG_D5: no longer CN6.20
- net FPGA_DEBUG_D6: no longer CN6.21
- net FPGA_DEBUG_D7: no longer CN6.22
- net FPGA_DEBUG_EN: no longer CN6.14
- net FPGA_UART_RX: no longer CN6.9
- net FPGA_UART_TX: no longer CN6.10
- net GND: now also CN3.P1, CN3.P17, CN3.P26, CN3.P32, CN3.P36, CN3.P44, CN3.P50, CN3.P8, CN3.SH1, CN3.SH2; no longer CN3.10, CN3.12, CN3.14, CN3.2, CN3.4, CN3.6, CN3.8, CN6.12, CN6.23, CN6.29, CN6.7, CN6.8
- net PWR_3V3_SLP: no longer C6.2, CN6.24, U3.3
- net PWR_FPGA_1V8: no longer CN6.11
- net PWR_SYS_3V3: now also C6.2, CN3.P27, U3.14, U3.3; no longer CN3.1, CN6.1
- net STP_NRESET: now also CN3.P6; no longer CN6.31
- net STP_SWCLK: now also CN3.P5; no longer CN6.28
- net STP_SWDIO: now also CN3.P4; no longer CN6.27
Routing:
- net PWR_3V3_SLP: track 59.0 -> 0.00 mm
- net PWR_FPGA_1V8: track 39.4 -> 0.00 mm
- net FPGA_JTAG_NRESET: track 37.4 -> 0.00 mm
- net FPGA_TDI: track 36.4 -> 0.00 mm, vias 1 -> 0
- net STP_SWDIO: track 35.7 -> 0.00 mm
- net FPGA_TDO: track 35.4 -> 0.00 mm, vias 1 -> 0
- net FPGA_TCK: track 34.1 -> 0.00 mm, vias 1 -> 0
- net STP_UART_TX: track 34.0 -> 0.00 mm
- net STP_SWCLK: track 33.5 -> 0.00 mm
- net FPGA_TMS: track 32.2 -> 0.00 mm, vias 1 -> 0
- net STP_UART_RX: track 31.7 -> 0.00 mm
- net FPGA_UART_TX: track 31.2 -> 0.00 mm
- net FPGA_UART_RX: track 27.5 -> 0.00 mm
- net FPGA_DEBUG_CLK: track 26.3 -> 0.00 mm
- net ESP32_UART_RX: track 0.00 -> 24.9 mm
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- removed copper zone on layer 1, net GND
- removed copper zone on layer 16, net GND
Other:
- board size 25 x 100 mm -> 120 x 50 mm

Commit message: SRST added to the debug port
Parts:
- removed C13: 0.1uF 16V, c_0603:0603
- removed U7: FT231X, ICs:SSOP20-4MM
- added C11, C12, C7, C8, C9: 0.1uF 16V, c_0603:0603
- added CN6, CN7: MICRO USB B, CONNECTORs:ZX62-B-5PA(33)
- added CN8: 2X4_HEADER, CONNECTORs:4X2_HEADER
- added D1: RED LED, OPTO:0603_POLAR
- added FB3: 150R 100MHz, INDUCTORS:1206
- added Q3: 2N7002, TRANSISTORs:SOT23-3
- added U4, U6: FT231X, ICs:SSOP20-4MM
- added U5: USBLC6-2SC6, ICs:SOT23-6
- C5: value 0.1uF 16V -> 2.2uF 25V; device c_0603:0603 -> CAPACITORS:0603
- CN2: value MICRO USB B -> JTAG PROG; device CONNECTORs:ZX62-B-5PA(33) -> CONNECTORs:2X7HEADER
- R1, R2: value 10R -> 4.7k
- moved CN2 117.0 mm to (-47.5, -17.0), turned to 270 degrees
- moved R2 110.4 mm to (-47.2, 12.1), turned to 90 degrees
- moved R1 105.9 mm to (-48.2, 5.38), turned to 270 degrees
- moved FB1 78.9 mm to (-3.75, -14.0), turned to 180 degrees
- moved U2 76.9 mm to (0.00, -14.0)
- moved C5 68.6 mm to (-1.50, -7.00), turned to 90 degrees
- moved C4 68.2 mm to (2.88, -14.0)
- moved C10 60.4 mm to (52.5, -7.00), turned to 90 degrees
- moved C1 22.5 mm to (15.4, -14.0)
- moved C2 22.5 mm to (11.0, -7.00)
- moved C3 22.5 mm to (12.2, -7.00)
- moved C6 22.5 mm to (14.1, 2.75)
- moved CN4 22.5 mm to (12.5, -23.0)
- moved FB2 22.5 mm to (8.75, -14.0)
- moved Q1 22.5 mm to (9.38, 7.25)
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Connections:
- net PSS_JTAG_TMS renamed FPGA_NPROG
- net STP_NRESET renamed PMC_NRESET
- net STP_SWCLK renamed PMC_SWCLK
- net STP_SWDIO renamed PMC_SWDIO
- removed net DEBUG_UART_RX: CN3.P34
- removed net DEBUG_UART_TX: CN3.P35
- removed net FPGA_GPIO_0: CN3.P9
- removed net FPGA_GPIO_1: CN3.P12
- removed net FPGA_GPIO_2: CN3.P14
- removed net FPGA_GPIO_3: CN3.P10
- removed net FPGA_GPIO_4: CN3.P13
- removed net FPGA_GPIO_5: CN3.P11
- removed net FPGA_GPIO_6: CN3.P15
- removed net FPGA_UART_RX: R1.2
- removed net FPGA_UART_TX: R2.2
- removed net N$25: CN2.1, FB1.1
- removed net N$28: CN2.2, U2.3
- removed net PSS_JTAG_MOD: CN3.P41
- removed net PSS_JTAG_NTRST: CN3.P40
- removed net PSS_JTAG_TCK: CN3.P42
- removed net PSS_JTAG_TDI: CN3.P39
- removed net PSS_JTAG_TDO: CN3.P38
- removed net PWR_3V3_SLP: CN1.1
- removed net PWR_DIG_1V8: CN3.P16, CN3.P45
- removed net PWR_FPGA_1V8: C5.2, U7.3
- removed net PWR_PSS_DCDC_1V8: CN3.P33, CN3.P37
- new net FPGA_DONE: CN3.P45, Q3.1, R1.1
- new net FPGA_NINIT: CN3.P44
- new net FPGA_PS_NSRST: CN2.8, CN3.P24
- new net FPGA_STATUS_D0: CN3.P28
- new net FPGA_STATUS_D1: CN3.P27
- new net FPGA_STATUS_D2: CN3.P26
- new net N$14: Q3.2, R2.1
- new net N$15: U2.6, U4.11
- new net N$16: CN7.2, U5.3
- new net N$17: C10.2, U6.13
- new net N$18: U5.4, U6.12
- new net N$19: U5.6, U6.11
- new net N$22: D1.K, R2.2
- new net PSS_DEBUG_UART_RX: CN3.P22, U4.20
- new net PSS_DEBUG_UART_TX: CN3.P21, U4.4
- new net PWR_SYS_1V8: C8.2, CN3.P20, U4.14, U4.3
- new net USB_VBUS1: C4.2, C7.2, FB1.2, U2.5, U4.15
- new net USB_VBUS2: C11.2, C9.2, FB3.2, U5.5, U6.15
- net BMS_I2C_SCL: now also CN3.P10, CN8.6; no longer CN3.P25
- net BMS_I2C_SDA: now also CN3.P11, CN8.7; no longer CN3.P24
- net BMS_NINT: now also CN3.P12, CN8.8; no longer CN3.P23
- net ESP32_EN: now also CN3.P15; no longer CN3.P28
- net ESP32_UART_RX: now also CN3.P17; no longer CN3.P30
- net ESP32_UART_TX: now also CN3.P16; no longer CN3.P29
- net ESP_IO0: now also CN3.P18; no longer CN3.P31
- net FPGA_DEBUG_CLK: now also CN3.P31, CN5.1; no longer CN5.10
- net FPGA_DEBUG_D0: now also CN3.P40, CN5.10; no longer CN5.8
- net FPGA_DEBUG_D1: now also CN3.P39, CN5.9; no longer CN5.7
- net FPGA_DEBUG_D2: now also CN3.P38, CN5.8; no longer CN5.6
- net FPGA_DEBUG_D3: now also CN3.P37, CN5.7; no longer CN5.5
- net FPGA_DEBUG_D4: now also CN3.P36, CN5.6; no longer CN5.4
- net FPGA_DEBUG_D5: now also CN3.P35, CN5.5; no longer CN5.3
- net FPGA_DEBUG_D6: now also CN3.P34, CN5.4; no longer CN5.2
- net FPGA_DEBUG_D7: now also CN3.P33, CN5.3; no longer CN5.1
- net FPGA_DEBUG_EN: now also CN3.P32, CN5.2; no longer CN5.9
- net FPGA_JTAG_TCK: now also CN2.12
- net FPGA_JTAG_TDI: now also CN2.10
- net FPGA_JTAG_TDO: now also CN2.11
- net FPGA_JTAG_TMS: now also CN2.13
- net GND: now also C11.1, C12.1, C7.1, C8.1, C9.1, CN2.1, CN2.2, CN2.3, CN2.4, CN2.6, CN2.7, CN3.P13, CN3.P19, CN3.P25, CN3.P29, CN3.P41, CN6.5, CN6.SH1, CN6.SH2, CN6.SH3, CN6.SH4, CN6.SH5, CN6.SH6, CN7.5, CN7.SH1, CN7.SH2, CN7.SH3, CN7.SH4, CN7.SH5, CN7.SH6, CN8.1, CN8.2, CN8.3, CN8.4, Q3.3, U4.16, U4.6, U5.2, U6.16, U6.6; no longer C13.1, CN2.SH1, CN2.SH2, CN2.SH3, CN2.SH4, CN2.SH5, CN2.SH6, CN3.P17, CN3.P26, CN3.P32, CN3.P36, CN3.P44, U7.16, U7.6
- net N$1: now also CN6.1, FB1.1; no longer CN2.3, U2.1
- net N$2: now also CN6.3, U2.1; no longer U2.6, U7.11
- net N$3: now also CN7.1, FB3.1; no longer U2.4, U7.12
- net N$4: now also CN7.3, U5.1; no longer C13.2, C4.2, FB1.2, U2.5, U7.15
- net N$5: now also CN6.2, U2.3; no longer C10.2, U7.13
- net N$6: now also C5.2, U4.13; no longer R1.1, U7.20
- net N$7: now also U2.4, U4.12; no longer R2.1, U7.4
- net PMC_UART_RX: now also U6.20
- net PMC_UART_TX: now also U6.4
- net PWR_SYS_1V8_SLP: now also C12.2, CN1.1, CN3.P9, CN8.5, U6.14, U6.3
- net PWR_SYS_3V3: now also CN2.14, CN3.P14, CN3.P30, CN3.P42, D1.A, R1.2; no longer CN3.P27
Routing:
- net PWR_SYS_3V3: track 8.69 -> 149.3 mm
- net PWR_SYS_1V8_SLP: track 0.00 -> 111.7 mm, vias 0 -> 1
- net FPGA_PS_NSRST: track 0.00 -> 91.5 mm
- net PMC_UART_RX: track 0.00 -> 62.5 mm
- net FPGA_JTAG_TDI: track 0.00 -> 58.4 mm
- net FPGA_DEBUG_D0: track 0.00 -> 57.0 mm
- net FPGA_JTAG_TCK: track 0.00 -> 56.8 mm, vias 0 -> 1
- net FPGA_JTAG_TDO: track 0.00 -> 56.7 mm
- net PMC_UART_TX: track 0.00 -> 56.3 mm, vias 0 -> 2
- net PMC_SWDIO: track 0.00 -> 55.8 mm
- net FPGA_DEBUG_D1: track 0.00 -> 54.9 mm
- net PMC_SWCLK: track 0.00 -> 53.8 mm
- net FPGA_DEBUG_D2: track 0.00 -> 52.9 mm
- net FPGA_JTAG_TMS: track 0.00 -> 51.9 mm, vias 0 -> 1
- net FPGA_DEBUG_D3: track 0.00 -> 50.9 mm
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- added copper zone on layer 2, net GND
Other:
- board text added: "FPGA DONE"

Commit message: Debug and power board ready for outputs
Routing:
- net FPGA_DEBUG_D6: track 48.5 -> 44.7 mm
Changed lines of the file:
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@@
 <wire x1="-4.25" y1="11.875" x2="-4.25" y2="17.5" width="0.15" layer="1"/>
 <wire x1="-8" y1="8.125" x2="-4.25" y2="11.875" width="0.15" layer="1"/>
-<wire x1="-17.565" y1="-20.73" x2="-14.885" y2="-18.05" width="0.15" layer="1"/>
 <wire x1="-17.565" y1="-20.73" x2="-14.835" y2="-18" width="0.15" layer="1"/>
 <wire x1="-14.835" y1="-18" x2="-13.125" y2="-18" width="0.15" layer="1"/>
@@
 <wire x1="8.875" y1="4" x2="4.75" y2="8.125" width="0.15" layer="1"/>
 <wire x1="4.75" y1="8.125" x2="4.75" y2="17.5" width="0.15" layer="1"/>
-<wire x1="13.4525" y1="1.0475" x2="10.5" y2="4" width="0.15" layer="1"/>
+<wire x1="12.975" y1="1.525" x2="12.92824375" y2="1.525" width="0.15" layer="1"/>
+<wire x1="12.92824375" y1="1.525" x2="12.65" y2="1.80324375" width="0.15" layer="1"/>
+<wire x1="12.65" y1="1.80324375" x2="12.65" y2="1.85" width="0.15" layer="1"/>
+<wire x1="13.4525" y1="1.0475" x2="12.975" y2="1.525" width="0.15" layer="1"/>
+<wire x1="12.65" y1="1.85" x2="10.5" y2="4" width="0.15" layer="1"/>
 </signal>
 <signal name="ESP32_UART_RX">
@@
 <contactref element="U4" pad="4"/>
 <wire x1="0.9525" y1="0.375" x2="0.9525" y2="1.0475" width="0.15" layer="1"/>
-<wire x1="0.9525" y1="1.0475" x2="0.125" y2="1.875" width="0.15" layer="1"/>
-<wire x1="0.125" y1="1.875" x2="0.125" y2="5" width="0.15" layer="1"/>
 <wire x1="2.625" y1="15" x2="2.25" y2="15.375" width="0.15" layer="1"/>
 <wire x1="2.25" y1="15.375" x2="2.25" y2="17.5" width="0.15" layer="1"/>
 <wire x1="0.125" y1="5" x2="2.625" y2="7.5" width="0.15" layer="1"/>
 <wire x1="2.625" y1="7.5" x2="2.625" y2="15" width="0.15" layer="1"/>
+<wire x1="0.4512" y1="1.5488" x2="0.43810625" y2="1.5488" width="0.15" layer="1"/>
+<wire x1="0.43810625" y1="1.5488" x2="0.125" y2="1.86190625" width="0.15" layer="1"/>
+<wire x1="0.9525" y1="1.0475" x2="0.4512" y2="1.5488" width="0.15" layer="1"/>
+<wire x1="0.125" y1="1.86190625" x2="0.125" y2="5" width="0.15" layer="1"/>
 </signal>
 <signal name="PMC_UART_TX">
@@
 <wire x1="11.75" y1="17.5" x2="11.75" y2="16.625" width="0.15" layer="1"/>
 <wire x1="48.375" y1="14.875" x2="54.5" y2="8.75" width="0.15" layer="1"/>
-<wire x1="54.5" y1="8.75" x2="54.875" y2="8.75" width="0.15" layer="1"/>
-<via x="54.875" y="8.75" extent="1-16" drill="0.3"/>
-<wire x1="54.875" y1="8.75" x2="54.125" y2="8" width="0.15" layer="16"/>
-<via x="54.125" y="8" extent="1-16" drill="0.3"/>
-<wire x1="54.125" y1="1.875" x2="55" y2="1" width="0.15" layer="1"/>
-<wire x1="55" y1="1" x2="55" y2="0.4225" width="0.15" layer="1"/>
+<wire x1="54.5" y1="8.75" x2="55" y2="8.75" width="0.15" layer="1"/>
+<via x="55" y="8.75" extent="1-16" drill="0.3"/>
+<wire x1="55" y1="8.75" x2="54.125" y2="7.875" width="0.15" layer="16"/>
+<via x="54.125" y="7.875" extent="1-16" drill="0.3"/>
+<wire x1="55" y1="0.4225" x2="55" y2="1" width="0.15" layer="1"/>
 <wire x1="55" y1="0.4225" x2="54.9525" y2="0.375" width="0.15" layer="1"/>
 <wire x1="11.75" y1="16.625" x2="13.5" y2="14.875" width="0.15" layer="1"/>
 <wire x1="13.5" y1="14.875" x2="48.375" y2="14.875" width="0.15" layer="1"/>
-<wire x1="54.125" y1="8" x2="54.125" y2="1.875" width="0.15" layer="1"/>
+<wire x1="54.4512" y1="1.5488" x2="54.43810625" y2="1.5488" width="0.15" layer="1"/>
+<wire x1="54.43810625" y1="1.5488" x2="54.125" y2="1.86190625" width="0.15" layer="1"/>
+<wire x1="55" y1="1" x2="54.4512" y2="1.5488" width="0.15" layer="1"/>
+<wire x1="54.125" y1="1.86190625" x2="54.125" y2="7.875" width="0.15" layer="1"/>
 </signal>
 <signal name="PMC_UART_RX">
@@
 <wire x1="8.5" y1="16.125" x2="9.25" y2="16.125" width="0.15" layer="1"/>
 <contactref element="CN8" pad="5"/>
-<wire x1="26.27" y1="-8.48" x2="26.375" y2="-8.375" width="0.15" layer="1"/>
 <wire x1="22.105" y1="-5.44" x2="24.045" y2="-3.5" width="0.5" layer="1"/>
 <wire x1="24.045" y1="-3.5" x2="26.375" y2="-3.5" width="0.5" layer="1"/>
