File: debug.sch (EAGLE design)
At the start: 24 parts, among them CN1 2X10 HEADER, CN2 MICRO USB B, CN3 14 PIN 2mm, CN4 MICRO USB B, CN5 2X10 HEADER, CN6 31 PIN FPC, U1 USBLC6-2SC6, U2 USBLC6-2SC6, U3 FT231X, U7 FT231X

Commit message: Thumb button connected to wakeup, diff pair lengths fixed
Parts:
- removed CN6: 31 PIN FPC, CONNECTORs:3-1734839-1
- removed R3: 10R, r_0603:CRCW060310R0FKTA
- added Q1, Q2: MMBT3904, TRANSISTORs:MMBT3904-7-F
- added R5: 10k, r_0603:ERJ3EKF1002V
- C10, C2: FARNELL 1845734 -> (none)
- CN3: value 14 PIN 2mm -> 50 PIN 0.5MM; device CONNECTORs:0878331420 -> CONNECTORs:FH52E-50S-0.5SH
- R4: value 10R -> 10k; device r_0603:CRCW060310R0FKTA -> r_0603:ERJ3EKF1002V
Connections:
- net N$13 renamed USB_VBUS
- removed net DEBUG_GPIO_0: CN6.30
- removed net FPGA_JTAG_NRESET: CN3.13, CN6.6
- removed net FPGA_TCK: CN3.5, CN6.2
- removed net FPGA_TDI: CN3.9, CN6.5
- removed net FPGA_TDO: CN3.7, CN6.4
- removed net FPGA_TMS: CN3.3, CN6.3
- removed net N$15: R3.1, U3.TXD
- removed net N$16: R4.1, U3.RXD
- removed net STP_UART_RX: CN6.26, R3.2
- removed net STP_UART_TX: CN6.25, R4.2
- new net BMS_I2C_SCL: CN3.P25
- new net BMS_I2C_SDA: CN3.P24
- new net BMS_NINT: CN3.P23
- new net DEBUG_UART_RX: CN3.P34
- new net DEBUG_UART_TX: CN3.P35
- new net ESP32_EN: CN3.P28, Q1.C
- new net ESP32_UART_!DTR: Q2.E, R4.2, U3.!DTR
- new net ESP32_UART_!RTS: Q1.E, R5.2, U3.!RTS
- new net ESP32_UART_RX: CN3.P30, U3.TXD
- new net ESP32_UART_TX: CN3.P29, U3.RXD
- new net ESP_IO0: CN3.P31, Q2.C
- new net FPGA_GPIO_0: CN3.P9
- new net FPGA_GPIO_1: CN3.P12
- new net FPGA_GPIO_2: CN3.P14
- new net FPGA_GPIO_3: CN3.P10
- new net FPGA_GPIO_4: CN3.P13
- new net FPGA_GPIO_5: CN3.P11
- new net FPGA_GPIO_6: CN3.P15
- new net FPGA_JTAG_TCK: CN3.P47
- new net FPGA_JTAG_TDI: CN3.P48
- new net FPGA_JTAG_TDO: CN3.P46
- new net FPGA_JTAG_TMS: CN3.P49
- new net N$100: Q2.B, R5.1
- new net N$99: Q1.B, R4.1
- new net PMC_UART_RX: CN3.P3
- new net PMC_UART_TX: CN3.P2
- new net PSS_JTAG_MOD: CN3.P41
- new net PSS_JTAG_NTRST: CN3.P40
- new net PSS_JTAG_TCK: CN3.P42
- new net PSS_JTAG_TDI: CN3.P39
- new net PSS_JTAG_TDO: CN3.P38
- new net PSS_JTAG_TMS: CN3.P43
- new net PWR_DIG_1V8: CN3.P16, CN3.P45
- new net PWR_PSS_DCDC_1V8: CN3.P33, CN3.P37
- new net PWR_SYS_1V8_SLP: CN3.P7
- net FPGA_DEBUG_CLK: no longer CN6.13
- net FPGA_DEBUG_D0: no longer CN6.15
- net FPGA_DEBUG_D1: no longer CN6.16
- net FPGA_DEBUG_D2: no longer CN6.17
- net FPGA_DEBUG_D3: no longer CN6.18
- net FPGA_DEBUG_D4: no longer CN6.19
- net FPGA_DEBUG_D5: no longer CN6.20
- net FPGA_DEBUG_D6: no longer CN6.21
- net FPGA_DEBUG_D7: no longer CN6.22
- net FPGA_DEBUG_EN: no longer CN6.14
- net FPGA_UART_RX: no longer CN6.9
- net FPGA_UART_TX: no longer CN6.10
- net GND: now also CN3.GND, CN3.P1, CN3.P17, CN3.P26, CN3.P32, CN3.P36, CN3.P44, CN3.P50, CN3.P8; no longer CN3.10, CN3.12, CN3.14, CN3.2, CN3.4, CN3.6, CN3.8, CN6.12, CN6.23, CN6.29, CN6.7, CN6.8
- net PWR_3V3_SLP: no longer C6.2, CN6.24, U3.VCCIO
- net PWR_FPGA_1V8: no longer CN6.11
- net PWR_SYS_3V3: now also C6.2, CN3.P27, U3.!RESET, U3.VCCIO; no longer CN3.1, CN6.1
- net STP_NRESET: now also CN3.P6; no longer CN6.31
- net STP_SWCLK: now also CN3.P5; no longer CN6.28
- net STP_SWDIO: now also CN3.P4; no longer CN6.27
Other:
- moved on the sheet: C1, C10, C13, C2, C3, C4, C5, C6, CN1, CN2, CN4, CN5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

Commit message: SRST added to the debug port
Parts:
- removed C13: 0.1uF 16V, c_0603:C0603C104K4RACTU
- removed U7: FT231X, ICs:FT231X
- added C11, C12, C7, C8: 0.1uF 16V, c_0603:CL10B104KO8WPNC
- added C9: 0.1uF 16V, c_0603:C0603C104K4RACTU
- added CN6, CN7: MICRO USB B, CONNECTORs:ZX62-B-5PA(33)
- added CN8: 2X4_HEADER, CONNECTORs:2X4_HEADER
- added D1: RED LED, OPTO:150060RS75000
- added FB3: 150R 100MHz, INDUCTORS:ILB1206ER151V
- added Q3: 2N7002, TRANSISTORs:2N7002P,215
- added U4, U6: FT231X, ICs:FT231X
- added U5: USBLC6-2SC6, ICs:USBLC6-2SC6
- C4: device c_0603:CL10B104KO8WPNC -> c_0603:C0603C104K4RACTU
- C5: value 0.1uF 16V -> 2.2uF 25V; device c_0603:CL10B104KO8WPNC -> CAPACITORS:GRM188R61E225KA12D; PRICE_PER (none) -> 0.0832; VALUE (none) -> 2.2uF 25V
- CN2: value MICRO USB B -> JTAG PROG; device CONNECTORs:ZX62-B-5PA(33) -> CONNECTORs:XILINXJTAG
- R1, R2: value 10R -> 4.7k; device r_0603:CRCW060310R0FKTA -> r_0603:CRCW06034K70FKEA
Connections:
- net PSS_JTAG_TMS renamed FPGA_NPROG
- net STP_NRESET renamed PMC_NRESET
- net STP_SWCLK renamed PMC_SWCLK
- net STP_SWDIO renamed PMC_SWDIO
- removed net DEBUG_UART_RX: CN3.P34
- removed net DEBUG_UART_TX: CN3.P35
- removed net FPGA_GPIO_0: CN3.P9
- removed net FPGA_GPIO_1: CN3.P12
- removed net FPGA_GPIO_2: CN3.P14
- removed net FPGA_GPIO_3: CN3.P10
- removed net FPGA_GPIO_4: CN3.P13
- removed net FPGA_GPIO_5: CN3.P11
- removed net FPGA_GPIO_6: CN3.P15
- removed net FPGA_UART_RX: R1.2
- removed net FPGA_UART_TX: R2.2
- removed net N$25: CN2.5V, FB1.1
- removed net N$28: CN2.D-, U2.D-_IN
- removed net PSS_JTAG_MOD: CN3.P41
- removed net PSS_JTAG_NTRST: CN3.P40
- removed net PSS_JTAG_TCK: CN3.P42
- removed net PSS_JTAG_TDI: CN3.P39
- removed net PSS_JTAG_TDO: CN3.P38
- removed net PWR_3V3_SLP: CN1.1
- removed net PWR_DIG_1V8: CN3.P16, CN3.P45
- removed net PWR_FPGA_1V8: C5.2, U7.VCCIO
- removed net PWR_PSS_DCDC_1V8: CN3.P33, CN3.P37
- new net FPGA_DONE: CN3.P45, Q3.G, R1.1
- new net FPGA_NINIT: CN3.P44
- new net FPGA_PS_NSRST: CN2.PS_NSRST, CN3.P24
- new net FPGA_STATUS_D0: CN3.P28
- new net FPGA_STATUS_D1: CN3.P27
- new net FPGA_STATUS_D2: CN3.P26
- new net N$14: Q3.D, R2.1
- new net N$15: U2.D+_OUT, U4.D+
- new net N$16: CN7.D-, U5.D-_IN
- new net N$17: C10.2, U6.3V3OUT
- new net N$18: U5.D-OUT, U6.D-
- new net N$19: U5.D+_OUT, U6.D+
- new net N$22: D1.K, R2.2
- new net PSS_DEBUG_UART_RX: CN3.P22, U4.TXD
- new net PSS_DEBUG_UART_TX: CN3.P21, U4.RXD
- new net PWR_SYS_1V8: C8.2, CN3.P20, U4.!RESET, U4.VCCIO
- new net USB_VBUS1: C4.2, C7.2, FB1.2, U2.VBUS, U4.VCC
- new net USB_VBUS2: C11.2, C9.2, FB3.2, U5.VBUS, U6.VCC
- net BMS_I2C_SCL: now also CN3.P10, CN8.6; no longer CN3.P25
- net BMS_I2C_SDA: now also CN3.P11, CN8.7; no longer CN3.P24
- net BMS_NINT: now also CN3.P12, CN8.8; no longer CN3.P23
- net ESP32_EN: now also CN3.P15; no longer CN3.P28
- net ESP32_UART_RX: now also CN3.P17; no longer CN3.P30
- net ESP32_UART_TX: now also CN3.P16; no longer CN3.P29
- net ESP_IO0: now also CN3.P18; no longer CN3.P31
- net FPGA_DEBUG_CLK: now also CN3.P31, CN5.1; no longer CN5.10
- net FPGA_DEBUG_D0: now also CN3.P40, CN5.10; no longer CN5.8
- net FPGA_DEBUG_D1: now also CN3.P39, CN5.9; no longer CN5.7
- net FPGA_DEBUG_D2: now also CN3.P38, CN5.8; no longer CN5.6
- net FPGA_DEBUG_D3: now also CN3.P37, CN5.7; no longer CN5.5
- net FPGA_DEBUG_D4: now also CN3.P36, CN5.6; no longer CN5.4
- net FPGA_DEBUG_D5: now also CN3.P35, CN5.5; no longer CN5.3
- net FPGA_DEBUG_D6: now also CN3.P34, CN5.4; no longer CN5.2
- net FPGA_DEBUG_D7: now also CN3.P33, CN5.3; no longer CN5.1
- net FPGA_DEBUG_EN: now also CN3.P32, CN5.2; no longer CN5.9
- net FPGA_JTAG_TCK: now also CN2.TCK
- net FPGA_JTAG_TDI: now also CN2.TDI
- net FPGA_JTAG_TDO: now also CN2.TDO
- net FPGA_JTAG_TMS: now also CN2.TMS
- net GND: now also C11.1, C12.1, C7.1, C8.1, C9.1, CN3.P13, CN3.P19, CN3.P25, CN3.P29, CN3.P41, CN6.GND, CN7.GND, CN8.1, CN8.2, CN8.3, CN8.4, Q3.S, U4.GND, U5.GND, U6.GND; no longer C13.1, CN3.P17, CN3.P26, CN3.P32, CN3.P36, CN3.P44, U7.GND
- net N$1: now also CN6.5V, FB1.1; no longer CN2.D+, U2.D+_IN
- net N$2: now also CN6.D+, U2.D+_IN; no longer U2.D+_OUT, U7.D+
- net N$3: now also CN7.5V, FB3.1; no longer U2.D-OUT, U7.D-
- net N$4: now also CN7.D+, U5.D+_IN; no longer C13.2, C4.2, FB1.2, U2.VBUS, U7.VCC
- net N$5: now also CN6.D-, U2.D-_IN; no longer C10.2, U7.3V3OUT
- net N$6: now also C5.2, U4.3V3OUT; no longer R1.1, U7.TXD
- net N$7: now also U2.D-OUT, U4.D-; no longer R2.1, U7.RXD
- net PMC_UART_RX: now also U6.TXD
- net PMC_UART_TX: now also U6.RXD
- net PWR_SYS_1V8_SLP: now also C12.2, CN1.1, CN3.P9, CN8.5, U6.!RESET, U6.VCCIO
- net PWR_SYS_3V3: now also CN2.VREF, CN3.P14, CN3.P30, CN3.P42, D1.A, R1.2; no longer CN3.P27
Other:
- moved on the sheet: C1, C10, C2, C3, C4, C5, C6, CN1, CN3, CN4, CN5, FB1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

Commit message: Debug and power board ready for outputs
Other:
- note added: "2023.07.25 - GSWDH LTD. CAMERA DEBUG PCB REVISION 1.0.0 DESIGN BY GEORGE WALLER, GSWDH LTD. GEORGEWALLER@GSWDH.CO.UK CONFIDENTIAL. FOR THE INTENDED READER ONLY."
- note removed: "YYYY.MM.DD - GSWDH LTD. CAMERA MAIN PCB REVISION 1.x.x DESIGN BY GEORGE WALLER, GSWDH LTD. GEORGEWALLER@GSWDH.CO.UK CONFIDENTIAL. FOR THE INTENDED READER ONLY."
Changed lines of the file:
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@@
 <description>TITLE</description>
 <plain>
-<text x="0" y="0" size="7.62" layer="97" font="vector" align="center">YYYY.MM.DD - GSWDH LTD.
-CAMERA MAIN PCB
-REVISION 1.x.x
+<text x="0" y="0" size="7.62" layer="97" font="vector" align="center">2023.07.25 - GSWDH LTD.
+CAMERA DEBUG PCB
+REVISION 1.0.0
 DESIGN BY GEORGE WALLER, GSWDH LTD.
 GEORGEWALLER@GSWDH.CO.UK
