File: main.sch (EAGLE design)
At the start: 562 parts, among them CN1 50 PIN 0.5MM, CN2 10067847-001RLF, CN3 632723300011, CN4 FF0881SA1, CN5 15PIN 0.5MM, CN6 31 PIN FPC, Q1 2N7002, Q2 FDN302P, Q3 2N7002, Q5 SI7489DP, SW2 TACT, SW3 TACT, SW4 TACT, SW5 TACT, SW7 TACT, SW8 SLIDE SPDT, U1 GMAX0505-DV, U10 TPS70950, U11 FT601Q, U12 CBTU02043, U13 MAX25300B, U14 ESP32, U15 MAX25300B, U16 INA180, U17 AP62301, U18 AP62301, U19 SCHMITT, U2 XC7Z014S-1CLG484C, U20 MAX25300B, U21 NOT, U22 MAX25300B, U23 SN74LVC1G3, U24 NAND, U25 EMC1812T, U26 BIPOLAR HALL, U27 LM2663, U28 ADS7867, U29 LM2663, U3 IS43TR16128CL-125KBLI, U30 LM2731X, U31 USBLC6-2SC6, U32 MAX1735, U33 MP2148, U34 TPS22917, U35 AP62301, U36 TLV61046A, U37 W25Q128JV, U38 TPS70918, U39 AP62301, U4 AP63300WU-7, U5 STM32L431RBT, U6 USB ESD, U7 ACT2861QI301-T, U8 TPS70918, U9 STUSB4500

Commit message: DDR3 length matched
Other:
- moved on the sheet: C62, C72, OSC1, R174, R175, R177, R97, R98, U37

Commit message: Some pullups added
Parts:
- added D15: BAT54S, DIODES:BAT54S-7-F
- added R103: 10k, r_0402:RC0402FR-0710KL
- added R105, R178, R179, R180, R181, R182: 2.2k, r_0402:RC0402FR-072K2L
- C154: value 1uF 25V -> 1uF 6.3V; device CAPACITORS:CL10A105KA8NNNC -> c_0402:C0402C105K9PACTU
- R85: value 26.7k -> 28k; device r_0603:CRCW060326K7FKEB -> r_0402:RC0402FR-0728KL
- R86: device r_0603:CRCW06032K00FKTA -> r_0402:RC0402FR-072KL
Connections:
- removed net N$134: U5.PB13
- net ACT_I2C_SCL: now also R179.1
- net ACT_I2C_SDA: now also R180.1
- net BMS_I2C_SCL: now also R105.1
- net BMS_I2C_SDA: now also R178.1
- net GND: now also D15.A, R103.1
- net MON_SYS_BUS_V: now also D15.AK
- net PSS_I2C_SCL: now also R182.1
- net PSS_I2C_SDA: now also R181.1
- net PWR_SYS_1V8: now also R181.2, R182.2
- net PWR_SYS_1V8_SLP: now also D15.K, R105.2, R178.2, R179.2, R180.2
- net STUSB_RESET: now also R103.2
Other:
- moved on the sheet: C154, R174, R175, R177, R85, R86, R98

Commit message: Clock for FTDI fixed and SD status pins moved
Parts:
- added R183, R184, R185, R186: 10k, r_0402:RC0402FR-0710KL
Connections:
- new net N$19: U2.IO_L13N_T2_MRCC_34
- new net N$31: U2.IO_L13P_T2_MRCC_34
- net BTN_BTMLEFT: now also R183.1
- net BTN_BTMRIGHT: now also R186.1
- net BTN_TOPLEFT: now also R185.1
- net BTN_TOPRIGHT: now also R184.1
- net FT_CLK: now also U2.IO_L11P_T1_SRCC_13; no longer U2.IO_L17P_T2_13
- net FT_D14: now also U2.IO_L11N_T1_SRCC_13; no longer U2.IO_L11P_T1_SRCC_13
- net FT_NOE: now also U2.IO_L17P_T2_13; no longer U2.IO_L11N_T1_SRCC_13
- net PSS_SD_CD: now also U2.IO_L6P_T0_13; no longer U2.PS_MIO34_501
- net PSS_SD_WP: now also U2.IO_L6N_T0_VREF_13; no longer U2.PS_MIO37_501
- net PWR_SYS_1V8: now also R186.2
- net PWR_SYS_3V3: now also R183.2, R184.2, R185.2
- net SEN_B_D12_N: now also U2.IO_L21N_T3_DQS_34; no longer U2.IO_L14N_T2_SRCC_34
- net SEN_B_D12_P: now also U2.IO_L21P_T3_DQS_34; no longer U2.IO_L14P_T2_SRCC_34
- net SEN_CLK_N: now also U2.IO_L14N_T2_SRCC_34; no longer U2.IO_L21N_T3_DQS_34
- net SEN_CLK_P: now also U2.IO_L14P_T2_SRCC_34; no longer U2.IO_L21P_T3_DQS_34

Commit message: DDR3 FPGA VRP/N pins fixed, pullups on the buttons corrected
Connections:
- net BTN_BTMLEFT: now also U2.PS_MIO33_501; no longer U2.PS_MIO0_500
- net BTN_TOPLEFT: now also U2.PS_MIO0_500; no longer U2.PS_MIO33_501
- net GND: now also R2.2; no longer R1.1
- net PWR_DDR3_1V35: now also R1.1; no longer R2.2
- net PWR_SYS_1V8: now also R183.2, R184.2; no longer R186.2
- net PWR_SYS_3V3: now also R186.2; no longer R183.2, R184.2
Other:
- moved on the sheet: R1, R2
Changed lines of the file:
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@@
 <attribute name="VALUE" x="-144.78" y="15.24" size="1.778" layer="96" align="center"/>
 </instance>
-<instance part="R1" gate="G$1" x="127" y="63.5" smashed="yes" rot="R90">
-<attribute name="NAME" x="124.46" y="63.5" size="1.27" layer="95" rot="R90" align="center"/>
-<attribute name="VALUE" x="129.54" y="63.5" size="1.27" layer="96" rot="R90" align="center"/>
-</instance>
-<instance part="R2" gate="G$1" x="127" y="81.28" smashed="yes" rot="R90">
-<attribute name="NAME" x="124.46" y="81.28" size="1.27" layer="95" rot="R90" align="center"/>
-<attribute name="VALUE" x="129.54" y="81.28" size="1.27" layer="96" rot="R90" align="center"/>
+<instance part="R1" gate="G$1" x="127" y="78.74" smashed="yes" rot="R270">
+<attribute name="NAME" x="129.54" y="78.74" size="1.27" layer="95" rot="R270" align="center"/>
+<attribute name="VALUE" x="124.46" y="78.74" size="1.27" layer="96" rot="R270" align="center"/>
+</instance>
+<instance part="R2" gate="G$1" x="124.46" y="63.5" smashed="yes" rot="R270">
+<attribute name="NAME" x="127" y="63.5" size="1.27" layer="95" rot="R270" align="center"/>
+<attribute name="VALUE" x="121.92" y="63.5" size="1.27" layer="96" rot="R270" align="center"/>
 </instance>
-<instance part="GND12" gate="G$1" x="127" y="53.34" smashed="yes">
-<attribute name="VALUE" x="127" y="50.8" size="1.778" layer="96" align="center"/>
+<instance part="GND12" gate="G$1" x="124.46" y="53.34" smashed="yes">
+<attribute name="VALUE" x="124.46" y="50.8" size="1.778" layer="96" align="center"/>
 </instance>
 <instance part="R3" gate="G$1" x="86.36" y="83.82" smashed="yes">
@@
 </segment>
 <segment>
-<pinref part="R1" gate="G$1" pin="1"/>
-<pinref part="GND12" gate="G$1" pin="GND"/>
-<wire x1="127" y1="55.88" x2="127" y2="58.42" width="0.1524" layer="91"/>
-</segment>
-<segment>
 <pinref part="R8" gate="G$1" pin="1"/>
 <pinref part="GND19" gate="G$1" pin="GND"/>
@@
 <pinref part="C278" gate="G$1" pin="1"/>
 </segment>
+<segment>
+<pinref part="GND12" gate="G$1" pin="GND"/>
+<pinref part="R2" gate="G$1" pin="2"/>
+<wire x1="124.46" y1="58.42" x2="124.46" y2="55.88" width="0.1524" layer="91"/>
+</segment>
 </net>
 <net name="FPGA_DONE" class="0">
@@
 <pinref part="U2" gate="G$1" pin="PS_DDR_VRN_502"/>
 <wire x1="43.18" y1="71.12" x2="127" y2="71.12" width="0.1524" layer="91"/>
-<wire x1="127" y1="71.12" x2="127" y2="68.58" width="0.1524" layer="91"/>
+<wire x1="127" y1="71.12" x2="127" y2="73.66" width="0.1524" layer="91"/>
 <pinref part="R1" gate="G$1" pin="2"/>
 </segment>
@@
 <segment>
 <pinref part="U2" gate="G$1" pin="PS_DDR_VRP_502"/>
-<wire x1="43.18" y1="73.66" x2="127" y2="73.66" width="0.1524" layer="91"/>
-<wire x1="127" y1="73.66" x2="127" y2="76.2" width="0.1524" layer="91"/>
+<wire x1="43.18" y1="73.66" x2="124.46" y2="73.66" width="0.1524" layer="91"/>
+<wire x1="124.46" y1="73.66" x2="124.46" y2="68.58" width="0.1524" layer="91"/>
 <pinref part="R2" gate="G$1" pin="1"/>
 </segment>
@@
 <net name="PWR_DDR3_1V35" class="0">
 <segment>
-<pinref part="R2" gate="G$1" pin="2"/>
-<wire x1="127" y1="86.36" x2="127" y2="88.9" width="0.1524" layer="91"/>
-<wire x1="127" y1="88.9" x2="157.48" y2="88.9" width="0.1524" layer="91"/>
-<label x="129.54" y="88.9" size="1.778" layer="95"/>
+<wire x1="127" y1="86.36" x2="157.48" y2="86.36" width="0.1524" layer="91"/>
+<label x="129.54" y="86.36" size="1.778" layer="95"/>
+<pinref part="R1" gate="G$1" pin="1"/>
+<wire x1="127" y1="83.82" x2="127" y2="86.36" width="0.1524" layer="91"/>
 </segment>
 <segment>
@@
 <net name="BTN_TOPLEFT" class="0">
 <segment>
-<pinref part="U2" gate="G$1" pin="PS_MIO33_501"/>
-<wire x1="81.28" y1="-27.94" x2="43.18" y2="-27.94" width="0.1524" layer="91"/>
-<label x="45.72" y="-27.94" size="1.778" layer="95"/>
+<pinref part="U2" gate="G$1" pin="PS_MIO0_500"/>
+<wire x1="43.18" y1="60.96" x2="81.28" y2="60.96" width="0.1524" layer="91"/>
+<label x="45.72" y="60.96" size="1.778" layer="95"/>
 </segment>
 </net>
@@
 </segment>
 </net>
-<net name="BTN_BTMLEFT" class="0">
-<segment>
-<pinref part="U2" gate="G$1" pin="PS_MIO0_500"/>
-<wire x1="43.18" y1="60.96" x2="81.28" y2="60.96" width="0.1524" layer="91"/>
-<label x="45.72" y="60.96" size="1.778" layer="95"/>
-</segment>
-</net>
 <net name="EVF_I2C_SCL" class="0">
 <segment>
@@
 </segment>
 </net>
+<net name="BTN_BTMLEFT" class="0">
+<segment>
+<pinref part="U2" gate="G$1" pin="PS_MIO33_501"/>
+<wire x1="81.28" y1="-27.94" x2="43.18" y2="-27.94" width="0.1524" layer="91"/>
+<label x="45.72" y="-27.94" size="1.778" layer="95"/>
+</segment>
+</net>
 </nets>
 </sheet>
@@
 </segment>
 <segment>
+<label x="134.62" y="30.48" size="1.778" layer="95"/>
 <pinref part="R185" gate="G$1" pin="2"/>
+<wire x1="104.14" y1="30.48" x2="116.84" y2="30.48" width="0.1524" layer="91"/>
+<wire x1="116.84" y1="30.48" x2="165.1" y2="30.48" width="0.1524" layer="91"/>
 <wire x1="104.14" y1="17.78" x2="104.14" y2="30.48" width="0.1524" layer="91"/>
-<wire x1="104.14" y1="30.48" x2="165.1" y2="30.48" width="0.1524" layer="91"/>
-<pinref part="R184" gate="G$1" pin="2"/>
-<wire x1="91.44" y1="17.78" x2="91.44" y2="30.48" width="0.1524" layer="91"/>
-<wire x1="91.44" y1="30.48" x2="104.14" y2="30.48" width="0.1524" layer="91"/>
-<junction x="104.14" y="30.48"/>
-<pinref part="R183" gate="G$1" pin="2"/>
-<wire x1="78.74" y1="17.78" x2="78.74" y2="30.48" width="0.1524" layer="91"/>
-<wire x1="78.74" y1="30.48" x2="91.44" y2="30.48" width="0.1524" layer="91"/>
-<junction x="91.44" y="30.48"/>
-<label x="134.62" y="30.48" size="1.778" layer="95"/>
+<pinref part="R186" gate="G$1" pin="2"/>
+<wire x1="116.84" y1="17.78" x2="116.84" y2="30.48" width="0.1524" layer="91"/>
+<junction x="116.84" y="30.48"/>
 </segment>
 </net>
@@
 </segment>
 <segment>
-<pinref part="R186" gate="G$1" pin="2"/>
-<wire x1="116.84" y1="17.78" x2="116.84" y2="27.94" width="0.1524" layer="91"/>
-<wire x1="116.84" y1="27.94" x2="165.1" y2="27.94" width="0.1524" layer="91"/>
+<wire x1="78.74" y1="27.94" x2="91.44" y2="27.94" width="0.1524" layer="91"/>
 <label x="134.62" y="27.94" size="1.778" layer="95"/>
+<pinref part="R183" gate="G$1" pin="2"/>
+<wire x1="91.44" y1="27.94" x2="165.1" y2="27.94" width="0.1524" layer="91"/>
+<wire x1="78.74" y1="17.78" x2="78.74" y2="27.94" width="0.1524" layer="91"/>
+<pinref part="R184" gate="G$1" pin="2"/>
+<wire x1="91.44" y1="17.78" x2="91.44" y2="27.94" width="0.1524" layer="91"/>
+<junction x="91.44" y="27.94"/>
 </segment>
 </net>

Commit message: Rev 1.0.0 ready for release
Other:
- note added: "2023.07.25 - GSWDH LTD. CAMERA MAIN PCB REVISION 1.0.0 DESIGN BY GEORGE WALLER, GSWDH LTD. GEORGEWALLER@GSWDH.CO.UK CONFIDENTIAL. FOR THE INTENDED READER ONLY."
- note removed: "YYYY.MM.DD - GSWDH LTD. CAMERA MAIN PCB REVISION 1.x.x DESIGN BY GEORGE WALLER, GSWDH LTD. GEORGEWALLER@GSWDH.CO.UK CONFIDENTIAL. FOR THE INTENDED READER ONLY."
Changed lines of the file:
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@@
 <description>TITLE</description>
 <plain>
-<text x="0" y="0" size="7.62" layer="97" font="vector" align="center">YYYY.MM.DD - GSWDH LTD.
+<text x="0" y="0" size="7.62" layer="97" font="vector" align="center">2023.07.25 - GSWDH LTD.
 CAMERA MAIN PCB
-REVISION 1.x.x
+REVISION 1.0.0
 DESIGN BY GEORGE WALLER, GSWDH LTD.
 GEORGEWALLER@GSWDH.CO.UK

Commit message: SRST added to the debug port
Connections:
- net PSS_NSRST: now also CN1.P27
Changed lines of the file:
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@@
+</segment>
+</net>
+<net name="PSS_NSRST" class="0">
+<segment>
+<pinref part="CN1" gate="G$1" pin="P27"/>
+<wire x1="15.24" y1="-5.08" x2="48.26" y2="-5.08" width="0.1524" layer="91"/>
+<label x="20.32" y="-5.08" size="1.778" layer="95"/>
 </segment>
 </net>

Commit message: Correct FPGA footprint routed. A lot of work to length match, optimise and review
Parts:
- removed C124, C126: 0.1uF 10V, c_0402:0402ZC104KAT2A
- C104, C123: value 0.1uF 10V -> 47uF 6.3V; device c_0402:0402ZC104KAT2A -> c_0603:06036D476MAT2A
Connections:
- removed net N$19: U2.IO_L13N_T2_MRCC_34
- removed net N$31: U2.IO_L13P_T2_MRCC_34
- net DDR_D0: now also U2.PS_DDR_DQ5_502; no longer U2.PS_DDR_DQ4_502
- net DDR_D2: now also U2.PS_DDR_DQ8_502; no longer U2.PS_DDR_DQ9_502
- net DDR_D4: now also U2.PS_DDR_DQ11_502; no longer U2.PS_DDR_DQ10_502
- net DDR_D6: now also U2.PS_DDR_DQ10_502; no longer U2.PS_DDR_DQ11_502
- net DDR_D8: now also U2.PS_DDR_DQ9_502; no longer U2.PS_DDR_DQ8_502
- net DDR_D9: now also U2.PS_DDR_DQ4_502; no longer U2.PS_DDR_DQ5_502
- net FT_BE0: now also U2.IO_L21N_T3_DQS_13; no longer U2.IO_L20N_T3_13
- net FT_BE1: now also U2.IO_L22P_T3_13; no longer U2.IO_L13N_T2_MRCC_13
- net FT_BE3: now also U2.IO_L22N_T3_13; no longer U2.IO_L21P_T3_DQS_13
- net FT_D0: now also U2.IO_L7P_T1_13; no longer U2.IO_L7N_T1_13
- net FT_D1: now also U2.IO_L7N_T1_13; no longer U2.IO_L7P_T1_13
- net FT_D10: now also U2.IO_L3N_T0_DQS_13; no longer U2.IO_L1P_T0_13
- net FT_D11: now also U2.IO_L9P_T1_DQS_13; no longer U2.IO_L10N_T1_13
- net FT_D12: now also U2.IO_L10N_T1_13; no longer U2.IO_L9P_T1_DQS_13
- net FT_D24: now also U2.IO_L20N_T3_13; no longer U2.IO_L21N_T3_DQS_13
- net FT_D29: now also U2.IO_L19N_T3_VREF_13; no longer U2.IO_0_13
- net FT_D3: now also U2.IO_L8P_T1_13; no longer U2.IO_L8N_T1_13
- net FT_D30: now also U2.IO_0_13; no longer U2.IO_L19N_T3_VREF_13
- net FT_D4: now also U2.IO_L8N_T1_13; no longer U2.IO_L8P_T1_13
- net FT_D6: now also U2.IO_L4P_T0_13; no longer U2.IO_L5P_T0_13
- net FT_D7: now also U2.IO_L5P_T0_13; no longer U2.IO_L4P_T0_13
- net FT_GPIO0: now also U2.IO_L2N_T0_13; no longer U2.IO_L2P_T0_13
- net FT_GPIO1: now also U2.IO_L1P_T0_13; no longer U2.IO_L3N_T0_DQS_13
- net FT_NRESET: now also U2.IO_L2P_T0_13; no longer U2.IO_L12N_T1_MRCC_13
- net FT_NSIWU: now also U2.IO_L13N_T2_MRCC_13; no longer U2.IO_L22P_T3_13
- net FT_NTXE: now also U2.IO_L21P_T3_DQS_13; no longer U2.IO_L22N_T3_13
- net FT_NWAKEUP: now also U2.IO_L12N_T1_MRCC_13; no longer U2.IO_L2N_T0_13
- net GND: no longer C124.1, C126.1
- net PWR_ANA_1V8: no longer C104.2
- net PWR_DDR3_1V35: now also C104.2, C123.2
- net PWR_SEN_0V7_EN: now also U2.PS_MIO36_501; no longer U2.PS_MIO47_501
- net PWR_SEN_N1V3A_EN: now also U2.PS_MIO47_501; no longer U2.PS_MIO36_501
- net PWR_SYS_1V8: no longer C123.2, C124.2, C126.2
Other:
- moved on the sheet: C104, C105, C123, C125, C127, C128, C129, C130

Commit message: button ADC is not attached to FPGA fabric
Connections:
- new net BADC_SPI_MISO: U2.IO_L18N_T2_34, U28.SDO
- new net BADC_SPI_NCS: U2.IO_L18P_T2_34, U28.!CS
- new net BADC_SPI_SCLK: U2.IO_L22P_T3_34, U28.SCLK
- net ADC_SPI_NCS: no longer U28.!CS
- net PSS_SPI_MISO: no longer U28.SDO
- net PSS_SPI_SCLK: no longer U28.SCLK
Changed lines of the file:
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@@
 </segment>
 </net>
+<net name="BADC_SPI_NCS" class="0">
+<segment>
+<pinref part="U2" gate="G$1" pin="IO_L18P_T2_34"/>
+<wire x1="-43.18" y1="-93.98" x2="-81.28" y2="-93.98" width="0.1524" layer="91"/>
+<label x="-78.74" y="-93.98" size="1.778" layer="95"/>
+</segment>
+</net>
+<net name="BADC_SPI_SCLK" class="0">
+<segment>
+<pinref part="U2" gate="G$1" pin="IO_L22P_T3_34"/>
+<wire x1="-43.18" y1="-114.3" x2="-81.28" y2="-114.3" width="0.1524" layer="91"/>
+<label x="-78.74" y="-114.3" size="1.778" layer="95"/>
+</segment>
+</net>
+<net name="BADC_SPI_MISO" class="0">
+<segment>
+<pinref part="U2" gate="G$1" pin="IO_L18N_T2_34"/>
+<wire x1="-43.18" y1="-91.44" x2="-81.28" y2="-91.44" width="0.1524" layer="91"/>
+<label x="-78.74" y="-91.44" size="1.778" layer="95"/>
+</segment>
+</net>
 </nets>
 </sheet>
@@
 <pinref part="CN6" gate="G$1" pin="12"/>
 </segment>
-<segment>
-<pinref part="U28" gate="G$1" pin="SCLK"/>
-<wire x1="180.34" y1="-76.2" x2="154.94" y2="-76.2" width="0.1524" layer="91"/>
-<label x="157.48" y="-76.2" size="1.778" layer="95"/>
-</segment>
 </net>
 <net name="PSS_SPI_MOSI" class="0">
@@
 </segment>
 </net>
-<net name="ADC_SPI_NCS" class="0">
-<segment>
-<pinref part="U28" gate="G$1" pin="!CS"/>
-<wire x1="180.34" y1="-73.66" x2="154.94" y2="-73.66" width="0.1524" layer="91"/>
-<label x="157.48" y="-73.66" size="1.778" layer="95"/>
-</segment>
-</net>
-<net name="PSS_SPI_MISO" class="0">
-<segment>
-<pinref part="U28" gate="G$1" pin="SDO"/>
-<wire x1="180.34" y1="-78.74" x2="154.94" y2="-78.74" width="0.1524" layer="91"/>
-<label x="157.48" y="-78.74" size="1.778" layer="95"/>
-</segment>
-</net>
 <net name="BMS_NINT" class="0">
 <segment>
@@
 </segment>
 </net>
+<net name="BADC_SPI_NCS" class="0">
+<segment>
+<pinref part="U28" gate="G$1" pin="!CS"/>
+<wire x1="187.96" y1="-73.66" x2="154.94" y2="-73.66" width="0.1524" layer="91"/>
+<label x="157.48" y="-73.66" size="1.778" layer="95"/>
+</segment>
+</net>
+<net name="BADC_SPI_SCLK" class="0">
+<segment>
+<pinref part="U28" gate="G$1" pin="SCLK"/>
+<wire x1="187.96" y1="-76.2" x2="154.94" y2="-76.2" width="0.1524" layer="91"/>
+<label x="157.48" y="-76.2" size="1.778" layer="95"/>
+</segment>
+</net>
+<net name="BADC_SPI_MISO" class="0">
+<segment>
+<pinref part="U28" gate="G$1" pin="SDO"/>
+<wire x1="187.96" y1="-78.74" x2="154.94" y2="-78.74" width="0.1524" layer="91"/>
+<label x="157.48" y="-78.74" size="1.778" layer="95"/>
+</segment>
+</net>
