File: main.sch (EAGLE design)
At the start: 572 parts, among them CN1 50 PIN 0.5MM, CN2 10067847-001RLF, CN3 632723300011, CN4 FF0881SA1, CN5 15PIN 0.5MM, CN6 31 PIN FPC, Q1 2N7002, Q2 FDN302P, Q3 2N7002, Q5 SI7489DP, SW2 TACT, SW3 TACT, SW4 TACT, SW5 TACT, SW7 TACT, SW8 SLIDE SPDT, U1 GMAX0505-DV, U10 TPS70950, U11 FT601Q, U12 CBTU02043, U13 MAX25300B, U14 ESP32, U15 MAX25300B, U16 INA180, U17 AP62301, U18 AP62301, U19 SCHMITT, U2 XC7Z014S-1CLG484C, U20 MAX25300B, U21 NOT, U22 MAX25300B, U23 SN74LVC1G3, U24 NAND, U25 EMC1812T, U26 BIPOLAR HALL, U27 LM2663, U28 ADS7867, U29 LM2663, U3 IS43TR16128CL-125KBLI, U30 LM2731X, U31 USBLC6-2SC6, U32 MAX1735, U33 MP2148, U34 TPS22917, U35 AP62301, U36 TLV61046A, U37 W25Q128JV, U38 TPS70918, U39 AP62301, U4 AP63300WU-7, U5 STM32L431RBT, U6 USB ESD, U7 ACT2861QI301-T, U8 TPS70918, U9 STUSB4500

Commit message: Updated schematic front page
Other:
- note added: "2023.09.01 - GSWDH LTD. CAMERA MAIN PCB REVISION 1.1.0 DESIGN BY GEORGE WALLER, GSWDH LTD. GEORGEWALLER@GSWDH.CO.UK CONFIDENTIAL. FOR THE INTENDED READER ONLY."
- note removed: "2023.07.25 - GSWDH LTD. CAMERA MAIN PCB REVISION 1.0.0 DESIGN BY GEORGE WALLER, GSWDH LTD. GEORGEWALLER@GSWDH.CO.UK CONFIDENTIAL. FOR THE INTENDED READER ONLY."
Changed lines of the file:
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@@
 <description>TITLE</description>
 <plain>
-<text x="0" y="0" size="7.62" layer="97" font="vector" align="center">2023.07.25 - GSWDH LTD.
+<text x="0" y="0" size="7.62" layer="97" font="vector" align="center">2023.09.01 - GSWDH LTD.
 CAMERA MAIN PCB
-REVISION 1.0.0
+REVISION 1.1.0
 DESIGN BY GEORGE WALLER, GSWDH LTD.
 GEORGEWALLER@GSWDH.CO.UK

Commit message: Added extra decoupling to the PLL PSU
Parts:
- removed MECH3, MECH4: 6mm x 3mm, MISC:MOUNTHOLE
- added C124: 47uF 6.3V, c_0603:06036D476MAT2A
Connections:
- net GND: now also C124.1
- net PWR_ANA_1V8: now also C124.2
Changed lines of the file:
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@@
 <part name="SW7" library="ELECTROMECH" deviceset="PTS830GM140_SMTR_LFS" device="" value="TACT"/>
 <part name="GND363" library="NETS" deviceset="GND" device=""/>
-<part name="MECH3" library="MISC" deviceset="MOUNTHOLE" device="" value="6mm x 3mm"/>
-<part name="MECH4" library="MISC" deviceset="MOUNTHOLE" device="" value="6mm x 3mm"/>
 <part name="U2" library="ICs" deviceset="XC7Z014S-1" device="CLG484C" value="XC7Z014S-1CLG484C"/>
 <part name="U3" library="ICs" deviceset="IS43TR16128CL-125KBLI" device="" value="IS43TR16128CL-125KBLI"/>
@@
 <part name="C123" library="c_0603" deviceset="06036D476MAT2A" device="" value="47uF 6.3V"/>
 <part name="GND205" library="NETS" deviceset="GND" device=""/>
+<part name="C124" library="c_0603" deviceset="06036D476MAT2A" device="" value="47uF 6.3V"/>
+<part name="GND206" library="NETS" deviceset="GND" device=""/>
 </parts>
 <sheets>
@@
 <attribute name="VALUE" x="165.1" y="-99.06" size="1.778" layer="96" align="center"/>
 </instance>
+<instance part="C124" gate="G$1" x="111.76" y="-200.66" smashed="yes" rot="R90">
+<attribute name="NAME" x="109.22" y="-200.66" size="1.27" layer="95" rot="R90" align="center"/>
+<attribute name="VALUE" x="114.3" y="-200.66" size="1.27" layer="96" rot="R90" align="center"/>
+</instance>
+<instance part="GND206" gate="G$1" x="111.76" y="-210.82" smashed="yes">
+<attribute name="VALUE" x="111.76" y="-213.36" size="1.778" layer="96" align="center"/>
+</instance>
 </instances>
 <busses>
@@
 <wire x1="165.1" y1="-93.98" x2="165.1" y2="-91.44" width="0.1524" layer="91"/>
 </segment>
+<segment>
+<pinref part="C124" gate="G$1" pin="1"/>
+<pinref part="GND206" gate="G$1" pin="GND"/>
+<wire x1="111.76" y1="-208.28" x2="111.76" y2="-205.74" width="0.1524" layer="91"/>
+</segment>
 </net>
 <net name="FPGA_DONE" class="0">
@@
 <segment>
 <pinref part="C105" gate="G$1" pin="2"/>
-<wire x1="104.14" y1="-193.04" x2="193.04" y2="-193.04" width="0.1524" layer="91"/>
+<wire x1="104.14" y1="-193.04" x2="111.76" y2="-193.04" width="0.1524" layer="91"/>
+<wire x1="111.76" y1="-193.04" x2="193.04" y2="-193.04" width="0.1524" layer="91"/>
 <wire x1="104.14" y1="-195.58" x2="104.14" y2="-193.04" width="0.1524" layer="91"/>
 <label x="170.18" y="-193.04" size="1.778" layer="95"/>
+<pinref part="C124" gate="G$1" pin="2"/>
+<wire x1="111.76" y1="-195.58" x2="111.76" y2="-193.04" width="0.1524" layer="91"/>
+<junction x="111.76" y="-193.04"/>
 </segment>
 </net>
@@
 <attribute name="VALUE" x="-35.56" y="-233.68" size="1.778" layer="96" align="center"/>
 </instance>
-<instance part="MECH3" gate="G$1" x="132.08" y="-266.7" smashed="yes">
-<attribute name="NAME" x="132.08" y="-263.144" size="1.27" layer="95" align="center"/>
-</instance>
-<instance part="MECH4" gate="G$1" x="132.08" y="-274.32" smashed="yes">
-<attribute name="NAME" x="132.08" y="-270.764" size="1.27" layer="95" align="center"/>
-</instance>
 <instance part="U17" gate="G$1" x="76.2" y="-165.1" smashed="yes">

Commit message: CN6 routed to new location closes #22
Parts:
- R95: device r_0603:CRCW06031M00FKEC -> r_0402:RC0402FR-071ML
Connections:
- net DDR_D0: now also U2.PS_DDR_DQ9_502; no longer U2.PS_DDR_DQ5_502
- net DDR_D8: now also U2.PS_DDR_DQ5_502; no longer U2.PS_DDR_DQ9_502
- net DDR_DQS0_N: now also U2.PS_DDR_DQS_N1_502; no longer U2.PS_DDR_DQS_N0_502
- net DDR_DQS0_P: now also U2.PS_DDR_DQS_P1_502; no longer U2.PS_DDR_DQS_P0_502
- net DDR_DQS1_N: now also U2.PS_DDR_DQS_N0_502; no longer U2.PS_DDR_DQS_N1_502
- net DDR_DQS1_P: now also U2.PS_DDR_DQS_P0_502; no longer U2.PS_DDR_DQS_P1_502

Commit message: Display is now connected to FPGA logic Closes #21
Connections:
- removed net ADC_SPI_NCS: U2.PS_MIO20_501
- new net DSP_SPI_MOSI: CN6.11, U2.IO_L1P_T0_AD0P_35
- new net DSP_SPI_SCLK: CN6.12, U2.IO_L1N_T0_AD0N_35
- net DSP_D_NC: now also U2.IO_L2P_T0_AD8P_35; no longer U2.PS_MIO42_501
- net DSP_NRESET: now also U2.IO_L3N_T0_DQS_AD1N_35; no longer U2.PS_MIO29_501
- net DSP_SPI_NCS: now also U2.IO_L3P_T0_DQS_AD1P_35; no longer U2.PS_MIO19_501
- net PSS_SPI_MISO: no longer U2.PS_MIO17_501
- net PSS_SPI_MOSI: no longer CN6.11, U2.PS_MIO21_501
- net PSS_SPI_SCLK: no longer CN6.12, U2.PS_MIO16_501
- net SEN_SPI_NCS: no longer U2.PS_MIO18_501
Changed lines of the file:
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@@
 </segment>
 </net>
-<net name="PSS_SPI_SCLK" class="0">
-<segment>
-<pinref part="U2" gate="G$1" pin="PS_MIO16_501"/>
-<wire x1="81.28" y1="15.24" x2="43.18" y2="15.24" width="0.1524" layer="91"/>
-<label x="45.72" y="15.24" size="1.778" layer="95"/>
-</segment>
-</net>
-<net name="PSS_SPI_MISO" class="0">
-<segment>
-<pinref part="U2" gate="G$1" pin="PS_MIO17_501"/>
-<wire x1="81.28" y1="12.7" x2="43.18" y2="12.7" width="0.1524" layer="91"/>
-<label x="45.72" y="12.7" size="1.778" layer="95"/>
-</segment>
-</net>
-<net name="SEN_SPI_NCS" class="0">
-<segment>
-<pinref part="U2" gate="G$1" pin="PS_MIO18_501"/>
-<wire x1="81.28" y1="10.16" x2="43.18" y2="10.16" width="0.1524" layer="91"/>
-<label x="45.72" y="10.16" size="1.778" layer="95"/>
-</segment>
-</net>
-<net name="DSP_SPI_NCS" class="0">
-<segment>
-<pinref part="U2" gate="G$1" pin="PS_MIO19_501"/>
-<wire x1="81.28" y1="7.62" x2="43.18" y2="7.62" width="0.1524" layer="91"/>
-<label x="45.72" y="7.62" size="1.778" layer="95"/>
-</segment>
-</net>
-<net name="PSS_SPI_MOSI" class="0">
-<segment>
-<pinref part="U2" gate="G$1" pin="PS_MIO21_501"/>
-<wire x1="81.28" y1="2.54" x2="43.18" y2="2.54" width="0.1524" layer="91"/>
-<label x="45.72" y="2.54" size="1.778" layer="95"/>
-</segment>
-</net>
 <net name="PSS_DEBUG_UART_RX" class="0">
 <segment>
@@
 </segment>
 </net>
-<net name="DSP_D_NC" class="0">
-<segment>
-<pinref part="U2" gate="G$1" pin="PS_MIO42_501"/>
-<wire x1="81.28" y1="-50.8" x2="43.18" y2="-50.8" width="0.1524" layer="91"/>
-<label x="45.72" y="-50.8" size="1.778" layer="95"/>
-</segment>
-</net>
-<net name="DSP_NRESET" class="0">
-<segment>
-<pinref part="U2" gate="G$1" pin="PS_MIO29_501"/>
-<wire x1="81.28" y1="-17.78" x2="43.18" y2="-17.78" width="0.1524" layer="91"/>
-<label x="45.72" y="-17.78" size="1.778" layer="95"/>
-</segment>
-</net>
 <net name="PWR_VDISP_EN" class="0">
 <segment>
@@
 </segment>
 </net>
-<net name="ADC_SPI_NCS" class="0">
-<segment>
-<pinref part="U2" gate="G$1" pin="PS_MIO20_501"/>
-<wire x1="43.18" y1="5.08" x2="81.28" y2="5.08" width="0.1524" layer="91"/>
-<label x="45.72" y="5.08" size="1.778" layer="95"/>
-</segment>
-</net>
 <net name="FT_D10" class="0">
 <segment>
@@
 </segment>
 </net>
+<net name="DSP_NRESET" class="0">
+<segment>
+<pinref part="U2" gate="G$1" pin="IO_L3N_T0_DQS_AD1N_35"/>
+<wire x1="-81.28" y1="-144.78" x2="-43.18" y2="-144.78" width="0.1524" layer="91"/>
+<label x="-78.74" y="-144.78" size="1.778" layer="95"/>
+</segment>
+</net>
+<net name="DSP_D_NC" class="0">
+<segment>
+<pinref part="U2" gate="G$1" pin="IO_L2P_T0_AD8P_35"/>
+<wire x1="-81.28" y1="-142.24" x2="-43.18" y2="-142.24" width="0.1524" layer="91"/>
+<label x="-78.74" y="-142.24" size="1.778" layer="95"/>
+</segment>
+</net>
+<net name="DSP_SPI_SCLK" class="0">
+<segment>
+<pinref part="U2" gate="G$1" pin="IO_L1N_T0_AD0N_35"/>
+<wire x1="-81.28" y1="-134.62" x2="-43.18" y2="-134.62" width="0.1524" layer="91"/>
+<label x="-78.74" y="-134.62" size="1.778" layer="95"/>
+</segment>
+</net>
+<net name="DSP_SPI_NCS" class="0">
+<segment>
+<pinref part="U2" gate="G$1" pin="IO_L3P_T0_DQS_AD1P_35"/>
+<wire x1="-81.28" y1="-147.32" x2="-43.18" y2="-147.32" width="0.1524" layer="91"/>
+<label x="-78.74" y="-147.32" size="1.778" layer="95"/>
+</segment>
+</net>
+<net name="DSP_SPI_MOSI" class="0">
+<segment>
+<pinref part="U2" gate="G$1" pin="IO_L1P_T0_AD0P_35"/>
+<wire x1="-43.18" y1="-137.16" x2="-81.28" y2="-137.16" width="0.1524" layer="91"/>
+<label x="-78.74" y="-137.16" size="1.778" layer="95"/>
+</segment>
+</net>
 </nets>
 </sheet>
@@
 </segment>
 </net>
-<net name="PSS_SPI_SCLK" class="0">
-<segment>
-<label x="121.92" y="210.82" size="1.778" layer="95"/>
-<wire x1="83.82" y1="210.82" x2="147.32" y2="210.82" width="0.1524" layer="91"/>
-<pinref part="CN6" gate="G$1" pin="12"/>
-</segment>
-</net>
-<net name="PSS_SPI_MOSI" class="0">
-<segment>
-<label x="121.92" y="213.36" size="1.778" layer="95"/>
-<wire x1="83.82" y1="213.36" x2="147.32" y2="213.36" width="0.1524" layer="91"/>
-<pinref part="CN6" gate="G$1" pin="11"/>
-</segment>
-</net>
 <net name="FPGA_DONE" class="0">
 <segment>
@@
 </segment>
 </net>
+<net name="DSP_SPI_MOSI" class="0">
+<segment>
+<label x="121.92" y="213.36" size="1.778" layer="95"/>
+<wire x1="83.82" y1="213.36" x2="147.32" y2="213.36" width="0.1524" layer="91"/>
+<pinref part="CN6" gate="G$1" pin="11"/>
+</segment>
+</net>
+<net name="DSP_SPI_SCLK" class="0">
+<segment>
+<label x="121.92" y="210.82" size="1.778" layer="95"/>
+<wire x1="83.82" y1="210.82" x2="147.32" y2="210.82" width="0.1524" layer="91"/>
+<pinref part="CN6" gate="G$1" pin="12"/>
+</segment>
+</net>

Commit message: STUSB4500 now has pullups
Parts:
- added R187, R188: 2.2k, r_0402:RC0402FR-072K2L
Connections:
- removed net STUSB_SCL: U5.PA7, U9.SCL
- removed net STUSB_SDA: U5.PB4, U9.SDA
- new net STUSB_I2C_SCL: R187.1, U5.PA7, U9.SCL
- new net STUSB_I2C_SDA: R188.1, U5.PB4, U9.SDA
- net PWR_SYS_1V8_SLP: now also R187.2, R188.2
Changed lines of the file:
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@@
 <part name="C124" library="c_0603" deviceset="06036D476MAT2A" device="" value="47uF 6.3V"/>
 <part name="GND206" library="NETS" deviceset="GND" device=""/>
+<part name="R187" library="r_0402" deviceset="RC0402FR-072K2L" device="" value="2.2k"/>
+<part name="R188" library="r_0402" deviceset="RC0402FR-072K2L" device="" value="2.2k"/>
 </parts>
 <sheets>
@@
 <attribute name="VALUE" x="53.34" y="-58.42" size="1.27" layer="96" rot="R90" align="center"/>
 </instance>
+<instance part="R187" gate="G$1" x="12.7" y="-58.42" smashed="yes" rot="R90">
+<attribute name="NAME" x="10.16" y="-58.42" size="1.27" layer="95" rot="R90" align="center"/>
+<attribute name="VALUE" x="15.24" y="-58.42" size="1.27" layer="96" rot="R90" align="center"/>
+</instance>
+<instance part="R188" gate="G$1" x="20.32" y="-58.42" smashed="yes" rot="R90">
+<attribute name="NAME" x="17.78" y="-58.42" size="1.27" layer="95" rot="R90" align="center"/>
+<attribute name="VALUE" x="22.86" y="-58.42" size="1.27" layer="96" rot="R90" align="center"/>
+</instance>
 </instances>
 <busses>
@@
 </segment>
 </net>
-<net name="STUSB_SCL" class="0">
+<net name="STUSB_I2C_SCL" class="0">
 <segment>
 <pinref part="U9" gate="G$1" pin="SCL"/>
@@
 <pinref part="U5" gate="G$1" pin="PA7"/>
 </segment>
+<segment>
+<pinref part="R187" gate="G$1" pin="1"/>
+<wire x1="12.7" y1="-63.5" x2="12.7" y2="-78.74" width="0.1524" layer="91"/>
+<wire x1="12.7" y1="-78.74" x2="83.82" y2="-78.74" width="0.1524" layer="91"/>
+<label x="53.34" y="-78.74" size="1.778" layer="95"/>
+</segment>
 </net>
-<net name="STUSB_SDA" class="0">
+<net name="STUSB_I2C_SDA" class="0">
 <segment>
 <pinref part="U9" gate="G$1" pin="SDA"/>
@@
 <label x="-99.06" y="93.98" size="1.778" layer="95"/>
 </segment>
+<segment>
+<pinref part="R188" gate="G$1" pin="1"/>
+<wire x1="20.32" y1="-63.5" x2="20.32" y2="-76.2" width="0.1524" layer="91"/>
+<wire x1="20.32" y1="-76.2" x2="83.82" y2="-76.2" width="0.1524" layer="91"/>
+<label x="53.34" y="-76.2" size="1.778" layer="95"/>
+</segment>
 </net>
 <net name="STUSB_PD0" class="0">
@@
 <junction x="50.8" y="-50.8"/>
 <label x="53.34" y="-50.8" size="1.778" layer="95"/>
+<pinref part="R187" gate="G$1" pin="2"/>
+<wire x1="12.7" y1="-53.34" x2="12.7" y2="-50.8" width="0.1524" layer="91"/>
+<wire x1="12.7" y1="-50.8" x2="20.32" y2="-50.8" width="0.1524" layer="91"/>
+<junction x="27.94" y="-50.8"/>
+<pinref part="R188" gate="G$1" pin="2"/>
+<wire x1="20.32" y1="-50.8" x2="27.94" y2="-50.8" width="0.1524" layer="91"/>
+<wire x1="20.32" y1="-53.34" x2="20.32" y2="-50.8" width="0.1524" layer="91"/>
+<junction x="20.32" y="-50.8"/>
 </segment>
 </net>

Commit message: STUSB4500 I2C orientation corrected and resistors added to facilitate reversing
Parts:
- added R189, R190: 10R, r_0402:RC0402FR-0710RL
Connections:
- new net STM_I2C2_SCL: R190.1, U5.PB4
- new net STM_I2C2_SDA: R189.1, U5.PA7
- net STUSB_I2C_SCL: now also R190.2; no longer U5.PA7
- net STUSB_I2C_SDA: now also R189.2; no longer U5.PB4
Changed lines of the file:
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@@
 <part name="R187" library="r_0402" deviceset="RC0402FR-072K2L" device="" value="2.2k"/>
 <part name="R188" library="r_0402" deviceset="RC0402FR-072K2L" device="" value="2.2k"/>
+<part name="R189" library="r_0402" deviceset="RC0402FR-0710RL" device="" value="10R"/>
+<part name="R190" library="r_0402" deviceset="RC0402FR-0710RL" device="" value="10R"/>
 </parts>
 <sheets>
@@
 <attribute name="VALUE" x="22.86" y="-58.42" size="1.27" layer="96" rot="R90" align="center"/>
 </instance>
+<instance part="R189" gate="G$1" x="-5.08" y="-76.2" smashed="yes">
+<attribute name="NAME" x="-5.08" y="-73.66" size="1.27" layer="95" align="center"/>
+<attribute name="VALUE" x="-5.08" y="-78.74" size="1.27" layer="96" align="center"/>
+</instance>
+<instance part="R190" gate="G$1" x="5.08" y="-81.28" smashed="yes">
+<attribute name="NAME" x="5.08" y="-78.74" size="1.27" layer="95" align="center"/>
+<attribute name="VALUE" x="5.08" y="-83.82" size="1.27" layer="96" align="center"/>
+</instance>
 </instances>
 <busses>
@@
 </segment>
 <segment>
-<wire x1="-101.6" y1="129.54" x2="-66.04" y2="129.54" width="0.1524" layer="91"/>
-<label x="-99.06" y="129.54" size="1.778" layer="95"/>
-<pinref part="U5" gate="G$1" pin="PA7"/>
-</segment>
-<segment>
 <pinref part="R187" gate="G$1" pin="1"/>
-<wire x1="12.7" y1="-63.5" x2="12.7" y2="-78.74" width="0.1524" layer="91"/>
-<wire x1="12.7" y1="-78.74" x2="83.82" y2="-78.74" width="0.1524" layer="91"/>
-<label x="53.34" y="-78.74" size="1.778" layer="95"/>
+<wire x1="12.7" y1="-63.5" x2="12.7" y2="-81.28" width="0.1524" layer="91"/>
+<wire x1="12.7" y1="-81.28" x2="83.82" y2="-81.28" width="0.1524" layer="91"/>
+<label x="53.34" y="-81.28" size="1.778" layer="95"/>
+<pinref part="R190" gate="G$1" pin="2"/>
+<wire x1="10.16" y1="-81.28" x2="12.7" y2="-81.28" width="0.1524" layer="91"/>
+<junction x="12.7" y="-81.28"/>
 </segment>
 </net>
@@
 </segment>
 <segment>
-<pinref part="U5" gate="G$1" pin="PB4"/>
-<wire x1="-101.6" y1="93.98" x2="-66.04" y2="93.98" width="0.1524" layer="91"/>
-<label x="-99.06" y="93.98" size="1.778" layer="95"/>
-</segment>
-<segment>
 <pinref part="R188" gate="G$1" pin="1"/>
 <wire x1="20.32" y1="-63.5" x2="20.32" y2="-76.2" width="0.1524" layer="91"/>
 <wire x1="20.32" y1="-76.2" x2="83.82" y2="-76.2" width="0.1524" layer="91"/>
 <label x="53.34" y="-76.2" size="1.778" layer="95"/>
+<pinref part="R189" gate="G$1" pin="2"/>
+<wire x1="0" y1="-76.2" x2="20.32" y2="-76.2" width="0.1524" layer="91"/>
+<junction x="20.32" y="-76.2"/>
 </segment>
 </net>
@@
 </segment>
 </net>
+<net name="STM_I2C2_SDA" class="0">
+<segment>
+<pinref part="R189" gate="G$1" pin="1"/>
+<wire x1="-10.16" y1="-76.2" x2="-40.64" y2="-76.2" width="0.1524" layer="91"/>
+<label x="-38.1" y="-76.2" size="1.778" layer="95"/>
+</segment>
+<segment>
+<wire x1="-101.6" y1="129.54" x2="-66.04" y2="129.54" width="0.1524" layer="91"/>
+<label x="-99.06" y="129.54" size="1.778" layer="95"/>
+<pinref part="U5" gate="G$1" pin="PA7"/>
+</segment>
+</net>
+<net name="STM_I2C2_SCL" class="0">
+<segment>
+<pinref part="R190" gate="G$1" pin="1"/>
+<wire x1="0" y1="-81.28" x2="-40.64" y2="-81.28" width="0.1524" layer="91"/>
+<label x="-38.1" y="-81.28" size="1.778" layer="95"/>
+</segment>
+<segment>
+<pinref part="U5" gate="G$1" pin="PB4"/>
+<wire x1="-101.6" y1="93.98" x2="-66.04" y2="93.98" width="0.1524" layer="91"/>
+<label x="-99.06" y="93.98" size="1.778" layer="95"/>
+</segment>
+</net>

Commit message: SPI fixed, FPGA LEDs fixed
Parts:
- OSC1: device CRYSTALS:KC2016Z33.0000C15XXK -> CRYSTALS:KC2016Z33.0000C1KX00
- R59, R79, R80: value 120 -> 2.2k; device r_0402:ERJ-2RKF1200X -> r_0402:RC0402FR-072K2L
Connections:
- removed net PSS_SPI_MISO: U1A.SPI_MISO
- removed net PSS_SPI_MOSI: U1A.SPI_MOSI
- removed net PSS_SPI_SCLK: U1A.SPI_SCLK
- new net SEN_SPI_MISO: U1A.SPI_MISO, U2.IO_L9N_T1_DQS_33
- new net SEN_SPI_MOSI: U1A.SPI_MOSI, U2.IO_L2N_T0_33
- new net SEN_SPI_SCLK: U1A.SPI_SCLK, U2.IO_0_33
- net SEN_SPI_NCS: now also U2.IO_L2P_T0_33
Changed lines of the file:
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@@
 <part name="R24" library="r_0603" deviceset="CRCW06032K00FKTA" device="" value="2k"/>
 <part name="GND102" library="NETS" deviceset="GND" device=""/>
-<part name="OSC1" library="CRYSTALS" deviceset="KC2016Z33.0000C15XXK" device="" value="33MHz"/>
+<part name="OSC1" library="CRYSTALS" deviceset="KC2016Z33.0000C1KX00" device="" value="33MHz"/>
 <part name="C72" library="c_0402" deviceset="0402ZC104KAT2A" device="" value="0.1uF 10V"/>
 <part name="GND74" library="NETS" deviceset="GND" device=""/>
@@
 <part name="D7" library="OPTO" deviceset="150060RS75000" device="" value="RED LED"/>
 <part name="D9" library="OPTO" deviceset="150060RS75000" device="" value="RED LED"/>
-<part name="R59" library="r_0402" deviceset="ERJ-2RKF1200X" device="" value="120"/>
-<part name="R79" library="r_0402" deviceset="ERJ-2RKF1200X" device="" value="120"/>
-<part name="R80" library="r_0402" deviceset="ERJ-2RKF1200X" device="" value="120"/>
+<part name="R59" library="r_0402" deviceset="RC0402FR-072K2L" device="" value="2.2k"/>
+<part name="R79" library="r_0402" deviceset="RC0402FR-072K2L" device="" value="2.2k"/>
+<part name="R80" library="r_0402" deviceset="RC0402FR-072K2L" device="" value="2.2k"/>
 <part name="C145" library="c_0603" deviceset="CL10B225KP8NFNC" device="" value="2.2uF 10V"/>
 <part name="GND211" library="NETS" deviceset="GND" device=""/>
@@
 </segment>
 </net>
+<net name="SEN_SPI_MOSI" class="0">
+<segment>
+<pinref part="U2" gate="G$1" pin="IO_L2N_T0_33"/>
+<wire x1="-43.18" y1="119.38" x2="-81.28" y2="119.38" width="0.1524" layer="91"/>
+<label x="-78.74" y="119.38" size="1.778" layer="95"/>
+</segment>
+</net>
+<net name="SEN_SPI_NCS" class="0">
+<segment>
+<pinref part="U2" gate="G$1" pin="IO_L2P_T0_33"/>
+<wire x1="-43.18" y1="116.84" x2="-81.28" y2="116.84" width="0.1524" layer="91"/>
+<label x="-78.74" y="116.84" size="1.778" layer="95"/>
+</segment>
+</net>
+<net name="SEN_SPI_MISO" class="0">
+<segment>
+<pinref part="U2" gate="G$1" pin="IO_L9N_T1_DQS_33"/>
+<wire x1="-43.18" y1="83.82" x2="-81.28" y2="83.82" width="0.1524" layer="91"/>
+<label x="-78.74" y="83.82" size="1.778" layer="95"/>
+</segment>
+</net>
+<net name="SEN_SPI_SCLK" class="0">
+<segment>
+<pinref part="U2" gate="G$1" pin="IO_0_33"/>
+<wire x1="-43.18" y1="127" x2="-81.28" y2="127" width="0.1524" layer="91"/>
+<label x="-78.74" y="127" size="1.778" layer="95"/>
+</segment>
+</net>
 </nets>
 </sheet>
@@
 </segment>
 </net>
-<net name="PSS_SPI_SCLK" class="0">
+<net name="SEN_SPI_SCLK" class="0">
 <segment>
 <wire x1="-114.3" y1="210.82" x2="-154.94" y2="210.82" width="0.1524" layer="91"/>
@@
 </segment>
 </net>
-<net name="PSS_SPI_MOSI" class="0">
+<net name="SEN_SPI_MOSI" class="0">
 <segment>
 <wire x1="-114.3" y1="208.28" x2="-154.94" y2="208.28" width="0.1524" layer="91"/>
@@
 </segment>
 </net>
-<net name="PSS_SPI_MISO" class="0">
+<net name="SEN_SPI_MISO" class="0">
 <segment>
 <wire x1="-114.3" y1="205.74" x2="-154.94" y2="205.74" width="0.1524" layer="91"/>
