File: main.sch (EAGLE design)
At the start: 597 parts, among them CN1 50 PIN 0.5MM, CN2 10067847-001RLF, CN3 632723300011, CN4 FF0881SA1, CN5 15PIN 0.5MM, CN6 31 PIN FPC, CN7 Mini Displayport, Q1 2N7002, Q2 FDN302P, Q3 2N7002, Q4 2N7002, Q5 SI7489DP, Q6 2N7002, SW2 TACT, SW3 TACT, SW4 TACT, SW5 TACT, SW7 TACT, SW8 SLIDE SPDT, U1 GMAX0505-DV, U10 RTL8211E, U11 PI4ULS3V204ZBEX, U13 MAX25300B, U14 ESP32, U15 MAX25300B, U16 INA180, U17 AP62301, U18 AP62301, U19 SCHMITT, U2 XC7Z014S-1CLG484C, U20 MAX25300B, U22 MAX25300B, U23 SN74LVC1G3, U24 NAND, U25 EMC1812T, U26 BIPOLAR HALL, U27 LM2663, U28 ADS7867, U29 LM2663, U3 IS43TR16128CL-125KBLI, U30 LM2731X, U31 USBLC6-2SC6, U32 MAX1735, U33 MP2148, U34 TPS22917, U35 AP62301, U36 TLV61046A, U37 W25Q128JV, U38 TPS70918, U39 AP62301, U4 AP63300WU-7, U40 ADJ BUCK, U5 STM32L431RBT, U6 USB 2.0 PHY, U7 ACT2861QI301-T, U8 TPS70950, U9 STUSB4500

Commit message: EVF connector now in the correct orientation. MIPI needs renaming and length matching
Connections:
- net EVF_MIPI_A_CLK_N: now also R112.2, R114.1, R116.2; no longer R15.2, R20.1, R27.2
- net EVF_MIPI_A_CLK_P: now also R110.2, R113.1, R115.2; no longer R14.2, R19.1, R21.2
- net EVF_MIPI_A_D0_N: now also R15.2, R20.1, R27.2; no longer R26.2, R66.1, R68.2
- net EVF_MIPI_A_D0_P: now also R14.2, R19.1, R21.2; no longer R25.2, R64.1, R67.2
- net EVF_MIPI_A_D1_N: now also R118.2, R124.1, R126.2; no longer R109.2, R70.2, R73.1
- net EVF_MIPI_A_D1_P: now also R117.2, R123.1, R125.2; no longer R69.2, R71.1, R96.2
- net EVF_MIPI_A_D2_N: now also R144.2, R146.1, R148.2; no longer R112.2, R114.1, R116.2
- net EVF_MIPI_A_D2_P: now also R143.2, R145.1, R147.2; no longer R110.2, R113.1, R115.2
- net EVF_MIPI_A_D3_N: now also R138.2, R140.1, R142.2; no longer R118.2, R124.1, R126.2
- net EVF_MIPI_A_D3_P: now also R134.2, R139.1, R141.2; no longer R117.2, R123.1, R125.2
- net EVF_MIPI_B_CLK_N: now also R156.2, R158.1, R160.2; no longer R128.2, R131.1, R133.2
- net EVF_MIPI_B_CLK_P: now also R155.2, R157.1, R159.2; no longer R127.2, R130.1, R132.2
- net EVF_MIPI_B_D0_N: now also R150.2, R152.1, R154.2; no longer R138.2, R140.1, R142.2
- net EVF_MIPI_B_D0_P: now also R149.2, R151.1, R153.2; no longer R134.2, R139.1, R141.2
- net EVF_MIPI_B_D1_N: now also R109.2, R70.2, R73.1; no longer R144.2, R146.1, R148.2
- net EVF_MIPI_B_D1_P: now also R69.2, R71.1, R96.2; no longer R143.2, R145.1, R147.2
- net EVF_MIPI_B_D2_N: now also R26.2, R66.1, R68.2; no longer R150.2, R152.1, R154.2
- net EVF_MIPI_B_D2_P: now also R25.2, R64.1, R67.2; no longer R149.2, R151.1, R153.2
- net EVF_MIPI_B_D3_N: now also R128.2, R131.1, R133.2; no longer R156.2, R158.1, R160.2
- net EVF_MIPI_B_D3_P: now also R127.2, R130.1, R132.2; no longer R155.2, R157.1, R159.2

Commit message: Adjusted PSS DEBUG UART Vio
Connections:
- net PWR_SYS_1V8: no longer CN1.P31
- net PWR_SYS_3V3: now also CN1.P31
Changed lines of the file:
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@@
 <junction x="116.84" y="30.48"/>
+</segment>
+<segment>
+<label x="20.32" y="-15.24" size="1.778" layer="95"/>
+<wire x1="15.24" y1="-15.24" x2="48.26" y2="-15.24" width="0.1524" layer="91"/>
+<pinref part="CN1" gate="G$1" pin="P31"/>
 </segment>
 </net>
@@
 </segment>
 <segment>
-<label x="20.32" y="-15.24" size="1.778" layer="95"/>
-<wire x1="15.24" y1="-15.24" x2="48.26" y2="-15.24" width="0.1524" layer="91"/>
-<pinref part="CN1" gate="G$1" pin="P31"/>
-</segment>
-<segment>

Commit message: Small bits
Connections:
- removed net N$95: R194.1, U10.LED0/PHY_AD0
- removed net N$96: R196.2, U10.LED1/PHY_AD1
- new net ETH_LED_ACT: CN7.CONFIG1, R194.1, U10.LED0/PHY_AD0
- new net ETH_LED_LNK: CN7.CONFIG2, R196.2, U10.LED1/PHY_AD1
- net PWR_SYS_3V3: now also CN7.HOT_PLUG_DECT
Other:
- note added: "VDDIO 1ms (min) VDD13AD+ VDD13D 1ms (min) VDD33A 1ms (min) Supply Array (VTXL etc.) 1ms (min) SYS_RST_N"
- note removed: "VDDIO 1ms (min) VDD13AD+VDD13D 1ms (min) VDD33A 1ms (min) Supply Array (VTXL etc.) 1ms (min) SYS_RST_N"
Changed lines of the file:
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@@
 <text x="0" y="-279.4" size="7.62" layer="97" font="vector" align="center">UNCONTROLLED WHEN PRINTED</text>
 <text x="0" y="279.4" size="7.62" layer="97" font="vector" align="center">UNCONTROLLED WHEN PRINTED</text>
-<text x="25.4" y="-264.16" size="5.08" layer="91">VDDIO
+<text x="139.7" y="-149.86" size="5.08" layer="91">VDDIO
 1ms (min)
-VDD13AD+VDD13D
+VDD13AD+
+VDD13D
 1ms (min)
 VDD33A
 1ms (min)
-Supply Array (VTXL etc.)
+Supply Array
+(VTXL etc.)
 1ms (min)
 SYS_RST_N</text>
-<text x="106.68" y="-266.7" size="5.08" layer="91">Voltage (V) Peak Current (mA)
+<text x="78.74" y="-264.16" size="5.08" layer="91">Voltage (V) Peak Current (mA)
 VDD33A 3.3 80
 VDD13D 1.3 250
@@
 <label x="-129.54" y="-50.8" size="1.778" layer="95"/>
 </segment>
+<segment>
+<pinref part="CN7" gate="G$1" pin="HOT_PLUG_DECT"/>
+<wire x1="109.22" y1="-81.28" x2="71.12" y2="-81.28" width="0.1524" layer="91"/>
+<label x="73.66" y="-81.28" size="1.778" layer="95"/>
+</segment>
 </net>
 <net name="USB_NRST" class="0">
@@
 </segment>
 </net>
-<net name="N$95" class="0">
+<net name="ETH_LED_ACT" class="0">
 <segment>
 <pinref part="U10" gate="G$1" pin="LED0/PHY_AD0"/>
@@
 <wire x1="10.16" y1="-104.14" x2="10.16" y2="-106.68" width="0.1524" layer="91"/>
 <junction x="10.16" y="-106.68"/>
+<label x="27.94" y="-106.68" size="1.778" layer="95"/>
+</segment>
+<segment>
+<pinref part="CN7" gate="G$1" pin="CONFIG1"/>
+<wire x1="109.22" y1="-73.66" x2="71.12" y2="-73.66" width="0.1524" layer="91"/>
+<label x="73.66" y="-73.66" size="1.778" layer="95"/>
 </segment>
 </net>
-<net name="N$96" class="0">
+<net name="ETH_LED_LNK" class="0">
 <segment>
 <pinref part="U10" gate="G$1" pin="LED1/PHY_AD1"/>
@@
 <wire x1="25.4" y1="-114.3" x2="25.4" y2="-109.22" width="0.1524" layer="91"/>
 <junction x="25.4" y="-109.22"/>
+<label x="27.94" y="-109.22" size="1.778" layer="95"/>
+</segment>
+<segment>
+<pinref part="CN7" gate="G$1" pin="CONFIG2"/>
+<wire x1="109.22" y1="-76.2" x2="71.12" y2="-76.2" width="0.1524" layer="91"/>
+<label x="73.66" y="-76.2" size="1.778" layer="95"/>
 </segment>
 </net>

Commit message: Planes implemented
Other:
- note added: "2023.11.28 - GSWDH LTD. CAMERA MAIN PCB REVISION 1.2.0 DESIGN BY GEORGE WALLER, GSWDH LTD. GEORGEWALLER@GSWDH.CO.UK CONFIDENTIAL. FOR THE INTENDED READER ONLY."
- note removed: "2023.11.20 - GSWDH LTD. CAMERA MAIN PCB REVISION 1.2.0 DESIGN BY GEORGE WALLER, GSWDH LTD. GEORGEWALLER@GSWDH.CO.UK CONFIDENTIAL. FOR THE INTENDED READER ONLY."
Changed lines of the file:
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@@
 <description>TITLE</description>
 <plain>
-<text x="0" y="0" size="7.62" layer="97" font="vector" align="center">2023.11.20 - GSWDH LTD.
+<text x="0" y="0" size="7.62" layer="97" font="vector" align="center">2023.11.28 - GSWDH LTD.
 CAMERA MAIN PCB
 REVISION 1.2.0

Commit message: Fixed ETH RX CTL and CLK bug. Mved USB and WTH resets to PL
Connections:
- removed net ETH_NRESET: R197.1, U10.PHYRSTB, U2.PS_MIO20_501
- removed net MIPI_DSI_B_HS_L3_N: R156.1, U2.IO_L18N_T2_33
- removed net MIPI_DSI_B_HS_L3_P: R155.1, U2.IO_L18P_T2_33
- new net ETH_NRST: R197.1, U10.PHYRSTB, U2.IO_L24N_T3_AD15N_35
- new net MIPI_DSI_B_HP_L3_N: R128.1, U2.IO_L23N_T3_33
- new net MIPI_DSI_B_HP_L3_P: R127.1, U2.IO_L23P_T3_33
- net ETH_RX_CLK: now also U10.RXC; no longer U10.RXCTL/PHY_AD
- net ETH_RX_CTL: now also U10.RXCTL/PHY_AD; no longer U10.RXC
- net MIPI_DSI_A_HS_CK_N: now also R112.1, U2.IO_L21N_T3_DQS_33; no longer R15.1, U2.IO_L19N_T3_VREF_33
- net MIPI_DSI_A_HS_CK_P: now also R110.1, U2.IO_L21P_T3_DQS_33; no longer R14.1, U2.IO_L19P_T3_33
- net MIPI_DSI_A_HS_L0_N: now also R15.1, U2.IO_L19N_T3_VREF_33; no longer R26.1, U2.IO_L11N_T1_SRCC_33
- net MIPI_DSI_A_HS_L0_P: now also R14.1, U2.IO_L19P_T3_33; no longer R25.1, U2.IO_L11P_T1_SRCC_33
- net MIPI_DSI_A_HS_L1_N: now also R118.1, U2.IO_L12N_T1_MRCC_33; no longer R70.1, U2.IO_L17N_T2_33
- net MIPI_DSI_A_HS_L1_P: now also R117.1, U2.IO_L12P_T1_MRCC_33; no longer R69.1, U2.IO_L17P_T2_33
- net MIPI_DSI_A_HS_L2_N: now also R144.1, U2.IO_L20N_T3_33; no longer R112.1, U2.IO_L21N_T3_DQS_33
- net MIPI_DSI_A_HS_L2_P: now also R143.1, U2.IO_L20P_T3_33; no longer R110.1, U2.IO_L21P_T3_DQS_33
- net MIPI_DSI_A_HS_L3_N: now also R138.1, U2.IO_L24N_T3_33; no longer R118.1, U2.IO_L12N_T1_MRCC_33
- net MIPI_DSI_A_HS_L3_P: now also R134.1, U2.IO_L24P_T3_33; no longer R117.1, U2.IO_L12P_T1_MRCC_33
- net MIPI_DSI_A_LP_CK_N: now also R116.1, U2.IO_L13N_T2_MRCC_33; no longer R27.1, U2.IO_L10N_T1_33
- net MIPI_DSI_A_LP_CK_P: now also R115.1, U2.IO_L13P_T2_MRCC_33; no longer R21.1, U2.IO_L10P_T1_33
- net MIPI_DSI_A_LP_L0_N: now also R27.1, U2.IO_L10N_T1_33; no longer R68.1, U2.IO_L7N_T1_33
- net MIPI_DSI_A_LP_L0_P: now also R21.1, U2.IO_L10P_T1_33; no longer R67.1, U2.IO_L7P_T1_33
- net MIPI_DSI_A_LP_L1_N: now also R126.1, U2.IO_L8N_T1_33; no longer R109.1, U2.IO_L3N_T0_DQS_33
- net MIPI_DSI_A_LP_L1_P: now also R125.1, U2.IO_L8P_T1_33; no longer R96.1, U2.IO_L3P_T0_DQS_33
- net MIPI_DSI_A_LP_L2_N: now also R148.1, U2.IO_L15N_T2_DQS_33; no longer R116.1, U2.IO_L13N_T2_MRCC_33
- net MIPI_DSI_A_LP_L2_P: now also R147.1, U2.IO_L15P_T2_DQS_33; no longer R115.1, U2.IO_L13P_T2_MRCC_33
- net MIPI_DSI_A_LP_L3_N: now also R142.1, U2.IO_L16N_T2_33; no longer R126.1, U2.IO_L8N_T1_33
- net MIPI_DSI_A_LP_L3_P: now also R141.1, U2.IO_L16P_T2_33; no longer R125.1, U2.IO_L8P_T1_33
- net MIPI_DSI_B_HS_CK_N: now also R156.1, U2.IO_L18N_T2_33; no longer R128.1, U2.IO_L23N_T3_33
- net MIPI_DSI_B_HS_CK_P: now also R155.1, U2.IO_L18P_T2_33; no longer R127.1, U2.IO_L23P_T3_33
- net MIPI_DSI_B_HS_L0_N: now also R150.1, U2.IO_L22N_T3_33; no longer R138.1, U2.IO_L24N_T3_33
- net MIPI_DSI_B_HS_L0_P: now also R149.1, U2.IO_L22P_T3_33; no longer R134.1, U2.IO_L24P_T3_33
- net MIPI_DSI_B_HS_L1_N: now also R70.1, U2.IO_L17N_T2_33; no longer R144.1, U2.IO_L20N_T3_33
- net MIPI_DSI_B_HS_L1_P: now also R69.1, U2.IO_L17P_T2_33; no longer R143.1, U2.IO_L20P_T3_33
- net MIPI_DSI_B_HS_L2_N: now also R26.1, U2.IO_L11N_T1_SRCC_33; no longer R150.1, U2.IO_L22N_T3_33
- net MIPI_DSI_B_HS_L2_P: now also R25.1, U2.IO_L11P_T1_SRCC_33; no longer R149.1, U2.IO_L22P_T3_33
- net MIPI_DSI_B_LP_CK_N: now also R160.1, U2.IO_L1N_T0_33; no longer R133.1, U2.IO_L5N_T0_33
- net MIPI_DSI_B_LP_CK_P: now also R159.1, U2.IO_L1P_T0_33; no longer R132.1, U2.IO_L5P_T0_33
- net MIPI_DSI_B_LP_L0_N: now also R154.1, U2.IO_L4N_T0_33; no longer R142.1, U2.IO_L16N_T2_33
- net MIPI_DSI_B_LP_L0_P: now also R153.1, U2.IO_L4P_T0_33; no longer R141.1, U2.IO_L16P_T2_33
- net MIPI_DSI_B_LP_L1_N: now also R109.1, U2.IO_L3N_T0_DQS_33; no longer R148.1, U2.IO_L15N_T2_DQS_33
- net MIPI_DSI_B_LP_L1_P: now also R96.1, U2.IO_L3P_T0_DQS_33; no longer R147.1, U2.IO_L15P_T2_DQS_33
- net MIPI_DSI_B_LP_L2_N: now also R68.1, U2.IO_L7N_T1_33; no longer R154.1, U2.IO_L4N_T0_33
- net MIPI_DSI_B_LP_L2_P: now also R67.1, U2.IO_L7P_T1_33; no longer R153.1, U2.IO_L4P_T0_33
- net MIPI_DSI_B_LP_L3_N: now also R133.1, U2.IO_L5N_T0_33; no longer R160.1, U2.IO_L1N_T0_33
- net MIPI_DSI_B_LP_L3_P: now also R132.1, U2.IO_L5P_T0_33; no longer R159.1, U2.IO_L1P_T0_33
- net PSS_SD_CD: now also U2.IO_L10N_T1_13
- net PSS_SD_WP: now also U2.IO_L11P_T1_SRCC_13
- net USB_NRST: now also U2.IO_L23N_T3_35; no longer U2.PS_MIO21_501

Commit message: BTN_THUMB connected directly to the PMC IO
Connections:
- net BTN_THUMB: now also U5.PD2
Changed lines of the file:
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@@
 <attribute name="VALUE" x="-119.38" y="185.42" size="1.27" layer="96" rot="R90" align="center"/>
 </instance>
-<instance part="GND68" gate="G$1" x="-121.92" y="175.26" smashed="yes"/>
+<instance part="GND68" gate="G$1" x="-121.92" y="175.26" smashed="yes">
+<attribute name="VALUE" x="-121.92" y="172.72" size="1.778" layer="96" align="center"/>
+</instance>
 <instance part="C29" gate="G$1" x="-114.3" y="185.42" smashed="yes" rot="R90">
 <attribute name="NAME" x="-116.84" y="185.42" size="1.27" layer="95" rot="R90" align="center"/>
@@
 <pinref part="U19" gate="G$1" pin="A"/>
 </segment>
-</net>
+<segment>
+<pinref part="U5" gate="G$1" pin="PD2"/>
+<wire x1="-142.24" y1="104.14" x2="-177.8" y2="104.14" width="0.1524" layer="91"/>
+<label x="-175.26" y="104.14" size="1.778" layer="95"/>
+</segment>
+</net>

Commit message: Updated the dates
Other:
- note added: "2024.02.14 - GSWDH LTD. CAMERA MAIN PCB REVISION 1.2.0 DESIGN BY GEORGE WALLER, GSWDH LTD. GEORGEWALLER@GSWDH.CO.UK CONFIDENTIAL. FOR THE INTENDED READER ONLY."
- note removed: "2023.11.28 - GSWDH LTD. CAMERA MAIN PCB REVISION 1.2.0 DESIGN BY GEORGE WALLER, GSWDH LTD. GEORGEWALLER@GSWDH.CO.UK CONFIDENTIAL. FOR THE INTENDED READER ONLY."
Changed lines of the file:
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@@
 <description>TITLE</description>
 <plain>
-<text x="0" y="0" size="7.62" layer="97" font="vector" align="center">2023.11.28 - GSWDH LTD.
+<text x="0" y="0" size="7.62" layer="97" font="vector" align="center">2024.02.14 - GSWDH LTD.
 CAMERA MAIN PCB
 REVISION 1.2.0

Commit message: New stuff
Parts:
- removed CN5: 15PIN 0.5MM, CONNECTORs:SFV15R-1STE1HLF
- removed CN7: Mini Displayport, CONNECTORs:2129320-3
- removed D1, D3: PESD5Z5.0, DIODES:PESD5Z5.0
- removed L7: 2.2uH 1.3A, INDUCTORS:CIG22L2R2MNE
- removed R189, R190: 10R, r_0402:RC0402FR-0710RL
- removed R198, R199, R200, R201, R202: 4.7k, r_0402:RC0402FR-074K7L
- removed R203: 1.5k, r_0402:RC0402FR-071K5L
- removed R204, R205: 2.2k, r_0402:RC0402FR-072K2L
- removed SW8: SLIDE SPDT, ELECTROMECH:EG1215AA
- removed TX1: 749020111A, PASSIVES:749020111A
- added C285, C287, C289, C291, C293, C295, C300, C303, C306: 4.7uF 6.3V, c_0402:04026D475KAT2A
- added C286, C288, C290, C292, C294, C296, C297, C301, C302, C304, C305, C308, C309, C310, C311, C312, C313, C314, C315, C316: 0.1uF 10V, c_0402:0402ZD104KAT2A
- added C298, C299: 0.22uF 16V, c_0402:0402YD224KAT2A
- added C307: 1uF 50V, c_0603:06035C105KAT2A
- added C317: 22uF 6.3V, c_1206:C1206C226K9RAC7800
- added C318: 2.2uF 10V, c_0402:0402ZD225KAT2A
- added U12, U21: ISO1044BDR, ICs:ISO1044BDR
- added U41, U42: 64GB eMMC, ICs:ZDEMDCM064G-95A8
- added U43: TPS70950, ICs:TPS70950DBVT
- added XTAL1: 30MHz 6pF, CRYSTALS:XRCGB30M000F3M00R0
- C102: value 0.1uF 16V -> 0.1uF 10V; device c_0603:C0603C104J4RAC7013 -> c_0402:0402ZD104KAT2A
- C103: value 10uF 10V -> 0.1uF 10V; device c_1206:C1206C106K8PACTU -> c_0402:0402ZD104KAT2A
- C107, C17, C77: value 4.7uF 6.3V -> 0.1uF 10V; device c_0402:04026D475KAT2A -> c_0402:0402ZD104KAT2A
- C111: value 0.1uF 10V -> 5.6pF 16V; device c_0402:0402ZD104KAT2A -> c_0402:0402YA5R6CAT2A
- C112: value 0.1uF 10V -> 4.7uF 6.3V; device c_0402:0402ZD104KAT2A -> c_0402:04026D475KAT2A
- C118, C119, C155, C280, C282: device c_0402:0402ZD104KAT2A -> c_0402:0402ZC104KAT2A
- C281: value 1nF 2kV -> 0.1uF 10V; device CAPACITORS:C1812C102KGRACAUTO -> c_0402:0402ZC104KAT2A
- C284, C60, C79, C80: device c_0402:0402ZC104KAT2A -> c_0402:0402ZD104KAT2A
- C61: value 1uF 50V -> 0.1uF 10V; device c_0603:06035C105KAT2A -> c_0402:0402ZD104KAT2A
- C76: value 2.2uF 10V -> 0.1uF 10V; device c_0603:CL10A225KP8NNNC -> c_0402:0402ZD104KAT2A
- C78: value 0.1uF 10V -> 5.6pF 16V; device c_0402:0402ZC104KAT2A -> c_0402:0402YA5R6CAT2A
- CN1: value 50 PIN 0.5MM -> X1321FR-2x20-C43D24; device CONNECTORs:FH52E-50S-0.5SH -> CONNECTORs:X1321FR-2X20-C43D24
- CN2: value 10067847-001RLF -> 15PIN 0.5MM; device CONNECTORs:10067847-001RLF -> CONNECTORs:SFV15R-1STE1HLF
- R102: value 2.2k -> 10R; device r_0402:RC0402FR-072K2L -> r_0402:RC0402FR-0710RL
- R181, R182: value 2.2k -> 120R; device r_0402:RC0402FR-072K2L -> r_0402:RC0402FR-07120RL
- R193: value 2.49k -> 1k; device r_0402:RC0402FR-072K49L -> r_0402:RC0402FR-071KL
- R194: value 4.7k -> 1k; device r_0402:RC0402FR-074K7L -> r_0402:RC0402FR-071KL
- R195: value 4.7k -> 20R; device r_0402:RC0402FR-074K7L -> r_0402:RC0402FR-0720RL
- R196: value 4.7k -> 10k; device r_0402:RC0402FR-074K7L -> r_0402:RC0402FR-0710KL
- R197: value 4.7k -> 4.99k; device r_0402:RC0402FR-074K7L -> r_0402:RC0402FR-074K99L
- R35: value 8.06k -> 1.6k; device r_0402:RC0402FR-078K06L -> r_0402:RC0402FR-071K6L
- R62, R63, R72, R75: value 75R -> 10k; device r_0603:CRCW060375R0FKEA -> r_0402:RC0402FR-0710KL
- R74: device r_0402:ERJ-2RKF1002X -> r_0402:RC0402FR-0710KL
- R78: value 10k -> 4.99k; device r_0402:ERJ-2RKF1002X -> r_0402:RC0402FR-074K99L
- U10: value RTL8211E -> 7498111120R; device ICs:RTL8211E-VB -> 7498111120R:7498111120R
- U11: value PI4ULS3V204ZBEX -> USBLC6-2SC6; device ICs:PI4ULS3V204 -> ICs:USBLC6-2SC6
- U26: value BIPOLAR HALL -> ISO1044BDR; device ICs:DRV5053VAQDBZT -> ICs:ISO1044BDR
- U28: value ADS7867 -> 88E1512; device ICs:ADS7867IDBVR -> ICs:88E1512-A0-NNP2I000
- U6: value USB 2.0 PHY -> FT601Q; device ICs:USB3320C -> ICs:FT601Q
- U8: value TPS70950 -> HD3SS3212; device ICs:TPS70950DBVT -> ICs:HD3SS3212IRKSR
Connections:
- net PSS_NRST renamed PSS_PS_POR
- removed net BADC_SPI_MISO: U2.IO_L18N_T2_34, U28.SDO
- removed net BADC_SPI_NCS: U2.IO_L18P_T2_34, U28.!CS
- removed net BADC_SPI_SCLK: U2.IO_L22P_T3_34, U28.SCLK
- removed net BUS_I2C_SCL: CN4.62, R182.1, U11.B2, U25.SCL
- removed net BUS_I2C_SDA: CN4.63, R181.1, U11.B1, U25.SDA
- removed net ETH_CLK: U10.CKXTAL1, U2.IO_L17N_T2_AD5N_35
- removed net ETH_CLK125M: U10.CLK125, U2.IO_L16P_T2_35
- removed net ETH_LED_ACT: CN7.CONFIG1, R194.1, U10.LED0/PHY_AD0
- removed net ETH_LED_LNK: CN7.CONFIG2, R196.2, U10.LED1/PHY_AD1
- removed net ETH_MD_0_N: TX1A.D-, U10.MDI_0_N
- removed net ETH_MD_0_P: TX1A.D+, U10.MDI_0_P
- removed net ETH_MD_1_N: TX1B.D-, U10.MDI_1_N
- removed net ETH_MD_1_P: TX1B.D+, U10.MDI_1_P
- removed net ETH_MD_2_N: TX1C.D-, U10.MDI_2_N
- removed net ETH_MD_2_P: TX1C.D+, U10.MDI_2_P
- removed net ETH_MD_3_N: TX1D.D-, U10.MDI_3_N
- removed net ETH_MD_3_P: TX1D.D+, U10.MDI_3_P
- removed net ETH_NINT: U10.INTB
- removed net ETH_NRST: R197.1, U10.PHYRSTB, U2.IO_L24N_T3_AD15N_35
- removed net ETH_TD_0_N: CN7.ML_LANE_2_P, TX1A.X-
- removed net ETH_TD_0_P: CN7.ML_LANE_2_N, TX1A.X+
- removed net ETH_TD_1_N: CN7.ML_LANE_1_P, TX1B.X-
- removed net ETH_TD_1_P: CN7.ML_LANE_1_N, TX1B.X+
- removed net ETH_TD_2_N: CN7.ML_LANE_3_P, TX1C.X-
- removed net ETH_TD_2_P: CN7.ML_LANE_3_N, TX1C.X+
- removed net ETH_TD_3_N: CN7.ML_LANE_0_P, TX1D.X-
- removed net ETH_TD_3_P: CN7.ML_LANE_0_N, TX1D.X+
- removed net FPGA_DEBUG_CLK: CN1.P20, U2.IO_L9N_T1_DQS_AD3N_35
- removed net FPGA_DEBUG_D0: CN1.P11, U2.IO_L18P_T2_AD13P_35
- removed net FPGA_DEBUG_D1: CN1.P12, U2.IO_L15P_T2_DQS_AD12P_35
- removed net FPGA_DEBUG_D2: CN1.P13, U2.IO_L13N_T2_MRCC_35
- removed net FPGA_DEBUG_D3: CN1.P14, U2.IO_L14N_T2_AD4N_SRCC_35
- removed net FPGA_DEBUG_D4: CN1.P15, U2.IO_L13P_T2_MRCC_35
- removed net FPGA_DEBUG_D5: CN1.P16, U2.IO_L10N_T1_AD11N_35
- removed net FPGA_DEBUG_D6: CN1.P17, U2.IO_L12N_T1_MRCC_35
- removed net FPGA_DEBUG_D7: CN1.P18, U2.IO_L10P_T1_AD11P_35
- removed net FPGA_DEBUG_EN: CN1.P19, U2.IO_L11N_T1_SRCC_35
- removed net FPGA_STATUS_D0: CN1.P23, U2.IO_L8N_T1_AD10N_35
- removed net FPGA_STATUS_D1: CN1.P24, U2.IO_L11P_T1_SRCC_35
- removed net FPGA_STATUS_D2: CN1.P25, U2.IO_L8P_T1_AD10P_35
- removed net N$101: L7.1, U10.REG_OUT
- removed net N$125: R63.1, TX1B.TX
- removed net N$128: C281.2, R62.2, R63.2, R72.2, R75.2
- removed net N$45: C118.2, C119.2, C155.2, C280.2, TX1A.TD, TX1B.TD, TX1C.TD, TX1D.TD
- removed net N$46: R35.2, U6.RBIAS
- removed net N$47: R61.2, U6.VBUS
- removed net N$55: R193.2, U10.RSET
- removed net N$97: R195.1, U10.LED2/RXDLY
- removed net PMC_PSS_FLAG: U2.IO_L7N_T1_13, U5.PB0
- removed net PSS_PMC_FLAG: U2.IO_L9N_T1_DQS_13, U5.PC5
- removed net PSS_PMC_UART_RX: U2.IO_L8N_T1_13, U5.PA3
- removed net PSS_PMC_UART_TX: U2.IO_L9P_T1_DQS_13, U5.PA2
- removed net PSS_SD_CD: CN2.CD, R74.1, U2.IO_L10N_T1_13
- removed net PSS_SD_CLK: CN2.CLK, U2.PS_MIO12_500
- removed net PSS_SD_CMD: CN2.CMD, U2.PS_MIO11_500
- removed net PSS_SD_D0: CN2.DAT0, U2.PS_MIO10_500
- removed net PSS_SD_D1: CN2.DAT1, U2.PS_MIO13_500
- removed net PSS_SD_D2: CN2.DAT2, U2.PS_MIO14_500
- removed net PSS_SD_D3: CN2.CD/DAT3, U2.PS_MIO15_500
- removed net PSS_SD_WP: CN2.WP, R78.1, U2.IO_L11P_T1_SRCC_13
- removed net PWR_ETH_1V0: C107.2, C108.2, C109.2, C111.2, C112.2, C113.2, L7.2, U10.AVDD10, U10.DVDD10
- removed net STM_I2C2_SCL: R190.1, U5.PB10
- removed net STM_I2C2_SDA: R189.1, U5.PB11
- removed net USB_CLK: U2.PS_MIO48_501, U6.CLKOUT
- removed net USB_D0: U2.PS_MIO44_501, U6.D0
- removed net USB_D1: U2.PS_MIO45_501, U6.D1
- removed net USB_D2: U2.PS_MIO46_501, U6.D2
- removed net USB_D3: U2.PS_MIO47_501, U6.D3
- removed net USB_D4: U2.PS_MIO40_501, U6.D4
- removed net USB_D5: U2.PS_MIO49_501, U6.D5
- removed net USB_D6: U2.PS_MIO50_501, U6.D6
- removed net USB_D7: U2.PS_MIO51_501, U6.D7
- removed net USB_DIR: U2.PS_MIO41_501, U6.DIR
- removed net USB_NRST: U2.IO_L23N_T3_35, U6.!RESET
- removed net USB_NXT: U2.PS_MIO43_501, U6.NXT
- removed net USB_REFCLK: U2.IO_L15N_T2_DQS_AD12N_35, U6.REFCLK
- removed net USB_STP: U2.PS_MIO42_501, U6.STP
- removed net USB_VBUS: C76.2, R61.1, U8.VOUT
- new net BTN_TOPRIGHT1: U2.PS_MIO41_501
- new net EMMC0_CLK: U2.IO_L16P_T2_35, U41.CLK
- new net EMMC0_CMD: U2.IO_L17N_T2_AD5N_35, U41.CMD
- new net EMMC0_D0: U2.IO_L8P_T1_AD10P_35, U41.D0
- new net EMMC0_D1: U2.IO_L2P_T0_AD8P_35, U41.D1
- new net EMMC0_D2: U2.IO_L1P_T0_AD0P_35, U41.D2
- new net EMMC0_D3: U2.IO_L4N_T0_35, U41.D3
- new net EMMC0_D4: U2.IO_L3N_T0_DQS_AD1N_35, U41.D4
- new net EMMC0_D5: U2.IO_L3P_T0_DQS_AD1P_35, U41.D5
- new net EMMC0_D6: U2.IO_L1N_T0_AD0N_35, U41.D6
- new net EMMC0_D7: U2.IO_L6N_T0_VREF_35, U41.D7
- new net EMMC0_DS: U2.IO_L12P_T1_MRCC_35, U41.DS
- new net EMMC0_NRESET: U2.IO_L14N_T2_AD4N_SRCC_35, U41.!RST
- new net EMMC1_CLK: U2.IO_L8N_T1_AD10N_35, U42.CLK
- new net EMMC1_CMD: U2.IO_L9N_T1_DQS_AD3N_35, U42.CMD
- new net EMMC1_D0: U2.IO_L13P_T2_MRCC_35, U42.D0
- new net EMMC1_D1: U2.IO_L12N_T1_MRCC_35, U42.D1
- new net EMMC1_D2: U2.IO_L18P_T2_AD13P_35, U42.D2
- new net EMMC1_D3: U2.IO_L10P_T1_AD11P_35, U42.D3
- new net EMMC1_D4: U2.IO_L10N_T1_AD11N_35, U42.D4
- new net EMMC1_D5: U2.IO_L13N_T2_MRCC_35, U42.D5
- new net EMMC1_D6: U2.IO_L15P_T2_DQS_AD12P_35, U42.D6
- new net EMMC1_D7: U2.IO_L15N_T2_DQS_AD12N_35, U42.D7
- new net EMMC1_DS: U2.IO_L11N_T1_SRCC_35, U42.DS
- new net EMMC1_NRESET: U2.IO_L11P_T1_SRCC_35, U42.!RST
- new net ESP_CANBUS_D: U14.IO19, U21.D
- new net ESP_CANBUS_R: U14.IO18, U21.R
- new net ETH_CLK_25MHZ: R195.2, U2.IO_L14P_T2_SRCC_33
- new net ETH_N_RESET: R196.1, U28.!RESET
- new net FT_BE0: U2.IO_L18P_T2_13, U6.BE0
- new net FT_BE1: U2.IO_L19P_T3_13, U6.BE1
- new net FT_BE2: U2.IO_L23P_T3_13, U6.BE2
- new net FT_BE3: U2.IO_L19N_T3_VREF_13, U6.BE3
- new net FT_CLK: U2.IO_L12P_T1_MRCC_13, U6.CLK
- new net FT_D0: U2.IO_L4N_T0_13, U6.D0
- new net FT_D1: U2.IO_L7N_T1_13, U6.D1
- new net FT_D10: U2.IO_L11P_T1_SRCC_13, U6.D10
- new net FT_D11: U2.IO_L11N_T1_SRCC_13, U6.D11
- new net FT_D12: U2.IO_L17P_T2_13, U6.D12
- new net FT_D13: U2.IO_L14P_T2_SRCC_13, U6.D13
- new net FT_D14: U2.IO_L17N_T2_13, U6.D14
- new net FT_D15: U2.IO_L14N_T2_SRCC_13, U6.D15
- new net FT_D16: U2.IO_L3N_T0_DQS_13, U6.D16
- new net FT_D17: U2.IO_L16P_T2_13, U6.D17
- new net FT_D18: U2.IO_L16N_T2_13, U6.D18
- new net FT_D19: U2.IO_L18N_T2_13, U6.D19
- new net FT_D2: U2.IO_L7P_T1_13, U6.D2
- new net FT_D20: U2.IO_L15P_T2_DQS_13, U6.D20
- new net FT_D21: U2.IO_L15N_T2_DQS_13, U6.D21
- new net FT_D22: U2.IO_L22P_T3_13, U6.D22
- new net FT_D23: U2.IO_L10N_T1_13, U6.D23
- new net FT_D24: U2.IO_L3P_T0_DQS_13, U6.D24
- new net FT_D25: U2.IO_L2N_T0_13, U6.D25
- new net FT_D26: U2.IO_L12N_T1_MRCC_13, U6.D26
- new net FT_D27: U2.IO_L23N_T3_13, U6.D27
- new net FT_D28: U2.IO_L13P_T2_MRCC_13, U6.D28
- new net FT_D29: U2.IO_L24P_T3_13, U6.D29
- new net FT_D3: U2.IO_L8N_T1_13, U6.D3
- new net FT_D30: U2.IO_L13N_T2_MRCC_13, U6.D30
- new net FT_D31: U2.IO_L24N_T3_13, U6.D31
- new net FT_D4: U2.IO_L8P_T1_13, U6.D4
- new net FT_D5: U2.IO_L9P_T1_DQS_13, U6.D5
- new net FT_D6: U2.IO_L4P_T0_13, U6.D6
- new net FT_D7: U2.IO_L5P_T0_13, U6.D7
- new net FT_D8: U2.IO_L10P_T1_13, U6.D8
- new net FT_D9: U2.IO_L9N_T1_DQS_13, U6.D9
- new net FT_N_OE: U2.IO_L6P_T0_13, U6.!OE
- new net FT_N_RD: U2.IO_0_13, U6.!RD
- new net FT_N_RESET: U2.IO_L5N_T0_13, U6.!RST
- new net FT_N_RXF: U2.IO_25_13, U6.!RXF
- new net FT_N_TXE: U2.IO_L2P_T0_13, U6.!TXE
- new net FT_N_WR: U2.IO_L6N_T0_VREF_13, U6.!WR
- new net FT_USB_SSRX_N: U6.RIDN, U8.A1N
- new net FT_USB_SSRX_P: U6.RIDP, U8.A1P
- new net FT_USB_SSTX_N: U6.TODN, U8.A0N
- new net FT_USB_SSTX_P: U6.TODP, U8.A0P
- new net FT_VBUS: C318.2, U43.VOUT, U6.VBUS
- new net N$104: R78.2, U28.RSET
- new net N$105: R193.1, U28.LED0
- new net N$108: R194.2, U10.G+
- new net N$122: U11.D+_OUT, U9.CC1, U9.CC1DB
- new net N$123: U11.D-OUT, U9.CC2, U9.CC2DB
- new net N$14: C114.2, U8.B0P
- new net N$141: C306.2, C308.2, C309.2, C310.2, C311.2, C312.2, U28.AVDD18, U28.AVDD18_OUT, U28.AVDDC18
- new net N$142: R102.1, U28.CONFIG
- new net N$143: R195.1, U28.XTAL_IN
- new net N$148: C116.2, U8.C0P
- new net N$149: C117.2, U8.C0N
- new net N$151: U10.TRD0-, U28.MDIN0
- new net N$152: R35.2, U6.RREF
- new net N$153: C78.2, U6.XI, XTAL1.P$2
- new net N$154: C111.2, U6.XO, XTAL1.P$1
- new net N$155: U10.TRD1+, U28.MDIP1
- new net N$156: U10.TRD1-, U28.MDIN1
- new net N$157: U10.TRD2+, U28.MDIP2
- new net N$158: U10.TRD2-, U28.MDIN2
- new net N$159: U10.TRD3+, U28.MDIP3
- new net N$160: U10.TRD3-, U28.MDIN3
- new net N$161: C283.2, C285.2, U41.VDD
- new net N$162: C290.2, C291.2, U42.VDD
- new net N$163: R63.2, U6.GPIO1
- new net N$164: R72.2, U6.GPIO0
- new net N$165: R74.1, U6.!WAKEUP
- new net N$166: R75.1, U6.!SIWU
- new net N$30: C115.2, U8.B0N
- new net N$8: U2.PS_DDR_A14_502
- new net PMC_CANBUS_D: U26.D, U5.PA12
- new net PMC_CANBUS_R: U26.R, U5.PA11
- new net PSS_CANBUS_D: U12.D, U2.PS_MIO15_500
- new net PSS_CANBUS_R: U12.R, U2.PS_MIO14_500
- new net PSS_JTAG_EN: CN1.P15, R170.1, R176.1
- new net PWR_FTDI_1V0: C15.2, C16.2, C17.2, C61.2, C76.2, C77.2, U6.AVDD, U6.DV10, U6.VD10
- new net SYS_CANBUS_H: CN1.P11, R181.2, R182.2, U12.CANH, U21.CANH, U26.CANH
- new net SYS_CANBUS_L: CN1.P12, R181.1, R182.1, U12.CANL, U21.CANL, U26.CANL
- new net USB_SSRX_N_A: CN3.RX1-, U8.B1N
- new net USB_SSRX_N_B: CN3.RX2-, U8.C1N
- new net USB_SSRX_P_A: CN3.RX1+, U8.B1P
- new net USB_SSRX_P_B: CN3.RX2+, U8.C1P
- new net USB_SSTX_N_A: C115.1, CN3.TX1-
- new net USB_SSTX_N_B: C117.1, CN3.TX2-
- new net USB_SSTX_P_A: C114.1, CN3.TX1+
- new net USB_SSTX_P_B: C116.1, CN3.TX2+
- new net USB_SW_N_OE: R62.1, U5.PB9, U8.!OE
- new net USB_SW_SEL: R61.2, U5.PB8, U8.SEL
- net ACT_I2C_SCL: now also U5.PB10; no longer R190.2
- net ACT_I2C_SDA: now also U5.PB11; no longer R189.2
- net BMS_I2C_SCL: now also CN1.P30, CN2.5; no longer CN1.P41, CN5.5
- net BMS_I2C_SDA: now also CN1.P29, CN2.6; no longer CN1.P40, CN5.6
- net BMS_NINT: now also CN2.7; no longer CN1.P39, CN5.7, U5.PA5
- net BMS_NPRESENT: now also CN2.10; no longer CN5.10
- net BTN_BTMLEFT: now also U2.PS_MIO16_501; no longer U2.IO_L21P_T3_DQS_13
- net BTN_BTMRIGHT: now also U2.PS_MIO27_501; no longer U2.IO_L15P_T2_DQS_13
- net BTN_THUMB: now also U2.PS_MIO20_501; no longer U2.IO_L16N_T2_13
- net BTN_TOPLEFT: now also U2.PS_MIO42_501; no longer U2.IO_L21N_T3_DQS_13
- net BTN_TOPRIGHT: now also U2.PS_MIO51_501; no longer U2.IO_L15N_T2_DQS_13
- net DSP_D_NC: now also U2.IO_L20P_T3_13; no longer U2.IO_L2P_T0_AD8P_35
- net DSP_NRESET: now also U2.IO_L21P_T3_DQS_13; no longer U2.IO_L3N_T0_DQS_AD1N_35
- net DSP_SPI_MOSI: now also U2.IO_L20N_T3_13; no longer U2.IO_L1P_T0_AD0P_35
- net DSP_SPI_NCS: now also U2.IO_L22N_T3_13; no longer U2.IO_L3P_T0_DQS_AD1P_35
- net DSP_SPI_SCLK: now also U2.IO_L21N_T3_DQS_13; no longer U2.IO_L1N_T0_AD0N_35
- net ESP32_EN: now also CN1.P25; no longer CN1.P36
- net ESP32_UART_RX: now also CN1.P23; no longer CN1.P34
- net ESP32_UART_TX: now also CN1.P24; no longer CN1.P35
- net ESP_IO0: now also CN1.P22; no longer CN1.P33
- net ESP_PSS_UART_RX: now also U2.PS_MIO12_500; no longer U2.IO_L18N_T2_AD13N_35
- net ESP_PSS_UART_TX: now also U2.PS_MIO13_500; no longer U2.IO_L16N_T2_35
- net ETH_MDC: now also R197.1, U28.MDC; no longer U10.MDC
- net ETH_MDIO: now also U28.MDIO; no longer R203.1, U10.MDIO
- net ETH_RX_CLK: now also U28.RX_CLK; no longer U10.RXC
- net ETH_RX_CTL: now also U28.RX_CTRL; no longer R202.2, U10.RXCTL/PHY_AD
- net ETH_RX_D0: now also U28.RXD0; no longer R201.1, U10.RXD0/SELRGV
- net ETH_RX_D1: now also U28.RXD1; no longer R200.1, U10.RXD1/TXDLY
- net ETH_RX_D2: now also U28.RXD2; no longer R199.1, U10.RX2/AN0
- net ETH_RX_D3: now also U28.RXD3; no longer R198.1, U10.RX3/AN1
- net ETH_TX_CLK: now also U28.TX_CLK; no longer U10.TXC
- net ETH_TX_CTL: now also U28.TX_CTRL; no longer U10.TXCTL
- net ETH_TX_D0: now also U28.TXD0; no longer U10.TXD0
- net ETH_TX_D1: now also U28.TXD1; no longer U10.TXD1
- net ETH_TX_D2: now also U28.TXD2; no longer U10.TXD2
- net ETH_TX_D3: now also U28.TXD3; no longer U10.TXD3
- net EVF_NRESET: now also U2.PS_MIO17_501; no longer U2.IO_L18P_T2_13
- net FPGA_DONE: no longer U5.PB9
- net FPGA_NINIT: no longer U5.PB8
- net FPGA_NPROG: no longer U5.PB12
- net GND: now also C285.1, C286.1, C287.1, C288.1, C289.1, C290.1, C291.1, C292.1, C293.1, C294.1, C295.1, C296.1, C297.1, C298.1, C299.1, C300.1, C301.1, C302.1, C303.1, C304.1, C305.1, C306.1, C307.1, C308.1, C309.1, C310.1, C311.1, C312.1, C313.1, C314.1, C315.1, C316.1, C317.1, C318.1, CN1.P13, CN1.P14, CN1.P21, CN1.P27, CN1.P39, CN1.P40, CN2.11, CN2.12, CN2.13, CN2.14, CN2.15, R102.2, R61.1, R63.1, R72.1, R78.1, U10.G-, U10.Y-, U12.GND1, U12.GND2, U21.GND1, U21.GND2, U26.GND1, U26.GND2, U41.GND, U42.GND, U43.GND; no longer C114.1, C115.1, C116.1, C117.1, CN1.GND, CN1.P22, CN1.P26, CN1.P38, CN1.P43, CN1.P50, CN2.GND, CN2.VSS, CN5.11, CN5.12, CN5.13, CN5.14, CN5.15, CN7.GND, CN7.SH, D1.A, D3.A, R170.1, R193.1, R196.1, R202.1, U10.CKXTAL2, U11.A3, U11.A4, U26.GND, U6.REFSEL0, U6.REFSEL2
- net N$106: now also R194.1, U28.LED1; no longer C79.2, R102.2, U28.VIN
- net N$107: now also R193.2, U10.Y+; no longer R102.1, U26.OUT
- net N$124: now also C303.2, C304.2, C305.2, U28.DVDD, U28.DVDD_OUT; no longer R62.1, TX1A.TX
- net N$126: now also C299.2, U28.REGCAP1; no longer R72.1, TX1C.TX
- net N$127: now also C298.2, U28.REGCAP2; no longer R75.1, TX1D.TX
- net N$70: now also U10.TRD0+, U28.MDIP0; no longer R170.2, R176.1, SW8.1
- net PMC_NRESET: now also CN1.P34; no longer CN1.P45
- net PMC_SWCLK: now also CN1.P35; no longer CN1.P46
- net PMC_SWDIO: now also CN1.P36; no longer CN1.P47
- net PMC_UART_RX: now also CN1.P37; no longer CN1.P48
- net PMC_UART_TX: now also CN1.P38; no longer CN1.P49
- net PSS_DEBUG_UART_RX: now also CN1.P18, U2.PS_MIO10_500; no longer CN1.P29, U2.PS_MIO22_501
- net PSS_DEBUG_UART_TX: now also CN1.P19, U2.PS_MIO11_500; no longer CN1.P30, U2.PS_MIO23_501
- net PSS_I2C_SCL: now also CN4.62, U2.IO_L20N_T3_AD6N_35, U25.SCL; no longer R205.1, U11.A2, U2.PS_MIO26_501
- net PSS_I2C_SDA: now also CN4.63, U2.IO_L5N_T0_AD9N_35, U25.SDA; no longer R204.1, U11.A1, U2.PS_MIO27_501
- net PSS_NSRST: now also CN1.P16; no longer CN1.P27
- net PWR_DIG_1V8_EN: now also U5.PB13; no longer U5.PA12
- net PWR_EVF_AVDD: now also C145.2, R81.2, U29.VIN
- net PWR_EVF_AVDD_EN: now also U2.IO_L6P_T0_35; no longer U2.IO_L21N_T3_DQS_AD14N_35
- net PWR_EVF_AVEE_EN: now also U2.IO_L2N_T0_AD8N_35; no longer U2.IO_L17P_T2_AD5P_35
- net PWR_SEN_0V7_EN: now also U2.IO_L4P_T0_35; no longer U2.IO_L21P_T3_DQS_AD14P_35
- net PWR_SEN_1V3_EN: now also U2.IO_L22N_T3_AD7N_35; no longer U2.IO_L22N_T3_13
- net PWR_SEN_3V3A_EN: now also U2.IO_L24N_T3_AD15N_35; no longer U2.IO_L22P_T3_13
- net PWR_SEN_3V6_EN: now also U2.IO_L19P_T3_35; no longer U2.IO_L20N_T3_AD6N_35
- net PWR_SEN_4V1_EN: now also U2.IO_25_35; no longer U2.IO_L5N_T0_AD9N_35
- net PWR_SEN_N1V3A_EN: now also U2.IO_0_35; no longer U2.IO_L14P_T2_AD4P_SRCC_35
- net PWR_SYS_1V8: now also C138.2, C139.2, C140.2, C141.2, C142.2, C143.2, C144.2, C286.2, C287.2, C292.2, C293.2, C296.2, C313.2, C314.2, C315.2, C60.2, R185.2, R186.2, R196.2, R197.2, U2.VCCO_35, U2.VCCO_MIO1_501, U28.VDDO, U28.VDDO_SEL, U41.VCCQ, U42.VCCQ; no longer C17.2, C258.2, C259.2, C260.2, C261.2, C262.2, C283.2, C284.2, C80.2, R181.2, R182.2, R74.2, R78.2, U11.VCCB, U2.VCCO_13, U28.VDD, U6.REFSEL1, U6.VDD18
- net PWR_SYS_1V8_SLP: now also C281.2, CN1.P31, CN1.P33, U26.VCC1; no longer CN1.P42, CN1.P44
- net PWR_SYS_3V3: now also C107.2, C108.2, C109.2, C112.2, C113.2, C119.2, C155.2, C157.2, C158.2, C258.2, C259.2, C260.2, C261.2, C262.2, C284.2, C288.2, C289.2, C294.2, C295.2, C297.2, C300.2, C301.2, C302.2, C316.2, C317.2, C79.2, C80.2, CN1.P20, R170.2, R62.2, R74.2, R75.2, U12.VCC1, U2.VCCO_13, U21.VCC1, U28.AVDD33, U28.REG_IN, U34.VIN, U41.VCC, U42.VCC, U6.VCC33, U6.VCCIO, U6.VDDA, U8.VCC; no longer C114.2, C115.2, C116.2, C117.2, C138.2, C139.2, C140.2, C141.2, C142.2, C143.2, C144.2, C15.2, C16.2, C282.2, C60.2, C77.2, C78.2, CN1.P21, CN1.P31, CN1.P37, CN2.VDD, CN7.HOT_PLUG_DECT, R185.2, R186.2, R194.2, R195.2, R197.2, R198.2, R199.2, R200.2, R201.2, R203.2, R204.2, R205.2, SW8.2, U10.AVDD33, U10.DVDD33, U10.ENSWREG, U10.VDDREG, U11.EN, U11.VCCA, U2.VCCO_35, U2.VCCO_MIO1_501, U26.VCC, U6.VBAT, U6.VDD33, U6.VDDIO
- net PWR_SYS_3V3_EN: now also U5.PB12; no longer U5.PA11
- net PWR_SYS_5V: now also C118.2, C280.2, C282.2, U12.VCC2, U21.VCC2, U26.VCC2; no longer C145.2, C157.2, C158.2, R81.2, U29.VIN, U34.VIN
- net PWR_USBC_VBUS: now also C307.2, U43.VIN; no longer C61.2, U8.EN, U8.VIN
- net PWR_VBAT: now also CN2.1, CN2.2, CN2.3, CN2.4; no longer CN5.1, CN5.2, CN5.3, CN5.4
- net PWR_VDISP_EN: now also U2.PS_MIO23_501; no longer U2.IO_L19P_T3_13
- net SEN_SPI_MISO: now also U2.IO_L21N_T3_DQS_AD14N_35; no longer U2.IO_L9N_T1_DQS_33
- net SEN_SPI_MOSI: now also U2.IO_L14P_T2_AD4P_SRCC_35; no longer U2.IO_L2P_T0_33
- net SEN_SPI_NCS: now also U2.IO_L16N_T2_35; no longer U2.IO_L2N_T0_33
- net SEN_SPI_SCLK: now also U2.IO_L18N_T2_AD13N_35; no longer U2.IO_0_33
- net SEN_SYS_NRESET: now also U2.IO_L22P_T3_AD7P_35; no longer U2.IO_L16P_T2_13
- net SEN_TDIG0: now also U2.IO_L21P_T3_DQS_AD14P_35; no longer U2.IO_L24N_T3_13
- net SEN_TDIG1: now also U2.IO_L17P_T2_AD5P_35; no longer U2.IO_L13N_T2_MRCC_13
- net SEN_TEXP0: now also U2.IO_L23N_T3_35; no longer U2.IO_L13P_T2_MRCC_13
- net SEN_TEXP1: now also U2.IO_L23P_T3_35; no longer U2.IO_L24P_T3_13
- net TMP_ALERT: no longer U2.IO_L12N_T1_MRCC_13
- net TMP_THERM: no longer U2.IO_L23N_T3_13
- net USBC_CC1: now also U11.D+_IN; no longer D3.K, U9.CC1, U9.CC1DB
- net USBC_CC2: now also U11.D-_IN; no longer D1.K, U9.CC2, U9.CC2DB
Other:
- note removed: "FT602Q"
- note removed: "GPIO ETC."
- note removed: "MIPI DSI"
- note removed: "SENSOR LVDS"
- moved on the sheet: C106, C107, C108, C109, C111, C112, C113, C114, C115, C116, C117, C145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
