File: ethernet.sch (EAGLE design)
At the start: 1 part, among them CN7 Mini Displayport

Commit message: Ethernet PCB done and small bits to main PCB
Parts:
- added CN1: 8P8C, CONNECTORs:MTJ-880X1
Connections:
- removed net ETH_LED_ACT: CN7.CONFIG1
- removed net ETH_LED_LNK: CN7.CONFIG2
- removed net PWR_SYS_3V3: CN7.HOT_PLUG_DECT
- net ETH_TD_0_N: now also CN1.A-
- net ETH_TD_0_P: now also CN1.A+
- net ETH_TD_1_N: now also CN1.B-
- net ETH_TD_1_P: now also CN1.B+
- net ETH_TD_2_N: now also CN1.C-
- net ETH_TD_2_P: now also CN1.C+
- net ETH_TD_3_N: now also CN1.D-
- net ETH_TD_3_P: now also CN1.D+
Other:
- moved on the sheet: CN7
Changed lines of the file:
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@@
 <parts>
 <part name="CN7" library="CONNECTORs" deviceset="2129320-3" device="" value="Mini Displayport"/>
-<part name="GND40" library="NETS" deviceset="GND" device=""/>
+<part name="CN1" library="CONNECTORs" deviceset="MTJ-880X1" device="" value="8P8C"/>
+<part name="GND1" library="NETS" deviceset="GND" device=""/>
 </parts>
 <sheets>
@@
 </plain>
 <instances>
-<instance part="CN7" gate="G$1" x="-93.98" y="0" smashed="yes">
-<attribute name="NAME" x="-106.68" y="40.64" size="1.778" layer="95"/>
-<attribute name="VALUE" x="-106.68" y="38.1" size="1.778" layer="96"/>
+<instance part="CN7" gate="G$1" x="-50.8" y="7.62" smashed="yes">
+<attribute name="NAME" x="-63.5" y="48.26" size="1.778" layer="95"/>
+<attribute name="VALUE" x="-63.5" y="45.72" size="1.778" layer="96"/>
 </instance>
-<instance part="GND40" gate="G$1" x="-93.98" y="-50.8" smashed="yes" rot="MR0">
-<attribute name="VALUE" x="-93.98" y="-53.34" size="1.778" layer="96" rot="MR0" align="center"/>
+<instance part="CN1" gate="G$1" x="55.88" y="15.24" smashed="yes">
+<attribute name="NAME" x="50.8" y="35.56" size="1.778" layer="95"/>
+<attribute name="VALUE" x="50.8" y="33.02" size="1.778" layer="96"/>
+</instance>
+<instance part="GND1" gate="G$1" x="-50.8" y="-40.64" smashed="yes">
+<attribute name="VALUE" x="-50.8" y="-43.18" size="1.778" layer="96" align="center"/>
 </instance>
 </instances>
@@
 </busses>
 <nets>
-<net name="GND" class="0">
-<segment>
-<pinref part="GND40" gate="G$1" pin="GND"/>
-<wire x1="-93.98" y1="-48.26" x2="-93.98" y2="-45.72" width="0.1524" layer="91"/>
-<wire x1="-93.98" y1="-45.72" x2="-96.52" y2="-45.72" width="0.1524" layer="91"/>
-<pinref part="CN7" gate="G$1" pin="SH"/>
-<wire x1="-96.52" y1="-45.72" x2="-96.52" y2="-40.64" width="0.1524" layer="91"/>
-<wire x1="-93.98" y1="-45.72" x2="-91.44" y2="-45.72" width="0.1524" layer="91"/>
-<junction x="-93.98" y="-45.72"/>
-<pinref part="CN7" gate="G$1" pin="GND"/>
-<wire x1="-91.44" y1="-45.72" x2="-91.44" y2="-40.64" width="0.1524" layer="91"/>
-</segment>
-</net>
-<net name="PWR_SYS_3V3" class="0">
-<segment>
-<pinref part="CN7" gate="G$1" pin="HOT_PLUG_DECT"/>
-<wire x1="-76.2" y1="-25.4" x2="-38.1" y2="-25.4" width="0.1524" layer="91"/>
-<label x="-40.64" y="-25.4" size="1.778" layer="95" rot="MR0"/>
-</segment>
-</net>
 <net name="ETH_TD_0_P" class="0">
 <segment>
 <pinref part="CN7" gate="G$1" pin="ML_LANE_2_N"/>
-<wire x1="-38.1" y1="2.54" x2="-76.2" y2="2.54" width="0.1524" layer="91"/>
-<label x="-40.64" y="2.54" size="1.778" layer="95" rot="MR0"/>
+<wire x1="5.08" y1="10.16" x2="-33.02" y2="10.16" width="0.1524" layer="91"/>
+<label x="2.54" y="10.16" size="1.778" layer="95" rot="MR0"/>
+</segment>
+<segment>
+<pinref part="CN1" gate="G$1" pin="A+"/>
+<wire x1="20.32" y1="27.94" x2="45.72" y2="27.94" width="0.1524" layer="91"/>
+<label x="22.86" y="27.94" size="1.778" layer="95"/>
 </segment>
 </net>
@@
 <segment>
 <pinref part="CN7" gate="G$1" pin="ML_LANE_2_P"/>
-<wire x1="-38.1" y1="5.08" x2="-76.2" y2="5.08" width="0.1524" layer="91"/>
-<label x="-40.64" y="5.08" size="1.778" layer="95" rot="MR0"/>
+<wire x1="5.08" y1="12.7" x2="-33.02" y2="12.7" width="0.1524" layer="91"/>
+<label x="2.54" y="12.7" size="1.778" layer="95" rot="MR0"/>
+</segment>
+<segment>
+<pinref part="CN1" gate="G$1" pin="A-"/>
+<wire x1="20.32" y1="25.4" x2="45.72" y2="25.4" width="0.1524" layer="91"/>
+<label x="22.86" y="25.4" size="1.778" layer="95"/>
 </segment>
 </net>
@@
 <segment>
 <pinref part="CN7" gate="G$1" pin="ML_LANE_1_N"/>
-<wire x1="-38.1" y1="10.16" x2="-76.2" y2="10.16" width="0.1524" layer="91"/>
-<label x="-40.64" y="10.16" size="1.778" layer="95" rot="MR0"/>
+<wire x1="5.08" y1="17.78" x2="-33.02" y2="17.78" width="0.1524" layer="91"/>
+<label x="2.54" y="17.78" size="1.778" layer="95" rot="MR0"/>
+</segment>
+<segment>
+<pinref part="CN1" gate="G$1" pin="B+"/>
+<wire x1="20.32" y1="20.32" x2="45.72" y2="20.32" width="0.1524" layer="91"/>
+<label x="22.86" y="20.32" size="1.778" layer="95"/>
 </segment>
 </net>
@@
 <segment>
 <pinref part="CN7" gate="G$1" pin="ML_LANE_1_P"/>
-<wire x1="-38.1" y1="12.7" x2="-76.2" y2="12.7" width="0.1524" layer="91"/>
-<label x="-40.64" y="12.7" size="1.778" layer="95" rot="MR0"/>
+<wire x1="5.08" y1="20.32" x2="-33.02" y2="20.32" width="0.1524" layer="91"/>
+<label x="2.54" y="20.32" size="1.778" layer="95" rot="MR0"/>
+</segment>
+<segment>
+<pinref part="CN1" gate="G$1" pin="B-"/>
+<wire x1="20.32" y1="17.78" x2="45.72" y2="17.78" width="0.1524" layer="91"/>
+<label x="22.86" y="17.78" size="1.778" layer="95"/>
 </segment>
 </net>
@@
 <segment>
 <pinref part="CN7" gate="G$1" pin="ML_LANE_3_N"/>
-<wire x1="-38.1" y1="-5.08" x2="-76.2" y2="-5.08" width="0.1524" layer="91"/>
-<label x="-40.64" y="-5.08" size="1.778" layer="95" rot="MR0"/>
+<wire x1="5.08" y1="2.54" x2="-33.02" y2="2.54" width="0.1524" layer="91"/>
+<label x="2.54" y="2.54" size="1.778" layer="95" rot="MR0"/>
+</segment>
+<segment>
+<pinref part="CN1" gate="G$1" pin="C+"/>
+<wire x1="20.32" y1="12.7" x2="45.72" y2="12.7" width="0.1524" layer="91"/>
+<label x="22.86" y="12.7" size="1.778" layer="95"/>
 </segment>
 </net>
@@
 <segment>
 <pinref part="CN7" gate="G$1" pin="ML_LANE_3_P"/>
-<wire x1="-38.1" y1="-2.54" x2="-76.2" y2="-2.54" width="0.1524" layer="91"/>
-<label x="-40.64" y="-2.54" size="1.778" layer="95" rot="MR0"/>
+<wire x1="5.08" y1="5.08" x2="-33.02" y2="5.08" width="0.1524" layer="91"/>
+<label x="2.54" y="5.08" size="1.778" layer="95" rot="MR0"/>
+</segment>
+<segment>
+<pinref part="CN1" gate="G$1" pin="C-"/>
+<wire x1="20.32" y1="10.16" x2="45.72" y2="10.16" width="0.1524" layer="91"/>
+<label x="22.86" y="10.16" size="1.778" layer="95"/>
 </segment>
 </net>
@@
 <segment>
 <pinref part="CN7" gate="G$1" pin="ML_LANE_0_N"/>
-<wire x1="-38.1" y1="17.78" x2="-76.2" y2="17.78" width="0.1524" layer="91"/>
-<label x="-40.64" y="17.78" size="1.778" layer="95" rot="MR0"/>
+<wire x1="5.08" y1="25.4" x2="-33.02" y2="25.4" width="0.1524" layer="91"/>
+<label x="2.54" y="25.4" size="1.778" layer="95" rot="MR0"/>
+</segment>
+<segment>
+<pinref part="CN1" gate="G$1" pin="D+"/>
+<wire x1="20.32" y1="5.08" x2="45.72" y2="5.08" width="0.1524" layer="91"/>
+<label x="22.86" y="5.08" size="1.778" layer="95"/>
 </segment>
 </net>
@@
 <segment>
 <pinref part="CN7" gate="G$1" pin="ML_LANE_0_P"/>
-<wire x1="-38.1" y1="20.32" x2="-76.2" y2="20.32" width="0.1524" layer="91"/>
-<label x="-40.64" y="20.32" size="1.778" layer="95" rot="MR0"/>
+<wire x1="5.08" y1="27.94" x2="-33.02" y2="27.94" width="0.1524" layer="91"/>
+<label x="2.54" y="27.94" size="1.778" layer="95" rot="MR0"/>
+</segment>
+<segment>
+<pinref part="CN1" gate="G$1" pin="D-"/>
+<wire x1="20.32" y1="2.54" x2="45.72" y2="2.54" width="0.1524" layer="91"/>
+<label x="22.86" y="2.54" size="1.778" layer="95"/>
 </segment>
 </net>
-<net name="ETH_LED_ACT" class="0">
+<net name="GND" class="0">
 <segment>
-<pinref part="CN7" gate="G$1" pin="CONFIG1"/>
-<wire x1="-76.2" y1="-17.78" x2="-38.1" y2="-17.78" width="0.1524" layer="91"/>
-<label x="-40.64" y="-17.78" size="1.778" layer="95" rot="MR0"/>
+<pinref part="CN7" gate="G$1" pin="SH"/>
+<wire x1="-53.34" y1="-33.02" x2="-53.34" y2="-35.56" width="0.1524" layer="91"/>
+<wire x1="-53.34" y1="-35.56" x2="-50.8" y2="-35.56" width="0.1524" layer="91"/>
+<pinref part="CN7" gate="G$1" pin="GND"/>
+<wire x1="-50.8" y1="-35.56" x2="-48.26" y2="-35.56" width="0.1524" layer="91"/>
+<wire x1="-48.26" y1="-35.56" x2="-48.26" y2="-33.02" width="0.1524" layer="91"/>
+<wire x1="-50.8" y1="-35.56" x2="-50.8" y2="-38.1" width="0.1524" layer="91"/>
+<junction x="-50.8" y="-35.56"/>
+<pinref part="GND1" gate="G$1" pin="GND"/>
 </segment>
 </net>
-<net name="ETH_LED_LNK" class="0">
-<segment>
-<pinref part="CN7" gate="G$1" pin="CONFIG2"/>
-<wire x1="-76.2" y1="-20.32" x2="-38.1" y2="-20.32" width="0.1524" layer="91"/>
-<label x="-40.64" y="-20.32" size="1.778" layer="95" rot="MR0"/>
-</segment>
-</net>

Commit message: Addition of an ethernet adapter PCB
Parts:
- removed CN7: Mini Displayport, CONNECTORs:2129320-3
- added MECH1, MECH2: 6mm x 3mm, MISC:MOUNTHOLE
- added TP1, TP10, TP11, TP12, TP2, TP3, TP4, TP5, TP6, TP7, TP8, TP9: TEST_POINT_SQUARE, MISC:TEST_POINT_SQUARE
- CN1: value 8P8C -> HFJ11-1G01ERL; device CONNECTORs:MTJ-880X1 -> CONNECTORs:HFJ11-1G01ERL
Connections:
- removed net ETH_TD_0_N: CN1.A-, CN7.ML_LANE_2_P
- removed net ETH_TD_0_P: CN1.A+, CN7.ML_LANE_2_N
- removed net ETH_TD_1_N: CN1.B-, CN7.ML_LANE_1_P
- removed net ETH_TD_1_P: CN1.B+, CN7.ML_LANE_1_N
- removed net ETH_TD_2_N: CN1.C-, CN7.ML_LANE_3_P
- removed net ETH_TD_2_P: CN1.C+, CN7.ML_LANE_3_N
- removed net ETH_TD_3_N: CN1.D-, CN7.ML_LANE_0_P
- removed net ETH_TD_3_P: CN1.D+, CN7.ML_LANE_0_N
- new net LED_AMBER: CN1AMBER.K, TP11.P$1
- new net LED_GREEN: CN1GREEN.A, TP10.P$1
- new net N$1: CN1JACK.TRD1+, TP1.P$1
- new net N$2: CN1JACK.TRD1-, TP2.P$1
- new net N$3: CN1JACK.TRD2+, TP3.P$1
- new net N$4: CN1JACK.TRD2-, TP4.P$1
- new net N$5: CN1JACK.TRD3+, TP5.P$1
- new net N$6: CN1JACK.TRD3-, TP6.P$1
- new net N$7: CN1JACK.TRD4+, TP7.P$1
- new net N$8: CN1JACK.TRD4-, TP8.P$1
- new net PWR_SYS_3V3: CN1AMBER.A, TP9.P$1
- net GND: now also CN1GREEN.K, CN1JACK.GND, TP12.P$1; no longer CN7.GND, CN7.SH
